File: hardware/vesc-bms.kicad_sch (KiCad schematic)
At the start: 0 parts

Commit message: Some work on Battery AFE and PSU
Other:
- added sheet Power Supply (power-supply.kicad_sch)
- sheet AFE ports: added BALANCE_EN; removed none
Changed lines of the file:
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@@
+    (stroke (width 0) (type default) (color 0 0 0 0))
+  )
+  (wire (pts (xy 69.85 106.68) (xy 90.17 106.68))
     (stroke (width 0) (type default) (color 0 0 0 0))
   )
@@
     )
   )
+  (sheet (at 57.15 104.14) (size 12.7 8.89) (fields_autoplaced)
+    (stroke (width 0.1524) (type solid) (color 0 0 0 0))
+    (fill (color 0 0 0 0.0000))
+    (property "Sheet name" "Power Supply" (id 0) (at 57.15 103.4284 0)
+      (effects (font (size 1.27 1.27)) (justify left bottom))
+    )
+    (property "Sheet file" "power-supply.kicad_sch" (id 1) (at 57.15 113.6146 0)
+      (effects (font (size 1.27 1.27)) (justify left top))
+    )
+    (pin "BAT_UVLO" output (at 69.85 106.68 0)
+      (effects (font (size 1.27 1.27)) (justify right))
+    )
+  )
   (sheet (at 186.69 68.58) (size 17.78 29.21) (fields_autoplaced)
     (stroke (width 0.1524) (type solid) (color 0 0 0 0))
@@
     )
   )
-  (sheet (at 96.52 100.33) (size 12.7 17.78) (fields_autoplaced)
+  (sheet (at 90.17 100.33) (size 16.51 16.51) (fields_autoplaced)
     (stroke (width 0.1524) (type solid) (color 0 0 0 0))
     (fill (color 0 0 0 0.0000))
-    (property "Sheet name" "AFE" (id 0) (at 96.52 99.6184 0)
+    (property "Sheet name" "AFE" (id 0) (at 90.17 99.6184 0)
       (effects (font (size 1.27 1.27)) (justify left bottom))
     )
-    (property "Sheet file" "afe.kicad_sch" (id 1) (at 96.52 118.6946 0)
+    (property "Sheet file" "afe.kicad_sch" (id 1) (at 90.17 117.4246 0)
       (effects (font (size 1.27 1.27)) (justify left top))
+    )
+    (pin "BALANCE_EN" input (at 90.17 106.68 180)
+      (effects (font (size 1.27 1.27)) (justify left))
     )
   )
@@
     (path "/a908ff77-32fe-48f6-8dc7-bc7bb4d76281" (page "3"))
     (path "/6e2b1342-9746-4a38-93af-9ab1059c6272" (page "4"))
+    (path "/600d3fd5-a2c8-411e-91ac-e4cbb4ace0f8" (page "5"))
   )
   (symbol_instances
@@
       (reference "#PWR0101") (unit 1) (value "+3.3V") (footprint "")
     )
+    (path "/a908ff77-32fe-48f6-8dc7-bc7bb4d76281/10c4b557-1888-4819-a69f-1afdc434805c"
+      (reference "#PWR?") (unit 1) (value "GND") (footprint "")
+    )
+    (path "/600d3fd5-a2c8-411e-91ac-e4cbb4ace0f8/3c777041-5cf1-41b0-926d-5f719e8273bc"
+      (reference "#PWR?") (unit 1) (value "GND") (footprint "")
+    )
+    (path "/a908ff77-32fe-48f6-8dc7-bc7bb4d76281/537e77f9-2ee5-4cf0-ae31-7c8471d3769e"
+      (reference "#PWR?") (unit 1) (value "GND") (footprint "")
+    )
+    (path "/a908ff77-32fe-48f6-8dc7-bc7bb4d76281/5ea30b86-8687-45af-84f8-9d6502383c30"
+      (reference "#PWR?") (unit 1) (value "+BATT") (footprint "")
+    )
+    (path "/a908ff77-32fe-48f6-8dc7-bc7bb4d76281/773a8d1f-955d-45b2-8bc3-fc5a688b9aa2"
+      (reference "#PWR?") (unit 1) (value "+5V") (footprint "")
+    )
+    (path "/600d3fd5-a2c8-411e-91ac-e4cbb4ace0f8/f318570c-d25f-4828-8a5f-09306e4d0123"
+      (reference "#PWR?") (unit 1) (value "+BATT") (footprint "")
+    )
+    (path "/a908ff77-32fe-48f6-8dc7-bc7bb4d76281/f41a26b3-fd69-4767-972c-6780f0774a62"
+      (reference "#PWR?") (unit 1) (value "+3.3V") (footprint "")
+    )
     (path "/1c5935ea-6f80-435f-8ae1-741f5546f8d9/3d53b2c0-0ab8-418a-a174-d479fe6d5385"
       (reference "C1") (unit 1) (value "DNP") (footprint "Capacitor_SMD:C_0603_1608Metric")
@@
       (reference "C10") (unit 1) (value "100n") (footprint "Capacitor_SMD:C_0603_1608Metric")
     )
+    (path "/600d3fd5-a2c8-411e-91ac-e4cbb4ace0f8/f55e1cba-f27b-4b04-9aa4-8502ed96b41b"
+      (reference "C?") (unit 1) (value "2.2u") (footprint "")
+    )
     (path "/1c5935ea-6f80-435f-8ae1-741f5546f8d9/b6cbb8ea-1784-4059-9a07-19b7c70fa644"
       (reference "J1") (unit 1) (value "Conn_ARM_JTAG_SWD_10") (footprint "Connector_PinHeader_1.27mm:PinHeader_2x05_P1.27mm_Vertical_SMD")
@@
       (reference "J4") (unit 1) (value "Conn_ARM_JTAG_SWD_10") (footprint "Connector_PinHeader_1.27mm:PinHeader_2x05_P1.27mm_Vertical_SMD")
     )
+    (path "/a908ff77-32fe-48f6-8dc7-bc7bb4d76281/7fc22c10-0052-435b-ac39-268c7141defb"
+      (reference "J?") (unit 1) (value "Conn_01x19_Male") (footprint "")
+    )
     (path "/1c5935ea-6f80-435f-8ae1-741f5546f8d9/21b9b2b5-ff97-447a-a56e-396f0ea09701"
       (reference "R1") (unit 1) (value "DNP") (footprint "Resistor_SMD:R_0603_1608Metric")
@@
       (reference "R5") (unit 1) (value "5.1k") (footprint "Resistor_SMD:R_0603_1608Metric")
     )
+    (path "/a908ff77-32fe-48f6-8dc7-bc7bb4d76281/39d14ca9-8bae-43d5-b4b7-a74d5b892d2f"
+      (reference "R?") (unit 1) (value "100") (footprint "")
+    )
+    (path "/a908ff77-32fe-48f6-8dc7-bc7bb4d76281/b0d717bf-2319-4285-9365-811d3b7c9f1b"
+      (reference "R?") (unit 1) (value "20k") (footprint "")
+    )
+    (path "/a908ff77-32fe-48f6-8dc7-bc7bb4d76281/c6042107-75c7-43d2-a4e9-7190df62e8cc"
+      (reference "R?") (unit 1) (value "5k") (footprint "")
+    )
+    (path "/600d3fd5-a2c8-411e-91ac-e4cbb4ace0f8/c9c79f4c-38dd-46dd-89b0-64d0a5910646"
+      (reference "R?") (unit 1) (value "100") (footprint "")
+    )
     (path "/1c5935ea-6f80-435f-8ae1-741f5546f8d9/fd1a8cd8-06e9-4d52-af0e-ed2b061904eb"
       (reference "SW1") (unit 1) (value "SW_Push") (footprint "Button_Switch_SMD:SW_SPST_CK_RS282G05A3")
@@
       (reference "U5") (unit 1) (value "E73-2G4M08S1C") (footprint "vesc-bms:E73-2G4M08S1C")
     )
+    (path "/600d3fd5-a2c8-411e-91ac-e4cbb4ace0f8/deb1b356-6b13-4777-a25c-1e6c644c15c0"
+      (reference "U?") (unit 1) (value "LM5164DDA") (footprint "Package_SO:HSOP-8-1EP_3.9x4.9mm_P1.27mm_EP2.41x3.1mm_ThermalVias")
+    )
     (path "/1c5935ea-6f80-435f-8ae1-741f5546f8d9/0827f1d0-8e1d-46d4-92fd-80f7ab36b847"

Commit message: Analog front end ready
Other:
- added sheet Thermal (thermal.kicad_sch)
- sheet AFE ports: added GPIO1, GPIO2, GPIO3, GPIO4, GPIO5, GPIO6, GPIO7, GPIO8, GPIO9; removed none
- sheet MCU ports: added SCL, SDA; removed none

Commit message: AFE SPI
Other:
- sheet AFE ports: added CS, SCK, SDI, SDO; removed none
- sheet MCU ports: added AFE_CS, AFE_MISO, AFE_MOSI, AFE_SCLK; removed none
Changed lines of the file:
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@@
+    (stroke (width 0) (type default) (color 0 0 0 0))
+  )
+  (wire (pts (xy 106.68 97.79) (xy 124.46 97.79))
     (stroke (width 0) (type default) (color 0 0 0 0))
   )
@@
     (stroke (width 0) (type default) (color 0 0 0 0))
   )
+  (wire (pts (xy 106.68 100.33) (xy 124.46 100.33))
+    (stroke (width 0) (type default) (color 0 0 0 0))
+  )
   (wire (pts (xy 152.4 78.74) (xy 186.69 78.74))
     (stroke (width 0) (type default) (color 0 0 0 0))
@@
     (stroke (width 0) (type default) (color 0 0 0 0))
   )
+  (wire (pts (xy 106.68 105.41) (xy 124.46 105.41))
+    (stroke (width 0) (type default) (color 0 0 0 0))
+  )
+  (wire (pts (xy 106.68 102.87) (xy 124.46 102.87))
+    (stroke (width 0) (type default) (color 0 0 0 0))
+  )
   (wire (pts (xy 71.12 64.77) (xy 124.46 64.77))
     (stroke (width 0) (type default) (color 0 0 0 0))
@@
       (effects (font (size 1.27 1.27)) (justify left))
     )
+    (pin "AFE_MISO" input (at 124.46 100.33 180)
+      (effects (font (size 1.27 1.27)) (justify left))
+    )
+    (pin "AFE_MOSI" output (at 124.46 97.79 180)
+      (effects (font (size 1.27 1.27)) (justify left))
+    )
+    (pin "AFE_SCLK" output (at 124.46 102.87 180)
+      (effects (font (size 1.27 1.27)) (justify left))
+    )
+    (pin "AFE_CS" output (at 124.46 105.41 180)
+      (effects (font (size 1.27 1.27)) (justify left))
+    )
   )
   (sheet (at 58.42 105.41) (size 12.7 5.08) (fields_autoplaced)
@@
       (effects (font (size 1.27 1.27)) (justify left))
     )
-  )
+    (pin "SDI" input (at 106.68 97.79 0)
+      (effects (font (size 1.27 1.27)) (justify right))
+    )
+    (pin "SDO" output (at 106.68 100.33 0)
+      (effects (font (size 1.27 1.27)) (justify right))
+    )
+    (pin "CS" input (at 106.68 105.41 0)
+      (effects (font (size 1.27 1.27)) (justify right))
+    )
+    (pin "SCK" input (at 106.68 102.87 0)
+      (effects (font (size 1.27 1.27)) (justify right))
+    )
+  )

Commit message: Status LEDs
Parts:
- added D?: Green, symbol Device:LED_Small
- added D?: Red, symbol Device:LED_Small
- added R? (x2): 220, symbol Device:R_Small
Connections:
- new net: D?.1 (K), R?.1 (x2)
- new net GND: R?.2, R?.2
- new net MCU/LED_GREEN: D?.2 (A)
- new net MCU/LED_RED: D?.2 (A)
Other:
- sheet MCU ports: added LED_GREEN, LED_RED; removed none
Changed lines of the file:
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@@
     (stroke (width 0) (type default) (color 0 0 0 0))
   )
-  (wire (pts (xy 106.68 97.79) (xy 124.46 97.79))
+  (wire (pts (xy 167.64 107.95) (xy 168.91 107.95))
+    (stroke (width 0) (type default) (color 0 0 0 0))
+  )
+  (wire (pts (xy 160.02 107.95) (xy 162.56 107.95))
+    (stroke (width 0) (type default) (color 0 0 0 0))
+  )
+  (wire (pts (xy 106.68 74.93) (xy 124.46 74.93))
     (stroke (width 0) (type default) (color 0 0 0 0))
   )
@@
     (stroke (width 0) (type default) (color 0 0 0 0))
   )
-  (wire (pts (xy 106.68 100.33) (xy 124.46 100.33))
+  (wire (pts (xy 167.64 124.46) (xy 168.91 124.46))
+    (stroke (width 0) (type default) (color 0 0 0 0))
+  )
+  (wire (pts (xy 106.68 77.47) (xy 124.46 77.47))
+    (stroke (width 0) (type default) (color 0 0 0 0))
+  )
+  (wire (pts (xy 168.91 124.46) (xy 168.91 125.73))
     (stroke (width 0) (type default) (color 0 0 0 0))
   )
@@
     (stroke (width 0) (type default) (color 0 0 0 0))
   )
+  (wire (pts (xy 160.02 124.46) (xy 162.56 124.46))
+    (stroke (width 0) (type default) (color 0 0 0 0))
+  )
+  (wire (pts (xy 168.91 107.95) (xy 168.91 109.22))
+    (stroke (width 0) (type default) (color 0 0 0 0))
+  )
   (wire (pts (xy 152.4 73.66) (xy 186.69 73.66))
     (stroke (width 0) (type default) (color 0 0 0 0))
@@
     (stroke (width 0) (type default) (color 0 0 0 0))
   )
-  (wire (pts (xy 106.68 105.41) (xy 124.46 105.41))
-    (stroke (width 0) (type default) (color 0 0 0 0))
-  )
-  (wire (pts (xy 106.68 102.87) (xy 124.46 102.87))
+  (wire (pts (xy 106.68 82.55) (xy 124.46 82.55))
+    (stroke (width 0) (type default) (color 0 0 0 0))
+  )
+  (wire (pts (xy 106.68 80.01) (xy 124.46 80.01))
     (stroke (width 0) (type default) (color 0 0 0 0))
   )
@@
     (stroke (width 0) (type default) (color 0 0 0 0))
   )
+  (wire (pts (xy 152.4 124.46) (xy 154.94 124.46))
+    (stroke (width 0) (type default) (color 0 0 0 0))
+  )
+  (wire (pts (xy 152.4 107.95) (xy 154.94 107.95))
+    (stroke (width 0) (type default) (color 0 0 0 0))
+  )
   (wire (pts (xy 71.12 107.95) (xy 90.17 107.95))
     (stroke (width 0) (type default) (color 0 0 0 0))
@@
   (wire (pts (xy 152.4 71.12) (xy 186.69 71.12))
     (stroke (width 0) (type default) (color 0 0 0 0))
+  )
+  (symbol (lib_id "Device:R_Small") (at 165.1 107.95 90) (unit 1)
+    (in_bom yes) (on_board yes)
+    (property "Reference" "R?" (id 0) (at 165.1 102.87 90))
+    (property "Value" "220" (id 1) (at 165.1 105.41 90))
+    (property "Footprint" "" (id 2) (at 165.1 107.95 0)
+      (effects (font (size 1.27 1.27)) hide)
+    )
+    (property "Datasheet" "~" (id 3) (at 165.1 107.95 0)
+      (effects (font (size 1.27 1.27)) hide)
+    )
+    (pin "1")
+    (pin "2")
+  )
+  (symbol (lib_id "Device:LED_Small") (at 157.48 124.46 180) (unit 1)
+    (in_bom yes) (on_board yes) (fields_autoplaced)
+    (property "Reference" "D?" (id 0) (at 157.4165 118.11 0))
+    (property "Value" "Green" (id 1) (at 157.4165 120.65 0))
+    (property "Footprint" "" (id 2) (at 157.48 124.46 90)
+      (effects (font (size 1.27 1.27)) hide)
+    )
+    (property "Datasheet" "~" (id 3) (at 157.48 124.46 90)
+      (effects (font (size 1.27 1.27)) hide)
+    )
+    (pin "1")
+    (pin "2")
+  )
+  (symbol (lib_id "power:GND") (at 168.91 125.73 0) (unit 1)
+    (in_bom yes) (on_board yes) (fields_autoplaced)
+    (property "Reference" "#PWR?" (id 0) (at 168.91 132.08 0)
+      (effects (font (size 1.27 1.27)) hide)
+    )
+    (property "Value" "GND" (id 1) (at 168.91 130.81 0))
+    (property "Footprint" "" (id 2) (at 168.91 125.73 0)
+      (effects (font (size 1.27 1.27)) hide)
+    )
+    (property "Datasheet" "" (id 3) (at 168.91 125.73 0)
+      (effects (font (size 1.27 1.27)) hide)
+    )
+    (pin "1")
+  )
+  (symbol (lib_id "power:GND") (at 168.91 109.22 0) (unit 1)
+    (in_bom yes) (on_board yes) (fields_autoplaced)
+    (property "Reference" "#PWR?" (id 0) (at 168.91 115.57 0)
+      (effects (font (size 1.27 1.27)) hide)
+    )
+    (property "Value" "GND" (id 1) (at 168.91 114.3 0))
+    (property "Footprint" "" (id 2) (at 168.91 109.22 0)
+      (effects (font (size 1.27 1.27)) hide)
+    )
+    (property "Datasheet" "" (id 3) (at 168.91 109.22 0)
+      (effects (font (size 1.27 1.27)) hide)
+    )
+    (pin "1")
+  )
+  (symbol (lib_id "Device:R_Small") (at 165.1 124.46 90) (unit 1)
+    (in_bom yes) (on_board yes)
+    (property "Reference" "R?" (id 0) (at 165.1 119.38 90))
+    (property "Value" "220" (id 1) (at 165.1 121.92 90))
+    (property "Footprint" "" (id 2) (at 165.1 124.46 0)
+      (effects (font (size 1.27 1.27)) hide)
+    )
+    (property "Datasheet" "~" (id 3) (at 165.1 124.46 0)
+      (effects (font (size 1.27 1.27)) hide)
+    )
+    (pin "1")
+    (pin "2")
+  )
+  (symbol (lib_id "Device:LED_Small") (at 157.48 107.95 180) (unit 1)
+    (in_bom yes) (on_board yes) (fields_autoplaced)
+    (property "Reference" "D?" (id 0) (at 157.4165 101.6 0))
+    (property "Value" "Red" (id 1) (at 157.4165 104.14 0))
+    (property "Footprint" "" (id 2) (at 157.48 107.95 90)
+      (effects (font (size 1.27 1.27)) hide)
+    )
+    (property "Datasheet" "~" (id 3) (at 157.48 107.95 90)
+      (effects (font (size 1.27 1.27)) hide)
+    )
+    (pin "1")
+    (pin "2")
   )
   (sheet (at 124.46 59.69) (size 27.94 77.47) (fields_autoplaced)
@@
       (effects (font (size 1.27 1.27)) (justify left))
     )
-    (pin "AFE_MISO" input (at 124.46 100.33 180)
-      (effects (font (size 1.27 1.27)) (justify left))
-    )
-    (pin "AFE_MOSI" output (at 124.46 97.79 180)
-      (effects (font (size 1.27 1.27)) (justify left))
-    )
-    (pin "AFE_SCLK" output (at 124.46 102.87 180)
-      (effects (font (size 1.27 1.27)) (justify left))
-    )
-    (pin "AFE_CS" output (at 124.46 105.41 180)
-      (effects (font (size 1.27 1.27)) (justify left))
+    (pin "AFE_MISO" input (at 124.46 77.47 180)
+      (effects (font (size 1.27 1.27)) (justify left))
+    )
+    (pin "AFE_MOSI" output (at 124.46 74.93 180)
+      (effects (font (size 1.27 1.27)) (justify left))
+    )
+    (pin "AFE_SCLK" output (at 124.46 80.01 180)
+      (effects (font (size 1.27 1.27)) (justify left))
+    )
+    (pin "AFE_CS" output (at 124.46 82.55 180)
+      (effects (font (size 1.27 1.27)) (justify left))
+    )
+    (pin "LED_RED" output (at 152.4 107.95 0)
+      (effects (font (size 1.27 1.27)) (justify right))
+    )
+    (pin "LED_GREEN" output (at 152.4 124.46 0)
+      (effects (font (size 1.27 1.27)) (justify right))
     )
   )
@@
       (effects (font (size 1.27 1.27)) (justify left))
     )
-    (pin "SDI" input (at 106.68 97.79 0)
-      (effects (font (size 1.27 1.27)) (justify right))
-    )
-    (pin "SDO" output (at 106.68 100.33 0)
-      (effects (font (size 1.27 1.27)) (justify right))
-    )
-    (pin "CS" input (at 106.68 105.41 0)
-      (effects (font (size 1.27 1.27)) (justify right))
-    )
-    (pin "SCK" input (at 106.68 102.87 0)
+    (pin "SDI" input (at 106.68 74.93 0)
+      (effects (font (size 1.27 1.27)) (justify right))
+    )
+    (pin "SDO" output (at 106.68 77.47 0)
+      (effects (font (size 1.27 1.27)) (justify right))
+    )
+    (pin "CS" input (at 106.68 82.55 0)
+      (effects (font (size 1.27 1.27)) (justify right))
+    )
+    (pin "SCK" input (at 106.68 80.01 0)
       (effects (font (size 1.27 1.27)) (justify right))
     )
@@
       (reference "#PWR038") (unit 1) (value "GND") (footprint "")
     )
+    (path "/67b76df2-8ce8-4dc6-bfe0-82a2412e7d29"
+      (reference "#PWR?") (unit 1) (value "GND") (footprint "")
+    )
+    (path "/853c3a08-c843-4b34-81c2-1d42d60076dc"
+      (reference "#PWR?") (unit 1) (value "GND") (footprint "")
+    )
     (path "/1c5935ea-6f80-435f-8ae1-741f5546f8d9/3d53b2c0-0ab8-418a-a174-d479fe6d5385"
       (reference "C1") (unit 1) (value "DNP") (footprint "Capacitor_SMD:C_0603_1608Metric")
@@
       (reference "C40") (unit 1) (value "2.2u") (footprint "")
     )
+    (path "/4fe5efad-76b7-4beb-a7a2-aa3d492ac76f"
+      (reference "D?") (unit 1) (value "Green") (footprint "")
+    )
+    (path "/e2704538-429c-4bfb-966d-1f0c6c110f6a"
+      (reference "D?") (unit 1) (value "Red") (footprint "")
+    )
     (path "/1c5935ea-6f80-435f-8ae1-741f5546f8d9/b6cbb8ea-1784-4059-9a07-19b7c70fa644"
       (reference "J1") (unit 1) (value "Conn_ARM_JTAG_SWD_10") (footprint "Connector_PinHeader_1.27mm:PinHeader_2x05_P1.27mm_Vertical_SMD")
@@
       (reference "R74") (unit 1) (value "33") (footprint "")
     )
+    (path "/00c1fef2-3215-41d1-9e45-4317a4aeb3fe"
+      (reference "R?") (unit 1) (value "220") (footprint "")
+    )
+    (path "/94457c82-22d1-458b-b4c4-6b45f4a4b8fd"
+      (reference "R?") (unit 1) (value "220") (footprint "")
+    )
     (path "/1c5935ea-6f80-435f-8ae1-741f5546f8d9/fd1a8cd8-06e9-4d52-af0e-ed2b061904eb"

Commit message: NTC sensors
Parts:
- removed D?: Green, symbol Device:LED_Small
- removed D?: Red, symbol Device:LED_Small
- removed R? (x2): 220, symbol Device:R_Small
Other:
- sheet MCU ports: added TEMP_0, TEMP_1, TEMP_2; removed LED_GREEN, LED_RED
- sheet Thermal ports: added TEMP_0, TEMP_1, TEMP_2; removed none

Commit message: Fix schematic
Other:
- sheet MCU ports: added none; removed TEMP_0, TEMP_1, TEMP_2
Changed lines of the file:
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@@
     (stroke (width 0) (type default) (color 0 0 0 0))
   )
-  (wire (pts (xy 71.12 58.42) (xy 124.46 58.42))
+  (wire (pts (xy 71.12 67.31) (xy 124.46 67.31))
     (stroke (width 0) (type default) (color 0 0 0 0))
   )
@@
     (stroke (width 0) (type default) (color 0 0 0 0))
   )
-  (wire (pts (xy 71.12 55.88) (xy 124.46 55.88))
+  (wire (pts (xy 71.12 64.77) (xy 124.46 64.77))
     (stroke (width 0) (type default) (color 0 0 0 0))
   )
@@
     (stroke (width 0) (type default) (color 0 0 0 0))
   )
-  (sheet (at 124.46 52.07) (size 27.94 85.09) (fields_autoplaced)
+  (sheet (at 124.46 62.23) (size 27.94 74.93) (fields_autoplaced)
     (stroke (width 0.1524) (type solid) (color 0 0 0 0))
     (fill (color 0 0 0 0.0000))
-    (property "Sheet name" "MCU" (id 0) (at 124.46 51.3584 0)
+    (property "Sheet name" "MCU" (id 0) (at 124.46 61.5184 0)
       (effects (font (size 1.27 1.27)) (justify left bottom))
     )
@@
       (effects (font (size 1.27 1.27)) (justify right))
     )
-    (pin "SCL" output (at 124.46 55.88 180)
-      (effects (font (size 1.27 1.27)) (justify left))
-    )
-    (pin "SDA" bidirectional (at 124.46 58.42 180)
+    (pin "SCL" output (at 124.46 64.77 180)
+      (effects (font (size 1.27 1.27)) (justify left))
+    )
+    (pin "SDA" bidirectional (at 124.46 67.31 180)
       (effects (font (size 1.27 1.27)) (justify left))
     )
@@
     )
     (pin "AFE_CS" output (at 124.46 82.55 180)
-      (effects (font (size 1.27 1.27)) (justify left))
-    )
-    (pin "TEMP_2" input (at 124.46 68.58 180)
-      (effects (font (size 1.27 1.27)) (justify left))
-    )
-    (pin "TEMP_0" input (at 124.46 63.5 180)
-      (effects (font (size 1.27 1.27)) (justify left))
-    )
-    (pin "TEMP_1" input (at 124.46 66.04 180)
       (effects (font (size 1.27 1.27)) (justify left))
     )
@@
       (reference "#PWR0104") (unit 1) (value "+3.3V") (footprint "")
     )
+    (path "/95476253-acbc-4b80-80be-f4a25f0f1538/fc1479f0-081a-4b3d-8813-844957f05f0a/581092af-1e76-44d7-837e-bd5acc6e1834"
+      (reference "#PWR?") (unit 1) (value "GND") (footprint "")
+    )
     (path "/95476253-acbc-4b80-80be-f4a25f0f1538/093546ac-4b32-4941-93d8-34442ea23c06/581092af-1e76-44d7-837e-bd5acc6e1834"
       (reference "#PWR?") (unit 1) (value "GND") (footprint "")
     )
-    (path "/95476253-acbc-4b80-80be-f4a25f0f1538/fc1479f0-081a-4b3d-8813-844957f05f0a/581092af-1e76-44d7-837e-bd5acc6e1834"
-      (reference "#PWR?") (unit 1) (value "GND") (footprint "")
-    )
     (path "/95476253-acbc-4b80-80be-f4a25f0f1538/ea0333f0-2b96-4936-8a1d-d23c72d3c285/581092af-1e76-44d7-837e-bd5acc6e1834"
       (reference "#PWR?") (unit 1) (value "GND") (footprint "")
@@
       (reference "C?") (unit 1) (value "10u") (footprint "")
     )
+    (path "/95476253-acbc-4b80-80be-f4a25f0f1538/093546ac-4b32-4941-93d8-34442ea23c06/31656d7d-9ae1-4c93-885b-4becbf380333"
+      (reference "C?") (unit 1) (value "10u") (footprint "")
+    )
     (path "/95476253-acbc-4b80-80be-f4a25f0f1538/ea0333f0-2b96-4936-8a1d-d23c72d3c285/31656d7d-9ae1-4c93-885b-4becbf380333"
       (reference "C?") (unit 1) (value "10u") (footprint "")
     )
-    (path "/95476253-acbc-4b80-80be-f4a25f0f1538/093546ac-4b32-4941-93d8-34442ea23c06/31656d7d-9ae1-4c93-885b-4becbf380333"
-      (reference "C?") (unit 1) (value "10u") (footprint "")
-    )
