File: hardware/vesc-bms.kicad_sch (KiCad schematic)
At the start: 0 parts

Commit message: Work on thermal
Parts:
- added J2: Load, symbol Connector_Generic:Conn_01x02
- added J3: Charger, symbol Connector_Generic:Conn_01x02
Other:
- added sheet Charger monitoring (charger_monitoring.kicad_sch)

Commit message: Fan ports
Connections:
- net GND: now reaches J3.2 (Pin_2)
Other:
- moved on the sheet: J3
Changed lines of the file:
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@@
+    (stroke (width 0) (type default))
+  )
+  (wire (pts (xy 46.99 66.04) (xy 46.99 67.31))
     (stroke (width 0) (type default))
   )
@@
   )
   (wire (pts (xy 199.39 80.01) (xy 233.68 80.01))
+    (stroke (width 0) (type default))
+  )
+  (wire (pts (xy 45.72 66.04) (xy 46.99 66.04))
     (stroke (width 0) (type default))
   )
@@
     )
   )
-  (symbol (lib_id "Connector_Generic:Conn_01x02") (at 40.64 68.58 0) (mirror y) (unit 1)
+  (symbol (lib_id "power:GND") (at 46.99 67.31 0) (unit 1)
+    (in_bom yes) (on_board yes) (dnp no) (fields_autoplaced)
+    (property "Reference" "#PWR064" (at 46.99 73.66 0)
+      (effects (font (size 1.27 1.27)) hide)
+    )
+    (property "Value" "GND" (at 46.99 72.39 0)
+      (effects (font (size 1.27 1.27)))
+    )
+    (property "Footprint" "" (at 46.99 67.31 0)
+      (effects (font (size 1.27 1.27)) hide)
+    )
+    (property "Datasheet" "" (at 46.99 67.31 0)
+      (effects (font (size 1.27 1.27)) hide)
+    )
+    (pin "1")
+    (instances
+      (project "vesc-bms"
+        (path "/3e668e3e-3e16-4665-a807-4735962c41d3"
+          (reference "#PWR064") (unit 1)
+        )
+      )
+    )
+  )
+  (symbol (lib_id "Connector_Generic:Conn_01x02") (at 40.64 63.5 0) (mirror y) (unit 1)
     (in_bom yes) (on_board yes) (dnp no)
-    (property "Reference" "J3" (at 41.91 63.5 0)
+    (property "Reference" "J3" (at 41.91 58.42 0)
       (effects (font (size 1.27 1.27)) (justify left))
     )
-    (property "Value" "Charger" (at 44.45 66.04 0)
+    (property "Value" "Charger" (at 44.45 60.96 0)
       (effects (font (size 1.27 1.27)) (justify left))
     )
-    (property "Footprint" "" (at 40.64 68.58 0)
+    (property "Footprint" "" (at 40.64 63.5 0)
       (effects (font (size 1.27 1.27)) hide)
     )
-    (property "Datasheet" "~" (at 40.64 68.58 0)
+    (property "Datasheet" "~" (at 40.64 63.5 0)
       (effects (font (size 1.27 1.27)) hide)
     )

Commit message: Charger monitor
Connections:
- net GND: now also J2.2 (Pin_2)
- net +BATT: now reaches J2.1 (Pin_1)
- net Charger monitoring/Chager+: now reaches J3.1 (Pin_1)
Other:
- sheet Charger monitoring ports: added Chager+, Charger_current; removed none
Changed lines of the file:
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@@
+    (stroke (width 0) (type default))
+  )
+  (wire (pts (xy 45.72 63.5) (xy 58.42 63.5))
     (stroke (width 0) (type default))
   )
@@
     (stroke (width 0) (type default))
   )
+  (wire (pts (xy 45.72 93.98) (xy 46.99 93.98))
+    (stroke (width 0) (type default))
+  )
   (wire (pts (xy 199.39 67.31) (xy 233.68 67.31))
     (stroke (width 0) (type default))
@@
   )
   (wire (pts (xy 199.39 64.77) (xy 233.68 64.77))
+    (stroke (width 0) (type default))
+  )
+  (wire (pts (xy 46.99 93.98) (xy 46.99 95.25))
     (stroke (width 0) (type default))
   )
@@
     )
   )
+  (symbol (lib_id "power:+BATT") (at 45.72 91.44 270) (unit 1)
+    (in_bom yes) (on_board yes) (dnp no) (fields_autoplaced)
+    (property "Reference" "#PWR070" (at 41.91 91.44 0)
+      (effects (font (size 1.27 1.27)) hide)
+    )
+    (property "Value" "+BATT" (at 49.53 92.075 90)
+      (effects (font (size 1.27 1.27)) (justify left))
+    )
+    (property "Footprint" "" (at 45.72 91.44 0)
+      (effects (font (size 1.27 1.27)) hide)
+    )
+    (property "Datasheet" "" (at 45.72 91.44 0)
+      (effects (font (size 1.27 1.27)) hide)
+    )
+    (pin "1")
+    (instances
+      (project "vesc-bms"
+        (path "/3e668e3e-3e16-4665-a807-4735962c41d3"
+          (reference "#PWR070") (unit 1)
+        )
+      )
+    )
+  )
   (symbol (lib_id "power:GND") (at 46.99 67.31 0) (unit 1)
     (in_bom yes) (on_board yes) (dnp no) (fields_autoplaced)
@@
     )
   )
+  (symbol (lib_id "power:GND") (at 46.99 95.25 0) (unit 1)
+    (in_bom yes) (on_board yes) (dnp no) (fields_autoplaced)
+    (property "Reference" "#PWR071" (at 46.99 101.6 0)
+      (effects (font (size 1.27 1.27)) hide)
+    )
+    (property "Value" "GND" (at 46.99 100.33 0)
+      (effects (font (size 1.27 1.27)))
+    )
+    (property "Footprint" "" (at 46.99 95.25 0)
+      (effects (font (size 1.27 1.27)) hide)
+    )
+    (property "Datasheet" "" (at 46.99 95.25 0)
+      (effects (font (size 1.27 1.27)) hide)
+    )
+    (pin "1")
+    (instances
+      (project "vesc-bms"
+        (path "/3e668e3e-3e16-4665-a807-4735962c41d3"
+          (reference "#PWR071") (unit 1)
+        )
+      )
+    )
+  )
   (symbol (lib_id "Connector_Generic:Conn_01x02") (at 40.64 63.5 0) (mirror y) (unit 1)
     (in_bom yes) (on_board yes) (dnp no)
@@
     )
   )
-  (sheet (at 58.42 57.15) (size 19.05 13.97) (fields_autoplaced)
+  (sheet (at 58.42 57.15) (size 31.75 13.97) (fields_autoplaced)
     (stroke (width 0.1524) (type solid))
     (fill (color 0 0 0 0.0000))
@@
       (effects (font (size 1.27 1.27)) hide)
     )
-    (instances
+    (pin "Charger_current" output (at 90.17 63.5 0)
+      (effects (font (size 1.27 1.27)) (justify right))
+    )
+    (pin "Chager+" input (at 58.42 63.5 180)
+      (effects (font (size 1.27 1.27)) (justify left))
+    )
+    (instances

Commit message: OLED screen
Parts:
- added J10: OLED, Connector_JST:JST_XH_B5B-XH-A_1x05_P2.50mm_Vertical, symbol Connector:Conn_01x05_Pin
Connections:
- net GND: now also J10.1 (Pin_1)
- net MCU/SCL: now also J10.2 (Pin_2)
- net MCU/SDA: now also J10.4 (Pin_4)
- new net +3.3V: J10.5 (Pin_5)
- new net MCU/OLED_RST: J10.3 (Pin_3)
Other:
- sheet MCU ports: added OLED_RST; removed none
Changed lines of the file:
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@@
 (kicad_sch (version 20230121) (generator eeschema)
   (paper "A4")
+  (junction (at 166.37 55.88) (diameter 0) (color 0 0 0 0)
+  )
+  (junction (at 165.1 53.34) (diameter 0) (color 0 0 0 0)
+  )
   (wire (pts (xy 118.11 63.5) (xy 137.16 63.5))
     (stroke (width 0) (type default))
   )
-  (wire (pts (xy 118.11 55.88) (xy 171.45 55.88))
+  (wire (pts (xy 118.11 55.88) (xy 166.37 55.88))
     (stroke (width 0) (type default))
   )
@@
     (stroke (width 0) (type default))
   )
+  (wire (pts (xy 165.1 33.02) (xy 179.07 33.02))
+    (stroke (width 0) (type default))
+  )
   (wire (pts (xy 45.72 63.5) (xy 58.42 63.5))
     (stroke (width 0) (type default))
@@
     (stroke (width 0) (type default))
   )
+  (wire (pts (xy 167.64 35.56) (xy 179.07 35.56))
+    (stroke (width 0) (type default))
+  )
   (wire (pts (xy 199.39 67.31) (xy 233.68 67.31))
     (stroke (width 0) (type default))
   )
+  (wire (pts (xy 166.37 55.88) (xy 171.45 55.88))
+    (stroke (width 0) (type default))
+  )
+  (wire (pts (xy 166.37 38.1) (xy 179.07 38.1))
+    (stroke (width 0) (type default))
+  )
   (wire (pts (xy 199.39 62.23) (xy 233.68 62.23))
     (stroke (width 0) (type default))
   )
+  (wire (pts (xy 167.64 58.42) (xy 167.64 35.56))
+    (stroke (width 0) (type default))
+  )
+  (wire (pts (xy 171.45 58.42) (xy 167.64 58.42))
+    (stroke (width 0) (type default))
+  )
   (wire (pts (xy 199.39 80.01) (xy 233.68 80.01))
     (stroke (width 0) (type default))
@@
     (stroke (width 0) (type default))
   )
-  (wire (pts (xy 118.11 53.34) (xy 171.45 53.34))
+  (wire (pts (xy 118.11 53.34) (xy 165.1 53.34))
     (stroke (width 0) (type default))
   )
@@
     (stroke (width 0) (type default))
   )
+  (wire (pts (xy 166.37 55.88) (xy 166.37 38.1))
+    (stroke (width 0) (type default))
+  )
   (wire (pts (xy 118.11 96.52) (xy 137.16 96.52))
     (stroke (width 0) (type default))
@@
     (stroke (width 0) (type default))
   )
+  (wire (pts (xy 165.1 53.34) (xy 171.45 53.34))
+    (stroke (width 0) (type default))
+  )
   (wire (pts (xy 46.99 93.98) (xy 46.99 95.25))
     (stroke (width 0) (type default))
@@
   (wire (pts (xy 118.11 68.58) (xy 137.16 68.58))
     (stroke (width 0) (type default))
+  )
+  (wire (pts (xy 165.1 53.34) (xy 165.1 33.02))
+    (stroke (width 0) (type default))
+  )
+  (symbol (lib_id "power:+3.3V") (at 179.07 40.64 90) (unit 1)
+    (in_bom yes) (on_board yes) (dnp no)
+    (property "Reference" "#PWR083" (at 182.88 40.64 0)
+      (effects (font (size 1.27 1.27)) hide)
+    )
+    (property "Value" "+3.3V" (at 175.26 40.64 90)
+      (effects (font (size 1.27 1.27)) (justify left))
+    )
+    (property "Footprint" "" (at 179.07 40.64 0)
+      (effects (font (size 1.27 1.27)) hide)
+    )
+    (property "Datasheet" "" (at 179.07 40.64 0)
+      (effects (font (size 1.27 1.27)) hide)
+    )
+    (pin "1")
+    (instances
+      (project "vesc-bms"
+        (path "/3e668e3e-3e16-4665-a807-4735962c41d3"
+          (reference "#PWR083") (unit 1)
+        )
+      )
+    )
   )
   (symbol (lib_id "Connector_Generic:Conn_01x02") (at 40.64 91.44 0) (mirror y) (unit 1)
@@
     )
   )
+  (symbol (lib_id "power:GND") (at 179.07 30.48 270) (unit 1)
+    (in_bom yes) (on_board yes) (dnp no)
+    (property "Reference" "#PWR082" (at 172.72 30.48 0)
+      (effects (font (size 1.27 1.27)) hide)
+    )
+    (property "Value" "GND" (at 175.26 30.48 90)
+      (effects (font (size 1.27 1.27)) (justify right))
+    )
+    (property "Footprint" "" (at 179.07 30.48 0)
+      (effects (font (size 1.27 1.27)) hide)
+    )
+    (property "Datasheet" "" (at 179.07 30.48 0)
+      (effects (font (size 1.27 1.27)) hide)
+    )
+    (pin "1")
+    (instances
+      (project "vesc-bms"
+        (path "/3e668e3e-3e16-4665-a807-4735962c41d3"
+          (reference "#PWR082") (unit 1)
+        )
+      )
+    )
+  )
   (symbol (lib_id "power:GND") (at 46.99 95.25 0) (unit 1)
     (in_bom yes) (on_board yes) (dnp no) (fields_autoplaced)
@@
         (path "/3e668e3e-3e16-4665-a807-4735962c41d3"
           (reference "#PWR071") (unit 1)
+        )
+      )
+    )
+  )
+  (symbol (lib_id "Connector:Conn_01x05_Pin") (at 184.15 35.56 0) (mirror y) (unit 1)
+    (in_bom yes) (on_board yes) (dnp no)
+    (property "Reference" "J10" (at 187.96 34.29 0)
+      (effects (font (size 1.27 1.27)))
+    )
+    (property "Value" "OLED" (at 187.96 36.83 0)
+      (effects (font (size 1.27 1.27)))
+    )
+    (property "Footprint" "Connector_JST:JST_XH_B5B-XH-A_1x05_P2.50mm_Vertical" (at 184.15 35.56 0)
+      (effects (font (size 1.27 1.27)) hide)
+    )
+    (property "Datasheet" "~" (at 184.15 35.56 0)
+      (effects (font (size 1.27 1.27)) hide)
+    )
+    (pin "1")
+    (pin "2")
+    (pin "3")
+    (pin "4")
+    (pin "5")
+    (instances
+      (project "vesc-bms"
+        (path "/3e668e3e-3e16-4665-a807-4735962c41d3"
+          (reference "J10") (unit 1)
         )
       )
@@
       (effects (font (size 1.27 1.27)) (justify left))
     )
+    (pin "OLED_RST" output (at 171.45 58.42 180)
+      (effects (font (size 1.27 1.27)) (justify left))
+    )
