File: hardware/afe.kicad_sch (KiCad schematic)
At the start: 1 part

Commit message: Define footprints
Parts:
- gave numbers to parts that had none: 1
Changed lines of the file:
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@@
   (symbol (lib_id "vesc-bms:LTC6813-1") (at 78.74 101.6 0) (unit 1)
     (in_bom yes) (on_board yes) (fields_autoplaced)
-    (property "Reference" "U?" (id 0) (at 80.7594 48.26 0)
+    (property "Reference" "U2" (id 0) (at 80.7594 48.26 0)
       (effects (font (size 1.27 1.27)) (justify left))
     )

Commit message: Added footprints and some LCSC part numbers
Parts:
- U2: LCSC (none) -> C2979142
Changed lines of the file:
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@@
+      (effects (font (size 1.27 1.27)) hide)
+    )
+    (property "LCSC" "C2979142" (id 4) (at 78.74 101.6 0)
       (effects (font (size 1.27 1.27)) hide)
     )

Commit message: Added bluetooth interface
Parts:
- added U?: BQ76200PW, Package_SO:TSSOP-16_4.4x5mm_P0.65mm, symbol Battery_Management:BQ76200PW
Changed lines of the file:
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@@
+    (pin "9")
+  )
+  (symbol (lib_id "Battery_Management:BQ76200PW") (at 208.28 64.77 0) (unit 1)
+    (in_bom yes) (on_board yes) (fields_autoplaced)
+    (property "Reference" "U?" (id 0) (at 210.2994 80.01 0)
+      (effects (font (size 1.27 1.27)) (justify left))
+    )
+    (property "Value" "BQ76200PW" (id 1) (at 210.2994 82.55 0)
+      (effects (font (size 1.27 1.27)) (justify left))
+    )
+    (property "Footprint" "Package_SO:TSSOP-16_4.4x5mm_P0.65mm" (id 2) (at 229.87 78.74 0)
+      (effects (font (size 1.27 1.27)) hide)
+    )
+    (property "Datasheet" "http://www.ti.com/lit/ds/symlink/bq76200.pdf" (id 3) (at 208.28 64.77 0)
+      (effects (font (size 1.27 1.27)) hide)
+    )
+    (pin "1")
+    (pin "10")
+    (pin "11")
+    (pin "12")
+    (pin "13")
+    (pin "14")
+    (pin "15")
+    (pin "16")
+    (pin "2")
+    (pin "3")
+    (pin "4")
+    (pin "5")
+    (pin "6")
+    (pin "7")
+    (pin "8")
     (pin "9")
   )

Commit message: Communication interfaces
Other:
- note added: "High-side enable/disable"
Changed lines of the file:
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@@
 (kicad_sch (version 20211123) (generator eeschema)
   (paper "A4")
+  (polyline (pts (xy 177.8 104.14) (xy 250.19 104.14))
+    (stroke (width 0) (type default) (color 0 0 0 0))
+  )
   (polyline (pts (xy 39.37 162.56) (xy 39.37 38.1))
     (stroke (width 0) (type default) (color 0 0 0 0))
@@
     (stroke (width 0) (type default) (color 0 0 0 0))
   )
+  (polyline (pts (xy 177.8 44.45) (xy 177.8 104.14))
+    (stroke (width 0) (type default) (color 0 0 0 0))
+  )
   (polyline (pts (xy 130.81 162.56) (xy 39.37 162.56))
     (stroke (width 0) (type default) (color 0 0 0 0))
   )
+  (polyline (pts (xy 177.8 44.45) (xy 250.19 44.45))
+    (stroke (width 0) (type default) (color 0 0 0 0))
+  )
+  (polyline (pts (xy 250.19 104.14) (xy 250.19 44.45))
+    (stroke (width 0) (type default) (color 0 0 0 0))
+  )
+  (text "High-side enable/disable" (at 179.07 41.91 0)
+    (effects (font (size 1.27 1.27)) (justify left bottom))
+  )
   (text "Analog Front-End" (at 40.64 36.83 0)

Commit message: BLE module
Parts:
- gave numbers to parts that had none: 1
Changed lines of the file:
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@@
   (symbol (lib_id "Battery_Management:BQ76200PW") (at 208.28 64.77 0) (unit 1)
     (in_bom yes) (on_board yes) (fields_autoplaced)
-    (property "Reference" "U?" (id 0) (at 210.2994 80.01 0)
+    (property "Reference" "U3" (id 0) (at 210.2994 80.01 0)
       (effects (font (size 1.27 1.27)) (justify left))
     )

Commit message: Some work on Battery AFE and PSU
Parts:
- added J?: Conn_01x19_Male, symbol Connector:Conn_01x19_Male
- added R?: 100, symbol Device:R_Small
- added R?: 20k, symbol Device:R_Small
- added R?: 5k, symbol Device:R_Small
Connections:
- net +BATT: now reaches U2.1 (V+)
- net +5V: now reaches U2.48 (VREG)
- net BALANCE_EN: now reaches U2.49 (DRIVE)
- net at U2.54 (SDO(NC)): now also R?.2
- net GND: now reaches U2.55 (ISOMD)
- net GND: now also R?.2
- net at U2.57 (IBIAS): now also U2.58 (ICMP), R?.1
- net at U2.63 (IMB): now also R?.1
- net at U2.64 (IPB): now also R?.2
- new net +3.3V: R?.1
Changed lines of the file:
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@@
 (kicad_sch (version 20211123) (generator eeschema)
   (paper "A4")
+  (junction (at 64.77 86.36) (diameter 0) (color 0 0 0 0)
+  )
   (polyline (pts (xy 177.8 104.14) (xy 250.19 104.14))
     (stroke (width 0) (type default) (color 0 0 0 0))
@@
     (stroke (width 0) (type default) (color 0 0 0 0))
   )
-  (polyline (pts (xy 39.37 38.1) (xy 130.81 38.1))
-    (stroke (width 0) (type default) (color 0 0 0 0))
-  )
-  (polyline (pts (xy 130.81 38.1) (xy 130.81 162.56))
+  (wire (pts (xy 54.61 96.52) (xy 54.61 99.06))
+    (stroke (width 0) (type default) (color 0 0 0 0))
+  )
+  (polyline (pts (xy 39.37 38.1) (xy 149.86 38.1))
+    (stroke (width 0) (type default) (color 0 0 0 0))
+  )
+  (wire (pts (xy 59.69 99.06) (xy 66.04 99.06))
+    (stroke (width 0) (type default) (color 0 0 0 0))
+  )
+  (wire (pts (xy 54.61 96.52) (xy 66.04 96.52))
+    (stroke (width 0) (type default) (color 0 0 0 0))
+  )
+  (polyline (pts (xy 149.86 38.1) (xy 149.86 162.56))
+    (stroke (width 0) (type default) (color 0 0 0 0))
+  )
+  (wire (pts (xy 46.99 86.36) (xy 64.77 86.36))
+    (stroke (width 0) (type default) (color 0 0 0 0))
+  )
+  (wire (pts (xy 64.77 86.36) (xy 66.04 86.36))
     (stroke (width 0) (type default) (color 0 0 0 0))
   )
@@
     (stroke (width 0) (type default) (color 0 0 0 0))
   )
-  (polyline (pts (xy 130.81 162.56) (xy 39.37 162.56))
+  (polyline (pts (xy 149.86 162.56) (xy 39.37 162.56))
+    (stroke (width 0) (type default) (color 0 0 0 0))
+  )
+  (wire (pts (xy 46.99 111.76) (xy 66.04 111.76))
+    (stroke (width 0) (type default) (color 0 0 0 0))
+  )
+  (wire (pts (xy 46.99 68.58) (xy 66.04 68.58))
+    (stroke (width 0) (type default) (color 0 0 0 0))
+  )
+  (wire (pts (xy 46.99 67.31) (xy 46.99 68.58))
     (stroke (width 0) (type default) (color 0 0 0 0))
   )
@@
     (stroke (width 0) (type default) (color 0 0 0 0))
   )
+  (wire (pts (xy 46.99 86.36) (xy 46.99 87.63))
+    (stroke (width 0) (type default) (color 0 0 0 0))
+  )
   (polyline (pts (xy 250.19 104.14) (xy 250.19 44.45))
+    (stroke (width 0) (type default) (color 0 0 0 0))
+  )
+  (wire (pts (xy 66.04 88.9) (xy 64.77 88.9))
+    (stroke (width 0) (type default) (color 0 0 0 0))
+  )
+  (wire (pts (xy 64.77 86.36) (xy 64.77 88.9))
+    (stroke (width 0) (type default) (color 0 0 0 0))
+  )
+  (wire (pts (xy 46.99 71.12) (xy 66.04 71.12))
+    (stroke (width 0) (type default) (color 0 0 0 0))
+  )
+  (wire (pts (xy 46.99 72.39) (xy 46.99 71.12))
+    (stroke (width 0) (type default) (color 0 0 0 0))
+  )
+  (wire (pts (xy 46.99 110.49) (xy 46.99 111.76))
     (stroke (width 0) (type default) (color 0 0 0 0))
   )
@@
   (text "Analog Front-End" (at 40.64 36.83 0)
     (effects (font (size 1.27 1.27)) (justify left bottom))
+  )
+  (hierarchical_label "BALANCE_EN" (shape input) (at 66.04 66.04 180)
+    (effects (font (size 1.27 1.27)) (justify right))
+  )
+  (symbol (lib_id "power:GND") (at 46.99 72.39 0) (unit 1)
+    (in_bom yes) (on_board yes) (fields_autoplaced)
+    (property "Reference" "#PWR?" (id 0) (at 46.99 78.74 0)
+      (effects (font (size 1.27 1.27)) hide)
+    )
+    (property "Value" "GND" (id 1) (at 46.99 77.47 0))
+    (property "Footprint" "" (id 2) (at 46.99 72.39 0)
+      (effects (font (size 1.27 1.27)) hide)
+    )
+    (property "Datasheet" "" (id 3) (at 46.99 72.39 0)
+      (effects (font (size 1.27 1.27)) hide)
+    )
+    (pin "1")
   )
   (symbol (lib_id "vesc-bms:LTC6813-1") (at 78.74 101.6 0) (unit 1)
@@
     (pin "9")
   )
+  (symbol (lib_id "Device:R_Small") (at 57.15 99.06 90) (unit 1)
+    (in_bom yes) (on_board yes)
+    (property "Reference" "R?" (id 0) (at 57.15 101.6 90))
+    (property "Value" "100" (id 1) (at 57.15 104.14 90))
+    (property "Footprint" "" (id 2) (at 57.15 99.06 0)
+      (effects (font (size 1.27 1.27)) hide)
+    )
+    (property "Datasheet" "~" (id 3) (at 57.15 99.06 0)
+      (effects (font (size 1.27 1.27)) hide)
+    )
+    (pin "1")
+    (pin "2")
+  )
   (symbol (lib_id "Battery_Management:BQ76200PW") (at 208.28 64.77 0) (unit 1)
     (in_bom yes) (on_board yes) (fields_autoplaced)
@@
     (pin "9")
   )
+  (symbol (lib_id "power:GND") (at 46.99 92.71 0) (unit 1)
+    (in_bom yes) (on_board yes) (fields_autoplaced)
+    (property "Reference" "#PWR?" (id 0) (at 46.99 99.06 0)
+      (effects (font (size 1.27 1.27)) hide)
+    )
+    (property "Value" "GND" (id 1) (at 46.99 97.79 0))
+    (property "Footprint" "" (id 2) (at 46.99 92.71 0)
+      (effects (font (size 1.27 1.27)) hide)
+    )
+    (property "Datasheet" "" (id 3) (at 46.99 92.71 0)
+      (effects (font (size 1.27 1.27)) hide)
+    )
+    (pin "1")
+  )
+  (symbol (lib_id "power:+BATT") (at 78.74 50.8 0) (unit 1)
+    (in_bom yes) (on_board yes) (fields_autoplaced)
+    (property "Reference" "#PWR?" (id 0) (at 78.74 54.61 0)
+      (effects (font (size 1.27 1.27)) hide)
+    )
+    (property "Value" "+BATT" (id 1) (at 78.74 45.72 0))
+    (property "Footprint" "" (id 2) (at 78.74 50.8 0)
+      (effects (font (size 1.27 1.27)) hide)
+    )
+    (property "Datasheet" "" (id 3) (at 78.74 50.8 0)
+      (effects (font (size 1.27 1.27)) hide)
+    )
+    (pin "1")
+  )
+  (symbol (lib_id "power:+5V") (at 46.99 67.31 0) (unit 1)
+    (in_bom yes) (on_board yes) (fields_autoplaced)
+    (property "Reference" "#PWR?" (id 0) (at 46.99 71.12 0)
+      (effects (font (size 1.27 1.27)) hide)
+    )
+    (property "Value" "+5V" (id 1) (at 46.99 62.23 0))
+    (property "Footprint" "" (id 2) (at 46.99 67.31 0)
+      (effects (font (size 1.27 1.27)) hide)
+    )
+    (property "Datasheet" "" (id 3) (at 46.99 67.31 0)
+      (effects (font (size 1.27 1.27)) hide)
+    )
+    (pin "1")
+  )
+  (symbol (lib_id "Connector:Conn_01x19_Male") (at 138.43 104.14 180) (unit 1)
+    (in_bom yes) (on_board yes) (fields_autoplaced)
+    (property "Reference" "J?" (id 0) (at 139.7 102.8699 0)
+      (effects (font (size 1.27 1.27)) (justify right))
+    )
+    (property "Value" "Conn_01x19_Male" (id 1) (at 139.7 105.4099 0)
+      (effects (font (size 1.27 1.27)) (justify right))
+    )
+    (property "Footprint" "" (id 2) (at 138.43 104.14 0)
+      (effects (font (size 1.27 1.27)) hide)
+    )
+    (property "Datasheet" "~" (id 3) (at 138.43 104.14 0)
+      (effects (font (size 1.27 1.27)) hide)
+    )
+    (pin "1")
+    (pin "10")
+    (pin "11")
+    (pin "12")
+    (pin "13")
+    (pin "14")
+    (pin "15")
+    (pin "16")
+    (pin "17")
+    (pin "18")
+    (pin "19")
+    (pin "2")
+    (pin "3")
+    (pin "4")
+    (pin "5")
+    (pin "6")
+    (pin "7")
+    (pin "8")
+    (pin "9")
+  )
+  (symbol (lib_id "Device:R_Small") (at 46.99 90.17 0) (unit 1)
+    (in_bom yes) (on_board yes) (fields_autoplaced)
+    (property "Reference" "R?" (id 0) (at 49.53 88.8999 0)
+      (effects (font (size 1.27 1.27)) (justify left))
+    )
+    (property "Value" "20k" (id 1) (at 49.53 91.4399 0)
+      (effects (font (size 1.27 1.27)) (justify left))
+    )
+    (property "Footprint" "" (id 2) (at 46.99 90.17 0)
+      (effects (font (size 1.27 1.27)) hide)
+    )
+    (property "Datasheet" "~" (id 3) (at 46.99 90.17 0)
+      (effects (font (size 1.27 1.27)) hide)
+    )
+    (pin "1")
+    (pin "2")
+  )
+  (symbol (lib_id "Device:R_Small") (at 46.99 107.95 0) (unit 1)
+    (in_bom yes) (on_board yes) (fields_autoplaced)
+    (property "Reference" "R?" (id 0) (at 49.53 106.6799 0)
+      (effects (font (size 1.27 1.27)) (justify left))
+    )
+    (property "Value" "5k" (id 1) (at 49.53 109.2199 0)
+      (effects (font (size 1.27 1.27)) (justify left))
+    )
+    (property "Footprint" "" (id 2) (at 46.99 107.95 0)
+      (effects (font (size 1.27 1.27)) hide)
+    )
+    (property "Datasheet" "~" (id 3) (at 46.99 107.95 0)
+      (effects (font (size 1.27 1.27)) hide)
+    )
+    (pin "1")
+    (pin "2")
+  )
+  (symbol (lib_id "power:+3.3V") (at 46.99 105.41 0) (unit 1)
+    (in_bom yes) (on_board yes) (fields_autoplaced)
+    (property "Reference" "#PWR?" (id 0) (at 46.99 109.22 0)
+      (effects (font (size 1.27 1.27)) hide)
+    )
+    (property "Value" "+3.3V" (id 1) (at 46.99 100.33 0))
+    (property "Footprint" "" (id 2) (at 46.99 105.41 0)
+      (effects (font (size 1.27 1.27)) hide)
+    )
+    (property "Datasheet" "" (id 3) (at 46.99 105.41 0)
+      (effects (font (size 1.27 1.27)) hide)
+    )
+    (pin "1")
+  )
 )

Commit message: Balance frontend
Parts:
- added C? (x19): C_Small, symbol Device:C_Small
- added R?: 100, symbol Device:R_Small
Connections:
- net GND: now also J?.1 (Pin_1), C?.2, R?.1
- net balance_front_end6/CELL_FILTERED: now reaches U2.10 (C14)
- net balance_front_end6/CELL_FILTERED: now also C?.1, C?.2
- net balance_front_end6/DISCHARGE_EN: now reaches U2.11 (S14)
- net balance_front_end5/CELL_FILTERED: now reaches U2.12 (C13)
- net balance_front_end5/CELL_FILTERED: now also C?.1, C?.2
- net balance_front_end5/DISCHARGE_EN: now reaches U2.13 (S13)
- net balance_front_end4/CELL_FILTERED: now reaches U2.14 (C12)
- net balance_front_end4/CELL_FILTERED: now also C?.1, C?.2
- net balance_front_end4/DISCHARGE_EN: now reaches U2.15 (S12)
- net balance_front_end10/CELL_FILTERED: now reaches U2.16 (C11)
- net balance_front_end10/CELL_FILTERED: now also C?.1, C?.2
- net balance_front_end10/DISCHARGE_EN: now reaches U2.17 (S11)
- net balance_front_end9/CELL_FILTERED: now reaches U2.18 (C10)
- net balance_front_end9/CELL_FILTERED: now also C?.1, C?.2
- net balance_front_end9/DISCHARGE_EN: now reaches U2.19 (S10)
- net balance_front_end/CELL_FILTERED: now reaches U2.2 (C18)
- net balance_front_end/CELL_FILTERED: now also C?.1
- net balance_front_end7/CELL_FILTERED: now reaches U2.20 (C9)
- net balance_front_end7/CELL_FILTERED: now also C?.1, C?.2
- net balance_front_end7/DISCHARGE_EN: now reaches U2.21 (S9)
- net balance_front_end11/CELL_FILTERED: now reaches U2.22 (C8)
- net balance_front_end11/CELL_FILTERED: now also C?.1, C?.2
- net balance_front_end11/DISCHARGE_EN: now reaches U2.23 (S8)
- net balance_front_end12/CELL_FILTERED: now reaches U2.24 (C7)
- net balance_front_end12/CELL_FILTERED: now also C?.1, C?.2
- net balance_front_end12/DISCHARGE_EN: now reaches U2.25 (S7)
- net balance_front_end8/CELL_FILTERED: now reaches U2.26 (C6)
- net balance_front_end8/CELL_FILTERED: now also C?.1, C?.2
- net balance_front_end8/DISCHARGE_EN: now reaches U2.27 (S6)
- net balance_front_end13/CELL_FILTERED: now reaches U2.28 (C5)
- net balance_front_end13/CELL_FILTERED: now also C?.1, C?.2
- net balance_front_end13/DISCHARGE_EN: now reaches U2.29 (S5)
- net balance_front_end/DISCHARGE_EN: now reaches U2.3 (S18)
- net balance_front_end16/CELL_FILTERED: now reaches U2.30 (C4)
- net balance_front_end16/CELL_FILTERED: now also C?.1, C?.2
- net balance_front_end16/DISCHARGE_EN: now reaches U2.31 (S4)
- net balance_front_end14/CELL_FILTERED: now reaches U2.32 (C3)
- net balance_front_end14/CELL_FILTERED: now also C?.1, C?.2
- net balance_front_end14/DISCHARGE_EN: now reaches U2.33 (S3)
- net balance_front_end15/CELL_FILTERED: now reaches U2.34 (C2)
- net balance_front_end15/CELL_FILTERED: now also C?.1, C?.2
- net balance_front_end15/DISCHARGE_EN: now reaches U2.35 (S2)
- net balance_front_end17/CELL_FILTERED: now reaches U2.36 (C1)
- net balance_front_end17/CELL_FILTERED: now also C?.1, C?.2
- net balance_front_end17/DISCHARGE_EN: now reaches U2.37 (S1)
- net at U2.38 (C0): now also C?.1, C?.2, R?.2
- net balance_front_end1/CELL_FILTERED: now reaches U2.4 (C17)
- net balance_front_end1/CELL_FILTERED: now also C?.1, C?.2
- net balance_front_end1/DISCHARGE_EN: now reaches U2.5 (S17)
- net balance_front_end2/CELL_FILTERED: now reaches U2.6 (C16)
- net balance_front_end2/CELL_FILTERED: now also C?.1, C?.2
- net balance_front_end2/DISCHARGE_EN: now reaches U2.7 (S16)
- net balance_front_end3/CELL_FILTERED: now reaches U2.8 (C15)
- net balance_front_end3/CELL_FILTERED: now also C?.1, C?.2
- net balance_front_end3/DISCHARGE_EN: now reaches U2.9 (S15)
- net balance_front_end7/CELL: now reaches J?.10 (Pin_10)
- net balance_front_end10/CELL-1: now reaches J?.11 (Pin_11)
- net balance_front_end10/CELL: now reaches J?.12 (Pin_12)
- net balance_front_end4/CELL: now reaches J?.13 (Pin_13)
- net balance_front_end5/CELL: now reaches J?.14 (Pin_14)
- net balance_front_end3/CELL-1: now reaches J?.15 (Pin_15)
- net balance_front_end2/CELL-1: now reaches J?.16 (Pin_16)
- net balance_front_end1/CELL-1: now reaches J?.17 (Pin_17)
- net balance_front_end/CELL-1: now reaches J?.18 (Pin_18)
- net balance_front_end/CELL: now reaches J?.19 (Pin_19)
- net balance_front_end15/CELL-1: now reaches J?.2 (Pin_2)
- net balance_front_end14/CELL-1: now reaches J?.3 (Pin_3)
- net balance_front_end14/CELL: now reaches J?.4 (Pin_4)
- net balance_front_end13/CELL-1: now reaches J?.5 (Pin_5)
- net balance_front_end13/CELL: now reaches J?.6 (Pin_6)
- net balance_front_end12/CELL-1: now reaches J?.7 (Pin_7)
- net balance_front_end11/CELL-1: now reaches J?.8 (Pin_8)
- net balance_front_end11/CELL: now reaches J?.9 (Pin_9)
Other:
- added sheet balance_front_end (balance_front_end.kicad_sch)
- added sheet balance_front_end1 (balance_front_end.kicad_sch)
- added sheet balance_front_end10 (balance_front_end.kicad_sch)
- added sheet balance_front_end11 (balance_front_end.kicad_sch)
- added sheet balance_front_end12 (balance_front_end.kicad_sch)
- added sheet balance_front_end13 (balance_front_end.kicad_sch)
- added sheet balance_front_end14 (balance_front_end.kicad_sch)
- added sheet balance_front_end15 (balance_front_end.kicad_sch)
- added sheet balance_front_end16 (balance_front_end.kicad_sch)
- added sheet balance_front_end17 (balance_front_end.kicad_sch)
- added sheet balance_front_end2 (balance_front_end.kicad_sch)
- added sheet balance_front_end3 (balance_front_end.kicad_sch)
- added sheet balance_front_end4 (balance_front_end.kicad_sch)
- added sheet balance_front_end5 (balance_front_end.kicad_sch)
- added sheet balance_front_end6 (balance_front_end.kicad_sch)
- added sheet balance_front_end7 (balance_front_end.kicad_sch)
- added sheet balance_front_end8 (balance_front_end.kicad_sch)
- added sheet balance_front_end9 (balance_front_end.kicad_sch)
- moved on the sheet: J?, U3

Commit message: Analog front end daisy chain
Parts:
- added C11, C12, C13, C14, C15, C16, C? (x2): DNP, symbol Device:C_Small
- added J2, J3: DNP, symbol Connector:Screw_Terminal_01x02
- added R11, R3, R4, R5, R6, R8: DNP, symbol Device:R_Small
- added R13, R9: 0, symbol Device:R_Small
- added TR?: DNP, Transformer_SMD:Transformer_Ethernet_Bourns_PT61017PEL, symbol vesc-bms:HM2102NLT
- C17, C18, C19, C20, C21, C22, C23, C24, C25, C26, C27, C28, C29, C30, C31, C32, C33, C34, C35: renamed from C?; value C_Small -> 10n
- gave numbers to parts that had none: 5
Connections:
- net +5V: now also R11.1
- net GND: now also R10.1, U2.59 (V-), U2.60 (V-), C11.2, C12.2, C?.2, C?.2, R9.2; no longer R10.2, U2.55 (ISOMD)
- net SDI: now reaches U2.53 (SDI(NC))
- net SDO: now reaches R12.2, U2.54 (SDO(NC))
- net CS: now reaches U2.61 (CSB(IMA))
- net CS: now also C15.1, R5.2, R8.2, TR?.14 (TX-)
- net SCK: now reaches U2.62 (SCK(IPA))
- net SCK: now also C16.2, R6.2, R8.1, TR?.16 (TX+)
- net at U2.63 (IMB): now also R7.2, C13.1, R3.2, TR?.9 (RX-); no longer R7.1
- net at U2.64 (IPB): now also R7.1, C14.2, R4.2, TR?.11 (RX+); no longer R7.2
- new net: C?.1, TR?.10 (C_RX)
- new net: R11.2, R9.1, U2.55 (ISOMD)
- new net: C12.1, C15.2, C16.1, R5.1, R6.1
- new net: R13.1, U2.57 (IBIAS)
- new net: R10.2, R13.2, U2.58 (ICMP)
- new net: J3.1 (Pin_1), TR?.1 (TD+)
- new net: C?.1, TR?.15 (C_TX)
- new net: J3.2 (Pin_2), TR?.3 (TD-)
- new net: J2.1 (Pin_1), TR?.6 (RD+)
- new net: J2.2 (Pin_2), TR?.8 (RD-)
- new net: C11.1, C13.2, C14.1, R3.1, R4.1
- no-connect marks 0 -> 3
Other:
- moved on the sheet: C17, C18, C19, C20, C21, C22, C23, C24, C25, C26, C27, C28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
