File: hardware/afe.kicad_sch (KiCad schematic)
At the start: 45 parts, among them J2 DNP, J3 DNP, J4 Conn_01x19_Male, U2 LTC6813-1, U3 BQ76200PW

Commit message: Analog front end ready
Parts:
- added C11, C12: 1u, symbol Device:C_Small
- added R3: DNP, symbol Device:R_Small
- added R4: 0, symbol Device:R_Small
- gave numbers to parts that had none: 3
- renumbered C11 to C15, C12 to C16, C13 to C17, C14 to C18, C15 to C19, C16 to C20, C17 to C21, C18 to C22, C19 to C23, C20 to C24, C21 to C25, C22 to C26, C23 to C27, C24 to C28, C25 to C29, C26 to C30, C27 to C31, C28 to C32, C29 to C33, C30 to C34, C31 to C35, C32 to C36, C33 to C37, C34 to C38, C35 to C39, R8 to R10, R9 to R11, R10 to R12, R11 to R13, R12 to R14, R13 to R15, R14 to R16, R3 to R5, R4 to R6, R5 to R7, R6 to R8, R7 to R9, U3 to U2, U2 to U3
Connections:
- net +5V: now also R3.1
- net GND: now also C11.1, C12.1, R4.2
- net GPIO1: now reaches U3.39 (GPIO1)
- net GPIO2: now reaches U3.40 (GPIO2)
- net GPIO3: now reaches U3.41 (GPIO3)
- net GPIO4: now reaches U3.42 (GPIO4)
- net GPIO5: now reaches U3.43 (GPIO5)
- net GPIO6: now reaches U3.44 (GPIO6)
- net GPIO7: now reaches U3.45 (GPIO7)
- net GPIO8: now reaches U3.46 (GPIO8)
- net GPIO9: now reaches U3.47 (GPIO9)
- net at U3.50 (VREF2): now also C12.2
- net at U3.51 (VREF1): now also C11.2
- net at U3.52 (DTEN): now also R3.2, R4.1
Other:
- moved on the sheet: R13

Commit message: NTC sensors
Parts:
- C11, C12, C13, C14, C15, C16, C17, C18, C19, C20, C21, C22, C23, C24, C25, C26, C27, C28, C29, C30, C31, C32, C33, C34, C35, C36, C37, C38, C39: footprint (none) -> Capacitor_SMD:C_0603_1608Metric
- renumbered R8 to R10, R9 to R11, R10 to R12, R11 to R13, R12 to R14, R13 to R15, R14 to R16, R15 to R17, R16 to R18, R3 to R5, R4 to R6, R5 to R7, R6 to R8, R7 to R9

Commit message: Annotate schematic
Parts:
- renumbered R8 to R10, R9 to R11, R10 to R12, R11 to R13, R12 to R14, R13 to R15, R14 to R16, R15 to R17, R16 to R18, R17 to R19, R18 to R20, R5 to R7, R6 to R8, R7 to R9
Changed lines of the file:
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@@
   (symbol (lib_id "Device:R_Small") (at 139.7 52.07 0) (unit 1)
     (in_bom yes) (on_board yes) (fields_autoplaced)
-    (property "Reference" "R15" (id 0) (at 142.24 50.7999 0)
+    (property "Reference" "R17" (id 0) (at 142.24 50.7999 0)
       (effects (font (size 1.27 1.27)) (justify left))
     )
@@
   (symbol (lib_id "power:GND") (at 129.54 54.61 0) (unit 1)
     (in_bom yes) (on_board yes)
-    (property "Reference" "#PWR022" (id 0) (at 129.54 60.96 0)
+    (property "Reference" "#PWR024" (id 0) (at 129.54 60.96 0)
       (effects (font (size 1.27 1.27)) hide)
     )
@@
   (symbol (lib_id "Device:R_Small") (at 119.38 100.33 180) (unit 1)
     (in_bom yes) (on_board yes)
-    (property "Reference" "R9" (id 0) (at 115.57 99.06 0))
+    (property "Reference" "R11" (id 0) (at 115.57 99.06 0))
     (property "Value" "DNP" (id 1) (at 115.57 101.6 0))
     (property "Footprint" "" (id 2) (at 119.38 100.33 0)
@@
   (symbol (lib_id "power:GND") (at 83.82 69.85 0) (unit 1)
     (in_bom yes) (on_board yes)
-    (property "Reference" "#PWR017" (id 0) (at 83.82 76.2 0)
+    (property "Reference" "#PWR019" (id 0) (at 83.82 76.2 0)
       (effects (font (size 1.27 1.27)) hide)
     )
@@
   (symbol (lib_id "Device:R_Small") (at 119.38 111.76 0) (unit 1)
     (in_bom yes) (on_board yes)
-    (property "Reference" "R10" (id 0) (at 115.57 110.49 0))
+    (property "Reference" "R12" (id 0) (at 115.57 110.49 0))
     (property "Value" "DNP" (id 1) (at 115.57 113.03 0))
     (property "Footprint" "" (id 2) (at 119.38 111.76 0)
@@
   (symbol (lib_id "power:GND") (at 113.03 53.34 0) (unit 1)
     (in_bom yes) (on_board yes)
-    (property "Reference" "#PWR020" (id 0) (at 113.03 59.69 0)
+    (property "Reference" "#PWR022" (id 0) (at 113.03 59.69 0)
       (effects (font (size 1.27 1.27)) hide)
     )
@@
   (symbol (lib_id "Device:R_Small") (at 124.46 105.41 180) (unit 1)
     (in_bom yes) (on_board yes)
-    (property "Reference" "R12" (id 0) (at 128.27 104.14 0))
+    (property "Reference" "R14" (id 0) (at 128.27 104.14 0))
     (property "Value" "DNP" (id 1) (at 128.27 106.68 0))
     (property "Footprint" "" (id 2) (at 124.46 105.41 0)
@@
   (symbol (lib_id "Device:R_Small") (at 124.46 78.74 180) (unit 1)
     (in_bom yes) (on_board yes)
-    (property "Reference" "R11" (id 0) (at 128.27 77.47 0))
+    (property "Reference" "R13" (id 0) (at 128.27 77.47 0))
     (property "Value" "100" (id 1) (at 128.27 80.01 0))
     (property "Footprint" "" (id 2) (at 124.46 78.74 0)
@@
   (symbol (lib_id "Device:R_Small") (at 236.22 125.73 90) (unit 1)
     (in_bom yes) (on_board yes)
-    (property "Reference" "R18" (id 0) (at 236.22 120.65 90))
+    (property "Reference" "R20" (id 0) (at 236.22 120.65 90))
     (property "Value" "100" (id 1) (at 236.22 123.19 90))
     (property "Footprint" "" (id 2) (at 236.22 125.73 0)
@@
   (symbol (lib_id "power:GND") (at 133.35 68.58 0) (unit 1)
     (in_bom yes) (on_board yes)
-    (property "Reference" "#PWR023" (id 0) (at 133.35 74.93 0)
+    (property "Reference" "#PWR025" (id 0) (at 133.35 74.93 0)
       (effects (font (size 1.27 1.27)) hide)
     )
@@
   (symbol (lib_id "power:+BATT") (at 163.83 31.75 0) (unit 1)
     (in_bom yes) (on_board yes) (fields_autoplaced)
-    (property "Reference" "#PWR025" (id 0) (at 163.83 35.56 0)
+    (property "Reference" "#PWR027" (id 0) (at 163.83 35.56 0)
       (effects (font (size 1.27 1.27)) hide)
     )
@@
   (symbol (lib_id "power:GND") (at 99.06 110.49 0) (unit 1)
     (in_bom yes) (on_board yes)
-    (property "Reference" "#PWR018" (id 0) (at 99.06 116.84 0)
+    (property "Reference" "#PWR020" (id 0) (at 99.06 116.84 0)
       (effects (font (size 1.27 1.27)) hide)
     )
@@
   (symbol (lib_id "Device:R_Small") (at 135.89 54.61 270) (unit 1)
     (in_bom yes) (on_board yes)
-    (property "Reference" "R13" (id 0) (at 132.08 50.8 90))
+    (property "Reference" "R15" (id 0) (at 132.08 50.8 90))
     (property "Value" "0" (id 1) (at 132.08 53.34 90))
     (property "Footprint" "" (id 2) (at 135.89 54.61 0)
@@
   (symbol (lib_id "power:+5V") (at 129.54 48.26 0) (unit 1)
     (in_bom yes) (on_board yes) (fields_autoplaced)
-    (property "Reference" "#PWR021" (id 0) (at 129.54 52.07 0)
+    (property "Reference" "#PWR023" (id 0) (at 129.54 52.07 0)
       (effects (font (size 1.27 1.27)) hide)
     )
@@
   (symbol (lib_id "Device:R_Small") (at 113.03 50.8 0) (unit 1)
     (in_bom yes) (on_board yes) (fields_autoplaced)
-    (property "Reference" "R6" (id 0) (at 115.57 49.5299 0)
+    (property "Reference" "R8" (id 0) (at 115.57 49.5299 0)
       (effects (font (size 1.27 1.27)) (justify left))
     )
@@
   (symbol (lib_id "Device:R_Small") (at 146.05 69.85 270) (unit 1)
     (in_bom yes) (on_board yes)
-    (property "Reference" "R17" (id 0) (at 146.05 72.39 90))
+    (property "Reference" "R19" (id 0) (at 146.05 72.39 90))
     (property "Value" "0" (id 1) (at 146.05 74.93 90))
     (property "Footprint" "" (id 2) (at 146.05 69.85 0)
@@
   (symbol (lib_id "power:GND") (at 101.6 85.09 0) (unit 1)
     (in_bom yes) (on_board yes)
-    (property "Reference" "#PWR019" (id 0) (at 101.6 91.44 0)
+    (property "Reference" "#PWR021" (id 0) (at 101.6 91.44 0)
       (effects (font (size 1.27 1.27)) hide)
     )
@@
   (symbol (lib_id "Device:R_Small") (at 138.43 67.31 90) (unit 1)
     (in_bom yes) (on_board yes)
-    (property "Reference" "R14" (id 0) (at 138.43 69.85 90))
+    (property "Reference" "R16" (id 0) (at 138.43 69.85 90))
     (property "Value" "20k" (id 1) (at 138.43 72.39 90))
     (property "Footprint" "" (id 2) (at 138.43 67.31 0)
@@
   (symbol (lib_id "Device:R_Small") (at 142.24 93.98 90) (unit 1)
     (in_bom yes) (on_board yes)
-    (property "Reference" "R16" (id 0) (at 142.24 96.52 90))
+    (property "Reference" "R18" (id 0) (at 142.24 96.52 90))
     (property "Value" "5k" (id 1) (at 142.24 99.06 90))
     (property "Footprint" "" (id 2) (at 142.24 93.98 0)
@@
   (symbol (lib_id "Device:R_Small") (at 119.38 85.09 0) (unit 1)
     (in_bom yes) (on_board yes)
-    (property "Reference" "R8" (id 0) (at 115.57 83.82 0))
+    (property "Reference" "R10" (id 0) (at 115.57 83.82 0))
     (property "Value" "DNP" (id 1) (at 115.57 86.36 0))
     (property "Footprint" "" (id 2) (at 119.38 85.09 0)
@@
   (symbol (lib_id "Device:R_Small") (at 119.38 73.66 180) (unit 1)
     (in_bom yes) (on_board yes)
-    (property "Reference" "R7" (id 0) (at 115.57 72.39 0))
+    (property "Reference" "R9" (id 0) (at 115.57 72.39 0))
     (property "Value" "DNP" (id 1) (at 115.57 74.93 0))
     (property "Footprint" "" (id 2) (at 119.38 73.66 0)
@@
   (symbol (lib_id "power:GND") (at 163.83 137.16 0) (unit 1)
     (in_bom yes) (on_board yes) (fields_autoplaced)
-    (property "Reference" "#PWR026" (id 0) (at 163.83 143.51 0)
+    (property "Reference" "#PWR028" (id 0) (at 163.83 143.51 0)
       (effects (font (size 1.27 1.27)) hide)
     )
@@
   (symbol (lib_id "power:+3.3V") (at 138.43 93.98 0) (unit 1)
     (in_bom yes) (on_board yes)
-    (property "Reference" "#PWR024" (id 0) (at 138.43 97.79 0)
+    (property "Reference" "#PWR026" (id 0) (at 138.43 97.79 0)
       (effects (font (size 1.27 1.27)) hide)
     )
@@
   (symbol (lib_id "Device:R_Small") (at 113.03 43.18 0) (unit 1)
     (in_bom yes) (on_board yes) (fields_autoplaced)
-    (property "Reference" "R5" (id 0) (at 115.57 41.9099 0)
-      (effects (font (size 1.27 1.27)) (justify left))
-    )
+    (property "Reference" "R7" (id 0) (at 115.57 41.9099 0)
+      (effects (font (size 1.27 1.27)) (justify left))
+    )

Commit message: MicroFit 3.0 for battery connector
Parts:
- J4: footprint (none) -> Connector_Molex:Molex_Micro-Fit_3.0_43045-2000_2x10_P3.00mm_Horizontal
Changed lines of the file:
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@@
       (effects (font (size 1.27 1.27)) (justify right))
     )
-    (property "Footprint" "" (id 2) (at 238.76 85.09 0)
+    (property "Footprint" "Connector_Molex:Molex_Micro-Fit_3.0_43045-2000_2x10_P3.00mm_Horizontal" (id 2) (at 238.76 85.09 0)
       (effects (font (size 1.27 1.27)) hide)
     )

Commit message: Current sensor
Parts:
- added C? (x2): 100n, symbol Device:C_Small
- added R?: 2.7k, symbol Device:R_Small
- added U?: ACS758xCB-050B-PFF, Sensor_Current:Allegro_CB_PFF, symbol Sensor_Current:ACS758xCB-050B-PFF
Connections:
- net +3.3V: now also C?.1, U?.1 (VCC)
- net GND: now also C?.2, C?.2, U?.2 (GND), U?.4 (IP+)
- new net: R?.1, U?.3 (VIOUT)
- new net -BATT: U?.5 (IP-)
- new net Current_sensor: C?.1, R?.2
Other:
- note added: "Total current sensing"
- moved on the sheet: U2

Commit message: DNP marks from new KiCAD
Parts:
- removed J2, J3: DNP, symbol Connector:Screw_Terminal_01x02
- removed R14: DNP, symbol Device:R_Small
- added C44: 100n, symbol Device:C_Small
- added J8, J9: RJ45, symbol Connector:RJ45
- added Q21: MMBT3904, Package_TO_SOT_SMD:SOT-23, symbol Transistor_BJT:MMBT3904
- C13, C14, C15, C16: value DNP -> 10n; now not fitted
- C17, C18, C19, C20: value DNP -> 100p; now not fitted
- R10, R11, R12, R9: value DNP -> 50
- R17, R7: value DNP -> 0; now not fitted
- TR1: value DNP -> HM2102NLT; now not fitted
Connections:
- net +5V: now also R13.1; no longer R17.1, R7.1, U3.48 (VREG)
- net GND: now also C44.2
- net at C17.1, R9.2, TR1.9 (RX-)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: no longer R13.2
- net at C18.2, R10.2, TR1.11 (RX+)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: no longer R13.1
- net BALANCE_EN: no longer names the net of U3.49 (DRIVE)
- net BALANCE_EN: now also Q21.1 (B)
- new net: Q21.3 (C), R13.2
- new net VREG: C44.1, Q21.2 (E), R17.1, R7.1, U3.48 (VREG)
Other:
- moved on the sheet: C11, C12, R10, R11, R12, R15, R16, R8, R9

Commit message: Work on thermal
Parts:
- removed C? (x2): 100n, symbol Device:C_Small
- removed R?: 2.7k, symbol Device:R_Small
- removed U2: BQ76200PW, Package_SO:TSSOP-16_4.4x5mm_P0.65mm, symbol Battery_Management:BQ76200PW
- removed U?: ACS758xCB-050B-PFF, Sensor_Current:Allegro_CB_PFF, symbol Sensor_Current:ACS758xCB-050B-PFF
- added C47: 100n, symbol Device:C_Small
- added R85: R_Small, symbol Device:R_Small
- added TH4: 100k, symbol Device:Thermistor_NTC
Connections:
- net GND: now also C47.2, TH4.2
- net Vref2: now reaches C12.2, U3.50 (VREF2)
- net Vref2: now also R85.1
- new net: C47.1, R85.2, TH4.1
Other:
- note added: "WDT can be used?"
- note added: "filter battery input"
- note added: "more caps?"
- note added: "power from battery to reduce noise"
- note removed: "Analog Front-End"
- note removed: "High-side enable/disable"
- note removed: "Total current sensing"
- moved on the sheet: C11, C12, C13, C14, C15, C16, C17, C18, C19, C20, C21, C22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
