File: hardware/afe.kicad_sch (KiCad schematic)
At the start: 52 parts, among them J4 Conn_01x19_Male, J8 RJ45, J9 RJ45, Q21 MMBT3904, U3 LTC6813-1

Commit message: AFE WDT pin
Parts:
- removed J8, J9: RJ45, symbol Connector:RJ45
- added J8: ISOSPI_OUT, symbol Connector:Conn_01x02_Pin
- added J9: ISOSPI_IN, symbol Connector:Conn_01x02_Pin
- added R86: 1M, symbol Device:R_Small
Connections:
- net CS: now also U3.62 (SCK(IPA)); no longer U3.61 (CSB(IMA))
- net SCK: now also U3.61 (CSB(IMA)); no longer U3.62 (SCK(IPA))
- net VREG: now also R86.1
- net WDT: now reaches U3.56 (WDT)
- net WDT: now also R86.2
- net at C17.1, R9.2, TR1.9 (RX-): now also U3.64 (IPB); no longer U3.63 (IMB)
- net at C18.2, R10.2, TR1.11 (RX+): now also U3.63 (IMB); no longer U3.64 (IPB)
- net at TR1.1 (TD+): now also J9.2 (Pin_2)
- net at TR1.3 (TD-): now also J9.1 (Pin_1)
- net at TR1.6 (RD+): now also J8.2 (Pin_2)
- net at TR1.8 (RD-): now also J8.1 (Pin_1)
- no-connect marks 3 -> 2
Other:
- note removed: "WDT can be used?"
- moved on the sheet: C13, C14, C15, C16, C17, C18, C19, C20, C47, R10, R11, R12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

Commit message: Fan ports
Parts:
- added C48: 10u, symbol Device:C_Small
Connections:
- net balance_front_end/CELL is gone; now on net +BATT: J4.19 (Pin_19)
- net GND: now also C48.2
- net VREG: now also C48.1
Other:
- note added: "Bypass cells for packs smaller than 18 S"
- note removed: "more caps?"
- moved on the sheet: C11, C12, R15, R17, R7, R8

Commit message: Improve AFE power supply filtering
Parts:
- added C54: 100n, symbol Device:C_Small
- C48: value 10u -> 1u
Connections:
- net GND: now also C54.2
- net at Q21.3 (C), R13.2: now also C54.1
Other:
- moved on the sheet: R13
Changed lines of the file:
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@@
   (junction (at 101.6 132.08) (diameter 0) (color 0 0 0 0)
+  )
+  (junction (at 101.6 29.21) (diameter 0) (color 0 0 0 0)
   )
   (junction (at 121.92 49.53) (diameter 0) (color 0 0 0 0)
@@
     (stroke (width 0) (type default))
   )
-  (wire (pts (xy 116.84 38.1) (xy 121.92 38.1))
+  (wire (pts (xy 97.79 29.21) (xy 101.6 29.21))
     (stroke (width 0) (type default))
   )
@@
     (stroke (width 0) (type default))
   )
+  (wire (pts (xy 121.92 29.21) (xy 121.92 38.1))
+    (stroke (width 0) (type default))
+  )
   (wire (pts (xy 176.53 82.55) (xy 189.23 82.55))
     (stroke (width 0) (type default))
@@
     (stroke (width 0) (type default))
   )
-  (wire (pts (xy 107.95 38.1) (xy 111.76 38.1))
+  (wire (pts (xy 88.9 29.21) (xy 92.71 29.21))
     (stroke (width 0) (type default))
   )
@@
     (stroke (width 0) (type default))
   )
-  (wire (pts (xy 107.95 36.83) (xy 107.95 38.1))
+  (wire (pts (xy 88.9 27.94) (xy 88.9 29.21))
     (stroke (width 0) (type default))
   )
@@
   )
   (wire (pts (xy 217.17 118.11) (xy 217.17 120.65))
+    (stroke (width 0) (type default))
+  )
+  (wire (pts (xy 101.6 29.21) (xy 121.92 29.21))
     (stroke (width 0) (type default))
   )
@@
     (effects (font (size 1.27 1.27)) (justify left bottom))
   )
-  (text "power from battery to reduce noise" (at 96.52 29.21 0)
+  (text "power from battery to reduce noise" (at 96.52 20.32 0)
     (effects (font (size 1.27 1.27)) (justify left bottom))
   )
@@
     )
   )
+  (symbol (lib_id "Device:C_Small") (at 101.6 31.75 0) (unit 1)
+    (in_bom yes) (on_board yes) (dnp no) (fields_autoplaced)
+    (property "Reference" "C54" (at 104.14 31.1213 0)
+      (effects (font (size 1.27 1.27)) (justify left))
+    )
+    (property "Value" "100n" (at 104.14 33.6613 0)
+      (effects (font (size 1.27 1.27)) (justify left))
+    )
+    (property "Footprint" "" (at 101.6 31.75 0)
+      (effects (font (size 1.27 1.27)) hide)
+    )
+    (property "Datasheet" "~" (at 101.6 31.75 0)
+      (effects (font (size 1.27 1.27)) hide)
+    )
+    (pin "1")
+    (pin "2")
+    (instances
+      (project "vesc-bms"
+        (path "/3e668e3e-3e16-4665-a807-4735962c41d3/a908ff77-32fe-48f6-8dc7-bc7bb4d76281"
+          (reference "C54") (unit 1)
+        )
+      )
+    )
+  )
   (symbol (lib_id "Device:C_Small") (at 180.34 72.39 0) (unit 1)
     (in_bom yes) (on_board yes) (dnp no) (fields_autoplaced)
@@
       (effects (font (size 1.27 1.27)) (justify left))
     )
-    (property "Value" "10u" (at 134.62 53.9813 0)
+    (property "Value" "1u" (at 134.62 53.9813 0)
       (effects (font (size 1.27 1.27)) (justify left))
     )
@@
     )
   )
+  (symbol (lib_id "power:GND") (at 101.6 34.29 0) (unit 1)
+    (in_bom yes) (on_board yes) (dnp no)
+    (property "Reference" "#PWR084" (at 101.6 40.64 0)
+      (effects (font (size 1.27 1.27)) hide)
+    )
+    (property "Value" "GND" (at 101.6 38.1 0)
+      (effects (font (size 1.27 1.27)))
+    )
+    (property "Footprint" "" (at 101.6 34.29 0)
+      (effects (font (size 1.27 1.27)) hide)
+    )
+    (property "Datasheet" "" (at 101.6 34.29 0)
+      (effects (font (size 1.27 1.27)) hide)
+    )
+    (pin "1")
+    (instances
+      (project "vesc-bms"
+        (path "/3e668e3e-3e16-4665-a807-4735962c41d3/a908ff77-32fe-48f6-8dc7-bc7bb4d76281"
+          (reference "#PWR084") (unit 1)
+        )
+      )
+    )
+  )
   (symbol (lib_id "Device:C_Small") (at 121.92 52.07 0) (unit 1)
     (in_bom yes) (on_board yes) (dnp no) (fields_autoplaced)
@@
     )
   )
-  (symbol (lib_id "power:+5V") (at 107.95 36.83 0) (unit 1)
-    (in_bom yes) (on_board yes) (dnp no) (fields_autoplaced)
-    (property "Reference" "#PWR051" (at 107.95 40.64 0)
-      (effects (font (size 1.27 1.27)) hide)
-    )
-    (property "Value" "+5V" (at 107.95 31.75 0)
-      (effects (font (size 1.27 1.27)))
-    )
-    (property "Footprint" "" (at 107.95 36.83 0)
-      (effects (font (size 1.27 1.27)) hide)
-    )
-    (property "Datasheet" "" (at 107.95 36.83 0)
+  (symbol (lib_id "power:+5V") (at 88.9 27.94 0) (unit 1)
+    (in_bom yes) (on_board yes) (dnp no) (fields_autoplaced)
+    (property "Reference" "#PWR051" (at 88.9 31.75 0)
+      (effects (font (size 1.27 1.27)) hide)
+    )
+    (property "Value" "+5V" (at 88.9 22.86 0)
+      (effects (font (size 1.27 1.27)))
+    )
+    (property "Footprint" "" (at 88.9 27.94 0)
+      (effects (font (size 1.27 1.27)) hide)
+    )
+    (property "Datasheet" "" (at 88.9 27.94 0)
       (effects (font (size 1.27 1.27)) hide)
     )
@@
     )
   )
-  (symbol (lib_id "Device:R_Small") (at 114.3 38.1 90) (unit 1)
-    (in_bom yes) (on_board yes) (dnp no) (fields_autoplaced)
-    (property "Reference" "R13" (at 114.3 33.02 90)
-      (effects (font (size 1.27 1.27)))
-    )
-    (property "Value" "100" (at 114.3 35.56 90)
-      (effects (font (size 1.27 1.27)))
-    )
-    (property "Footprint" "" (at 114.3 38.1 0)
-      (effects (font (size 1.27 1.27)) hide)
-    )
-    (property "Datasheet" "~" (at 114.3 38.1 0)
-      (effects (font (size 1.27 1.27)) hide)
-    )
+  (symbol (lib_id "Device:R_Small") (at 95.25 29.21 90) (unit 1)
+    (in_bom yes) (on_board yes) (dnp no) (fields_autoplaced)
+    (property "Reference" "R13" (at 95.25 24.13 90)
+      (effects (font (size 1.27 1.27)))
+    )
+    (property "Value" "100" (at 95.25 26.67 90)
+      (effects (font (size 1.27 1.27)))
+    )
+    (property "Footprint" "" (at 95.25 29.21 0)
+      (effects (font (size 1.27 1.27)) hide)
+    )
+    (property "Datasheet" "~" (at 95.25 29.21 0)
+      (effects (font (size 1.27 1.27)) hide)
+    )

Commit message: Charge monitor complete
Parts:
- added C334: 100n, symbol Device:C_Small
- added R316: R_Small, symbol Device:R_Small
- renumbered C11 to C301, C14 to C302, C13 to C303, C12 to C304, C15 to C305, C16 to C306, C17 to C307, C18 to C308, C19 to C309, C20 to C310, C54 to C311, C47 to C312, C44 to C313, C48 to C314, C21 to C315, C22 to C316, C23 to C317, C24 to C318, C25 to C319, C26 to C320, C27 to C321, C28 to C322, C29 to C323, C30 to C324, C31 to C325, C32 to C326, C33 to C327, C34 to C328, C35 to C329, C36 to C330, C37 to C331, C38 to C332, C39 to C333, J8 to J301, J9 to J302, J4 to J303, Q21 to Q301, R7 to R301, R8 to R302, R17 to R303, R15 to R304, R13 to R305, R16 to R306, R86 to R307, R9 to R308, R10 to R309, R11 to R310, R12 to R311, R19 to R312, R85 to R313, R18 to R314, R20 to R315, TH4 to TH301, TR1 to TR301, U3 to U301
Connections:
- net +5V is gone; now on net +BATT: R305.1
- net GND: now also C334.2
- net at R313.2, TH301.1: now also C334.1, R316.1; no longer C312.1
- new net: C312.1, R316.2
Other:
- note removed: "Bypass cells for packs smaller than 18 S"
- note removed: "power from battery to reduce noise"
- moved on the sheet: C312

Commit message: Total current sense and buzzer
Connections:
- net +BATT: no longer J303.19 (Pin_19)
- new net BAT+: J303.19 (Pin_19)
Changed lines of the file:
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@@
   (junction (at 180.34 90.17) (diameter 0) (color 0 0 0 0)
-  )
-  (junction (at 232.41 49.53) (diameter 0) (color 0 0 0 0)
   )
   (junction (at 101.6 137.16) (diameter 0) (color 0 0 0 0)
@@
   (hierarchical_label "GPIO1" (shape input) (at 151.13 110.49 180) (fields_autoplaced)
     (effects (font (size 1.27 1.27)) (justify right))
+  )
+  (hierarchical_label "BAT+" (shape input) (at 232.41 49.53 0) (fields_autoplaced)
+    (effects (font (size 1.27 1.27)) (justify left))
   )
   (hierarchical_label "GPIO4" (shape input) (at 151.13 118.11 180) (fields_autoplaced)
@@
         )
       )
-    )
-  )
-  (symbol (lib_id "power:+BATT") (at 232.41 49.53 0) (unit 1)
-    (in_bom yes) (on_board yes) (dnp no) (fields_autoplaced)
-    (property "Reference" "#PWR0318" (at 232.41 53.34 0)
-      (effects (font (size 1.27 1.27)) hide)
-    )
-    (property "Value" "+BATT" (at 232.41 44.45 0)
-      (effects (font (size 1.27 1.27)))
-    )
-    (property "Footprint" "" (at 232.41 49.53 0)
-      (effects (font (size 1.27 1.27)) hide)
-    )
-    (property "Datasheet" "" (at 232.41 49.53 0)
-      (effects (font (size 1.27 1.27)) hide)
-    )
-    (pin "1")
-    (instances
-      (project "vesc-bms"
-        (path "/3e668e3e-3e16-4665-a807-4735962c41d3/a908ff77-32fe-48f6-8dc7-bc7bb4d76281"
-          (reference "#PWR0318") (unit 1)
-        )
-      )
