File: hardware/comms.kicad_sch (KiCad schematic)
At the start: 1 part

Commit message: Communication interfaces
Parts:
- added J?: USB_C_Receptacle_USB2.0, symbol Connector:USB_C_Receptacle_USB2.0
- added J?: CAN, symbol Connector:Screw_Terminal_01x02
- added R?: 120, symbol Device:R_Small
- added R? (x2): 5.1k, symbol Device:R
- added U?: MCP2562-E-SN, Package_SO:SOIC-8_3.9x4.9mm_P1.27mm, symbol Interface_CAN_LIN:MCP2562-E-SN
Connections:
- net +3.3V: now also U?.5 (Vio)
- net GND: now also J?.A1 (GND), J?.A12 (GND), J?.B1 (GND), J?.B12 (GND), J?.S1 (SHIELD), R?.2, R?.2, U?.2 (VSS)
- new net: J?.A5 (CC1), R?.1
- new net: J?.B5 (CC2), R?.1
- new net: J?.1 (Pin_1), R?.1, U?.7 (CANH)
- new net: J?.2 (Pin_2), R?.2, U?.6 (CANL)
- new net +5V: U?.3 (VDD)
- new net CAN_EN: U?.8 (STBY)
- new net CAN_RX: U?.4 (RXD)
- new net CAN_TX: U?.1 (TXD)
- new net USB_DN: J?.A7 (D-), J?.B7 (D-)
- new net USB_DP: J?.A6 (D+), J?.B6 (D+)
- new net VBUS: J?.A4 (VBUS), J?.A9 (VBUS), J?.B4 (VBUS), J?.B9 (VBUS)
- no-connect marks 3 -> 5
Other:
- note added: "CAN interface"
- note added: "USB"
- moved on the sheet: J?

Commit message: BLE module
Parts:
- removed J?: BLE, symbol Connector:Conn_ARM_JTAG_SWD_10
- added J?: Conn_ARM_JTAG_SWD_10, symbol Connector:Conn_ARM_JTAG_SWD_10
- added U?: E73-2G4M08S1C, vesc-bms:E73-2G4M08S1C, symbol vesc-bms:E73-2G4M08S1C
Connections:
- net +3.3V: now also J?.1 (VTref)
- net GND: now also J?.3 (GND), J?.5 (GND), J?.9 (GNDDetect), U?.21 (GND), U?.24 (GND), U?.5 (GND)
- net NRF5x_SWCLK: now also J?.4 (SWDCLK/TCK), U?.39 (SWDCLK)
- net NRF5x_SWDIO: now also J?.2 (SWDIO/TMS), U?.37 (SWDIO)
- new net: J?.10 (~{RESET}), U?.26 (P0.18\RESET)
- no-connect marks 5 -> 4
Other:
- moved on the sheet: J?, R?, U?

Commit message: BLE module
Parts:
- J4: renamed from J?; footprint (none) -> Connector_PinHeader_1.27mm:PinHeader_2x05_P1.27mm_Vertical_SMD
- R3, R4, R5: renamed from R?; footprint (none) -> Resistor_SMD:R_0603_1608Metric
- gave numbers to parts that had none: 4
Connections:
- net +3.3V: now also U5.19 (VDD), U5.23 (VDDH)
- net BLE_RX: now reaches U5.33 (P0.13)
- net BLE_TX: now reaches U5.35 (P0.24)
- no-connect marks 4 -> 36
Other:
- moved on the sheet: J4, U5

Commit message: Analog front end daisy chain
Parts:
- renumbered J2 to J5, J3 to J6, J4 to J7, R3 to R15, R4 to R16, R5 to R17
Changed lines of the file:
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@@
   (symbol (lib_id "Connector:USB_C_Receptacle_USB2.0") (at 68.58 124.46 0) (unit 1)
     (in_bom yes) (on_board yes) (fields_autoplaced)
-    (property "Reference" "J2" (id 0) (at 68.58 101.6 0))
+    (property "Reference" "J5" (id 0) (at 68.58 101.6 0))
     (property "Value" "USB_C_Receptacle_USB2.0" (id 1) (at 68.58 104.14 0))
     (property "Footprint" "" (id 2) (at 72.39 124.46 0)
@@
   (symbol (lib_id "power:GND") (at 104.14 125.73 0) (unit 1)
     (in_bom yes) (on_board yes) (fields_autoplaced)
-    (property "Reference" "#PWR020" (id 0) (at 104.14 132.08 0)
+    (property "Reference" "#PWR028" (id 0) (at 104.14 132.08 0)
       (effects (font (size 1.27 1.27)) hide)
     )
@@
   (symbol (lib_id "Device:R_Small") (at 99.06 67.31 0) (unit 1)
     (in_bom yes) (on_board yes) (fields_autoplaced)
-    (property "Reference" "R3" (id 0) (at 101.6 66.0399 0)
+    (property "Reference" "R15" (id 0) (at 101.6 66.0399 0)
       (effects (font (size 1.27 1.27)) (justify left))
     )
@@
   (symbol (lib_id "power:+3.3V") (at 58.42 66.04 0) (unit 1)
     (in_bom yes) (on_board yes) (fields_autoplaced)
-    (property "Reference" "#PWR015" (id 0) (at 58.42 69.85 0)
+    (property "Reference" "#PWR023" (id 0) (at 58.42 69.85 0)
       (effects (font (size 1.27 1.27)) hide)
     )
@@
   (symbol (lib_id "power:+3.3V") (at 175.26 82.55 0) (unit 1)
     (in_bom yes) (on_board yes) (fields_autoplaced)
-    (property "Reference" "#PWR021" (id 0) (at 175.26 86.36 0)
+    (property "Reference" "#PWR029" (id 0) (at 175.26 86.36 0)
       (effects (font (size 1.27 1.27)) hide)
     )
@@
   (symbol (lib_id "power:GND") (at 175.26 114.3 0) (unit 1)
     (in_bom yes) (on_board yes) (fields_autoplaced)
-    (property "Reference" "#PWR022" (id 0) (at 175.26 120.65 0)
+    (property "Reference" "#PWR030" (id 0) (at 175.26 120.65 0)
       (effects (font (size 1.27 1.27)) hide)
     )
@@
   (symbol (lib_id "power:GND") (at 229.87 125.73 0) (unit 1)
     (in_bom yes) (on_board yes) (fields_autoplaced)
-    (property "Reference" "#PWR023" (id 0) (at 229.87 132.08 0)
+    (property "Reference" "#PWR032" (id 0) (at 229.87 132.08 0)
       (effects (font (size 1.27 1.27)) hide)
     )
@@
   (symbol (lib_id "power:GND") (at 68.58 149.86 0) (unit 1)
     (in_bom yes) (on_board yes) (fields_autoplaced)
-    (property "Reference" "#PWR016" (id 0) (at 68.58 156.21 0)
+    (property "Reference" "#PWR024" (id 0) (at 68.58 156.21 0)
       (effects (font (size 1.27 1.27)) hide)
     )
@@
   (symbol (lib_id "Device:R") (at 99.06 120.65 0) (unit 1)
     (in_bom yes) (on_board yes) (fields_autoplaced)
-    (property "Reference" "R4" (id 0) (at 101.6 119.3799 0)
+    (property "Reference" "R16" (id 0) (at 101.6 119.3799 0)
       (effects (font (size 1.27 1.27)) (justify left))
     )
@@
   (symbol (lib_id "power:GND") (at 83.82 77.47 0) (unit 1)
     (in_bom yes) (on_board yes) (fields_autoplaced)
-    (property "Reference" "#PWR018" (id 0) (at 83.82 83.82 0)
+    (property "Reference" "#PWR026" (id 0) (at 83.82 83.82 0)
       (effects (font (size 1.27 1.27)) hide)
     )
@@
   (symbol (lib_id "power:+3.3V") (at 228.6 58.42 0) (unit 1)
     (in_bom yes) (on_board yes) (fields_autoplaced)
-    (property "Reference" "#PWR0101" (id 0) (at 228.6 62.23 0)
+    (property "Reference" "#PWR031" (id 0) (at 228.6 62.23 0)
       (effects (font (size 1.27 1.27)) hide)
     )
@@
   (symbol (lib_id "Device:R") (at 107.95 120.65 0) (unit 1)
     (in_bom yes) (on_board yes) (fields_autoplaced)
-    (property "Reference" "R5" (id 0) (at 110.49 119.3799 0)
+    (property "Reference" "R17" (id 0) (at 110.49 119.3799 0)
       (effects (font (size 1.27 1.27)) (justify left))
     )
@@
   (symbol (lib_id "Connector:Screw_Terminal_01x02") (at 111.76 66.04 0) (unit 1)
     (in_bom yes) (on_board yes) (fields_autoplaced)
-    (property "Reference" "J3" (id 0) (at 114.3 66.0399 0)
+    (property "Reference" "J6" (id 0) (at 114.3 66.0399 0)
       (effects (font (size 1.27 1.27)) (justify left))
     )
@@
   (symbol (lib_id "power:VBUS") (at 86.36 107.95 0) (unit 1)
     (in_bom yes) (on_board yes) (fields_autoplaced)
-    (property "Reference" "#PWR019" (id 0) (at 86.36 111.76 0)
+    (property "Reference" "#PWR027" (id 0) (at 86.36 111.76 0)
       (effects (font (size 1.27 1.27)) hide)
     )
@@
   (symbol (lib_id "power:+5V") (at 83.82 57.15 0) (unit 1)
     (in_bom yes) (on_board yes) (fields_autoplaced)
-    (property "Reference" "#PWR017" (id 0) (at 83.82 60.96 0)
+    (property "Reference" "#PWR025" (id 0) (at 83.82 60.96 0)
       (effects (font (size 1.27 1.27)) hide)
     )
@@
   (symbol (lib_id "Connector:Conn_ARM_JTAG_SWD_10") (at 175.26 97.79 0) (unit 1)
     (in_bom yes) (on_board yes) (fields_autoplaced)
-    (property "Reference" "J4" (id 0) (at 163.83 96.5199 0)
+    (property "Reference" "J7" (id 0) (at 163.83 96.5199 0)
       (effects (font (size 1.27 1.27)) (justify right))
     )

Commit message: Analog front end ready
Parts:
- renumbered R15 to R17, R16 to R18, R17 to R19
Changed lines of the file:
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@@
   (symbol (lib_id "power:GND") (at 104.14 125.73 0) (unit 1)
     (in_bom yes) (on_board yes) (fields_autoplaced)
-    (property "Reference" "#PWR028" (id 0) (at 104.14 132.08 0)
+    (property "Reference" "#PWR030" (id 0) (at 104.14 132.08 0)
       (effects (font (size 1.27 1.27)) hide)
     )
@@
   (symbol (lib_id "Device:R_Small") (at 99.06 67.31 0) (unit 1)
     (in_bom yes) (on_board yes) (fields_autoplaced)
-    (property "Reference" "R15" (id 0) (at 101.6 66.0399 0)
+    (property "Reference" "R17" (id 0) (at 101.6 66.0399 0)
       (effects (font (size 1.27 1.27)) (justify left))
     )
@@
   (symbol (lib_id "power:+3.3V") (at 58.42 66.04 0) (unit 1)
     (in_bom yes) (on_board yes) (fields_autoplaced)
-    (property "Reference" "#PWR023" (id 0) (at 58.42 69.85 0)
+    (property "Reference" "#PWR025" (id 0) (at 58.42 69.85 0)
       (effects (font (size 1.27 1.27)) hide)
     )
@@
   (symbol (lib_id "power:+3.3V") (at 175.26 82.55 0) (unit 1)
     (in_bom yes) (on_board yes) (fields_autoplaced)
-    (property "Reference" "#PWR029" (id 0) (at 175.26 86.36 0)
+    (property "Reference" "#PWR031" (id 0) (at 175.26 86.36 0)
       (effects (font (size 1.27 1.27)) hide)
     )
@@
   (symbol (lib_id "power:GND") (at 175.26 114.3 0) (unit 1)
     (in_bom yes) (on_board yes) (fields_autoplaced)
-    (property "Reference" "#PWR030" (id 0) (at 175.26 120.65 0)
+    (property "Reference" "#PWR032" (id 0) (at 175.26 120.65 0)
       (effects (font (size 1.27 1.27)) hide)
     )
@@
   (symbol (lib_id "power:GND") (at 229.87 125.73 0) (unit 1)
     (in_bom yes) (on_board yes) (fields_autoplaced)
-    (property "Reference" "#PWR032" (id 0) (at 229.87 132.08 0)
+    (property "Reference" "#PWR034" (id 0) (at 229.87 132.08 0)
       (effects (font (size 1.27 1.27)) hide)
     )
@@
   (symbol (lib_id "power:GND") (at 68.58 149.86 0) (unit 1)
     (in_bom yes) (on_board yes) (fields_autoplaced)
-    (property "Reference" "#PWR024" (id 0) (at 68.58 156.21 0)
+    (property "Reference" "#PWR026" (id 0) (at 68.58 156.21 0)
       (effects (font (size 1.27 1.27)) hide)
     )
@@
   (symbol (lib_id "Device:R") (at 99.06 120.65 0) (unit 1)
     (in_bom yes) (on_board yes) (fields_autoplaced)
-    (property "Reference" "R16" (id 0) (at 101.6 119.3799 0)
+    (property "Reference" "R18" (id 0) (at 101.6 119.3799 0)
       (effects (font (size 1.27 1.27)) (justify left))
     )
@@
   (symbol (lib_id "power:GND") (at 83.82 77.47 0) (unit 1)
     (in_bom yes) (on_board yes) (fields_autoplaced)
-    (property "Reference" "#PWR026" (id 0) (at 83.82 83.82 0)
+    (property "Reference" "#PWR028" (id 0) (at 83.82 83.82 0)
       (effects (font (size 1.27 1.27)) hide)
     )
@@
   (symbol (lib_id "power:+3.3V") (at 228.6 58.42 0) (unit 1)
     (in_bom yes) (on_board yes) (fields_autoplaced)
-    (property "Reference" "#PWR031" (id 0) (at 228.6 62.23 0)
+    (property "Reference" "#PWR033" (id 0) (at 228.6 62.23 0)
       (effects (font (size 1.27 1.27)) hide)
     )
@@
   (symbol (lib_id "Device:R") (at 107.95 120.65 0) (unit 1)
     (in_bom yes) (on_board yes) (fields_autoplaced)
-    (property "Reference" "R17" (id 0) (at 110.49 119.3799 0)
+    (property "Reference" "R19" (id 0) (at 110.49 119.3799 0)
       (effects (font (size 1.27 1.27)) (justify left))
     )
@@
   (symbol (lib_id "power:VBUS") (at 86.36 107.95 0) (unit 1)
     (in_bom yes) (on_board yes) (fields_autoplaced)
-    (property "Reference" "#PWR027" (id 0) (at 86.36 111.76 0)
+    (property "Reference" "#PWR029" (id 0) (at 86.36 111.76 0)
       (effects (font (size 1.27 1.27)) hide)
     )
@@
   (symbol (lib_id "power:+5V") (at 83.82 57.15 0) (unit 1)
     (in_bom yes) (on_board yes) (fields_autoplaced)
-    (property "Reference" "#PWR025" (id 0) (at 83.82 60.96 0)
-      (effects (font (size 1.27 1.27)) hide)
-    )
+    (property "Reference" "#PWR027" (id 0) (at 83.82 60.96 0)
+      (effects (font (size 1.27 1.27)) hide)
+    )

Commit message: NTC sensors
Parts:
- renumbered R17 to R19, R18 to R20, R19 to R21
Changed lines of the file:
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@@
   (symbol (lib_id "power:GND") (at 104.14 125.73 0) (unit 1)
     (in_bom yes) (on_board yes) (fields_autoplaced)
-    (property "Reference" "#PWR030" (id 0) (at 104.14 132.08 0)
+    (property "Reference" "#PWR032" (id 0) (at 104.14 132.08 0)
       (effects (font (size 1.27 1.27)) hide)
     )
@@
   (symbol (lib_id "Device:R_Small") (at 99.06 67.31 0) (unit 1)
     (in_bom yes) (on_board yes) (fields_autoplaced)
-    (property "Reference" "R17" (id 0) (at 101.6 66.0399 0)
+    (property "Reference" "R19" (id 0) (at 101.6 66.0399 0)
       (effects (font (size 1.27 1.27)) (justify left))
     )
@@
   (symbol (lib_id "power:+3.3V") (at 58.42 66.04 0) (unit 1)
     (in_bom yes) (on_board yes) (fields_autoplaced)
-    (property "Reference" "#PWR025" (id 0) (at 58.42 69.85 0)
+    (property "Reference" "#PWR027" (id 0) (at 58.42 69.85 0)
       (effects (font (size 1.27 1.27)) hide)
     )
@@
   (symbol (lib_id "power:+3.3V") (at 175.26 82.55 0) (unit 1)
     (in_bom yes) (on_board yes) (fields_autoplaced)
-    (property "Reference" "#PWR031" (id 0) (at 175.26 86.36 0)
+    (property "Reference" "#PWR033" (id 0) (at 175.26 86.36 0)
       (effects (font (size 1.27 1.27)) hide)
     )
@@
   (symbol (lib_id "power:GND") (at 175.26 114.3 0) (unit 1)
     (in_bom yes) (on_board yes) (fields_autoplaced)
-    (property "Reference" "#PWR032" (id 0) (at 175.26 120.65 0)
+    (property "Reference" "#PWR034" (id 0) (at 175.26 120.65 0)
       (effects (font (size 1.27 1.27)) hide)
     )
@@
   (symbol (lib_id "power:GND") (at 229.87 125.73 0) (unit 1)
     (in_bom yes) (on_board yes) (fields_autoplaced)
-    (property "Reference" "#PWR034" (id 0) (at 229.87 132.08 0)
+    (property "Reference" "#PWR036" (id 0) (at 229.87 132.08 0)
       (effects (font (size 1.27 1.27)) hide)
     )
@@
   (symbol (lib_id "power:GND") (at 68.58 149.86 0) (unit 1)
     (in_bom yes) (on_board yes) (fields_autoplaced)
-    (property "Reference" "#PWR026" (id 0) (at 68.58 156.21 0)
+    (property "Reference" "#PWR028" (id 0) (at 68.58 156.21 0)
       (effects (font (size 1.27 1.27)) hide)
     )
@@
   (symbol (lib_id "Device:R") (at 99.06 120.65 0) (unit 1)
     (in_bom yes) (on_board yes) (fields_autoplaced)
-    (property "Reference" "R18" (id 0) (at 101.6 119.3799 0)
+    (property "Reference" "R20" (id 0) (at 101.6 119.3799 0)
       (effects (font (size 1.27 1.27)) (justify left))
     )
@@
   (symbol (lib_id "power:GND") (at 83.82 77.47 0) (unit 1)
     (in_bom yes) (on_board yes) (fields_autoplaced)
-    (property "Reference" "#PWR028" (id 0) (at 83.82 83.82 0)
+    (property "Reference" "#PWR030" (id 0) (at 83.82 83.82 0)
       (effects (font (size 1.27 1.27)) hide)
     )
@@
   (symbol (lib_id "power:+3.3V") (at 228.6 58.42 0) (unit 1)
     (in_bom yes) (on_board yes) (fields_autoplaced)
-    (property "Reference" "#PWR033" (id 0) (at 228.6 62.23 0)
+    (property "Reference" "#PWR035" (id 0) (at 228.6 62.23 0)
       (effects (font (size 1.27 1.27)) hide)
     )
@@
   (symbol (lib_id "Device:R") (at 107.95 120.65 0) (unit 1)
     (in_bom yes) (on_board yes) (fields_autoplaced)
-    (property "Reference" "R19" (id 0) (at 110.49 119.3799 0)
+    (property "Reference" "R21" (id 0) (at 110.49 119.3799 0)
       (effects (font (size 1.27 1.27)) (justify left))
     )
@@
   (symbol (lib_id "power:VBUS") (at 86.36 107.95 0) (unit 1)
     (in_bom yes) (on_board yes) (fields_autoplaced)
-    (property "Reference" "#PWR029" (id 0) (at 86.36 111.76 0)
+    (property "Reference" "#PWR031" (id 0) (at 86.36 111.76 0)
       (effects (font (size 1.27 1.27)) hide)
     )
@@
   (symbol (lib_id "power:+5V") (at 83.82 57.15 0) (unit 1)
     (in_bom yes) (on_board yes) (fields_autoplaced)
-    (property "Reference" "#PWR027" (id 0) (at 83.82 60.96 0)
-      (effects (font (size 1.27 1.27)) hide)
-    )
+    (property "Reference" "#PWR029" (id 0) (at 83.82 60.96 0)
+      (effects (font (size 1.27 1.27)) hide)
+    )

Commit message: Annotate schematic
Parts:
- renumbered R19 to R21, R20 to R22, R21 to R23
Changed lines of the file:
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@@
   (symbol (lib_id "power:GND") (at 104.14 125.73 0) (unit 1)
     (in_bom yes) (on_board yes) (fields_autoplaced)
-    (property "Reference" "#PWR032" (id 0) (at 104.14 132.08 0)
+    (property "Reference" "#PWR034" (id 0) (at 104.14 132.08 0)
       (effects (font (size 1.27 1.27)) hide)
     )
@@
   (symbol (lib_id "Device:R_Small") (at 99.06 67.31 0) (unit 1)
     (in_bom yes) (on_board yes) (fields_autoplaced)
-    (property "Reference" "R19" (id 0) (at 101.6 66.0399 0)
+    (property "Reference" "R21" (id 0) (at 101.6 66.0399 0)
       (effects (font (size 1.27 1.27)) (justify left))
     )
@@
   (symbol (lib_id "power:+3.3V") (at 58.42 66.04 0) (unit 1)
     (in_bom yes) (on_board yes) (fields_autoplaced)
-    (property "Reference" "#PWR027" (id 0) (at 58.42 69.85 0)
+    (property "Reference" "#PWR029" (id 0) (at 58.42 69.85 0)
       (effects (font (size 1.27 1.27)) hide)
     )
@@
   (symbol (lib_id "power:+3.3V") (at 175.26 82.55 0) (unit 1)
     (in_bom yes) (on_board yes) (fields_autoplaced)
-    (property "Reference" "#PWR033" (id 0) (at 175.26 86.36 0)
+    (property "Reference" "#PWR035" (id 0) (at 175.26 86.36 0)
       (effects (font (size 1.27 1.27)) hide)
     )
@@
   (symbol (lib_id "power:GND") (at 175.26 114.3 0) (unit 1)
     (in_bom yes) (on_board yes) (fields_autoplaced)
-    (property "Reference" "#PWR034" (id 0) (at 175.26 120.65 0)
+    (property "Reference" "#PWR036" (id 0) (at 175.26 120.65 0)
       (effects (font (size 1.27 1.27)) hide)
     )
@@
   (symbol (lib_id "power:GND") (at 229.87 125.73 0) (unit 1)
     (in_bom yes) (on_board yes) (fields_autoplaced)
-    (property "Reference" "#PWR036" (id 0) (at 229.87 132.08 0)
+    (property "Reference" "#PWR038" (id 0) (at 229.87 132.08 0)
       (effects (font (size 1.27 1.27)) hide)
     )
@@
   (symbol (lib_id "power:GND") (at 68.58 149.86 0) (unit 1)
     (in_bom yes) (on_board yes) (fields_autoplaced)
-    (property "Reference" "#PWR028" (id 0) (at 68.58 156.21 0)
+    (property "Reference" "#PWR030" (id 0) (at 68.58 156.21 0)
       (effects (font (size 1.27 1.27)) hide)
     )
@@
   (symbol (lib_id "Device:R") (at 99.06 120.65 0) (unit 1)
     (in_bom yes) (on_board yes) (fields_autoplaced)
-    (property "Reference" "R20" (id 0) (at 101.6 119.3799 0)
+    (property "Reference" "R22" (id 0) (at 101.6 119.3799 0)
       (effects (font (size 1.27 1.27)) (justify left))
     )
@@
   (symbol (lib_id "power:GND") (at 83.82 77.47 0) (unit 1)
     (in_bom yes) (on_board yes) (fields_autoplaced)
-    (property "Reference" "#PWR030" (id 0) (at 83.82 83.82 0)
+    (property "Reference" "#PWR032" (id 0) (at 83.82 83.82 0)
       (effects (font (size 1.27 1.27)) hide)
     )
@@
   (symbol (lib_id "power:+3.3V") (at 228.6 58.42 0) (unit 1)
     (in_bom yes) (on_board yes) (fields_autoplaced)
-    (property "Reference" "#PWR035" (id 0) (at 228.6 62.23 0)
+    (property "Reference" "#PWR037" (id 0) (at 228.6 62.23 0)
       (effects (font (size 1.27 1.27)) hide)
     )
@@
   (symbol (lib_id "Device:R") (at 107.95 120.65 0) (unit 1)
     (in_bom yes) (on_board yes) (fields_autoplaced)
-    (property "Reference" "R21" (id 0) (at 110.49 119.3799 0)
+    (property "Reference" "R23" (id 0) (at 110.49 119.3799 0)
       (effects (font (size 1.27 1.27)) (justify left))
     )
@@
   (symbol (lib_id "power:VBUS") (at 86.36 107.95 0) (unit 1)
     (in_bom yes) (on_board yes) (fields_autoplaced)
-    (property "Reference" "#PWR031" (id 0) (at 86.36 111.76 0)
+    (property "Reference" "#PWR033" (id 0) (at 86.36 111.76 0)
       (effects (font (size 1.27 1.27)) hide)
     )
@@
   (symbol (lib_id "power:+5V") (at 83.82 57.15 0) (unit 1)
     (in_bom yes) (on_board yes) (fields_autoplaced)
-    (property "Reference" "#PWR029" (id 0) (at 83.82 60.96 0)
-      (effects (font (size 1.27 1.27)) hide)
-    )
+    (property "Reference" "#PWR031" (id 0) (at 83.82 60.96 0)
+      (effects (font (size 1.27 1.27)) hide)
+    )
