File: hardware/comms.kicad_sch (KiCad schematic)
At the start: 8 parts, among them J5 USB_C_Receptacle_USB2.0, J6 CAN, J7 Conn_ARM_JTAG_SWD_10, U4 MCP2562-E-SN, U5 E73-2G4M08S1C

Commit message: Fan ports
Parts:
- added U2: nRF52840, Package_DFN_QFN:Nordic_AQFN-73-1EP_7x7mm_P0.5mm, symbol MCU_Nordic:nRF52840
Connections:
- new net: U2.A22 (VDD), U2.AD14 (VDD), U2.AD23 (VDD), U2.B1 (VDD), U2.W1 (VDD)
- new net: U2.B7 (VSS), U2.EP (VSS)
Other:
- note added: "To be replaced by a discrete circuit"
Changed lines of the file:
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@@
+    (effects (font (size 1.27 1.27)) (justify left bottom))
+  )
+  (text "To be replaced by a discrete circuit" (at 153.67 63.5 0)
     (effects (font (size 1.27 1.27)) (justify left bottom))
   )
@@
         )
       )
+    )
+  )
+  (symbol (lib_id "MCU_Nordic:nRF52840") (at 359.41 78.74 0) (unit 1)
+    (in_bom yes) (on_board yes) (dnp no) (fields_autoplaced)
+    (property "Reference" "U2" (at 363.9059 147.32 0)
+      (effects (font (size 1.27 1.27)) (justify left))
+    )
+    (property "Value" "nRF52840" (at 363.9059 149.86 0)
+      (effects (font (size 1.27 1.27)) (justify left))
+    )
+    (property "Footprint" "Package_DFN_QFN:Nordic_AQFN-73-1EP_7x7mm_P0.5mm" (at 359.41 152.4 0)
+      (effects (font (size 1.27 1.27)) hide)
+    )
+    (property "Datasheet" "http://infocenter.nordicsemi.com/topic/com.nordic.infocenter.nrf52/dita/nrf52/chips/nrf52840.html" (at 342.9 30.48 0)
+      (effects (font (size 1.27 1.27)) hide)
+    )
+    (pin "A10")
+    (pin "A12")
+    (pin "A14")
+    (pin "A16")
+    (pin "A18")
+    (pin "A20")
+    (pin "A22")
+    (pin "A23")
+    (pin "A8")
+    (pin "AA24")
+    (pin "AB2")
+    (pin "AC11")
+    (pin "AC13")
+    (pin "AC15")
+    (pin "AC17")
+    (pin "AC19")
+    (pin "AC21")
+    (pin "AC24")
+    (pin "AC5")
+    (pin "AC9")
+    (pin "AD10")
+    (pin "AD12")
+    (pin "AD14")
+    (pin "AD16")
+    (pin "AD18")
+    (pin "AD2")
+    (pin "AD20")
+    (pin "AD22")
+    (pin "AD23")
+    (pin "AD4")
+    (pin "AD6")
+    (pin "AD8")
+    (pin "B1")
+    (pin "B11")
+    (pin "B13")
+    (pin "B15")
+    (pin "B17")
+    (pin "B19")
+    (pin "B24")
+    (pin "B3")
+    (pin "B5")
+    (pin "B7")
+    (pin "B9")
+    (pin "C1")
+    (pin "D2")
+    (pin "D23")
+    (pin "E24")
+    (pin "EP")
+    (pin "F2")
+    (pin "F23")
+    (pin "G1")
+    (pin "H2")
+    (pin "H23")
+    (pin "J1")
+    (pin "J24")
+    (pin "K2")
+    (pin "L1")
+    (pin "L24")
+    (pin "M2")
+    (pin "N1")
+    (pin "N24")
+    (pin "P2")
+    (pin "P23")
+    (pin "R1")
+    (pin "R24")
+    (pin "T2")
+    (pin "T23")
+    (pin "U1")
+    (pin "U24")
+    (pin "V23")
+    (pin "W1")
+    (pin "W24")
+    (pin "Y2")
+    (pin "Y23")
+    (instances
+      (project "vesc-bms"
+        (path "/3e668e3e-3e16-4665-a807-4735962c41d3/6e2b1342-9746-4a38-93af-9ab1059c6272"
+          (reference "U2") (unit 1)
+        )
+      )

Commit message: Remove left over IC
Parts:
- removed U2: nRF52840, Package_DFN_QFN:Nordic_AQFN-73-1EP_7x7mm_P0.5mm, symbol MCU_Nordic:nRF52840
Changed lines of the file:
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@@
-    )
-  )
-  (symbol (lib_id "MCU_Nordic:nRF52840") (at 359.41 78.74 0) (unit 1)
-    (in_bom yes) (on_board yes) (dnp no) (fields_autoplaced)
-    (property "Reference" "U2" (at 363.9059 147.32 0)
-      (effects (font (size 1.27 1.27)) (justify left))
-    )
-    (property "Value" "nRF52840" (at 363.9059 149.86 0)
-      (effects (font (size 1.27 1.27)) (justify left))
-    )
-    (property "Footprint" "Package_DFN_QFN:Nordic_AQFN-73-1EP_7x7mm_P0.5mm" (at 359.41 152.4 0)
-      (effects (font (size 1.27 1.27)) hide)
-    )
-    (property "Datasheet" "http://infocenter.nordicsemi.com/topic/com.nordic.infocenter.nrf52/dita/nrf52/chips/nrf52840.html" (at 342.9 30.48 0)
-      (effects (font (size 1.27 1.27)) hide)
-    )
-    (pin "A10")
-    (pin "A12")
-    (pin "A14")
-    (pin "A16")
-    (pin "A18")
-    (pin "A20")
-    (pin "A22")
-    (pin "A23")
-    (pin "A8")
-    (pin "AA24")
-    (pin "AB2")
-    (pin "AC11")
-    (pin "AC13")
-    (pin "AC15")
-    (pin "AC17")
-    (pin "AC19")
-    (pin "AC21")
-    (pin "AC24")
-    (pin "AC5")
-    (pin "AC9")
-    (pin "AD10")
-    (pin "AD12")
-    (pin "AD14")
-    (pin "AD16")
-    (pin "AD18")
-    (pin "AD2")
-    (pin "AD20")
-    (pin "AD22")
-    (pin "AD23")
-    (pin "AD4")
-    (pin "AD6")
-    (pin "AD8")
-    (pin "B1")
-    (pin "B11")
-    (pin "B13")
-    (pin "B15")
-    (pin "B17")
-    (pin "B19")
-    (pin "B24")
-    (pin "B3")
-    (pin "B5")
-    (pin "B7")
-    (pin "B9")
-    (pin "C1")
-    (pin "D2")
-    (pin "D23")
-    (pin "E24")
-    (pin "EP")
-    (pin "F2")
-    (pin "F23")
-    (pin "G1")
-    (pin "H2")
-    (pin "H23")
-    (pin "J1")
-    (pin "J24")
-    (pin "K2")
-    (pin "L1")
-    (pin "L24")
-    (pin "M2")
-    (pin "N1")
-    (pin "N24")
-    (pin "P2")
-    (pin "P23")
-    (pin "R1")
-    (pin "R24")
-    (pin "T2")
-    (pin "T23")
-    (pin "U1")
-    (pin "U24")
-    (pin "V23")
-    (pin "W1")
-    (pin "W24")
-    (pin "Y2")
-    (pin "Y23")
-    (instances
-      (project "vesc-bms"
-        (path "/3e668e3e-3e16-4665-a807-4735962c41d3/6e2b1342-9746-4a38-93af-9ab1059c6272"
-          (reference "U2") (unit 1)
-        )
-      )
     )
   )

Commit message: Charge monitor complete
Parts:
- renumbered J5 to J401, J6 to J402, J7 to J403, R21 to R401, R22 to R402, R23 to R403, U4 to U401, U5 to U402
Changed lines of the file:
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@@
   (symbol (lib_id "Connector:USB_C_Receptacle_USB2.0") (at 68.58 124.46 0) (unit 1)
     (in_bom yes) (on_board yes) (dnp no) (fields_autoplaced)
-    (property "Reference" "J5" (at 68.58 101.6 0)
+    (property "Reference" "J401" (at 68.58 101.6 0)
       (effects (font (size 1.27 1.27)))
     )
@@
       (project "vesc-bms"
         (path "/3e668e3e-3e16-4665-a807-4735962c41d3/6e2b1342-9746-4a38-93af-9ab1059c6272"
-          (reference "J5") (unit 1)
+          (reference "J401") (unit 1)
         )
       )
@@
   (symbol (lib_id "power:GND") (at 104.14 125.73 0) (unit 1)
     (in_bom yes) (on_board yes) (dnp no) (fields_autoplaced)
-    (property "Reference" "#PWR034" (at 104.14 132.08 0)
+    (property "Reference" "#PWR0406" (at 104.14 132.08 0)
       (effects (font (size 1.27 1.27)) hide)
     )
@@
       (project "vesc-bms"
         (path "/3e668e3e-3e16-4665-a807-4735962c41d3/6e2b1342-9746-4a38-93af-9ab1059c6272"
-          (reference "#PWR034") (unit 1)
+          (reference "#PWR0406") (unit 1)
         )
       )
@@
   (symbol (lib_id "Device:R_Small") (at 99.06 67.31 0) (unit 1)
     (in_bom yes) (on_board yes) (dnp no) (fields_autoplaced)
-    (property "Reference" "R21" (at 101.6 66.0399 0)
+    (property "Reference" "R401" (at 101.6 66.0399 0)
       (effects (font (size 1.27 1.27)) (justify left))
     )
@@
       (project "vesc-bms"
         (path "/3e668e3e-3e16-4665-a807-4735962c41d3/6e2b1342-9746-4a38-93af-9ab1059c6272"
-          (reference "R21") (unit 1)
+          (reference "R401") (unit 1)
         )
       )
@@
   (symbol (lib_id "power:+3.3V") (at 58.42 66.04 0) (unit 1)
     (in_bom yes) (on_board yes) (dnp no) (fields_autoplaced)
-    (property "Reference" "#PWR029" (at 58.42 69.85 0)
+    (property "Reference" "#PWR0401" (at 58.42 69.85 0)
       (effects (font (size 1.27 1.27)) hide)
     )
@@
       (project "vesc-bms"
         (path "/3e668e3e-3e16-4665-a807-4735962c41d3/6e2b1342-9746-4a38-93af-9ab1059c6272"
-          (reference "#PWR029") (unit 1)
+          (reference "#PWR0401") (unit 1)
         )
       )
@@
   (symbol (lib_id "power:+3.3V") (at 175.26 82.55 0) (unit 1)
     (in_bom yes) (on_board yes) (dnp no) (fields_autoplaced)
-    (property "Reference" "#PWR035" (at 175.26 86.36 0)
+    (property "Reference" "#PWR0407" (at 175.26 86.36 0)
       (effects (font (size 1.27 1.27)) hide)
     )
@@
       (project "vesc-bms"
         (path "/3e668e3e-3e16-4665-a807-4735962c41d3/6e2b1342-9746-4a38-93af-9ab1059c6272"
-          (reference "#PWR035") (unit 1)
+          (reference "#PWR0407") (unit 1)
         )
       )
@@
   (symbol (lib_id "power:GND") (at 175.26 114.3 0) (unit 1)
     (in_bom yes) (on_board yes) (dnp no) (fields_autoplaced)
-    (property "Reference" "#PWR036" (at 175.26 120.65 0)
+    (property "Reference" "#PWR0408" (at 175.26 120.65 0)
       (effects (font (size 1.27 1.27)) hide)
     )
@@
       (project "vesc-bms"
         (path "/3e668e3e-3e16-4665-a807-4735962c41d3/6e2b1342-9746-4a38-93af-9ab1059c6272"
-          (reference "#PWR036") (unit 1)
+          (reference "#PWR0408") (unit 1)
         )
       )
@@
   (symbol (lib_id "power:GND") (at 229.87 125.73 0) (unit 1)
     (in_bom yes) (on_board yes) (dnp no) (fields_autoplaced)
-    (property "Reference" "#PWR038" (at 229.87 132.08 0)
+    (property "Reference" "#PWR0410" (at 229.87 132.08 0)
       (effects (font (size 1.27 1.27)) hide)
     )
@@
       (project "vesc-bms"
         (path "/3e668e3e-3e16-4665-a807-4735962c41d3/6e2b1342-9746-4a38-93af-9ab1059c6272"
-          (reference "#PWR038") (unit 1)
+          (reference "#PWR0410") (unit 1)
         )
       )
@@
   (symbol (lib_id "power:GND") (at 68.58 149.86 0) (unit 1)
     (in_bom yes) (on_board yes) (dnp no) (fields_autoplaced)
-    (property "Reference" "#PWR030" (at 68.58 156.21 0)
+    (property "Reference" "#PWR0402" (at 68.58 156.21 0)
       (effects (font (size 1.27 1.27)) hide)
     )
@@
       (project "vesc-bms"
         (path "/3e668e3e-3e16-4665-a807-4735962c41d3/6e2b1342-9746-4a38-93af-9ab1059c6272"
-          (reference "#PWR030") (unit 1)
+          (reference "#PWR0402") (unit 1)
         )
       )
@@
   (symbol (lib_id "Device:R") (at 99.06 120.65 0) (unit 1)
     (in_bom yes) (on_board yes) (dnp no) (fields_autoplaced)
-    (property "Reference" "R22" (at 101.6 119.3799 0)
+    (property "Reference" "R402" (at 101.6 119.3799 0)
       (effects (font (size 1.27 1.27)) (justify left))
     )
@@
       (project "vesc-bms"
         (path "/3e668e3e-3e16-4665-a807-4735962c41d3/6e2b1342-9746-4a38-93af-9ab1059c6272"
-          (reference "R22") (unit 1)
+          (reference "R402") (unit 1)
         )
       )
@@
   (symbol (lib_id "power:GND") (at 83.82 77.47 0) (unit 1)
     (in_bom yes) (on_board yes) (dnp no) (fields_autoplaced)
-    (property "Reference" "#PWR032" (at 83.82 83.82 0)
+    (property "Reference" "#PWR0404" (at 83.82 83.82 0)
       (effects (font (size 1.27 1.27)) hide)
     )
@@
       (project "vesc-bms"
         (path "/3e668e3e-3e16-4665-a807-4735962c41d3/6e2b1342-9746-4a38-93af-9ab1059c6272"
-          (reference "#PWR032") (unit 1)
+          (reference "#PWR0404") (unit 1)
         )
       )
@@
   (symbol (lib_id "vesc-bms:E73-2G4M08S1C") (at 229.87 92.71 0) (unit 1)
     (in_bom yes) (on_board yes) (dnp no) (fields_autoplaced)
-    (property "Reference" "U5" (at 231.8894 125.73 0)
+    (property "Reference" "U402" (at 231.8894 125.73 0)
       (effects (font (size 1.27 1.27)) (justify left))
     )
@@
       (project "vesc-bms"
         (path "/3e668e3e-3e16-4665-a807-4735962c41d3/6e2b1342-9746-4a38-93af-9ab1059c6272"
-          (reference "U5") (unit 1)
+          (reference "U402") (unit 1)
         )
       )
@@
   (symbol (lib_id "power:+3.3V") (at 228.6 58.42 0) (unit 1)
     (in_bom yes) (on_board yes) (dnp no) (fields_autoplaced)
-    (property "Reference" "#PWR037" (at 228.6 62.23 0)
+    (property "Reference" "#PWR0409" (at 228.6 62.23 0)
       (effects (font (size 1.27 1.27)) hide)
     )
@@
       (project "vesc-bms"
         (path "/3e668e3e-3e16-4665-a807-4735962c41d3/6e2b1342-9746-4a38-93af-9ab1059c6272"
-          (reference "#PWR037") (unit 1)
+          (reference "#PWR0409") (unit 1)
         )
       )
@@
   (symbol (lib_id "Device:R") (at 107.95 120.65 0) (unit 1)
     (in_bom yes) (on_board yes) (dnp no) (fields_autoplaced)
-    (property "Reference" "R23" (at 110.49 119.3799 0)
+    (property "Reference" "R403" (at 110.49 119.3799 0)
       (effects (font (size 1.27 1.27)) (justify left))
     )
@@
       (project "vesc-bms"
         (path "/3e668e3e-3e16-4665-a807-4735962c41d3/6e2b1342-9746-4a38-93af-9ab1059c6272"
-          (reference "R23") (unit 1)
+          (reference "R403") (unit 1)
         )
       )
@@
   (symbol (lib_id "Interface_CAN_LIN:MCP2562-E-SN") (at 83.82 67.31 0) (unit 1)
     (in_bom yes) (on_board yes) (dnp no) (fields_autoplaced)
-    (property "Reference" "U4" (at 85.8394 54.61 0)
+    (property "Reference" "U401" (at 85.8394 54.61 0)
       (effects (font (size 1.27 1.27)) (justify left))
     )
@@
       (project "vesc-bms"
         (path "/3e668e3e-3e16-4665-a807-4735962c41d3/6e2b1342-9746-4a38-93af-9ab1059c6272"
-          (reference "U4") (unit 1)
+          (reference "U401") (unit 1)
         )
       )
@@
   (symbol (lib_id "Connector:Screw_Terminal_01x02") (at 111.76 66.04 0) (unit 1)
     (in_bom yes) (on_board yes) (dnp no) (fields_autoplaced)
-    (property "Reference" "J6" (at 114.3 66.0399 0)
+    (property "Reference" "J402" (at 114.3 66.0399 0)
       (effects (font (size 1.27 1.27)) (justify left))
     )
@@
       (project "vesc-bms"
         (path "/3e668e3e-3e16-4665-a807-4735962c41d3/6e2b1342-9746-4a38-93af-9ab1059c6272"
-          (reference "J6") (unit 1)
+          (reference "J402") (unit 1)
         )
       )
@@
   (symbol (lib_id "power:VBUS") (at 86.36 107.95 0) (unit 1)
     (in_bom yes) (on_board yes) (dnp no) (fields_autoplaced)
-    (property "Reference" "#PWR033" (at 86.36 111.76 0)
+    (property "Reference" "#PWR0405" (at 86.36 111.76 0)
       (effects (font (size 1.27 1.27)) hide)
     )
@@
       (project "vesc-bms"
         (path "/3e668e3e-3e16-4665-a807-4735962c41d3/6e2b1342-9746-4a38-93af-9ab1059c6272"
-          (reference "#PWR033") (unit 1)
+          (reference "#PWR0405") (unit 1)
         )
       )
@@
   (symbol (lib_id "power:+5V") (at 83.82 57.15 0) (unit 1)
     (in_bom yes) (on_board yes) (dnp no) (fields_autoplaced)
-    (property "Reference" "#PWR031" (at 83.82 60.96 0)
+    (property "Reference" "#PWR0403" (at 83.82 60.96 0)
       (effects (font (size 1.27 1.27)) hide)
     )
@@
       (project "vesc-bms"
         (path "/3e668e3e-3e16-4665-a807-4735962c41d3/6e2b1342-9746-4a38-93af-9ab1059c6272"
-          (reference "#PWR031") (unit 1)
+          (reference "#PWR0403") (unit 1)
         )
       )
@@
   (symbol (lib_id "Connector:Conn_ARM_JTAG_SWD_10") (at 175.26 97.79 0) (unit 1)
     (in_bom yes) (on_board yes) (dnp no) (fields_autoplaced)
-    (property "Reference" "J7" (at 163.83 96.5199 0)
+    (property "Reference" "J403" (at 163.83 96.5199 0)
       (effects (font (size 1.27 1.27)) (justify right))
     )
@@
       (project "vesc-bms"
         (path "/3e668e3e-3e16-4665-a807-4735962c41d3/6e2b1342-9746-4a38-93af-9ab1059c6272"
-          (reference "J7") (unit 1)
-        )
-      )
+          (reference "J403") (unit 1)
+        )
+      )
