File: hardware/comms.kicad_sch (KiCad schematic)
At the start: 8 parts, among them J401 USB_C_Receptacle_USB2.0, J402 CAN, J403 Conn_ARM_JTAG_SWD_10, U401 MCP2562-E-SN, U402 E73-2G4M08S1C

Commit message: BAT to 12V converter
Other:
- company: (none) -> GreenMobi
- title: (none) -> GreenMobi BMS
Changed lines of the file:
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@@
 (kicad_sch (version 20230121) (generator eeschema)
   (paper "A4")
+  (title_block
+    (title "GreenMobi BMS")
+    (date "2024-02-09")
+    (rev "ALPHA")
+    (company "GreenMobi")
+  )
   (junction (at 175.26 113.03) (diameter 0) (color 0 0 0 0)
   )

Commit message: Voltage regulators
Other:
- note removed: "To be replaced by a discrete circuit"
Changed lines of the file:
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@@
-    (effects (font (size 1.27 1.27)) (justify left bottom))
-  )
-  (text "To be replaced by a discrete circuit" (at 153.67 63.5 0)
     (effects (font (size 1.27 1.27)) (justify left bottom))
   )

Commit message: Fix some ERC issues
Parts:
- renumbered J401 to J10, J402 to J11, J403 to J12, R401 to R13, R402 to R14, R403 to R15, U401 to U4, U402 to U5
Changed lines of the file:
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@@
   (symbol (lib_id "Connector:USB_C_Receptacle_USB2.0") (at 68.58 124.46 0) (unit 1)
     (in_bom yes) (on_board yes) (dnp no) (fields_autoplaced)
-    (property "Reference" "J401" (at 68.58 101.6 0)
+    (property "Reference" "J10" (at 68.58 101.6 0)
       (effects (font (size 1.27 1.27)))
     )
@@
       (project "greenmobi-bms"
         (path "/3e668e3e-3e16-4665-a807-4735962c41d3/6e2b1342-9746-4a38-93af-9ab1059c6272"
-          (reference "J401") (unit 1)
+          (reference "J10") (unit 1)
         )
       )
@@
   (symbol (lib_id "power:GND") (at 104.14 125.73 0) (unit 1)
     (in_bom yes) (on_board yes) (dnp no) (fields_autoplaced)
-    (property "Reference" "#PWR0406" (at 104.14 132.08 0)
+    (property "Reference" "#PWR041" (at 104.14 132.08 0)
       (effects (font (size 1.27 1.27)) hide)
     )
@@
       (project "greenmobi-bms"
         (path "/3e668e3e-3e16-4665-a807-4735962c41d3/6e2b1342-9746-4a38-93af-9ab1059c6272"
-          (reference "#PWR0406") (unit 1)
+          (reference "#PWR041") (unit 1)
         )
       )
@@
   (symbol (lib_id "Device:R_Small") (at 99.06 67.31 0) (unit 1)
     (in_bom yes) (on_board yes) (dnp no) (fields_autoplaced)
-    (property "Reference" "R401" (at 101.6 66.0399 0)
+    (property "Reference" "R13" (at 101.6 66.0399 0)
       (effects (font (size 1.27 1.27)) (justify left))
     )
@@
       (project "greenmobi-bms"
         (path "/3e668e3e-3e16-4665-a807-4735962c41d3/6e2b1342-9746-4a38-93af-9ab1059c6272"
-          (reference "R401") (unit 1)
+          (reference "R13") (unit 1)
         )
       )
@@
   (symbol (lib_id "power:+3.3V") (at 58.42 66.04 0) (unit 1)
     (in_bom yes) (on_board yes) (dnp no) (fields_autoplaced)
-    (property "Reference" "#PWR0401" (at 58.42 69.85 0)
+    (property "Reference" "#PWR036" (at 58.42 69.85 0)
       (effects (font (size 1.27 1.27)) hide)
     )
@@
       (project "greenmobi-bms"
         (path "/3e668e3e-3e16-4665-a807-4735962c41d3/6e2b1342-9746-4a38-93af-9ab1059c6272"
-          (reference "#PWR0401") (unit 1)
+          (reference "#PWR036") (unit 1)
         )
       )
@@
   (symbol (lib_id "power:+3.3V") (at 175.26 82.55 0) (unit 1)
     (in_bom yes) (on_board yes) (dnp no) (fields_autoplaced)
-    (property "Reference" "#PWR0407" (at 175.26 86.36 0)
+    (property "Reference" "#PWR042" (at 175.26 86.36 0)
       (effects (font (size 1.27 1.27)) hide)
     )
@@
       (project "greenmobi-bms"
         (path "/3e668e3e-3e16-4665-a807-4735962c41d3/6e2b1342-9746-4a38-93af-9ab1059c6272"
-          (reference "#PWR0407") (unit 1)
+          (reference "#PWR042") (unit 1)
         )
       )
@@
   (symbol (lib_id "power:GND") (at 175.26 114.3 0) (unit 1)
     (in_bom yes) (on_board yes) (dnp no) (fields_autoplaced)
-    (property "Reference" "#PWR0408" (at 175.26 120.65 0)
+    (property "Reference" "#PWR043" (at 175.26 120.65 0)
       (effects (font (size 1.27 1.27)) hide)
     )
@@
       (project "greenmobi-bms"
         (path "/3e668e3e-3e16-4665-a807-4735962c41d3/6e2b1342-9746-4a38-93af-9ab1059c6272"
-          (reference "#PWR0408") (unit 1)
+          (reference "#PWR043") (unit 1)
         )
       )
@@
   (symbol (lib_id "power:GND") (at 229.87 125.73 0) (unit 1)
     (in_bom yes) (on_board yes) (dnp no) (fields_autoplaced)
-    (property "Reference" "#PWR0410" (at 229.87 132.08 0)
+    (property "Reference" "#PWR045" (at 229.87 132.08 0)
       (effects (font (size 1.27 1.27)) hide)
     )
@@
       (project "greenmobi-bms"
         (path "/3e668e3e-3e16-4665-a807-4735962c41d3/6e2b1342-9746-4a38-93af-9ab1059c6272"
-          (reference "#PWR0410") (unit 1)
+          (reference "#PWR045") (unit 1)
         )
       )
@@
   (symbol (lib_id "power:GND") (at 68.58 149.86 0) (unit 1)
     (in_bom yes) (on_board yes) (dnp no) (fields_autoplaced)
-    (property "Reference" "#PWR0402" (at 68.58 156.21 0)
+    (property "Reference" "#PWR037" (at 68.58 156.21 0)
       (effects (font (size 1.27 1.27)) hide)
     )
@@
       (project "greenmobi-bms"
         (path "/3e668e3e-3e16-4665-a807-4735962c41d3/6e2b1342-9746-4a38-93af-9ab1059c6272"
-          (reference "#PWR0402") (unit 1)
+          (reference "#PWR037") (unit 1)
         )
       )
@@
   (symbol (lib_id "Device:R") (at 99.06 120.65 0) (unit 1)
     (in_bom yes) (on_board yes) (dnp no) (fields_autoplaced)
-    (property "Reference" "R402" (at 101.6 119.3799 0)
+    (property "Reference" "R14" (at 101.6 119.3799 0)
       (effects (font (size 1.27 1.27)) (justify left))
     )
@@
       (project "greenmobi-bms"
         (path "/3e668e3e-3e16-4665-a807-4735962c41d3/6e2b1342-9746-4a38-93af-9ab1059c6272"
-          (reference "R402") (unit 1)
+          (reference "R14") (unit 1)
         )
       )
@@
   (symbol (lib_id "power:GND") (at 83.82 77.47 0) (unit 1)
     (in_bom yes) (on_board yes) (dnp no) (fields_autoplaced)
-    (property "Reference" "#PWR0404" (at 83.82 83.82 0)
+    (property "Reference" "#PWR039" (at 83.82 83.82 0)
       (effects (font (size 1.27 1.27)) hide)
     )
@@
       (project "greenmobi-bms"
         (path "/3e668e3e-3e16-4665-a807-4735962c41d3/6e2b1342-9746-4a38-93af-9ab1059c6272"
-          (reference "#PWR0404") (unit 1)
+          (reference "#PWR039") (unit 1)
         )
       )
@@
   (symbol (lib_id "vesc-bms:E73-2G4M08S1C") (at 229.87 92.71 0) (unit 1)
     (in_bom yes) (on_board yes) (dnp no) (fields_autoplaced)
-    (property "Reference" "U402" (at 231.8894 125.73 0)
+    (property "Reference" "U5" (at 231.8894 125.73 0)
       (effects (font (size 1.27 1.27)) (justify left))
     )
@@
       (project "greenmobi-bms"
         (path "/3e668e3e-3e16-4665-a807-4735962c41d3/6e2b1342-9746-4a38-93af-9ab1059c6272"
-          (reference "U402") (unit 1)
+          (reference "U5") (unit 1)
         )
       )
@@
   (symbol (lib_id "power:+3.3V") (at 228.6 58.42 0) (unit 1)
     (in_bom yes) (on_board yes) (dnp no) (fields_autoplaced)
-    (property "Reference" "#PWR0409" (at 228.6 62.23 0)
+    (property "Reference" "#PWR044" (at 228.6 62.23 0)
       (effects (font (size 1.27 1.27)) hide)
     )
@@
       (project "greenmobi-bms"
         (path "/3e668e3e-3e16-4665-a807-4735962c41d3/6e2b1342-9746-4a38-93af-9ab1059c6272"
-          (reference "#PWR0409") (unit 1)
+          (reference "#PWR044") (unit 1)
         )
       )
@@
   (symbol (lib_id "Device:R") (at 107.95 120.65 0) (unit 1)
     (in_bom yes) (on_board yes) (dnp no) (fields_autoplaced)
-    (property "Reference" "R403" (at 110.49 119.3799 0)
+    (property "Reference" "R15" (at 110.49 119.3799 0)
       (effects (font (size 1.27 1.27)) (justify left))
     )
@@
       (project "greenmobi-bms"
         (path "/3e668e3e-3e16-4665-a807-4735962c41d3/6e2b1342-9746-4a38-93af-9ab1059c6272"
-          (reference "R403") (unit 1)
+          (reference "R15") (unit 1)
         )
       )
@@
   (symbol (lib_id "Interface_CAN_LIN:MCP2562-E-SN") (at 83.82 67.31 0) (unit 1)
     (in_bom yes) (on_board yes) (dnp no) (fields_autoplaced)
-    (property "Reference" "U401" (at 85.8394 54.61 0)
+    (property "Reference" "U4" (at 85.8394 54.61 0)
       (effects (font (size 1.27 1.27)) (justify left))
     )
@@
       (project "greenmobi-bms"
         (path "/3e668e3e-3e16-4665-a807-4735962c41d3/6e2b1342-9746-4a38-93af-9ab1059c6272"
-          (reference "U401") (unit 1)
+          (reference "U4") (unit 1)
         )
       )
@@
   (symbol (lib_id "Connector:Screw_Terminal_01x02") (at 111.76 66.04 0) (unit 1)
     (in_bom yes) (on_board yes) (dnp no) (fields_autoplaced)
-    (property "Reference" "J402" (at 114.3 66.0399 0)
+    (property "Reference" "J11" (at 114.3 66.0399 0)
       (effects (font (size 1.27 1.27)) (justify left))
     )
@@
       (project "greenmobi-bms"
         (path "/3e668e3e-3e16-4665-a807-4735962c41d3/6e2b1342-9746-4a38-93af-9ab1059c6272"
-          (reference "J402") (unit 1)
+          (reference "J11") (unit 1)
         )
       )
@@
   (symbol (lib_id "power:VBUS") (at 86.36 107.95 0) (unit 1)
     (in_bom yes) (on_board yes) (dnp no) (fields_autoplaced)
-    (property "Reference" "#PWR0405" (at 86.36 111.76 0)
+    (property "Reference" "#PWR040" (at 86.36 111.76 0)
       (effects (font (size 1.27 1.27)) hide)
     )
@@
       (project "greenmobi-bms"
         (path "/3e668e3e-3e16-4665-a807-4735962c41d3/6e2b1342-9746-4a38-93af-9ab1059c6272"
-          (reference "#PWR0405") (unit 1)
+          (reference "#PWR040") (unit 1)
         )
       )
@@
   (symbol (lib_id "power:+5V") (at 83.82 57.15 0) (unit 1)
     (in_bom yes) (on_board yes) (dnp no) (fields_autoplaced)
-    (property "Reference" "#PWR0403" (at 83.82 60.96 0)
+    (property "Reference" "#PWR038" (at 83.82 60.96 0)
       (effects (font (size 1.27 1.27)) hide)
     )
@@
       (project "greenmobi-bms"
         (path "/3e668e3e-3e16-4665-a807-4735962c41d3/6e2b1342-9746-4a38-93af-9ab1059c6272"
-          (reference "#PWR0403") (unit 1)
+          (reference "#PWR038") (unit 1)
         )
       )
@@
   (symbol (lib_id "Connector:Conn_ARM_JTAG_SWD_10") (at 175.26 97.79 0) (unit 1)
     (in_bom yes) (on_board yes) (dnp no) (fields_autoplaced)
-    (property "Reference" "J403" (at 163.83 96.5199 0)
+    (property "Reference" "J12" (at 163.83 96.5199 0)
       (effects (font (size 1.27 1.27)) (justify right))
     )
@@
       (project "greenmobi-bms"
         (path "/3e668e3e-3e16-4665-a807-4735962c41d3/6e2b1342-9746-4a38-93af-9ab1059c6272"
-          (reference "J403") (unit 1)
-        )
-      )
+          (reference "J12") (unit 1)
+        )
+      )

Commit message: Remove BLE module to increase efficiency
Parts:
- removed J10: USB_C_Receptacle_USB2.0, symbol Connector:USB_C_Receptacle_USB2.0
- removed J12: Conn_ARM_JTAG_SWD_10, Connector_PinHeader_1.27mm:PinHeader_2x05_P1.27mm_Vertical_SMD, symbol Connector:Conn_ARM_JTAG_SWD_10
- removed U5: E73-2G4M08S1C, vesc-bms:E73-2G4M08S1C, symbol vesc-bms:E73-2G4M08S1C
- added J23: USB_C_Receptacle_USB2.0_14P, symbol Connector:USB_C_Receptacle_USB2.0_14P
Connections:
- net GND: now also J23.A1 (GND), J23.A12 (GND), J23.B1 (GND), J23.B12 (GND), J23.S1 (SHIELD)
- net USB_DN: now also J23.A7 (D-), J23.B7 (D-)
- net USB_DP: now also J23.A6 (D+), J23.B6 (D+)
- net VBUS: now also J23.A4 (VBUS), J23.A9 (VBUS), J23.B4 (VBUS), J23.B9 (VBUS)
- net at R15.1: now also J23.A5 (CC1)
- net at R14.1: now also J23.B5 (CC2)
- no-connect marks 36 -> 0
Other:
- note removed: "Bluetooth module"

Commit message: Assigned some footprints
Parts:
- renumbered J23 to J10
Changed lines of the file:
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@@
   (symbol (lib_id "power:GND") (at 104.14 125.73 0) (unit 1)
     (in_bom yes) (on_board yes) (dnp no) (fields_autoplaced)
-    (property "Reference" "#PWR041" (at 104.14 132.08 0)
+    (property "Reference" "#PWR042" (at 104.14 132.08 0)
       (effects (font (size 1.27 1.27)) hide)
     )
@@
       (project "greenmobi-bms"
         (path "/3e668e3e-3e16-4665-a807-4735962c41d3/6e2b1342-9746-4a38-93af-9ab1059c6272"
-          (reference "#PWR041") (unit 1)
+          (reference "#PWR042") (unit 1)
         )
       )
@@
   (symbol (lib_id "power:+3.3V") (at 58.42 66.04 0) (unit 1)
     (in_bom yes) (on_board yes) (dnp no) (fields_autoplaced)
-    (property "Reference" "#PWR036" (at 58.42 69.85 0)
+    (property "Reference" "#PWR037" (at 58.42 69.85 0)
       (effects (font (size 1.27 1.27)) hide)
     )
@@
       (project "greenmobi-bms"
         (path "/3e668e3e-3e16-4665-a807-4735962c41d3/6e2b1342-9746-4a38-93af-9ab1059c6272"
-          (reference "#PWR036") (unit 1)
+          (reference "#PWR037") (unit 1)
         )
       )
@@
   (symbol (lib_id "Connector:USB_C_Receptacle_USB2.0_14P") (at 68.58 124.46 0) (unit 1)
     (in_bom yes) (on_board yes) (dnp no) (fields_autoplaced)
-    (property "Reference" "J23" (at 68.58 101.6 0)
+    (property "Reference" "J10" (at 68.58 101.6 0)
       (effects (font (size 1.27 1.27)))
     )
@@
       (project "greenmobi-bms"
         (path "/3e668e3e-3e16-4665-a807-4735962c41d3/6e2b1342-9746-4a38-93af-9ab1059c6272"
-          (reference "J23") (unit 1)
+          (reference "J10") (unit 1)
         )
       )
@@
   (symbol (lib_id "power:GND") (at 68.58 149.86 0) (unit 1)
     (in_bom yes) (on_board yes) (dnp no) (fields_autoplaced)
-    (property "Reference" "#PWR037" (at 68.58 156.21 0)
+    (property "Reference" "#PWR038" (at 68.58 156.21 0)
       (effects (font (size 1.27 1.27)) hide)
     )
@@
       (project "greenmobi-bms"
         (path "/3e668e3e-3e16-4665-a807-4735962c41d3/6e2b1342-9746-4a38-93af-9ab1059c6272"
-          (reference "#PWR037") (unit 1)
+          (reference "#PWR038") (unit 1)
         )
       )
@@
   (symbol (lib_id "power:GND") (at 83.82 77.47 0) (unit 1)
     (in_bom yes) (on_board yes) (dnp no) (fields_autoplaced)
-    (property "Reference" "#PWR039" (at 83.82 83.82 0)
+    (property "Reference" "#PWR040" (at 83.82 83.82 0)
       (effects (font (size 1.27 1.27)) hide)
     )
@@
       (project "greenmobi-bms"
         (path "/3e668e3e-3e16-4665-a807-4735962c41d3/6e2b1342-9746-4a38-93af-9ab1059c6272"
-          (reference "#PWR039") (unit 1)
+          (reference "#PWR040") (unit 1)
         )
       )
@@
   (symbol (lib_id "power:VBUS") (at 86.36 107.95 0) (unit 1)
     (in_bom yes) (on_board yes) (dnp no) (fields_autoplaced)
-    (property "Reference" "#PWR040" (at 86.36 111.76 0)
+    (property "Reference" "#PWR041" (at 86.36 111.76 0)
       (effects (font (size 1.27 1.27)) hide)
     )
@@
       (project "greenmobi-bms"
         (path "/3e668e3e-3e16-4665-a807-4735962c41d3/6e2b1342-9746-4a38-93af-9ab1059c6272"
-          (reference "#PWR040") (unit 1)
+          (reference "#PWR041") (unit 1)
         )
       )
@@
   (symbol (lib_id "power:+5V") (at 83.82 57.15 0) (unit 1)
     (in_bom yes) (on_board yes) (dnp no) (fields_autoplaced)
-    (property "Reference" "#PWR038" (at 83.82 60.96 0)
+    (property "Reference" "#PWR039" (at 83.82 60.96 0)
       (effects (font (size 1.27 1.27)) hide)
     )
@@
       (project "greenmobi-bms"
         (path "/3e668e3e-3e16-4665-a807-4735962c41d3/6e2b1342-9746-4a38-93af-9ab1059c6272"
-          (reference "#PWR038") (unit 1)
-        )
-      )
+          (reference "#PWR039") (unit 1)
+        )
+      )
