File: hardware/balance_front_end.kicad_sch (KiCad schematic)
At the start: 4 parts, among them Q1 BSS308PE

Commit message: Analog front end ready
Parts:
- renumbered R19 to R21, R20 to R22, R21 to R23
Changed lines of the file:
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@@
   (symbol (lib_id "Device:R_Small") (at 146.05 92.71 90) (unit 1)
     (in_bom yes) (on_board yes)
-    (property "Reference" "R20" (id 0) (at 146.05 87.63 90))
+    (property "Reference" "R22" (id 0) (at 146.05 87.63 90))
     (property "Value" "100" (id 1) (at 146.05 90.17 90))
     (property "Footprint" "" (id 2) (at 146.05 92.71 0)
@@
   (symbol (lib_id "Device:R_Small") (at 139.7 101.6 90) (unit 1)
     (in_bom yes) (on_board yes)
-    (property "Reference" "R19" (id 0) (at 139.7 96.52 90))
+    (property "Reference" "R21" (id 0) (at 139.7 96.52 90))
     (property "Value" "33k" (id 1) (at 139.7 99.06 90))
     (property "Footprint" "" (id 2) (at 139.7 101.6 0)
@@
   (symbol (lib_id "Device:R_Small") (at 152.4 110.49 0) (unit 1)
     (in_bom yes) (on_board yes) (fields_autoplaced)
-    (property "Reference" "R21" (id 0) (at 154.94 109.2199 0)
+    (property "Reference" "R23" (id 0) (at 154.94 109.2199 0)
       (effects (font (size 1.27 1.27)) (justify left))
     )

Commit message: NTC sensors
Parts:
- renumbered R21 to R23, R22 to R24, R23 to R25
Changed lines of the file:
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@@
   (symbol (lib_id "Device:R_Small") (at 146.05 92.71 90) (unit 1)
     (in_bom yes) (on_board yes)
-    (property "Reference" "R22" (id 0) (at 146.05 87.63 90))
+    (property "Reference" "R24" (id 0) (at 146.05 87.63 90))
     (property "Value" "100" (id 1) (at 146.05 90.17 90))
     (property "Footprint" "" (id 2) (at 146.05 92.71 0)
@@
   (symbol (lib_id "Device:R_Small") (at 139.7 101.6 90) (unit 1)
     (in_bom yes) (on_board yes)
-    (property "Reference" "R21" (id 0) (at 139.7 96.52 90))
+    (property "Reference" "R23" (id 0) (at 139.7 96.52 90))
     (property "Value" "33k" (id 1) (at 139.7 99.06 90))
     (property "Footprint" "" (id 2) (at 139.7 101.6 0)
@@
   (symbol (lib_id "Device:R_Small") (at 152.4 110.49 0) (unit 1)
     (in_bom yes) (on_board yes) (fields_autoplaced)
-    (property "Reference" "R23" (id 0) (at 154.94 109.2199 0)
+    (property "Reference" "R25" (id 0) (at 154.94 109.2199 0)
       (effects (font (size 1.27 1.27)) (justify left))
     )

Commit message: Annotate schematic
Parts:
- renumbered Q1 to Q3, R23 to R25, R24 to R26, R25 to R27
Changed lines of the file:
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@@
   (symbol (lib_id "Device:R_Small") (at 146.05 92.71 90) (unit 1)
     (in_bom yes) (on_board yes)
-    (property "Reference" "R24" (id 0) (at 146.05 87.63 90))
+    (property "Reference" "R26" (id 0) (at 146.05 87.63 90))
     (property "Value" "100" (id 1) (at 146.05 90.17 90))
     (property "Footprint" "" (id 2) (at 146.05 92.71 0)
@@
   (symbol (lib_id "vesc-bms:BSS308PE") (at 149.86 101.6 0) (unit 1)
     (in_bom yes) (on_board yes) (fields_autoplaced)
-    (property "Reference" "Q1" (id 0) (at 156.21 100.3299 0)
+    (property "Reference" "Q3" (id 0) (at 156.21 100.3299 0)
       (effects (font (size 1.27 1.27)) (justify left))
     )
@@
   (symbol (lib_id "Device:R_Small") (at 139.7 101.6 90) (unit 1)
     (in_bom yes) (on_board yes)
-    (property "Reference" "R23" (id 0) (at 139.7 96.52 90))
+    (property "Reference" "R25" (id 0) (at 139.7 96.52 90))
     (property "Value" "33k" (id 1) (at 139.7 99.06 90))
     (property "Footprint" "" (id 2) (at 139.7 101.6 0)
@@
   (symbol (lib_id "Device:R_Small") (at 152.4 110.49 0) (unit 1)
     (in_bom yes) (on_board yes) (fields_autoplaced)
-    (property "Reference" "R25" (id 0) (at 154.94 109.2199 0)
+    (property "Reference" "R27" (id 0) (at 154.94 109.2199 0)
       (effects (font (size 1.27 1.27)) (justify left))
     )

Commit message: Update design to KiCAD v7
Parts:
- renumbered Q3 to Q12, R25 to R52, R26 to R53, R27 to R54

Commit message: DNP marks from new KiCAD
Other:
- note added: "~10mA balance current"
Changed lines of the file:
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@@
     (stroke (width 0) (type default))
+  )
+  (text "~10mA balance current" (at 168.91 101.6 0)
+    (effects (font (size 1.27 1.27)) (justify left bottom))
   )
   (hierarchical_label "DISCHARGE_EN" (shape input) (at 137.16 101.6 180) (fields_autoplaced)

Commit message: Fan ports
Parts:
- renumbered Q12 to Q3, R52 to R25, R53 to R26, R54 to R27

Commit message: Charge monitor complete
Parts:
- renumbered Q3 to Q1501, R25 to R1501, R26 to R1502, R27 to R1503

Commit message: Total current sense and buzzer
Parts:
- renumbered Q1501 to Q601, R1501 to R601, R1502 to R602, R1503 to R603
