File: hardware/balance_front_end.kicad_sch (KiCad schematic)
At the start: 5 parts, among them Q601 BSS308PE

Commit message: BAT to 12V converter
Other:
- company: (none) -> GreenMobi
- title: (none) -> GreenMobi BMS
