File: hardware/balance_front_end.kicad_sch (KiCad schematic)
At the start: 5 parts, among them Q4 BSS308PE

Commit message: Remove BLE module to increase efficiency
Parts:
- removed Q4: BSS308PE, Package_TO_SOT_SMD:SOT-23, symbol vesc-bms:BSS308PE
- added Q35: BSS308PE, Package_TO_SOT_SMD:SOT-23, symbol greenmobi-bms:BSS308PE
- renumbered R9 to R78, R10 to R79, R11 to R80, R12 to R81
Connections:
- net CELL: now also Q35.3 (D)
- net at R78.2, R79.2: now also Q35.1 (G)
- net at R79.1, R81.1: now also Q35.2 (S)

Commit message: Assigned some footprints
Parts:
- renumbered Q35 to Q4, R79 to R10, R80 to R11, R81 to R12, R78 to R9

Commit message: Fix orientation of balance FET
Parts:
- renumbered Q4 to Q14, R9 to R78, R10 to R79, R11 to R80, R12 to R81
Connections:
- net CELL: now also Q14.2 (S); no longer Q14.3 (D)
- net at R79.1, R81.1: now also Q14.3 (D); no longer Q14.2 (S)
