File: hardware/charger_monitoring.kicad_sch (KiCad schematic)
At the start: 5 parts, among them U2 BQ76200PW, U9 ACS724xLCTR-30AU

Commit message: Charger monitor
Parts:
- added C49: 1n, symbol Device:C_Small
Connections:
- net GND: now also C49.2
- net Chager+: now reaches U9.1 (IP+), U9.2 (IP+)
- net +BATT: now reaches U9.3 (IP-), U9.4 (IP-)
- net at U9.6 (FILTER): now also C49.1
Changed lines of the file:
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@@
   (junction (at 124.46 90.17) (diameter 0) (color 0 0 0 0)
+  )
+  (wire (pts (xy 102.87 92.71) (xy 105.41 92.71))
+    (stroke (width 0) (type default))
   )
   (polyline (pts (xy 153.67 125.73) (xy 153.67 72.39))
@@
     (stroke (width 0) (type default))
   )
+  (wire (pts (xy 105.41 92.71) (xy 105.41 93.98))
+    (stroke (width 0) (type default))
+  )
   (polyline (pts (xy 156.21 121.92) (xy 228.6 121.92))
     (stroke (width 0) (type default))
@@
     (effects (font (size 1.27 1.27)) (justify left))
   )
+  (hierarchical_label "Chager+" (shape input) (at 82.55 85.09 180) (fields_autoplaced)
+    (effects (font (size 1.27 1.27)) (justify right))
+  )
   (symbol (lib_id "power:GND") (at 92.71 100.33 0) (unit 1)
     (in_bom yes) (on_board yes) (dnp no) (fields_autoplaced)
@@
         (path "/3e668e3e-3e16-4665-a807-4735962c41d3/b1abebf7-38b9-44bd-9506-7ade495be8e0"
           (reference "C46") (unit 1)
+        )
+      )
+    )
+  )
+  (symbol (lib_id "Device:C_Small") (at 105.41 96.52 0) (unit 1)
+    (in_bom yes) (on_board yes) (dnp no) (fields_autoplaced)
+    (property "Reference" "C49" (at 107.95 95.8913 0)
+      (effects (font (size 1.27 1.27)) (justify left))
+    )
+    (property "Value" "1n" (at 107.95 98.4313 0)
+      (effects (font (size 1.27 1.27)) (justify left))
+    )
+    (property "Footprint" "" (at 105.41 96.52 0)
+      (effects (font (size 1.27 1.27)) hide)
+    )
+    (property "Datasheet" "~" (at 105.41 96.52 0)
+      (effects (font (size 1.27 1.27)) hide)
+    )
+    (pin "1")
+    (pin "2")
+    (instances
+      (project "vesc-bms"
+        (path "/3e668e3e-3e16-4665-a807-4735962c41d3/b1abebf7-38b9-44bd-9506-7ade495be8e0"
+          (reference "C49") (unit 1)
         )
       )
@@
         (path "/3e668e3e-3e16-4665-a807-4735962c41d3/b1abebf7-38b9-44bd-9506-7ade495be8e0"
           (reference "U9") (unit 1)
+        )
+      )
+    )
+  )
+  (symbol (lib_id "power:+BATT") (at 82.55 95.25 90) (unit 1)
+    (in_bom yes) (on_board yes) (dnp no) (fields_autoplaced)
+    (property "Reference" "#PWR068" (at 86.36 95.25 0)
+      (effects (font (size 1.27 1.27)) hide)
+    )
+    (property "Value" "+BATT" (at 78.74 95.885 90)
+      (effects (font (size 1.27 1.27)) (justify left))
+    )
+    (property "Footprint" "" (at 82.55 95.25 0)
+      (effects (font (size 1.27 1.27)) hide)
+    )
+    (property "Datasheet" "" (at 82.55 95.25 0)
+      (effects (font (size 1.27 1.27)) hide)
+    )
+    (pin "1")
+    (instances
+      (project "vesc-bms"
+        (path "/3e668e3e-3e16-4665-a807-4735962c41d3/b1abebf7-38b9-44bd-9506-7ade495be8e0"
+          (reference "#PWR068") (unit 1)
         )
       )
@@
         )
       )
+    )
+  )
+  (symbol (lib_id "power:GND") (at 105.41 99.06 0) (unit 1)
+    (in_bom yes) (on_board yes) (dnp no) (fields_autoplaced)
+    (property "Reference" "#PWR?" (at 105.41 105.41 0)
+      (effects (font (size 1.27 1.27)) hide)
+    )
+    (property "Value" "GND" (at 105.41 104.14 0)
+      (effects (font (size 1.27 1.27)))
+    )
+    (property "Footprint" "" (at 105.41 99.06 0)
+      (effects (font (size 1.27 1.27)) hide)
+    )
+    (property "Datasheet" "" (at 105.41 99.06 0)
+      (effects (font (size 1.27 1.27)) hide)
+    )
+    (pin "1")
+    (instances
+      (project "vesc-bms"
+        (path "/3e668e3e-3e16-4665-a807-4735962c41d3/a908ff77-32fe-48f6-8dc7-bc7bb4d76281"
+          (reference "#PWR?") (unit 1)
+        )
+        (path "/3e668e3e-3e16-4665-a807-4735962c41d3/b1abebf7-38b9-44bd-9506-7ade495be8e0"
+          (reference "#PWR069") (unit 1)
+        )
+      )

Commit message: Initial work on High side switch
Parts:
- added C50: 10n, symbol Device:C_Small
- added C51: 470n, symbol Device:C_Small
- added Q23, Q24: IPT015N10N5, Package_TO_SOT_SMD:Infineon_PG-HSOF-8-1, symbol Transistor_FET:IPT015N10N5
- added Q25: IRFR120NTRPBF, Package_TO_SOT_SMD:TO-252-2, symbol vesc-bms:IRFR120NTRPBF
- added R89: 100, symbol Device:R_Small
- added R90, R91, R92: 10, symbol Device:R
Connections:
- net +BATT: now also Q24.2 (S), R89.1, R90.1, R91.1, R92.1; no longer U9.3 (IP-), U9.4 (IP-)
- net GND: now also U2.9 (VSS), C50.2
- net at U2.1 (VDDCP): now also C51.1
- net at U2.11 (PACK): now also C51.2
- net at U2.12 (DSG): now also Q23.1 (G)
- net at U2.14 (PCHG): now also Q25.1 (G)
- net at U2.16 (CHG): now also Q24.1 (G)
- net at U2.2 (BAT): now also C50.1, R89.2
- net CHG_EN: now reaches U2.4 (CHG_EN)
- net CP_EN: now reaches U2.5 (CP_EN)
- net DSG_EN: now reaches U2.6 (DSG_EN)
- net PMON_EN: now reaches U2.7 (PMON_EN)
- net PCHG_EN: now reaches U2.8 (PCHG_EN)
- new net: Q25.2 (D), R90.2, R91.2, R92.2
- new net: U9.3 (IP-), U9.4 (IP-)
- new net: Q23.3 (D), Q24.3 (D), Q25.3 (S)
- new net PACK+: Q23.2 (S)
Other:
- note removed: "24A max"
- note removed: "7.5A typ"
- moved on the sheet: C49, C?, R?, U2, U9

Commit message: Charger enable circiut and more ext NTC
Parts:
- added R93, R94, R95: 10, Resistor_SMD:R_2010_5025Metric, symbol Device:R
- R90, R91, R92: footprint (none) -> Resistor_SMD:R_2010_5025Metric
Connections:
- net +BATT: now also U9.3 (IP-), U9.4 (IP-); no longer Q24.2 (S), R90.1, R91.1, R92.1
- net Chager+: now also Q24.2 (S), R90.1, R91.1, R92.1, R93.1, R94.1, R95.1; no longer U9.1 (IP+), U9.2 (IP+)
- net at Q25.2 (D), R90.2, R91.2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: now also R93.2, R94.2
- net PACK+ renamed Charger_s
- net Charger_s: now also U9.1 (IP+), U9.2 (IP+)
Other:
- moved on the sheet: C49, C?, Q23, Q24, Q25, R90, R91, R92, R?, U9

Commit message: Charge monitor complete
Parts:
- removed R93, R94: 10, Resistor_SMD:R_2010_5025Metric, symbol Device:R
- added C2806: 100n, symbol Device:C_Small
- added C2807: 10n, symbol Device:C_Small
- added R2803: 100k, symbol Device:R_Small
- added R2804: 3.9k, symbol Device:R_Small
- added R2805: 1k, symbol Device:R_Small
- added R2810, R2811, R2812: 10M, symbol Device:R_Small
- added R2813: 100, symbol Device:R_Small
- R2806: renamed from R95; value 10 -> 1k; footprint Resistor_SMD:R_2010_5025Metric -> Resistor_SMD:R_2512_6332Metric
- R2807: renamed from R92; value 10 -> 1k; footprint Resistor_SMD:R_2010_5025Metric -> Resistor_SMD:R_2512_6332Metric
- R2808: renamed from R90; value 10 -> 1k; footprint Resistor_SMD:R_2010_5025Metric -> Resistor_SMD:R_2512_6332Metric
- R2809: renamed from R91; value 10 -> 1k; footprint Resistor_SMD:R_2010_5025Metric -> Resistor_SMD:R_2512_6332Metric
- renumbered C49 to C2802, C50 to C2803, C51 to C2805, Q25 to Q2801, Q24 to Q2802, Q23 to Q2803, R89 to R2801, U9 to U2801
Connections:
- net +BATT: no longer R2801.1
- net Charger_s: now also Q2802.2 (S), R2801.1, R2806.1, R2807.1, R2810.1; no longer Q2803.2 (S)
- net GND: now also C2806.2, C2807.2, R2804.2
- net at Q2801.2 (D), R2808.2, R2809.2: no longer R2807.2
- net at R2806.2: now also R2807.2, R2808.1, R2809.1
- net at Q2802.1 (G), U2.16 (CHG): now also R2810.2
- net at Q2801.3 (S), Q2802.3 (D), Q2803.3 (D): now also R2811.1, R2812.1
- net at C2803.1, R2801.2, U2.2 (BAT): now also C2805.2
- net at U2.10 (PACKDIV): now also R2803.1
- net at U2.11 (PACK): now also C2807.1, R2813.1; no longer C2805.2
- net at Q2803.1 (G), U2.12 (DSG): now also R2812.2
- net at Q2801.1 (G), U2.14 (PCHG): now also R2811.2
- removed net Chager+: Q2802.2 (S), R2806.1, R2807.1, R2808.1, R2809.1
- new net: R2803.2, R2804.1, R2805.1
- new net Charger: Q2803.2 (S), R2813.2
- new net PACK_V: C2806.1, R2805.2
Other:
- note added: "Max 80V (18S)"
- moved on the sheet: C2802, C2803, C2805, C?, Q2801, Q2802, Q2803, R2801, R2806, R2807, R2808, R2809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

Commit message: Total current sense and buzzer
Connections:
- net +BATT renamed BAT+
Changed lines of the file:
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@@
+    (effects (font (size 1.27 1.27)) (justify right))
+  )
+  (hierarchical_label "BAT+" (shape output) (at 76.2 154.94 180) (fields_autoplaced)
     (effects (font (size 1.27 1.27)) (justify right))
   )
@@
         )
       )
-    )
-  )
-  (symbol (lib_id "power:+BATT") (at 76.2 154.94 90) (unit 1)
-    (in_bom yes) (on_board yes) (dnp no) (fields_autoplaced)
-    (property "Reference" "#PWR02803" (at 80.01 154.94 0)
-      (effects (font (size 1.27 1.27)) hide)
-    )
-    (property "Value" "+BATT" (at 72.39 155.575 90)
-      (effects (font (size 1.27 1.27)) (justify left))
-    )
-    (property "Footprint" "" (at 76.2 154.94 0)
-      (effects (font (size 1.27 1.27)) hide)
-    )
-    (property "Datasheet" "" (at 76.2 154.94 0)
-      (effects (font (size 1.27 1.27)) hide)
-    )
-    (pin "1")
-    (instances
-      (project "vesc-bms"
-        (path "/3e668e3e-3e16-4665-a807-4735962c41d3/b1abebf7-38b9-44bd-9506-7ade495be8e0"
-          (reference "#PWR02803") (unit 1)
-        )
-      )
