File: hardware/charger_monitoring.kicad_sch (KiCad schematic)
At the start: 24 parts, among them Q2801 IRFR120NTRPBF, Q2802 IPT015N10N5, Q2803 IPT015N10N5, U2802 BQ76200PW, U4 ACS770xCB-050B-PFF

Commit message: Fix OLED pinout and add HDC1080
Other:
- moved on the sheet: C2803, C2805, C2806, C2807, Q2801, Q2802, Q2803, R2801, R2803, R2804, R2805, R2806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

Commit message: Charger connector
Parts:
- removed U4: ACS770xCB-050B-PFF, Sensor_Current:Allegro_CB_PFF, symbol Sensor_Current:ACS770xCB-050B-PFF
- added U2: ACS770xCB-050U-PFF, Sensor_Current:Allegro_CB_PFF, symbol Sensor_Current:ACS770xCB-050U-PFF
Connections:
- net +3.3V: now also U2.1 (VCC)
- net BAT+: now also U2.5 (IP-)
- net Charger_s: now also U2.4 (IP+)
- net GND: now also U2.2 (GND)
- net at R2802.1: now also U2.3 (VIOUT)
Changed lines of the file:
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@@
-    )
-  )
-  (symbol (lib_id "Sensor_Current:ACS770xCB-050B-PFF") (at 86.36 149.86 0) (unit 1)
-    (in_bom yes) (on_board yes) (dnp no)
-    (property "Reference" "U4" (at 88.9 140.97 0)
-      (effects (font (size 1.27 1.27)))
-    )
-    (property "Value" "ACS770xCB-050B-PFF" (at 97.79 143.51 0)
-      (effects (font (size 1.27 1.27)))
-    )
-    (property "Footprint" "Sensor_Current:Allegro_CB_PFF" (at 86.36 149.86 0)
-      (effects (font (size 1.27 1.27)) hide)
-    )
-    (property "Datasheet" "http://www.allegromicro.com/~/media/Files/Datasheets/ACS758-Datasheet.ashx?la=en" (at 86.36 149.86 0)
-      (effects (font (size 1.27 1.27)) hide)
-    )
-    (pin "4")
-    (pin "5")
-    (pin "1")
-    (pin "3")
-    (pin "2")
-    (instances
-      (project "greenmobi-bms"
-        (path "/3e668e3e-3e16-4665-a807-4735962c41d3/b1abebf7-38b9-44bd-9506-7ade495be8e0"
-          (reference "U4") (unit 1)
-        )
-      )
     )
   )
@@
         )
       )
+    )
+  )
+  (symbol (lib_id "Sensor_Current:ACS770xCB-050U-PFF") (at 86.36 149.86 0) (unit 1)
+    (in_bom yes) (on_board yes) (dnp no)
+    (property "Reference" "U2" (at 88.9 140.97 0)
+      (effects (font (size 1.27 1.27)))
+    )
+    (property "Value" "ACS770xCB-050U-PFF" (at 97.79 143.51 0)
+      (effects (font (size 1.27 1.27)))
+    )
+    (property "Footprint" "Sensor_Current:Allegro_CB_PFF" (at 86.36 149.86 0)
+      (effects (font (size 1.27 1.27)) hide)
+    )
+    (property "Datasheet" "http://www.allegromicro.com/~/media/Files/Datasheets/ACS758-Datasheet.ashx?la=en" (at 86.36 149.86 0)
+      (effects (font (size 1.27 1.27)) hide)
+    )
+    (pin "1")
+    (pin "4")
+    (pin "3")
+    (pin "2")
+    (pin "5")
+    (instances
+      (project "greenmobi-bms"
+        (path "/3e668e3e-3e16-4665-a807-4735962c41d3/b1abebf7-38b9-44bd-9506-7ade495be8e0"
+          (reference "U2") (unit 1)
+        )
+      )

Commit message: BAT to 12V converter
Other:
- company: (none) -> GreenMobi
- title: (none) -> GreenMobi BMS
Changed lines of the file:
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@@
 (kicad_sch (version 20230121) (generator eeschema)
   (paper "A4")
+  (title_block
+    (title "GreenMobi BMS")
+    (date "2024-02-09")
+    (rev "ALPHA")
+    (company "GreenMobi")
+  )
   (junction (at 167.64 35.56) (diameter 0) (color 0 0 0 0)
   )

Commit message: Fix some ERC issues
Parts:
- renumbered C2801 to C66, C2804 to C67, C2806 to C68, C2805 to C69, C2807 to C70, C2803 to C71, Q2803 to Q20, Q2802 to Q21, Q2801 to Q22, R2812 to R108, R2802 to R109, R2811 to R110, R2810 to R111, R2808 to R112, R2809 to R113, R2806 to R114, R2807 to R115, R2805 to R116, R2803 to R117, R2804 to R118, R2813 to R119, R2801 to R120, U2 to U10, U2802 to U11

Commit message: Remove BLE module to increase efficiency
Parts:
- removed Q22: IRFR120NTRPBF, Package_TO_SOT_SMD:TO-252-2, symbol vesc-bms:IRFR120NTRPBF
- added Q4: IRFR120NTRPBF, Package_TO_SOT_SMD:TO-252-2, symbol greenmobi-bms:IRFR120NTRPBF
Connections:
- net at R112.2, R113.2: now also Q4.2 (D)
- net at Q20.3 (D), Q21.3 (D), R108.1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: now also Q4.3 (S)
- net at R110.2, U11.14 (PCHG): now also Q4.1 (G)
Changed lines of the file:
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@@
     (company "GreenMobi")
   )
+  (junction (at 132.08 43.18) (diameter 0) (color 0 0 0 0)
+  )
   (junction (at 167.64 35.56) (diameter 0) (color 0 0 0 0)
   )
@@
   )
   (junction (at 118.11 149.86) (diameter 0) (color 0 0 0 0)
-  )
-  (junction (at 132.08 43.18) (diameter 0) (color 0 0 0 0)
   )
   (junction (at 104.14 78.74) (diameter 0) (color 0 0 0 0)
@@
     (stroke (width 0) (type default))
   )
-  (wire (pts (xy 125.73 35.56) (xy 104.14 35.56))
+  (wire (pts (xy 104.14 35.56) (xy 125.73 35.56))
     (stroke (width 0) (type default))
   )
@@
         (path "/3e668e3e-3e16-4665-a807-4735962c41d3/b1abebf7-38b9-44bd-9506-7ade495be8e0"
           (reference "R120") (unit 1)
+        )
+      )
+    )
+  )
+  (symbol (lib_id "power:PWR_FLAG") (at 215.9 58.42 0) (unit 1)
+    (in_bom yes) (on_board yes) (dnp no) (fields_autoplaced)
+    (property "Reference" "#FLG08" (at 215.9 56.515 0)
+      (effects (font (size 1.27 1.27)) hide)
+    )
+    (property "Value" "PWR_FLAG" (at 215.9 53.34 0)
+      (effects (font (size 1.27 1.27)) hide)
+    )
+    (property "Footprint" "" (at 215.9 58.42 0)
+      (effects (font (size 1.27 1.27)) hide)
+    )
+    (property "Datasheet" "~" (at 215.9 58.42 0)
+      (effects (font (size 1.27 1.27)) hide)
+    )
+    (pin "1")
+    (instances
+      (project "greenmobi-bms"
+        (path "/3e668e3e-3e16-4665-a807-4735962c41d3/b1abebf7-38b9-44bd-9506-7ade495be8e0"
+          (reference "#FLG08") (unit 1)
         )
       )
@@
     )
   )
-  (symbol (lib_id "vesc-bms:IRFR120NTRPBF") (at 132.08 38.1 270) (mirror x) (unit 1)
-    (in_bom yes) (on_board yes) (dnp no) (fields_autoplaced)
-    (property "Reference" "Q22" (at 132.08 29.21 90)
+  (symbol (lib_id "power:PWR_FLAG") (at 189.23 44.45 0) (unit 1)
+    (in_bom yes) (on_board yes) (dnp no) (fields_autoplaced)
+    (property "Reference" "#FLG09" (at 189.23 42.545 0)
+      (effects (font (size 1.27 1.27)) hide)
+    )
+    (property "Value" "PWR_FLAG" (at 189.23 39.37 0)
+      (effects (font (size 1.27 1.27)) hide)
+    )
+    (property "Footprint" "" (at 189.23 44.45 0)
+      (effects (font (size 1.27 1.27)) hide)
+    )
+    (property "Datasheet" "~" (at 189.23 44.45 0)
+      (effects (font (size 1.27 1.27)) hide)
+    )
+    (pin "1")
+    (instances
+      (project "greenmobi-bms"
+        (path "/3e668e3e-3e16-4665-a807-4735962c41d3/b1abebf7-38b9-44bd-9506-7ade495be8e0"
+          (reference "#FLG09") (unit 1)
+        )
+      )
+    )
+  )
+  (symbol (lib_id "Device:C_Small") (at 74.93 173.99 0) (unit 1)
+    (in_bom yes) (on_board yes) (dnp no) (fields_autoplaced)
+    (property "Reference" "C66" (at 77.47 172.7262 0)
+      (effects (font (size 1.27 1.27)) (justify left))
+    )
+    (property "Value" "100n" (at 77.47 175.2662 0)
+      (effects (font (size 1.27 1.27)) (justify left))
+    )
+    (property "Footprint" "" (at 74.93 173.99 0)
+      (effects (font (size 1.27 1.27)) hide)
+    )
+    (property "Datasheet" "~" (at 74.93 173.99 0)
+      (effects (font (size 1.27 1.27)) hide)
+    )
+    (pin "1")
+    (pin "2")
+    (instances
+      (project "greenmobi-bms"
+        (path "/3e668e3e-3e16-4665-a807-4735962c41d3/b1abebf7-38b9-44bd-9506-7ade495be8e0"
+          (reference "C66") (unit 1)
+        )
+      )
+    )
+  )
+  (symbol (lib_id "power:GND") (at 195.58 93.98 0) (mirror y) (unit 1)
+    (in_bom yes) (on_board yes) (dnp no) (fields_autoplaced)
+    (property "Reference" "#PWR0104" (at 195.58 100.33 0)
+      (effects (font (size 1.27 1.27)) hide)
+    )
+    (property "Value" "GND" (at 195.58 99.06 0)
+      (effects (font (size 1.27 1.27)))
+    )
+    (property "Footprint" "" (at 195.58 93.98 0)
+      (effects (font (size 1.27 1.27)) hide)
+    )
+    (property "Datasheet" "" (at 195.58 93.98 0)
+      (effects (font (size 1.27 1.27)) hide)
+    )
+    (pin "1")
+    (instances
+      (project "greenmobi-bms"
+        (path "/3e668e3e-3e16-4665-a807-4735962c41d3/b1abebf7-38b9-44bd-9506-7ade495be8e0"
+          (reference "#PWR0104") (unit 1)
+        )
+      )
+    )
+  )
+  (symbol (lib_id "Device:C_Small") (at 215.9 62.23 0) (mirror y) (unit 1)
+    (in_bom yes) (on_board yes) (dnp no) (fields_autoplaced)
+    (property "Reference" "C71" (at 213.36 61.6013 0)
+      (effects (font (size 1.27 1.27)) (justify left))
+    )
+    (property "Value" "10n" (at 213.36 64.1413 0)
+      (effects (font (size 1.27 1.27)) (justify left))
+    )
+    (property "Footprint" "" (at 215.9 62.23 0)
+      (effects (font (size 1.27 1.27)) hide)
+    )
+    (property "Datasheet" "~" (at 215.9 62.23 0)
+      (effects (font (size 1.27 1.27)) hide)
+    )
+    (pin "1")
+    (pin "2")
+    (instances
+      (project "greenmobi-bms"
+        (path "/3e668e3e-3e16-4665-a807-4735962c41d3/b1abebf7-38b9-44bd-9506-7ade495be8e0"
+          (reference "C71") (unit 1)
+        )
+      )
+    )
+  )
+  (symbol (lib_id "Device:R_Small") (at 104.14 72.39 0) (mirror y) (unit 1)
+    (in_bom yes) (on_board yes) (dnp no) (fields_autoplaced)
+    (property "Reference" "R108" (at 101.6 71.12 0)
+      (effects (font (size 1.27 1.27)) (justify left))
+    )
+    (property "Value" "10M" (at 101.6 73.66 0)
+      (effects (font (size 1.27 1.27)) (justify left))
+    )
+    (property "Footprint" "" (at 104.14 72.39 0)
+      (effects (font (size 1.27 1.27)) hide)
+    )
+    (property "Datasheet" "~" (at 104.14 72.39 0)
+      (effects (font (size 1.27 1.27)) hide)
+    )
+    (pin "1")
+    (pin "2")
+    (instances
+      (project "greenmobi-bms"
+        (path "/3e668e3e-3e16-4665-a807-4735962c41d3/b1abebf7-38b9-44bd-9506-7ade495be8e0"
+          (reference "R108") (unit 1)
+        )
+      )
+    )
+  )
+  (symbol (lib_id "greenmobi-bms:IRFR120NTRPBF") (at 132.08 38.1 270) (mirror x) (unit 1)
+    (in_bom yes) (on_board yes) (dnp no) (fields_autoplaced)
+    (property "Reference" "Q4" (at 132.08 29.21 90)
       (effects (font (size 1.27 1.27)))
     )
@@
       (effects (font (size 1.27 1.27)) (justify left) hide)
     )
-    (pin "1")
-    (pin "2")
     (pin "3")
-    (instances
-      (project "greenmobi-bms"
-        (path "/3e668e3e-3e16-4665-a807-4735962c41d3/b1abebf7-38b9-44bd-9506-7ade495be8e0"
-          (reference "Q22") (unit 1)
-        )
-      )
-    )
-  )
-  (symbol (lib_id "Device:C_Small") (at 74.93 173.99 0) (unit 1)
-    (in_bom yes) (on_board yes) (dnp no) (fields_autoplaced)
-    (property "Reference" "C66" (at 77.47 172.7262 0)
-      (effects (font (size 1.27 1.27)) (justify left))
-    )
-    (property "Value" "100n" (at 77.47 175.2662 0)
-      (effects (font (size 1.27 1.27)) (justify left))
-    )
-    (property "Footprint" "" (at 74.93 173.99 0)
-      (effects (font (size 1.27 1.27)) hide)
-    )
-    (property "Datasheet" "~" (at 74.93 173.99 0)
-      (effects (font (size 1.27 1.27)) hide)
-    )
-    (pin "1")
-    (pin "2")
-    (instances
-      (project "greenmobi-bms"
-        (path "/3e668e3e-3e16-4665-a807-4735962c41d3/b1abebf7-38b9-44bd-9506-7ade495be8e0"
-          (reference "C66") (unit 1)
-        )
-      )
-    )
-  )
-  (symbol (lib_id "power:GND") (at 195.58 93.98 0) (mirror y) (unit 1)
-    (in_bom yes) (on_board yes) (dnp no) (fields_autoplaced)
-    (property "Reference" "#PWR0104" (at 195.58 100.33 0)
-      (effects (font (size 1.27 1.27)) hide)
-    )
-    (property "Value" "GND" (at 195.58 99.06 0)
-      (effects (font (size 1.27 1.27)))
-    )
-    (property "Footprint" "" (at 195.58 93.98 0)
-      (effects (font (size 1.27 1.27)) hide)
-    )
-    (property "Datasheet" "" (at 195.58 93.98 0)
-      (effects (font (size 1.27 1.27)) hide)
-    )
-    (pin "1")
-    (instances
-      (project "greenmobi-bms"
-        (path "/3e668e3e-3e16-4665-a807-4735962c41d3/b1abebf7-38b9-44bd-9506-7ade495be8e0"
-          (reference "#PWR0104") (unit 1)
-        )
-      )
-    )
-  )
-  (symbol (lib_id "Device:C_Small") (at 215.9 62.23 0) (mirror y) (unit 1)
-    (in_bom yes) (on_board yes) (dnp no) (fields_autoplaced)
-    (property "Reference" "C71" (at 213.36 61.6013 0)
-      (effects (font (size 1.27 1.27)) (justify left))
-    )
-    (property "Value" "10n" (at 213.36 64.1413 0)
-      (effects (font (size 1.27 1.27)) (justify left))
-    )
-    (property "Footprint" "" (at 215.9 62.23 0)
-      (effects (font (size 1.27 1.27)) hide)
-    )
-    (property "Datasheet" "~" (at 215.9 62.23 0)
-      (effects (font (size 1.27 1.27)) hide)
-    )
-    (pin "1")
-    (pin "2")
-    (instances
-      (project "greenmobi-bms"
-        (path "/3e668e3e-3e16-4665-a807-4735962c41d3/b1abebf7-38b9-44bd-9506-7ade495be8e0"
-          (reference "C71") (unit 1)
-        )
-      )
-    )
-  )
-  (symbol (lib_id "Device:R_Small") (at 104.14 72.39 0) (mirror y) (unit 1)
-    (in_bom yes) (on_board yes) (dnp no) (fields_autoplaced)
-    (property "Reference" "R108" (at 101.6 71.12 0)
-      (effects (font (size 1.27 1.27)) (justify left))
-    )
-    (property "Value" "10M" (at 101.6 73.66 0)
-      (effects (font (size 1.27 1.27)) (justify left))
-    )
-    (property "Footprint" "" (at 104.14 72.39 0)
-      (effects (font (size 1.27 1.27)) hide)
-    )
-    (property "Datasheet" "~" (at 104.14 72.39 0)
-      (effects (font (size 1.27 1.27)) hide)
-    )
-    (pin "1")
-    (pin "2")
-    (instances
-      (project "greenmobi-bms"
-        (path "/3e668e3e-3e16-4665-a807-4735962c41d3/b1abebf7-38b9-44bd-9506-7ade495be8e0"
-          (reference "R108") (unit 1)
-        )
-      )
+    (pin "1")
+    (pin "2")
+    (instances
+      (project "greenmobi-bms"
+        (path "/3e668e3e-3e16-4665-a807-4735962c41d3/b1abebf7-38b9-44bd-9506-7ade495be8e0"
+          (reference "Q4") (unit 1)
+        )
+      )

Commit message: Assigned some footprints
Parts:
- renumbered Q4 to Q22, U11 to U10, U10 to U9
Changed lines of the file:
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@@
   (symbol (lib_id "power:GND") (at 176.53 100.33 0) (mirror y) (unit 1)
     (in_bom yes) (on_board yes) (dnp no) (fields_autoplaced)
-    (property "Reference" "#PWR0102" (at 176.53 106.68 0)
+    (property "Reference" "#PWR0107" (at 176.53 106.68 0)
       (effects (font (size 1.27 1.27)) hide)
     )
@@
       (project "greenmobi-bms"
         (path "/3e668e3e-3e16-4665-a807-4735962c41d3/b1abebf7-38b9-44bd-9506-7ade495be8e0"
-          (reference "#PWR0102") (unit 1)
+          (reference "#PWR0107") (unit 1)
         )
       )
@@
   (symbol (lib_id "power:GND") (at 86.36 157.48 0) (unit 1)
     (in_bom yes) (on_board yes) (dnp no) (fields_autoplaced)
-    (property "Reference" "#PWR099" (at 86.36 163.83 0)
+    (property "Reference" "#PWR0104" (at 86.36 163.83 0)
       (effects (font (size 1.27 1.27)) hide)
     )
@@
       (project "greenmobi-bms"
         (path "/3e668e3e-3e16-4665-a807-4735962c41d3/b1abebf7-38b9-44bd-9506-7ade495be8e0"
-          (reference "#PWR099") (unit 1)
+          (reference "#PWR0104") (unit 1)
         )
       )
@@
   (symbol (lib_id "power:GND") (at 152.4 100.33 0) (mirror y) (unit 1)
     (in_bom yes) (on_board yes) (dnp no) (fields_autoplaced)
-    (property "Reference" "#PWR0101" (at 152.4 106.68 0)
+    (property "Reference" "#PWR0106" (at 152.4 106.68 0)
       (effects (font (size 1.27 1.27)) hide)
     )
@@
       (project "greenmobi-bms"
         (path "/3e668e3e-3e16-4665-a807-4735962c41d3/b1abebf7-38b9-44bd-9506-7ade495be8e0"
-          (reference "#PWR0101") (unit 1)
+          (reference "#PWR0106") (unit 1)
         )
       )
@@
   (symbol (lib_id "power:GND") (at 74.93 176.53 0) (unit 1)
     (in_bom yes) (on_board yes) (dnp no) (fields_autoplaced)
-    (property "Reference" "#PWR097" (at 74.93 182.88 0)
+    (property "Reference" "#PWR0102" (at 74.93 182.88 0)
       (effects (font (size 1.27 1.27)) hide)
     )
@@
       (project "greenmobi-bms"
         (path "/3e668e3e-3e16-4665-a807-4735962c41d3/b1abebf7-38b9-44bd-9506-7ade495be8e0"
-          (reference "#PWR097") (unit 1)
+          (reference "#PWR0102") (unit 1)
         )
       )
@@
   (symbol (lib_id "power:PWR_FLAG") (at 215.9 58.42 0) (unit 1)
     (in_bom yes) (on_board yes) (dnp no) (fields_autoplaced)
-    (property "Reference" "#FLG08" (at 215.9 56.515 0)
+    (property "Reference" "#FLG09" (at 215.9 56.515 0)
       (effects (font (size 1.27 1.27)) hide)
     )
@@
       (project "greenmobi-bms"
         (path "/3e668e3e-3e16-4665-a807-4735962c41d3/b1abebf7-38b9-44bd-9506-7ade495be8e0"
-          (reference "#FLG08") (unit 1)
+          (reference "#FLG09") (unit 1)
         )
       )
@@
   (symbol (lib_id "power:+3.3V") (at 74.93 171.45 0) (unit 1)
     (in_bom yes) (on_board yes) (dnp no) (fields_autoplaced)
-    (property "Reference" "#PWR096" (at 74.93 175.26 0)
+    (property "Reference" "#PWR0101" (at 74.93 175.26 0)
       (effects (font (size 1.27 1.27)) hide)
     )
@@
       (project "greenmobi-bms"
         (path "/3e668e3e-3e16-4665-a807-4735962c41d3/b1abebf7-38b9-44bd-9506-7ade495be8e0"
-          (reference "#PWR096") (unit 1)
+          (reference "#PWR0101") (unit 1)
         )
       )
@@
   (symbol (lib_id "Battery_Management:BQ76200PW") (at 195.58 78.74 0) (mirror y) (unit 1)
     (in_bom yes) (on_board yes) (dnp no) (fields_autoplaced)
-    (property "Reference" "U11" (at 193.5606 93.98 0)
+    (property "Reference" "U10" (at 193.5606 93.98 0)
       (effects (font (size 1.27 1.27)) (justify left))
     )
@@
       (project "greenmobi-bms"
         (path "/3e668e3e-3e16-4665-a807-4735962c41d3/b1abebf7-38b9-44bd-9506-7ade495be8e0"
-          (reference "U11") (unit 1)
+          (reference "U10") (unit 1)
         )
       )
@@
   (symbol (lib_id "power:PWR_FLAG") (at 189.23 44.45 0) (unit 1)
     (in_bom yes) (on_board yes) (dnp no) (fields_autoplaced)
-    (property "Reference" "#FLG09" (at 189.23 42.545 0)
+    (property "Reference" "#FLG08" (at 189.23 42.545 0)
       (effects (font (size 1.27 1.27)) hide)
     )
@@
       (project "greenmobi-bms"
         (path "/3e668e3e-3e16-4665-a807-4735962c41d3/b1abebf7-38b9-44bd-9506-7ade495be8e0"
-          (reference "#FLG09") (unit 1)
+          (reference "#FLG08") (unit 1)
         )
       )
@@
   (symbol (lib_id "power:GND") (at 195.58 93.98 0) (mirror y) (unit 1)
     (in_bom yes) (on_board yes) (dnp no) (fields_autoplaced)
-    (property "Reference" "#PWR0104" (at 195.58 100.33 0)
+    (property "Reference" "#PWR0109" (at 195.58 100.33 0)
       (effects (font (size 1.27 1.27)) hide)
     )
@@
       (project "greenmobi-bms"
         (path "/3e668e3e-3e16-4665-a807-4735962c41d3/b1abebf7-38b9-44bd-9506-7ade495be8e0"
-          (reference "#PWR0104") (unit 1)
+          (reference "#PWR0109") (unit 1)
         )
       )
@@
   (symbol (lib_id "greenmobi-bms:IRFR120NTRPBF") (at 132.08 38.1 270) (mirror x) (unit 1)
     (in_bom yes) (on_board yes) (dnp no) (fields_autoplaced)
-    (property "Reference" "Q4" (at 132.08 29.21 90)
+    (property "Reference" "Q22" (at 132.08 29.21 90)
       (effects (font (size 1.27 1.27)))
     )
@@
       (project "greenmobi-bms"
         (path "/3e668e3e-3e16-4665-a807-4735962c41d3/b1abebf7-38b9-44bd-9506-7ade495be8e0"
-          (reference "Q4") (unit 1)
+          (reference "Q22") (unit 1)
         )
       )
@@
   (symbol (lib_id "power:+3.3V") (at 86.36 142.24 0) (unit 1)
     (in_bom yes) (on_board yes) (dnp no) (fields_autoplaced)
-    (property "Reference" "#PWR098" (at 86.36 146.05 0)
+    (property "Reference" "#PWR0103" (at 86.36 146.05 0)
       (effects (font (size 1.27 1.27)) hide)
     )
@@
       (project "greenmobi-bms"
         (path "/3e668e3e-3e16-4665-a807-4735962c41d3/b1abebf7-38b9-44bd-9506-7ade495be8e0"
-          (reference "#PWR098") (unit 1)
+          (reference "#PWR0103") (unit 1)
         )
       )
@@
   (symbol (lib_id "Sensor_Current:ACS770xCB-050U-PFF") (at 86.36 149.86 0) (unit 1)
     (in_bom yes) (on_board yes) (dnp no)
-    (property "Reference" "U10" (at 88.9 140.97 0)
+    (property "Reference" "U9" (at 88.9 140.97 0)
       (effects (font (size 1.27 1.27)))
     )
@@
       (project "greenmobi-bms"
         (path "/3e668e3e-3e16-4665-a807-4735962c41d3/b1abebf7-38b9-44bd-9506-7ade495be8e0"
-          (reference "U10") (unit 1)
+          (reference "U9") (unit 1)
         )
       )
@@
   (symbol (lib_id "power:GND") (at 215.9 64.77 0) (mirror y) (unit 1)
     (in_bom yes) (on_board yes) (dnp no) (fields_autoplaced)
-    (property "Reference" "#PWR0105" (at 215.9 71.12 0)
+    (property "Reference" "#PWR0110" (at 215.9 71.12 0)
       (effects (font (size 1.27 1.27)) hide)
     )
@@
       (project "greenmobi-bms"
         (path "/3e668e3e-3e16-4665-a807-4735962c41d3/b1abebf7-38b9-44bd-9506-7ade495be8e0"
+          (reference "#PWR0110") (unit 1)
+        )
+      )
+    )
+  )
+  (symbol (lib_id "power:GND") (at 118.11 156.21 0) (unit 1)
+    (in_bom yes) (on_board yes) (dnp no) (fields_autoplaced)
+    (property "Reference" "#PWR0105" (at 118.11 162.56 0)
+      (effects (font (size 1.27 1.27)) hide)
+    )
+    (property "Value" "GND" (at 118.11 161.29 0)
+      (effects (font (size 1.27 1.27)))
+    )
+    (property "Footprint" "" (at 118.11 156.21 0)
+      (effects (font (size 1.27 1.27)) hide)
+    )
+    (property "Datasheet" "" (at 118.11 156.21 0)
+      (effects (font (size 1.27 1.27)) hide)
+    )
+    (pin "1")
+    (instances
+      (project "greenmobi-bms"
+        (path "/3e668e3e-3e16-4665-a807-4735962c41d3/b1abebf7-38b9-44bd-9506-7ade495be8e0"
           (reference "#PWR0105") (unit 1)
         )
@@
     )
   )
-  (symbol (lib_id "power:GND") (at 118.11 156.21 0) (unit 1)
-    (in_bom yes) (on_board yes) (dnp no) (fields_autoplaced)
-    (property "Reference" "#PWR0100" (at 118.11 162.56 0)
-      (effects (font (size 1.27 1.27)) hide)
-    )
-    (property "Value" "GND" (at 118.11 161.29 0)
-      (effects (font (size 1.27 1.27)))
-    )
-    (property "Footprint" "" (at 118.11 156.21 0)
-      (effects (font (size 1.27 1.27)) hide)
-    )
-    (property "Datasheet" "" (at 118.11 156.21 0)
-      (effects (font (size 1.27 1.27)) hide)
-    )
-    (pin "1")
-    (instances
-      (project "greenmobi-bms"
-        (path "/3e668e3e-3e16-4665-a807-4735962c41d3/b1abebf7-38b9-44bd-9506-7ade495be8e0"
-          (reference "#PWR0100") (unit 1)
-        )
-      )
-    )
-  )
   (symbol (lib_id "power:GND") (at 189.23 50.8 0) (mirror y) (unit 1)
     (in_bom yes) (on_board yes) (dnp no) (fields_autoplaced)
-    (property "Reference" "#PWR0103" (at 189.23 57.15 0)
+    (property "Reference" "#PWR0108" (at 189.23 57.15 0)
       (effects (font (size 1.27 1.27)) hide)
     )
@@
       (project "greenmobi-bms"
         (path "/3e668e3e-3e16-4665-a807-4735962c41d3/b1abebf7-38b9-44bd-9506-7ade495be8e0"
-          (reference "#PWR0103") (unit 1)
-        )
-      )
+          (reference "#PWR0108") (unit 1)
+        )
+      )
