File: hardware/thermal.kicad_sch (KiCad schematic)
At the start: 2 parts, among them U7 HDC1080

Commit message: NTC sensors
Parts:
- removed TH1: Thermistor_NTC, symbol Device:Thermistor_NTC
Other:
- added sheet NTC (ntc.kicad_sch)
- added sheet NTC1 (ntc.kicad_sch)
- added sheet NTC2 (ntc.kicad_sch)
Changed lines of the file:
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@@
     (effects (font (size 1.27 1.27)) (justify left))
+  )
+  (hierarchical_label "TEMP_2" (shape output) (at 144.78 101.6 180)
+    (effects (font (size 1.27 1.27)) (justify right))
+  )
+  (hierarchical_label "TEMP_0" (shape output) (at 144.78 88.9 180)
+    (effects (font (size 1.27 1.27)) (justify right))
   )
   (hierarchical_label "SCL" (shape input) (at 195.58 92.71 0)
     (effects (font (size 1.27 1.27)) (justify left))
   )
+  (hierarchical_label "TEMP_1" (shape output) (at 144.78 95.25 180)
+    (effects (font (size 1.27 1.27)) (justify right))
+  )
   (symbol (lib_id "power:+3.3V") (at 185.42 87.63 0) (unit 1)
     (in_bom yes) (on_board yes) (fields_autoplaced)
-    (property "Reference" "#PWR037" (id 0) (at 185.42 91.44 0)
+    (property "Reference" "#PWR039" (id 0) (at 185.42 91.44 0)
       (effects (font (size 1.27 1.27)) hide)
     )
@@
   (symbol (lib_id "power:GND") (at 185.42 102.87 0) (unit 1)
     (in_bom yes) (on_board yes) (fields_autoplaced)
-    (property "Reference" "#PWR038" (id 0) (at 185.42 109.22 0)
+    (property "Reference" "#PWR040" (id 0) (at 185.42 109.22 0)
       (effects (font (size 1.27 1.27)) hide)
     )
@@
     (pin "7")
   )
-  (symbol (lib_id "Device:Thermistor_NTC") (at 138.43 96.52 0) (unit 1)
-    (in_bom yes) (on_board yes) (fields_autoplaced)
-    (property "Reference" "TH1" (id 0) (at 140.97 95.5674 0)
+  (sheet (at 144.78 92.71) (size 12.7 5.08) (fields_autoplaced)
+    (stroke (width 0.1524) (type solid) (color 0 0 0 0))
+    (fill (color 0 0 0 0.0000))
+    (property "Sheet name" "NTC1" (id 0) (at 144.78 91.9984 0)
+      (effects (font (size 1.27 1.27)) (justify left bottom) hide)
+    )
+    (property "Sheet file" "ntc.kicad_sch" (id 1) (at 144.78 98.3746 0)
+      (effects (font (size 1.27 1.27)) (justify left top) hide)
+    )
+    (pin "TEMP" output (at 144.78 95.25 180)
       (effects (font (size 1.27 1.27)) (justify left))
     )
-    (property "Value" "Thermistor_NTC" (id 1) (at 140.97 98.1074 0)
+  )
+  (sheet (at 144.78 99.06) (size 12.7 5.08) (fields_autoplaced)
+    (stroke (width 0.1524) (type solid) (color 0 0 0 0))
+    (fill (color 0 0 0 0.0000))
+    (property "Sheet name" "NTC2" (id 0) (at 144.78 98.3484 0)
+      (effects (font (size 1.27 1.27)) (justify left bottom) hide)
+    )
+    (property "Sheet file" "ntc.kicad_sch" (id 1) (at 144.78 104.7246 0)
+      (effects (font (size 1.27 1.27)) (justify left top))
+    )
+    (pin "TEMP" output (at 144.78 101.6 180)
       (effects (font (size 1.27 1.27)) (justify left))
     )
-    (property "Footprint" "" (id 2) (at 138.43 95.25 0)
-      (effects (font (size 1.27 1.27)) hide)
+  )
+  (sheet (at 144.78 86.36) (size 12.7 5.08) (fields_autoplaced)
+    (stroke (width 0.1524) (type solid) (color 0 0 0 0))
+    (fill (color 0 0 0 0.0000))
+    (property "Sheet name" "NTC" (id 0) (at 144.78 85.6484 0)
+      (effects (font (size 1.27 1.27)) (justify left bottom))
     )
-    (property "Datasheet" "~" (id 3) (at 138.43 95.25 0)
-      (effects (font (size 1.27 1.27)) hide)
+    (property "Sheet file" "ntc.kicad_sch" (id 1) (at 144.78 92.0246 0)
+      (effects (font (size 1.27 1.27)) (justify left top) hide)
     )
-    (pin "1")
-    (pin "2")
+    (pin "TEMP" output (at 144.78 88.9 180)
+      (effects (font (size 1.27 1.27)) (justify left))
+    )
   )
 )

Commit message: Fan ports
Parts:
- added M1: Fan_4pin, Connector:FanPinHeader_1x04_P2.54mm_Vertical, symbol Motor:Fan_4pin
- added M2: Fan, Connector_JST:JST_XH_B2B-XH-A_1x02_P2.50mm_Vertical, symbol Motor:Fan
- added Q22: AO3401A, Package_TO_SOT_SMD:SOT-23, symbol Transistor_FET:AO3401A
- added R87: 1k, symbol Device:R_Small
- added R88: 100k, symbol Device:R_Small
Connections:
- net GND: now also M1.1 (-), M2.2 (-)
- new net: Q22.1 (G), R87.2, R88.2
- new net: M1.2 (+), M2.1 (+), Q22.3 (D)
- new net +12V: Q22.2 (S), R88.1
- new net Fan_EN: R87.1
- new net Fan_PWM: M1.4 (PWM)
- new net Fan_Tacho: M1.3 (Tacho)

Commit message: Fan freewheeling
Parts:
- added D3: SM4007, Diode_THT:D_DO-41_SOD81_P7.62mm_Horizontal, symbol Diode:SM4007
Connections:
- net GND: now also D3.2 (A)
- net at M1.2 (+), M2.1 (+), Q22.3 (D): now also D3.1 (K)
Changed lines of the file:
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@@
   (junction (at 76.2 88.9) (diameter 0) (color 0 0 0 0)
   )
+  (junction (at 107.95 95.25) (diameter 0) (color 0 0 0 0)
+  )
   (wire (pts (xy 71.12 88.9) (xy 76.2 88.9))
     (stroke (width 0) (type default))
@@
     (stroke (width 0) (type default))
   )
+  (wire (pts (xy 120.65 95.25) (xy 107.95 95.25))
+    (stroke (width 0) (type default))
+  )
   (wire (pts (xy 76.2 80.01) (xy 76.2 78.74))
     (stroke (width 0) (type default))
@@
     (stroke (width 0) (type default))
   )
+  (wire (pts (xy 120.65 99.06) (xy 120.65 95.25))
+    (stroke (width 0) (type default))
+  )
   (wire (pts (xy 76.2 78.74) (xy 87.63 78.74))
     (stroke (width 0) (type default))
@@
   )
   (wire (pts (xy 87.63 78.74) (xy 87.63 83.82))
+    (stroke (width 0) (type default))
+  )
+  (wire (pts (xy 120.65 106.68) (xy 120.65 109.22))
     (stroke (width 0) (type default))
   )
@@
         )
       )
+    )
+  )
+  (symbol (lib_name "GND_2") (lib_id "power:GND") (at 120.65 109.22 0) (unit 1)
+    (in_bom yes) (on_board yes) (dnp no) (fields_autoplaced)
+    (property "Reference" "#PWR075" (at 120.65 115.57 0)
+      (effects (font (size 1.27 1.27)) hide)
+    )
+    (property "Value" "GND" (at 120.65 114.3 0)
+      (effects (font (size 1.27 1.27)))
+    )
+    (property "Footprint" "" (at 120.65 109.22 0)
+      (effects (font (size 1.27 1.27)) hide)
+    )
+    (property "Datasheet" "" (at 120.65 109.22 0)
+      (effects (font (size 1.27 1.27)) hide)
+    )
+    (pin "1")
+    (instances
+      (project "vesc-bms"
+        (path "/3e668e3e-3e16-4665-a807-4735962c41d3/95476253-acbc-4b80-80be-f4a25f0f1538"
+          (reference "#PWR075") (unit 1)
+        )
+      )
+    )
+  )
+  (symbol (lib_id "Diode:SM4007") (at 120.65 102.87 270) (unit 1)
+    (in_bom yes) (on_board yes) (dnp no) (fields_autoplaced)
+    (property "Reference" "D3" (at 123.19 102.235 90)
+      (effects (font (size 1.27 1.27)) (justify left))
+    )
+    (property "Value" "SM4007" (at 123.19 104.775 90)
+      (effects (font (size 1.27 1.27)) (justify left))
+    )
+    (property "Footprint" "Diode_THT:D_DO-41_SOD81_P7.62mm_Horizontal" (at 116.205 102.87 0)
+      (effects (font (size 1.27 1.27)) hide)
+    )
+    (property "Datasheet" "http://cdn-reichelt.de/documents/datenblatt/A400/SMD1N400%23DIO.pdf" (at 120.65 102.87 0)
+      (effects (font (size 1.27 1.27)) hide)
+    )
+    (property "Sim.Device" "D" (at 120.65 102.87 0)
+      (effects (font (size 1.27 1.27)) hide)
+    )
+    (property "Sim.Pins" "1=K 2=A" (at 120.65 102.87 0)
+      (effects (font (size 1.27 1.27)) hide)
+    )
+    (pin "1")
+    (pin "2")
+    (instances
+      (project "vesc-bms"
+        (path "/3e668e3e-3e16-4665-a807-4735962c41d3/95476253-acbc-4b80-80be-f4a25f0f1538"
+          (reference "D3") (unit 1)
+        )
+      )

Commit message: Charger enable circiut and more ext NTC
Other:
- added sheet NTC3 (ntc.kicad_sch)
- added sheet NTC4 (ntc.kicad_sch)
Changed lines of the file:
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@@
     (effects (font (size 1.27 1.27)) (justify right))
   )
-  (hierarchical_label "TEMP_2" (shape output) (at 144.78 101.6 180) (fields_autoplaced)
-    (effects (font (size 1.27 1.27)) (justify right))
-  )
-  (hierarchical_label "TEMP_0" (shape output) (at 144.78 88.9 180) (fields_autoplaced)
+  (hierarchical_label "TEMP_3" (shape output) (at 144.78 101.6 180) (fields_autoplaced)
+    (effects (font (size 1.27 1.27)) (justify right))
+  )
+  (hierarchical_label "TEMP_5" (shape output) (at 144.78 114.3 180) (fields_autoplaced)
+    (effects (font (size 1.27 1.27)) (justify right))
+  )
+  (hierarchical_label "TEMP_1" (shape output) (at 144.78 88.9 180) (fields_autoplaced)
     (effects (font (size 1.27 1.27)) (justify right))
   )
@@
     (effects (font (size 1.27 1.27)) (justify left))
   )
-  (hierarchical_label "TEMP_1" (shape output) (at 144.78 95.25 180) (fields_autoplaced)
+  (hierarchical_label "TEMP_2" (shape output) (at 144.78 95.25 180) (fields_autoplaced)
     (effects (font (size 1.27 1.27)) (justify right))
   )
   (hierarchical_label "Fan_Tacho" (shape input) (at 62.23 101.6 180) (fields_autoplaced)
+    (effects (font (size 1.27 1.27)) (justify right))
+  )
+  (hierarchical_label "TEMP_4" (shape output) (at 144.78 107.95 180) (fields_autoplaced)
     (effects (font (size 1.27 1.27)) (justify right))
   )
@@
     )
   )
+  (sheet (at 144.78 105.41) (size 12.7 5.08) (fields_autoplaced)
+    (stroke (width 0.1524) (type solid))
+    (fill (color 0 0 0 0.0000))
+    (property "Sheetname" "NTC4" (at 144.78 104.6984 0)
+      (effects (font (size 1.27 1.27)) (justify left bottom) hide)
+    )
+    (property "Sheetfile" "ntc.kicad_sch" (at 144.78 111.0746 0)
+      (effects (font (size 1.27 1.27)) (justify left top) hide)
+    )
+    (pin "TEMP" output (at 144.78 107.95 180)
+      (effects (font (size 1.27 1.27)) (justify left))
+    )
+    (instances
+      (project "vesc-bms"
+        (path "/3e668e3e-3e16-4665-a807-4735962c41d3/95476253-acbc-4b80-80be-f4a25f0f1538" (page "30"))
+      )
+    )
+  )
   (sheet (at 144.78 99.06) (size 12.7 5.08) (fields_autoplaced)
     (stroke (width 0.1524) (type solid))
     (fill (color 0 0 0 0.0000))
-    (property "Sheetname" "NTC2" (at 144.78 98.3484 0)
+    (property "Sheetname" "NTC3" (at 144.78 98.3484 0)
       (effects (font (size 1.27 1.27)) (justify left bottom) hide)
     )
     (property "Sheetfile" "ntc.kicad_sch" (at 144.78 104.7246 0)
+      (effects (font (size 1.27 1.27)) (justify left top) hide)
+    )
+    (pin "TEMP" output (at 144.78 101.6 180)
+      (effects (font (size 1.27 1.27)) (justify left))
+    )
+    (instances
+      (project "vesc-bms"
+        (path "/3e668e3e-3e16-4665-a807-4735962c41d3/95476253-acbc-4b80-80be-f4a25f0f1538" (page "29"))
+      )
+    )
+  )
+  (sheet (at 144.78 111.76) (size 12.7 5.08) (fields_autoplaced)
+    (stroke (width 0.1524) (type solid))
+    (fill (color 0 0 0 0.0000))
+    (property "Sheetname" "NTC2" (at 144.78 111.0484 0)
+      (effects (font (size 1.27 1.27)) (justify left bottom) hide)
+    )
+    (property "Sheetfile" "ntc.kicad_sch" (at 144.78 117.4246 0)
       (effects (font (size 1.27 1.27)) (justify left top))
     )
-    (pin "TEMP" output (at 144.78 101.6 180)
-      (effects (font (size 1.27 1.27)) (justify left))
-    )
+    (pin "TEMP" output (at 144.78 114.3 180)
+      (effects (font (size 1.27 1.27)) (justify left))
+    )

Commit message: Charge monitor complete
Parts:
- renumbered D3 to D2401, M1 to M2401, M2 to M2402, Q22 to Q2401, R87 to R2401, R88 to R2402, U7 to U2401
Changed lines of the file:
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@@
   (symbol (lib_id "Device:R_Small") (at 68.58 88.9 90) (unit 1)
     (in_bom yes) (on_board yes) (dnp no) (fields_autoplaced)
-    (property "Reference" "R87" (at 68.58 83.82 90)
+    (property "Reference" "R2401" (at 68.58 83.82 90)
       (effects (font (size 1.27 1.27)))
     )
@@
       (project "vesc-bms"
         (path "/3e668e3e-3e16-4665-a807-4735962c41d3/95476253-acbc-4b80-80be-f4a25f0f1538"
-          (reference "R87") (unit 1)
+          (reference "R2401") (unit 1)
         )
       )
@@
   (symbol (lib_id "power:+3.3V") (at 185.42 87.63 0) (unit 1)
     (in_bom yes) (on_board yes) (dnp no) (fields_autoplaced)
-    (property "Reference" "#PWR041" (at 185.42 91.44 0)
+    (property "Reference" "#PWR02405" (at 185.42 91.44 0)
       (effects (font (size 1.27 1.27)) hide)
     )
@@
       (project "vesc-bms"
         (path "/3e668e3e-3e16-4665-a807-4735962c41d3/95476253-acbc-4b80-80be-f4a25f0f1538"
-          (reference "#PWR041") (unit 1)
+          (reference "#PWR02405") (unit 1)
         )
       )
@@
   (symbol (lib_id "power:GND") (at 185.42 102.87 0) (unit 1)
     (in_bom yes) (on_board yes) (dnp no) (fields_autoplaced)
-    (property "Reference" "#PWR042" (at 185.42 109.22 0)
+    (property "Reference" "#PWR02406" (at 185.42 109.22 0)
       (effects (font (size 1.27 1.27)) hide)
     )
@@
       (project "vesc-bms"
         (path "/3e668e3e-3e16-4665-a807-4735962c41d3/95476253-acbc-4b80-80be-f4a25f0f1538"
-          (reference "#PWR042") (unit 1)
+          (reference "#PWR02406") (unit 1)
         )
       )
@@
   (symbol (lib_id "power:+12V") (at 87.63 77.47 0) (unit 1)
     (in_bom yes) (on_board yes) (dnp no) (fields_autoplaced)
-    (property "Reference" "#PWR067" (at 87.63 81.28 0)
+    (property "Reference" "#PWR02401" (at 87.63 81.28 0)
       (effects (font (size 1.27 1.27)) hide)
     )
@@
       (project "vesc-bms"
         (path "/3e668e3e-3e16-4665-a807-4735962c41d3/95476253-acbc-4b80-80be-f4a25f0f1538"
-          (reference "#PWR067") (unit 1)
+          (reference "#PWR02401") (unit 1)
         )
       )
@@
   (symbol (lib_id "Motor:Fan_4pin") (at 87.63 104.14 0) (unit 1)
     (in_bom yes) (on_board yes) (dnp no) (fields_autoplaced)
-    (property "Reference" "M1" (at 92.71 103.505 0)
+    (property "Reference" "M2401" (at 92.71 103.505 0)
       (effects (font (size 1.27 1.27)) (justify left))
     )
@@
       (project "vesc-bms"
         (path "/3e668e3e-3e16-4665-a807-4735962c41d3/95476253-acbc-4b80-80be-f4a25f0f1538"
-          (reference "M1") (unit 1)
+          (reference "M2401") (unit 1)
         )
       )
@@
   (symbol (lib_name "GND_1") (lib_id "power:GND") (at 87.63 109.22 0) (unit 1)
     (in_bom yes) (on_board yes) (dnp no) (fields_autoplaced)
-    (property "Reference" "#PWR063" (at 87.63 115.57 0)
+    (property "Reference" "#PWR02402" (at 87.63 115.57 0)
       (effects (font (size 1.27 1.27)) hide)
     )
@@
       (project "vesc-bms"
         (path "/3e668e3e-3e16-4665-a807-4735962c41d3/95476253-acbc-4b80-80be-f4a25f0f1538"
-          (reference "#PWR063") (unit 1)
+          (reference "#PWR02402") (unit 1)
         )
       )
@@
   (symbol (lib_name "GND_2") (lib_id "power:GND") (at 120.65 109.22 0) (unit 1)
     (in_bom yes) (on_board yes) (dnp no) (fields_autoplaced)
-    (property "Reference" "#PWR075" (at 120.65 115.57 0)
+    (property "Reference" "#PWR02404" (at 120.65 115.57 0)
       (effects (font (size 1.27 1.27)) hide)
     )
@@
       (project "vesc-bms"
         (path "/3e668e3e-3e16-4665-a807-4735962c41d3/95476253-acbc-4b80-80be-f4a25f0f1538"
-          (reference "#PWR075") (unit 1)
+          (reference "#PWR02404") (unit 1)
         )
       )
@@
   (symbol (lib_id "Diode:SM4007") (at 120.65 102.87 270) (unit 1)
     (in_bom yes) (on_board yes) (dnp no) (fields_autoplaced)
-    (property "Reference" "D3" (at 123.19 102.235 90)
+    (property "Reference" "D2401" (at 123.19 102.235 90)
       (effects (font (size 1.27 1.27)) (justify left))
     )
@@
       (project "vesc-bms"
         (path "/3e668e3e-3e16-4665-a807-4735962c41d3/95476253-acbc-4b80-80be-f4a25f0f1538"
-          (reference "D3") (unit 1)
+          (reference "D2401") (unit 1)
         )
       )
@@
   (symbol (lib_id "Transistor_FET:AO3401A") (at 85.09 88.9 0) (mirror x) (unit 1)
     (in_bom yes) (on_board yes) (dnp no)
-    (property "Reference" "Q22" (at 91.44 88.265 0)
+    (property "Reference" "Q2401" (at 91.44 88.265 0)
       (effects (font (size 1.27 1.27)) (justify left))
     )
@@
       (project "vesc-bms"
         (path "/3e668e3e-3e16-4665-a807-4735962c41d3/95476253-acbc-4b80-80be-f4a25f0f1538"
-          (reference "Q22") (unit 1)
+          (reference "Q2401") (unit 1)
         )
       )
@@
   (symbol (lib_id "Sensor_Humidity:HDC1080") (at 187.96 95.25 0) (unit 1)
     (in_bom yes) (on_board yes) (dnp no) (fields_autoplaced)
-    (property "Reference" "U7" (at 179.07 93.9799 0)
+    (property "Reference" "U2401" (at 179.07 93.9799 0)
       (effects (font (size 1.27 1.27)) (justify right))
     )
@@
       (project "vesc-bms"
         (path "/3e668e3e-3e16-4665-a807-4735962c41d3/95476253-acbc-4b80-80be-f4a25f0f1538"
-          (reference "U7") (unit 1)
+          (reference "U2401") (unit 1)
         )
       )
@@
   (symbol (lib_id "Motor:Fan") (at 107.95 104.14 0) (unit 1)
     (in_bom yes) (on_board yes) (dnp no) (fields_autoplaced)
-    (property "Reference" "M2" (at 113.03 103.505 0)
+    (property "Reference" "M2402" (at 113.03 103.505 0)
       (effects (font (size 1.27 1.27)) (justify left))
     )
@@
       (project "vesc-bms"
         (path "/3e668e3e-3e16-4665-a807-4735962c41d3/95476253-acbc-4b80-80be-f4a25f0f1538"
-          (reference "M2") (unit 1)
+          (reference "M2402") (unit 1)
         )
       )
@@
   (symbol (lib_id "Device:R_Small") (at 76.2 82.55 0) (unit 1)
     (in_bom yes) (on_board yes) (dnp no) (fields_autoplaced)
-    (property "Reference" "R88" (at 78.74 81.915 0)
+    (property "Reference" "R2402" (at 78.74 81.915 0)
       (effects (font (size 1.27 1.27)) (justify left))
     )
@@
       (project "vesc-bms"
         (path "/3e668e3e-3e16-4665-a807-4735962c41d3/95476253-acbc-4b80-80be-f4a25f0f1538"
-          (reference "R88") (unit 1)
+          (reference "R2402") (unit 1)
         )
       )
@@
   (symbol (lib_name "GND_1") (lib_id "power:GND") (at 107.95 109.22 0) (unit 1)
     (in_bom yes) (on_board yes) (dnp no) (fields_autoplaced)
-    (property "Reference" "#PWR066" (at 107.95 115.57 0)
+    (property "Reference" "#PWR02403" (at 107.95 115.57 0)
       (effects (font (size 1.27 1.27)) hide)
     )
@@
       (project "vesc-bms"
         (path "/3e668e3e-3e16-4665-a807-4735962c41d3/95476253-acbc-4b80-80be-f4a25f0f1538"
-          (reference "#PWR066") (unit 1)
-        )
-      )
+          (reference "#PWR02403") (unit 1)
+        )
+      )

Commit message: Total current sense and buzzer
Other:
- removed sheet NTC2
- removed sheet NTC4
Changed lines of the file:
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@@
-    (effects (font (size 1.27 1.27)) (justify right))
-  )
-  (hierarchical_label "TEMP_5" (shape output) (at 144.78 114.3 180) (fields_autoplaced)
     (effects (font (size 1.27 1.27)) (justify right))
   )
@@
   )
   (hierarchical_label "Fan_Tacho" (shape input) (at 62.23 101.6 180) (fields_autoplaced)
-    (effects (font (size 1.27 1.27)) (justify right))
-  )
-  (hierarchical_label "TEMP_4" (shape output) (at 144.78 107.95 180) (fields_autoplaced)
     (effects (font (size 1.27 1.27)) (justify right))
   )
@@
     )
   )
-  (sheet (at 144.78 105.41) (size 12.7 5.08) (fields_autoplaced)
-    (stroke (width 0.1524) (type solid))
-    (fill (color 0 0 0 0.0000))
-    (property "Sheetname" "NTC4" (at 144.78 104.6984 0)
-      (effects (font (size 1.27 1.27)) (justify left bottom) hide)
-    )
-    (property "Sheetfile" "ntc.kicad_sch" (at 144.78 111.0746 0)
-      (effects (font (size 1.27 1.27)) (justify left top) hide)
-    )
-    (pin "TEMP" output (at 144.78 107.95 180)
-      (effects (font (size 1.27 1.27)) (justify left))
-    )
-    (instances
-      (project "vesc-bms"
-        (path "/3e668e3e-3e16-4665-a807-4735962c41d3/95476253-acbc-4b80-80be-f4a25f0f1538" (page "30"))
-      )
-    )
-  )
   (sheet (at 144.78 99.06) (size 12.7 5.08) (fields_autoplaced)
     (stroke (width 0.1524) (type solid))
@@
       )
     )
-  )
-  (sheet (at 144.78 111.76) (size 12.7 5.08) (fields_autoplaced)
-    (stroke (width 0.1524) (type solid))
-    (fill (color 0 0 0 0.0000))
-    (property "Sheetname" "NTC2" (at 144.78 111.0484 0)
-      (effects (font (size 1.27 1.27)) (justify left bottom) hide)
-    )
-    (property "Sheetfile" "ntc.kicad_sch" (at 144.78 117.4246 0)
-      (effects (font (size 1.27 1.27)) (justify left top))
-    )
-    (pin "TEMP" output (at 144.78 114.3 180)
-      (effects (font (size 1.27 1.27)) (justify left))
-    )
-    (instances
-      (project "vesc-bms"
-        (path "/3e668e3e-3e16-4665-a807-4735962c41d3/95476253-acbc-4b80-80be-f4a25f0f1538" (page "27"))
-      )
-    )
