File: hardware/greenmobi-bms.kicad_sch (KiCad schematic)
At the start: 11 parts, among them J1 Power, J101 CHG+, J102 BAT+, J103 OLED, J104 Barrel_Jack, J105 PACK-, J106 BAT-, U2 ACS770xCB-200B-PFF

Commit message: Changed back to a unified design
Other:
- removed sheet ISOSPI interface
- added sheet Frontend (frontend.kicad_sch)
Changed lines of the file:
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@@
     (pin "1")
     (instances
-      (project "greenmobi-bms-controller"
+      (project "greenmobi-bms"
         (path "/3e668e3e-3e16-4665-a807-4735962c41d3"
           (reference "#PWR0105") (unit 1)
@@
     (pin "1")
     (instances
-      (project "greenmobi-bms-controller"
+      (project "greenmobi-bms"
         (path "/3e668e3e-3e16-4665-a807-4735962c41d3"
           (reference "#PWR0101") (unit 1)
@@
     (pin "1")
     (instances
-      (project "greenmobi-bms-controller"
+      (project "greenmobi-bms"
         (path "/3e668e3e-3e16-4665-a807-4735962c41d3"
           (reference "J101") (unit 1)
@@
     (pin "1")
     (instances
-      (project "greenmobi-bms-controller"
+      (project "greenmobi-bms"
         (path "/3e668e3e-3e16-4665-a807-4735962c41d3"
           (reference "J1") (unit 1)
@@
     (pin "2")
     (instances
-      (project "greenmobi-bms-controller"
+      (project "greenmobi-bms"
         (path "/3e668e3e-3e16-4665-a807-4735962c41d3"
           (reference "R101") (unit 1)
@@
     (pin "2")
     (instances
-      (project "greenmobi-bms-controller"
+      (project "greenmobi-bms"
         (path "/3e668e3e-3e16-4665-a807-4735962c41d3"
           (reference "J104") (unit 1)
@@
     (pin "1")
     (instances
-      (project "greenmobi-bms-controller"
+      (project "greenmobi-bms"
         (path "/3e668e3e-3e16-4665-a807-4735962c41d3"
           (reference "#PWR01") (unit 1)
@@
     (pin "2")
     (instances
-      (project "greenmobi-bms-controller"
+      (project "greenmobi-bms"
         (path "/3e668e3e-3e16-4665-a807-4735962c41d3"
           (reference "C101") (unit 1)
@@
     (pin "1")
     (instances
-      (project "greenmobi-bms-controller"
+      (project "greenmobi-bms"
         (path "/3e668e3e-3e16-4665-a807-4735962c41d3"
           (reference "#PWR0107") (unit 1)
@@
     (pin "1")
     (instances
-      (project "greenmobi-bms-controller"
+      (project "greenmobi-bms"
         (path "/3e668e3e-3e16-4665-a807-4735962c41d3"
           (reference "#PWR0102") (unit 1)
@@
     (pin "1")
     (instances
-      (project "greenmobi-bms-controller"
+      (project "greenmobi-bms"
         (path "/3e668e3e-3e16-4665-a807-4735962c41d3"
           (reference "#PWR0104") (unit 1)
@@
     (pin "1")
     (instances
-      (project "greenmobi-bms-controller"
+      (project "greenmobi-bms"
         (path "/3e668e3e-3e16-4665-a807-4735962c41d3"
           (reference "#PWR0108") (unit 1)
@@
     (pin "2")
     (instances
-      (project "greenmobi-bms-controller"
+      (project "greenmobi-bms"
         (path "/3e668e3e-3e16-4665-a807-4735962c41d3"
           (reference "U2") (unit 1)
@@
     (pin "1")
     (instances
-      (project "greenmobi-bms-controller"
+      (project "greenmobi-bms"
         (path "/3e668e3e-3e16-4665-a807-4735962c41d3"
           (reference "#PWR0111") (unit 1)
@@
     (pin "5")
     (instances
-      (project "greenmobi-bms-controller"
+      (project "greenmobi-bms"
         (path "/3e668e3e-3e16-4665-a807-4735962c41d3"
           (reference "J103") (unit 1)
@@
     (pin "1")
     (instances
-      (project "greenmobi-bms-controller"
+      (project "greenmobi-bms"
         (path "/3e668e3e-3e16-4665-a807-4735962c41d3"
           (reference "J102") (unit 1)
@@
     (pin "1")
     (instances
-      (project "greenmobi-bms-controller"
+      (project "greenmobi-bms"
         (path "/3e668e3e-3e16-4665-a807-4735962c41d3"
           (reference "J105") (unit 1)
@@
     (pin "1")
     (instances
-      (project "greenmobi-bms-controller"
+      (project "greenmobi-bms"
         (path "/3e668e3e-3e16-4665-a807-4735962c41d3"
           (reference "#PWR0106") (unit 1)
@@
     (pin "1")
     (instances
-      (project "greenmobi-bms-controller"
+      (project "greenmobi-bms"
         (path "/3e668e3e-3e16-4665-a807-4735962c41d3"
           (reference "J106") (unit 1)
@@
     (pin "1")
     (instances
-      (project "greenmobi-bms-controller"
+      (project "greenmobi-bms"
         (path "/3e668e3e-3e16-4665-a807-4735962c41d3"
           (reference "#PWR0110") (unit 1)
@@
     (pin "2")
     (instances
-      (project "greenmobi-bms-controller"
+      (project "greenmobi-bms"
         (path "/3e668e3e-3e16-4665-a807-4735962c41d3"
           (reference "C103") (unit 1)
         )
+      )
+    )
+  )
+  (sheet (at 127 69.85) (size 30.48 20.32) (fields_autoplaced)
+    (stroke (width 0.1524) (type solid))
+    (fill (color 0 0 0 0.0000))
+    (property "Sheetname" "Frontend" (at 127 69.1384 0)
+      (effects (font (size 1.27 1.27)) (justify left bottom))
+    )
+    (property "Sheetfile" "frontend.kicad_sch" (at 127 90.7546 0)
+      (effects (font (size 1.27 1.27)) (justify left top))
+    )
+    (instances
+      (project "greenmobi-bms"
+        (path "/3e668e3e-3e16-4665-a807-4735962c41d3" (page "6"))
       )
     )
@@
     )
     (instances
-      (project "greenmobi-bms-controller"
+      (project "greenmobi-bms"
         (path "/3e668e3e-3e16-4665-a807-4735962c41d3" (page "2"))
-      )
-    )
-  )
-  (sheet (at 130.81 71.12) (size 34.29 20.32) (fields_autoplaced)
-    (stroke (width 0.1524) (type solid))
-    (fill (color 0 0 0 0.0000))
-    (property "Sheetname" "ISOSPI interface" (at 130.81 70.4084 0)
-      (effects (font (size 1.27 1.27)) (justify left bottom))
-    )
-    (property "Sheetfile" "isospi_interface.kicad_sch" (at 130.81 92.0246 0)
-      (effects (font (size 1.27 1.27)) (justify left top))
-    )
-    (pin "CS" input (at 165.1 83.82 0)
-      (effects (font (size 1.27 1.27)) (justify right))
-    )
-    (pin "MISO" output (at 165.1 78.74 0)
-      (effects (font (size 1.27 1.27)) (justify right))
-    )
-    (pin "SCK" input (at 165.1 81.28 0)
-      (effects (font (size 1.27 1.27)) (justify right))
-    )
-    (pin "MOSI" input (at 165.1 76.2 0)
-      (effects (font (size 1.27 1.27)) (justify right))
-    )
-    (instances
-      (project "greenmobi-bms-controller"
-        (path "/3e668e3e-3e16-4665-a807-4735962c41d3" (page "6"))
       )
     )
@@
     )
     (instances
-      (project "greenmobi-bms-controller"
+      (project "greenmobi-bms"
         (path "/3e668e3e-3e16-4665-a807-4735962c41d3" (page "5"))
       )
@@
     )
     (instances
-      (project "greenmobi-bms-controller"
+      (project "greenmobi-bms"
         (path "/3e668e3e-3e16-4665-a807-4735962c41d3" (page "4"))
       )
@@
     )
     (instances
-      (project "greenmobi-bms-controller"
+      (project "greenmobi-bms"
         (path "/3e668e3e-3e16-4665-a807-4735962c41d3" (page "28"))
       )

Commit message: Fix OLED pinout and add HDC1080
Parts:
- removed J103: OLED, Connector_JST:JST_XH_B5B-XH-A_1x05_P2.50mm_Vertical, symbol Connector:Conn_01x05_Pin
- added C26: 100n, symbol Device:C_Small
- added J11: Conn_01x04_Socket, symbol Connector:Conn_01x04_Socket
- added U5: HDC1080, Package_SON:Texas_PWSON-N6, symbol Sensor_Humidity:HDC1080
Connections:
- net +3.3V: now also C26.1, J11.2 (Pin_2), U5.5 (VCC)
- net GND: now also C26.2, J11.1 (Pin_1), U5.2 (GND)
- net MCU/SCL: now also J11.3 (Pin_3), U5.6 (SCL)
- net MCU/SDA: now also J11.4 (Pin_4), U5.1 (SDA)

Commit message: Wire up the AFE
Other:
- sheet Frontend ports: added 5V_IN, CS, SCK, SDI, SDO, WDT; removed none
- sheet MCU ports: added AFE_WDT; removed OLED_RST
Changed lines of the file:
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@@
+    (stroke (width 0) (type default))
+  )
+  (wire (pts (xy 165.1 87.63) (xy 182.88 87.63))
     (stroke (width 0) (type default))
   )
@@
     )
   )
-  (sheet (at 140.97 100.33) (size 30.48 20.32) (fields_autoplaced)
+  (sheet (at 149.86 73.66) (size 15.24 16.51) (fields_autoplaced)
     (stroke (width 0.1524) (type solid))
     (fill (color 0 0 0 0.0000))
-    (property "Sheetname" "Frontend" (at 140.97 99.6184 0)
+    (property "Sheetname" "Frontend" (at 149.86 72.9484 0)
       (effects (font (size 1.27 1.27)) (justify left bottom))
     )
-    (property "Sheetfile" "frontend.kicad_sch" (at 140.97 121.2346 0)
+    (property "Sheetfile" "frontend.kicad_sch" (at 149.86 90.7546 0)
       (effects (font (size 1.27 1.27)) (justify left top))
+    )
+    (pin "5V_IN" input (at 149.86 76.2 180)
+      (effects (font (size 1.27 1.27)) (justify left))
+    )
+    (pin "WDT" output (at 165.1 87.63 0)
+      (effects (font (size 1.27 1.27)) (justify right))
+    )
+    (pin "SCK" input (at 165.1 81.28 0)
+      (effects (font (size 1.27 1.27)) (justify right))
+    )
+    (pin "CS" input (at 165.1 83.82 0)
+      (effects (font (size 1.27 1.27)) (justify right))
+    )
+    (pin "SDI" input (at 165.1 76.2 0)
+      (effects (font (size 1.27 1.27)) (justify right))
+    )
+    (pin "SDO" output (at 165.1 78.74 0)
+      (effects (font (size 1.27 1.27)) (justify right))
     )
     (instances
@@
       (effects (font (size 1.27 1.27)) (justify left))
     )
-    (pin "OLED_RST" output (at 182.88 71.12 180)
-      (effects (font (size 1.27 1.27)) (justify left))
-    )
+    (pin "AFE_WDT" input (at 182.88 87.63 180)
+      (effects (font (size 1.27 1.27)) (justify left))
+    )

Commit message: Charger connector
Parts:
- removed U2: ACS770xCB-200B-PFF, Sensor_Current:Allegro_CB_PFF, symbol Sensor_Current:ACS770xCB-200B-PFF
- added J12: CHG-, TestPoint:TestPoint_Pad_4.0x4.0mm, symbol Connector_Generic:Conn_01x01
- added U6: ACS770xCB-100B-PFF, Sensor_Current:Allegro_CB_PFF, symbol Sensor_Current:ACS770xCB-100B-PFF
Connections:
- net +3.3V: now also U6.1 (VCC)
- net GND: now also J12.1 (Pin_1), U6.2 (GND), U6.4 (IP+)
- net at R101.1: now also U6.3 (VIOUT)
- net at J106.1 (Pin_1): now also U6.5 (IP-)
Other:
- sheet MCU ports: added Total_current; removed none
Changed lines of the file:
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@@
+    (stroke (width 0) (type default))
+  )
+  (wire (pts (xy 48.26 33.02) (xy 52.07 33.02))
     (stroke (width 0) (type default))
   )
@@
   (text "Place close to ADC input" (at 92.71 147.32 0)
     (effects (font (size 1.27 1.27) bold) (justify left bottom))
+  )
+  (hierarchical_label "Total_current" (shape input) (at 182.88 97.79 180) (fields_autoplaced)
+    (effects (font (size 1.27 1.27)) (justify right))
   )
   (hierarchical_label "Total_current" (shape output) (at 115.57 129.54 0) (fields_autoplaced)
@@
     )
   )
+  (symbol (lib_id "Connector_Generic:Conn_01x01") (at 43.18 33.02 180) (unit 1)
+    (in_bom yes) (on_board yes) (dnp no) (fields_autoplaced)
+    (property "Reference" "J12" (at 43.18 26.67 0)
+      (effects (font (size 1.27 1.27)))
+    )
+    (property "Value" "CHG-" (at 43.18 29.21 0)
+      (effects (font (size 1.27 1.27)))
+    )
+    (property "Footprint" "TestPoint:TestPoint_Pad_4.0x4.0mm" (at 43.18 33.02 0)
+      (effects (font (size 1.27 1.27)) hide)
+    )
+    (property "Datasheet" "~" (at 43.18 33.02 0)
+      (effects (font (size 1.27 1.27)) hide)
+    )
+    (pin "1")
+    (instances
+      (project "greenmobi-bms"
+        (path "/3e668e3e-3e16-4665-a807-4735962c41d3"
+          (reference "J12") (unit 1)
+        )
+      )
+    )
+  )
   (symbol (lib_id "power:GND") (at 125.73 171.45 0) (unit 1)
     (in_bom yes) (on_board yes) (dnp no) (fields_autoplaced)
@@
         (path "/3e668e3e-3e16-4665-a807-4735962c41d3"
           (reference "#PWR016") (unit 1)
+        )
+      )
+    )
+  )
+  (symbol (lib_id "power:GND") (at 52.07 33.02 0) (unit 1)
+    (in_bom yes) (on_board yes) (dnp no) (fields_autoplaced)
+    (property "Reference" "#PWR020" (at 52.07 39.37 0)
+      (effects (font (size 1.27 1.27)) hide)
+    )
+    (property "Value" "GND" (at 52.07 38.1 0)
+      (effects (font (size 1.27 1.27)))
+    )
+    (property "Footprint" "" (at 52.07 33.02 0)
+      (effects (font (size 1.27 1.27)) hide)
+    )
+    (property "Datasheet" "" (at 52.07 33.02 0)
+      (effects (font (size 1.27 1.27)) hide)
+    )
+    (pin "1")
+    (instances
+      (project "greenmobi-bms"
+        (path "/3e668e3e-3e16-4665-a807-4735962c41d3"
+          (reference "#PWR020") (unit 1)
         )
       )
@@
     )
   )
-  (symbol (lib_id "Sensor_Current:ACS770xCB-200B-PFF") (at 72.39 129.54 0) (unit 1)
+  (symbol (lib_id "power:GND") (at 53.34 114.3 0) (unit 1)
+    (in_bom yes) (on_board yes) (dnp no) (fields_autoplaced)
+    (property "Reference" "#PWR0111" (at 53.34 120.65 0)
+      (effects (font (size 1.27 1.27)) hide)
+    )
+    (property "Value" "GND" (at 53.34 119.38 0)
+      (effects (font (size 1.27 1.27)))
+    )
+    (property "Footprint" "" (at 53.34 114.3 0)
+      (effects (font (size 1.27 1.27)) hide)
+    )
+    (property "Datasheet" "" (at 53.34 114.3 0)
+      (effects (font (size 1.27 1.27)) hide)
+    )
+    (pin "1")
+    (instances
+      (project "greenmobi-bms"
+        (path "/3e668e3e-3e16-4665-a807-4735962c41d3"
+          (reference "#PWR0111") (unit 1)
+        )
+      )
+    )
+  )
+  (symbol (lib_id "Sensor_Current:ACS770xCB-100B-PFF") (at 72.39 129.54 0) (unit 1)
     (in_bom yes) (on_board yes) (dnp no)
-    (property "Reference" "U2" (at 74.93 120.65 0)
-      (effects (font (size 1.27 1.27)))
-    )
-    (property "Value" "ACS770xCB-200B-PFF" (at 83.82 123.19 0)
+    (property "Reference" "U6" (at 74.93 120.65 0)
+      (effects (font (size 1.27 1.27)))
+    )
+    (property "Value" "ACS770xCB-100B-PFF" (at 83.82 123.19 0)
       (effects (font (size 1.27 1.27)))
     )
@@
       (effects (font (size 1.27 1.27)) hide)
     )
-    (pin "5")
-    (pin "1")
     (pin "3")
     (pin "4")
+    (pin "5")
     (pin "2")
-    (instances
-      (project "greenmobi-bms"
-        (path "/3e668e3e-3e16-4665-a807-4735962c41d3"
-          (reference "U2") (unit 1)
-        )
-      )
-    )
-  )
-  (symbol (lib_id "power:GND") (at 53.34 114.3 0) (unit 1)
-    (in_bom yes) (on_board yes) (dnp no) (fields_autoplaced)
-    (property "Reference" "#PWR0111" (at 53.34 120.65 0)
-      (effects (font (size 1.27 1.27)) hide)
-    )
-    (property "Value" "GND" (at 53.34 119.38 0)
-      (effects (font (size 1.27 1.27)))
-    )
-    (property "Footprint" "" (at 53.34 114.3 0)
-      (effects (font (size 1.27 1.27)) hide)
-    )
-    (property "Datasheet" "" (at 53.34 114.3 0)
-      (effects (font (size 1.27 1.27)) hide)
-    )
-    (pin "1")
-    (instances
-      (project "greenmobi-bms"
-        (path "/3e668e3e-3e16-4665-a807-4735962c41d3"
-          (reference "#PWR0111") (unit 1)
+    (pin "1")
+    (instances
+      (project "greenmobi-bms"
+        (path "/3e668e3e-3e16-4665-a807-4735962c41d3"
+          (reference "U6") (unit 1)
         )
       )
@@
       (effects (font (size 1.27 1.27)) (justify left))
     )
+    (pin "Total_current" input (at 182.88 97.79 180)
+      (effects (font (size 1.27 1.27)) (justify left))
+    )

Commit message: BAT to 12V converter
Other:
- company: (none) -> GreenMobi
- title: (none) -> GreenMobi BMS
Changed lines of the file:
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@@
 (kicad_sch (version 20230121) (generator eeschema)
   (paper "A4")
+  (title_block
+    (title "GreenMobi BMS")
+    (date "2024-02-09")
+    (rev "ALPHA")
+    (company "GreenMobi")
+  )
   (junction (at 49.53 114.3) (diameter 0) (color 0 0 0 0)
   )

Commit message: Add option to power AFE from 5V on board regulator
Other:
- sheet Frontend ports: added none; removed 5V_IN
Changed lines of the file:
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@@
       (effects (font (size 1.27 1.27)) (justify left top))
-    )
-    (pin "5V_IN" input (at 149.86 76.2 180)
-      (effects (font (size 1.27 1.27)) (justify left))
     )
     (pin "WDT" output (at 165.1 87.63 0)

Commit message: Fix some ERC issues
Parts:
- renumbered C101 to C1, C103 to C2, C26 to C3, J12 to J1, J101 to J2, J104 to J3, J102 to J4, J105 to J5, J106 to J6, J1 to J7, J11 to J8, R101 to R1, U6 to U1, U5 to U2
Other:
- sheet Power Supply ports: added none; removed BAT_UVLO

Commit message: Add MCU connections
Other:
- sheet MCU ports: added CHG_EN, CP_EN, Charger_current, Charger_voltage, DSG_EN, PCHG_EN, PMON_EN; removed none
Changed lines of the file:
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@@
     (effects (font (size 1.27 1.27) bold) (justify left bottom))
   )
-  (hierarchical_label "Total_current" (shape input) (at 182.88 97.79 180) (fields_autoplaced)
-    (effects (font (size 1.27 1.27)) (justify right))
-  )
-  (hierarchical_label "Total_current" (shape output) (at 115.57 129.54 0) (fields_autoplaced)
-    (effects (font (size 1.27 1.27)) (justify left))
+  (label "CHG_EN" (at 182.88 104.14 180) (fields_autoplaced)
+    (effects (font (size 1.27 1.27)) (justify right bottom))
+  )
+  (label "CHG_EN" (at 101.6 59.69 0) (fields_autoplaced)
+    (effects (font (size 1.27 1.27)) (justify left bottom))
+  )
+  (label "Charger_voltage" (at 182.88 100.33 180) (fields_autoplaced)
+    (effects (font (size 1.27 1.27)) (justify right bottom))
+  )
+  (label "Charger_current" (at 101.6 54.61 0) (fields_autoplaced)
+    (effects (font (size 1.27 1.27)) (justify left bottom))
+  )
+  (label "CP_EN" (at 182.88 106.68 180) (fields_autoplaced)
+    (effects (font (size 1.27 1.27)) (justify right bottom))
+  )
+  (label "PCHG_EN" (at 182.88 111.76 180) (fields_autoplaced)
+    (effects (font (size 1.27 1.27)) (justify right bottom))
+  )
+  (label "Charger_voltage" (at 101.6 52.07 0) (fields_autoplaced)
+    (effects (font (size 1.27 1.27)) (justify left bottom))
+  )
+  (label "CP_EN" (at 101.6 62.23 0) (fields_autoplaced)
+    (effects (font (size 1.27 1.27)) (justify left bottom))
+  )
+  (label "DSG_EN" (at 101.6 64.77 0) (fields_autoplaced)
+    (effects (font (size 1.27 1.27)) (justify left bottom))
+  )
+  (label "PMON_EN" (at 182.88 114.3 180) (fields_autoplaced)
+    (effects (font (size 1.27 1.27)) (justify right bottom))
+  )
+  (label "Total_current" (at 182.88 97.79 180) (fields_autoplaced)
+    (effects (font (size 1.27 1.27)) (justify right bottom))
+  )
+  (label "Charger_current" (at 182.88 95.25 180) (fields_autoplaced)
+    (effects (font (size 1.27 1.27)) (justify right bottom))
+  )
+  (label "DSG_EN" (at 182.88 109.22 180) (fields_autoplaced)
+    (effects (font (size 1.27 1.27)) (justify right bottom))
+  )
+  (label "PCHG_EN" (at 101.6 67.31 0) (fields_autoplaced)
+    (effects (font (size 1.27 1.27)) (justify left bottom))
+  )
+  (label "Total_current" (at 115.57 129.54 0) (fields_autoplaced)
+    (effects (font (size 1.27 1.27)) (justify left bottom))
+  )
+  (label "PMON_EN" (at 101.6 69.85 0) (fields_autoplaced)
+    (effects (font (size 1.27 1.27)) (justify left bottom))
   )
   (symbol (lib_id "power:+3.3V") (at 190.5 43.18 90) (unit 1)
@@
       (effects (font (size 1.27 1.27)) (justify left))
     )
+    (pin "CHG_EN" input (at 182.88 104.14 180)
+      (effects (font (size 1.27 1.27)) (justify left))
+    )
+    (pin "DSG_EN" input (at 182.88 109.22 180)
+      (effects (font (size 1.27 1.27)) (justify left))
+    )
+    (pin "CP_EN" input (at 182.88 106.68 180)
+      (effects (font (size 1.27 1.27)) (justify left))
+    )
+    (pin "PCHG_EN" input (at 182.88 111.76 180)
+      (effects (font (size 1.27 1.27)) (justify left))
+    )
+    (pin "PMON_EN" input (at 182.88 114.3 180)
+      (effects (font (size 1.27 1.27)) (justify left))
+    )
+    (pin "Charger_current" input (at 182.88 95.25 180)
+      (effects (font (size 1.27 1.27)) (justify left))
+    )
+    (pin "Charger_voltage" input (at 182.88 100.33 180)
+      (effects (font (size 1.27 1.27)) (justify left))
+    )
     (instances
       (project "greenmobi-bms"
@@
       (effects (font (size 1.27 1.27)) (justify right))
     )
-    (pin "CP_EN" input (at 101.6 64.77 0)
+    (pin "CP_EN" input (at 101.6 62.23 0)
       (effects (font (size 1.27 1.27)) (justify right))
     )
@@
       (effects (font (size 1.27 1.27)) (justify right))
     )
-    (pin "PMON_EN" input (at 101.6 62.23 0)
-      (effects (font (size 1.27 1.27)) (justify right))
-    )
-    (pin "DSG_EN" input (at 101.6 67.31 0)
-      (effects (font (size 1.27 1.27)) (justify right))
-    )
-    (pin "PCHG_EN" input (at 101.6 69.85 0)
-      (effects (font (size 1.27 1.27)) (justify right))
-    )
+    (pin "PMON_EN" input (at 101.6 69.85 0)
+      (effects (font (size 1.27 1.27)) (justify right))
+    )
+    (pin "DSG_EN" input (at 101.6 64.77 0)
+      (effects (font (size 1.27 1.27)) (justify right))
+    )
+    (pin "PCHG_EN" input (at 101.6 67.31 0)
+      (effects (font (size 1.27 1.27)) (justify right))
+    )
