File: hardware/greenmobi-bms.kicad_sch (KiCad schematic)
At the start: 24 parts, among them J1 CHG-, J10 USB_C_Receptacle_USB2.0_14P, J11 CAN, J2 CHG+, J3 Barrel_Jack, J4 BAT+, J5 PACK-, J6 BAT-, J7 Power, J8 PACK+, M1 Fan, Q27 AO3401A, U1 ACS770xCB-100B-PFF, U2 HDC1080, U4 MCP2562-E-SN

Commit message: Added shunt amplifier
Parts:
- removed J3: Barrel_Jack, symbol Connector:Barrel_Jack
- removed J7: Power, symbol Connector_Generic:Conn_01x02
- removed U1: ACS770xCB-100B-PFF, Sensor_Current:Allegro_CB_PFF, symbol Sensor_Current:ACS770xCB-100B-PFF
- added C63, C72: 100n, symbol Device:C_Small
- added R102, R93: 1k, symbol Device:R_Small
- added R91: 0.2m, symbol Device:R_Small
- added U12: INA181, Package_TO_SOT_SMD:SOT-23-6, symbol Amplifier_Current:INA181
Connections:
- net +3.3VP: now also U12.6 (V+)
- net GND: now also C63.2, C72.2, R102.1, R91.2, U12.2 (GND)
- net at R1.1: now also U12.1
- net at J6.1 (Pin_1): now also R91.1, R93.1
- net Charger monitoring/PACK+ renamed PACK+
- new net: C72.1, R102.2, U12.3 (+)
- new net: C63.1, R93.2, U12.4 (-)
Other:
- sheet MCU ports: added 12V_OUT_EN; removed none
- sheet Power Supply ports: added 12V_OUT_EN; removed none
- note added: "Missing reference voltage"
- moved on the sheet: C1, J1, J2, J4, J5, J6, J8

Commit message: Tune Charger current and MOSFET fix orientation
Parts:
- removed Q27: AO3401A, Package_TO_SOT_SMD:SOT-23, symbol Transistor_FET:AO3401A
- added Q27: AO3400A, Package_TO_SOT_SMD:SOT-23, symbol Transistor_FET:AO3400A
Connections:
- net GND: now also Q27.2 (S)
- net at D3.2 (A), M1.2 (-): now also Q27.3 (D)
- net at R68.1: now also Q27.1 (G)
Changed lines of the file:
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@@
-	)
-	(symbol
-		(lib_id "Transistor_FET:AO3401A")
-		(at 151.13 129.54 180)
-		(unit 1)
-		(exclude_from_sim no)
-		(in_bom yes)
-		(on_board yes)
-		(dnp no)
-		(property "Reference" "Q27"
-			(at 144.78 130.81 0)
-			(effects
-				(font
-					(size 1.27 1.27)
-				)
-				(justify left)
-			)
-		)
-		(property "Value" "AO3401A"
-			(at 144.78 128.27 0)
-			(effects
-				(font
-					(size 1.27 1.27)
-				)
-				(justify left)
-			)
-		)
-		(property "Footprint" "Package_TO_SOT_SMD:SOT-23"
-			(at 146.05 127.635 0)
-			(effects
-				(font
-					(size 1.27 1.27)
-					(italic yes)
-				)
-				(justify left)
-				(hide yes)
-			)
-		)
-		(property "Datasheet" "http://www.aosmd.com/pdfs/datasheet/AO3401A.pdf"
-			(at 146.05 125.73 0)
-			(effects
-				(font
-					(size 1.27 1.27)
-				)
-				(justify left)
-				(hide yes)
-			)
-		)
-		(property "Description" ""
-			(at 151.13 129.54 0)
-			(effects
-				(font
-					(size 1.27 1.27)
-				)
-				(hide yes)
-			)
-		)
-		(pin "2"
-		)
-		(pin "1"
-		)
-		(pin "3"
-		)
-		(instances
-			(project "greenmobi-bms"
-				(path "/3e668e3e-3e16-4665-a807-4735962c41d3"
-					(reference "Q27")
-					(unit 1)
-				)
-			)
-		)
 	)
 	(symbol
@@
 					(unit 1)
 				)
+			)
+		)
+	)
+	(symbol
+		(lib_id "Transistor_FET:AO3400A")
+		(at 151.13 129.54 0)
+		(mirror y)
+		(unit 1)
+		(exclude_from_sim no)
+		(in_bom yes)
+		(on_board yes)
+		(dnp no)
+		(fields_autoplaced yes)
+		(property "Reference" "Q27"
+			(at 144.78 128.2699 0)
+			(effects
+				(font
+					(size 1.27 1.27)
+				)
+				(justify left)
+			)
+		)
+		(property "Value" "AO3400A"
+			(at 144.78 130.8099 0)
+			(effects
+				(font
+					(size 1.27 1.27)
+				)
+				(justify left)
+			)
+		)
+		(property "Footprint" "Package_TO_SOT_SMD:SOT-23"
+			(at 146.05 131.445 0)
+			(effects
+				(font
+					(size 1.27 1.27)
+					(italic yes)
+				)
+				(justify left)
+				(hide yes)
+			)
+		)
+		(property "Datasheet" "http://www.aosmd.com/pdfs/datasheet/AO3400A.pdf"
+			(at 146.05 133.35 0)
+			(effects
+				(font
+					(size 1.27 1.27)
+				)
+				(justify left)
+				(hide yes)
+			)
+		)
+		(property "Description" "30V Vds, 5.7A Id, N-Channel MOSFET, SOT-23"
+			(at 151.13 129.54 0)
+			(effects
+				(font
+					(size 1.27 1.27)
+				)
+				(hide yes)
+			)
+		)
+		(pin "1"
+		)
+		(pin "3"
+		)
+		(pin "2"
+		)
+		(instances
+			(project "greenmobi-bms"
+				(path "/3e668e3e-3e16-4665-a807-4735962c41d3"
+					(reference "Q27")
+					(unit 1)
+				)

Commit message: Initiated sourcing
Parts:
- C63, C72: footprint (none) -> Capacitor_SMD:C_0402_1005Metric
Changed lines of the file:
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@@
 			)
 		)
-		(property "Footprint" ""
+		(property "Footprint" "Capacitor_SMD:C_0402_1005Metric"
 			(at 43.18 137.16 0)
 			(effects
@@
 			)
 		)
-		(property "Footprint" ""
+		(property "Footprint" "Capacitor_SMD:C_0402_1005Metric"
 			(at 29.21 137.16 0)
 			(effects

Commit message: More sourcing components
Parts:
- J10: footprint (none) -> Connector_USB:USB_C_Receptacle_Palconn_UTC16-G
- J11: footprint (none) -> Connector_Phoenix_MC:PhoenixContact_MCV_1,5_2-G-3.5_1x02_P3.50mm_Vertical
- M1: footprint (none) -> Connector_JST:JST_PH_B2B-PH-SM4-TB_1x02-1MP_P2.00mm_Vertical
- R1: footprint (none) -> Resistor_SMD:R_0402_1005Metric
Changed lines of the file:
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@@
 			)
 		)
-		(property "Footprint" ""
+		(property "Footprint" "Resistor_SMD:R_0402_1005Metric"
 			(at 99.06 129.54 0)
 			(effects
@@
 			)
 		)
-		(property "Footprint" ""
+		(property "Footprint" "Connector_JST:JST_PH_B2B-PH-SM4-TB_1x02-1MP_P2.00mm_Vertical"
 			(at 148.59 117.856 0)
 			(effects
@@
 			)
 		)
-		(property "Footprint" ""
+		(property "Footprint" "Connector_USB:USB_C_Receptacle_Palconn_UTC16-G"
 			(at 234.315 64.77 0)
 			(effects
@@
 			)
 		)
-		(property "Footprint" ""
+		(property "Footprint" "Connector_Phoenix_MC:PhoenixContact_MCV_1,5_2-G-3.5_1x02_P3.50mm_Vertical"
 			(at 271.78 125.095 0)
 			(effects

Commit message: Improved Currrent Sensors
Parts:
- removed C63, C72: 100n, Capacitor_SMD:C_0402_1005Metric, symbol Device:C_Small
- removed J11: CAN, Connector_Phoenix_MC:PhoenixContact_MCV_1,5_2-G-3.5_1x02_P3.50mm_Vertical, symbol Connector:Screw_Terminal_01x02
- added C59: 8u, symbol Device:C_Small
- added J3: CAN, Connector_Phoenix_MC:PhoenixContact_MCV_1,5_2-G-3.5_1x02_P3.50mm_Vertical, symbol Connector_Generic:Conn_01x02
- R102, R93: value 1k -> 10
Connections:
- net at R102.2, U12.3 (+): now also C59.2
- net at R13.1, U4.7 (CANH): now also J3.1 (Pin_1)
- net at R13.2, U4.6 (CANL): now also J3.2 (Pin_2)
- net at R93.2, U12.4 (-): now also C59.1
- net ADC_REF: now reaches U12.5 (REF)
Other:
- sheet MCU ports: added ADC_REF; removed none
- note added: "Total Current Sensor"
- note removed: "Missing reference voltage"
- moved on the sheet: C1, C2, J1, J10, J2, J4, J5, J6, J8, R1, R102, R13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

Commit message: Charger monitoring
Parts:
- added U9: REF3012, Package_TO_SOT_SMD:SOT-23, symbol Reference_Voltage:REF3012
Connections:
- net +3.3V: no longer C1.1
- net +3.3VP: now also C1.1, U9.1 (IN)
- net GND: now also U9.3 (GND)
- net ADC_REF: no longer names the net of U12.5 (REF)
- net ADC_REF: now also U9.2 (OUT)
Other:
- sheet MCU ports: added none; removed ADC_REF

Commit message: Ongoing work on high side switch
Other:
- sheet Charger monitoring ports: added none; removed BAT+
- moved on the sheet: J4, J8
Changed lines of the file:
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@@
 	)
 	(junction
-		(at 46.99 71.12)
+		(at 36.83 29.21)
 		(diameter 0)
 		(color 0 0 0 0)
@@
 	(wire
 		(pts
-			(xy 67.31 62.23) (xy 54.61 62.23)
-		)
-		(stroke
-			(width 0)
-			(type default)
-		)
-	)
-	(wire
-		(pts
 			(xy 162.56 129.54) (xy 171.45 129.54)
 		)
@@
 	(wire
 		(pts
-			(xy 60.96 83.82) (xy 45.72 83.82)
+			(xy 45.72 67.31) (xy 67.31 67.31)
 		)
 		(stroke
@@
 	(wire
 		(pts
-			(xy 46.99 71.12) (xy 45.72 71.12)
+			(xy 36.83 29.21) (xy 35.56 29.21)
 		)
 		(stroke
@@
 	(wire
 		(pts
-			(xy 67.31 67.31) (xy 60.96 67.31)
-		)
-		(stroke
-			(width 0)
-			(type default)
-		)
-	)
-	(wire
-		(pts
-			(xy 46.99 71.12) (xy 54.61 71.12)
+			(xy 36.83 29.21) (xy 44.45 29.21)
 		)
 		(stroke
@@
 	(wire
 		(pts
-			(xy 60.96 67.31) (xy 60.96 83.82)
-		)
-		(stroke
-			(width 0)
-			(type default)
-		)
-	)
-	(wire
-		(pts
 			(xy 170.18 48.26) (xy 170.18 62.23)
 		)
@@
 	(wire
 		(pts
-			(xy 54.61 62.23) (xy 54.61 71.12)
-		)
-		(stroke
-			(width 0)
-			(type default)
-		)
-	)
-	(wire
-		(pts
 			(xy 245.11 57.15) (xy 260.35 57.15)
 		)
@@
 	)
 	(label "PACK+"
-		(at 46.99 83.82 0)
+		(at 46.99 67.31 0)
 		(fields_autoplaced yes)
 		(effects
@@
 	(symbol
 		(lib_id "power:+BATT")
-		(at 46.99 71.12 0)
+		(at 36.83 29.21 0)
 		(unit 1)
 		(exclude_from_sim no)
@@
 		(fields_autoplaced yes)
 		(property "Reference" "#PWR01"
-			(at 46.99 74.93 0)
+			(at 36.83 33.02 0)
 			(effects
 				(font
@@
 		)
 		(property "Value" "+BATT"
-			(at 46.99 66.04 0)
+			(at 36.83 24.13 0)
 			(effects
 				(font
@@
 		)
 		(property "Footprint" ""
-			(at 46.99 71.12 0)
+			(at 36.83 29.21 0)
 			(effects
 				(font
@@
 		)
 		(property "Datasheet" ""
-			(at 46.99 71.12 0)
+			(at 36.83 29.21 0)
 			(effects
 				(font
@@
 		)
 		(property "Description" ""
-			(at 46.99 71.12 0)
+			(at 36.83 29.21 0)
 			(effects
 				(font
@@
 	(symbol
 		(lib_id "Connector_Generic:Conn_01x01")
-		(at 40.64 83.82 180)
+		(at 40.64 67.31 180)
 		(unit 1)
 		(exclude_from_sim no)
@@
 		(fields_autoplaced yes)
 		(property "Reference" "J8"
-			(at 40.64 77.47 0)
+			(at 40.64 60.96 0)
 			(effects
 				(font
@@
 		)
 		(property "Value" "PACK+"
-			(at 40.64 80.01 0)
+			(at 40.64 63.5 0)
 			(effects
 				(font
@@
 		)
 		(property "Footprint" "TestPoint:TestPoint_Pad_4.0x4.0mm"
-			(at 40.64 83.82 0)
+			(at 40.64 67.31 0)
 			(effects
 				(font
@@
 		)
 		(property "Datasheet" "~"
-			(at 40.64 83.82 0)
+			(at 40.64 67.31 0)
 			(effects
 				(font
@@
 		)
 		(property "Description" ""
-			(at 40.64 83.82 0)
+			(at 40.64 67.31 0)
 			(effects
 				(font
@@
 	(symbol
 		(lib_id "Connector_Generic:Conn_01x01")
-		(at 40.64 71.12 180)
+		(at 30.48 29.21 180)
 		(unit 1)
 		(exclude_from_sim no)
@@
 		(fields_autoplaced yes)
 		(property "Reference" "J4"
-			(at 40.64 64.77 0)
+			(at 30.48 22.86 0)
 			(effects
 				(font
@@
 		)
 		(property "Value" "BAT+"
-			(at 40.64 67.31 0)
+			(at 30.48 25.4 0)
 			(effects
 				(font
@@
 		)
 		(property "Footprint" "TestPoint:TestPoint_Pad_4.0x4.0mm"
-			(at 40.64 71.12 0)
+			(at 30.48 29.21 0)
 			(effects
 				(font
@@
 		)
 		(property "Datasheet" "~"
-			(at 40.64 71.12 0)
+			(at 30.48 29.21 0)
 			(effects
 				(font
@@
 		)
 		(property "Description" ""
-			(at 40.64 71.12 0)
+			(at 30.48 29.21 0)
 			(effects
 				(font
@@
 	(symbol
 		(lib_id "power:PWR_FLAG")
-		(at 46.99 71.12 180)
+		(at 36.83 29.21 180)
 		(unit 1)
 		(exclude_from_sim no)
@@
 		(fields_autoplaced yes)
 		(property "Reference" "#FLG01"
-			(at 46.99 73.025 0)
+			(at 36.83 31.115 0)
 			(effects
 				(font
@@
 		)
 		(property "Value" "PWR_FLAG"
-			(at 46.99 76.2 0)
+			(at 36.83 34.29 0)
 			(effects
 				(font
@@
 		)
 		(property "Footprint" ""
-			(at 46.99 71.12 0)
+			(at 36.83 29.21 0)
 			(effects
 				(font
@@
 		)
 		(property "Datasheet" "~"
-			(at 46.99 71.12 0)
+			(at 36.83 29.21 0)
 			(effects
 				(font
@@
 		)
 		(property "Description" ""
-			(at 46.99 71.12 0)
+			(at 36.83 29.21 0)
 			(effects
 				(font
@@
 			(effects
 				(font
-					(size 1.27 1.27)
-				)
-				(justify left)
-			)
-		)
-		(pin "BAT+" output
-			(at 67.31 62.23 180)
-			(effects
-				(font

Commit message: Changed MCU and AFE
Connections:
- net GND: no longer J1.1 (Pin_1)
Other:
- sheet Charger monitoring ports: added none; removed CHG_EN, CP_EN, DSG_EN, PACK+, PACK_V, PCHG_EN, PMON_EN
- moved on the sheet: J1, J2, J4, J8
