File: hardware/greenmobi-bms.kicad_sch (KiCad schematic)
At the start: 14 parts, among them J3 EN, J6 USB_C_Receptacle_USB2.0_14P, J7 CAN, U1 TJA1042T-3

Commit message: package sizes set and AFE layout
Parts:
- J3: symbol Connector_Generic:Conn_01x02 -> Connector_Generic_MountingPin:Conn_01x02_MountingPin
- J6: value USB_C_Receptacle_USB2.0_14P -> USB; symbol Connector:USB_C_Receptacle_USB2.0_14P -> Connector:USB_C_Receptacle_USB2.0_16P
Connections:
- net Frontend/Shutdown: now also J3.1 (Pin_1); no longer J3.2 (Pin_2)
- net GND: now also J3.2 (Pin_2), J3.MP (MountPin); no longer J3.1 (Pin_1)
- net CAN-: now reaches R3.2, U1.6 (CANL)
- net CAN-: now also J7.1 (Pin_1); no longer J7.2 (Pin_2)
- net CAN+: now reaches R3.1, U1.7 (CANH)
- net CAN+: now also J7.2 (Pin_2); no longer J7.1 (Pin_1)
- no-connect marks 2 -> 4
Other:
- moved on the sheet: J7
Changed lines of the file:
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@@
 	)
 	(rectangle
-		(start 21.59 29.21)
+		(start 20.32 29.21)
 		(end 52.197 52.07)
 		(stroke
@@
 	)
 	(junction
+		(at 31.75 44.45)
+		(diameter 0)
+		(color 0 0 0 0)
+	)
+	(junction
 		(at 62.23 39.37)
 		(diameter 0)
@@
 	)
 	(no_connect
+		(at 196.85 91.44)
+	)
+	(no_connect
 		(at 25.4 59.69)
 	)
@@
 		(at 196.85 60.96)
 	)
+	(no_connect
+		(at 196.85 88.9)
+	)
 	(wire
 		(pts
@@
 	(wire
 		(pts
+			(xy 222.25 120.65) (xy 222.25 125.73)
+		)
+		(stroke
+			(width 0)
+			(type default)
+		)
+	)
+	(wire
+		(pts
 			(xy 100.33 90.17) (xy 118.11 90.17)
 		)
@@
 	(wire
 		(pts
+			(xy 217.17 120.65) (xy 222.25 120.65)
+		)
+		(stroke
+			(width 0)
+			(type default)
+		)
+	)
+	(wire
+		(pts
 			(xy 172.72 68.58) (xy 172.72 66.04)
 		)
@@
 	(wire
 		(pts
+			(xy 29.21 46.99) (xy 29.21 44.45)
+		)
+		(stroke
+			(width 0)
+			(type default)
+		)
+	)
+	(wire
+		(pts
 			(xy 207.01 134.62) (xy 209.55 134.62)
 		)
@@
 	(wire
 		(pts
+			(xy 29.21 44.45) (xy 31.75 44.45)
+		)
+		(stroke
+			(width 0)
+			(type default)
+		)
+	)
+	(wire
+		(pts
 			(xy 104.14 38.1) (xy 104.14 39.37)
 		)
@@
 		(pts
 			(xy 172.72 77.47) (xy 176.53 77.47)
+		)
+		(stroke
+			(width 0)
+			(type default)
+		)
+	)
+	(wire
+		(pts
+			(xy 26.67 46.99) (xy 29.21 46.99)
 		)
 		(stroke
@@
 	(label "USB_DP"
 		(at 195.58 76.2 180)
+		(effects
+			(font
+				(size 1.27 1.27)
+			)
+			(justify right bottom)
+		)
+	)
+	(label "CAN+"
+		(at 209.55 129.54 90)
+		(effects
+			(font
+				(size 1.27 1.27)
+			)
+			(justify left bottom)
+		)
+	)
+	(label "CAN-"
+		(at 209.55 134.62 270)
 		(effects
 			(font
@@
 	)
 	(symbol
-		(lib_id "Connector:USB_C_Receptacle_USB2.0_14P")
+		(lib_id "Connector:USB_C_Receptacle_USB2.0_16P")
 		(at 212.09 76.2 0)
 		(mirror y)
@@
 		(fields_autoplaced yes)
 		(property "Reference" "J6"
-			(at 212.09 53.34 0)
-			(effects
-				(font
-					(size 1.27 1.27)
-				)
-			)
-		)
-		(property "Value" "USB_C_Receptacle_USB2.0_14P"
-			(at 212.09 55.88 0)
-			(effects
-				(font
-					(size 1.27 1.27)
-				)
+			(at 223.52 74.9299 0)
+			(effects
+				(font
+					(size 1.27 1.27)
+				)
+				(justify right)
+			)
+		)
+		(property "Value" "USB"
+			(at 223.52 77.4699 0)
+			(effects
+				(font
+					(size 1.27 1.27)
+				)
+				(justify right)
 			)
 		)
@@
 			)
 		)
-		(property "Description" "USB 2.0-only 14P Type-C Receptacle connector"
+		(property "Description" "USB 2.0-only 16P Type-C Receptacle connector"
 			(at 212.09 76.2 0)
 			(effects
@@
 			)
 		)
-		(property "Sim.Device" ""
-			(at 212.09 76.2 0)
-			(effects
-				(font
-					(size 1.27 1.27)
-				)
-			)
-		)
-		(property "Sim.Pins" ""
-			(at 212.09 76.2 0)
-			(effects
-				(font
-					(size 1.27 1.27)
-				)
-			)
-		)
 		(pin "S1"
 		)
@@
 		)
 		(pin "B9"
+		)
+		(pin "B8"
+		)
+		(pin "A8"
 		)
 		(instances
@@
 	)
 	(symbol
-		(lib_id "Connector_Generic:Conn_01x02")
-		(at 26.67 41.91 180)
+		(lib_id "Connector_Generic_MountingPin:Conn_01x02_MountingPin")
+		(at 26.67 39.37 0)
+		(mirror y)
 		(unit 1)
 		(exclude_from_sim no)
@@
 		(on_board yes)
 		(dnp no)
-		(fields_autoplaced yes)
 		(property "Reference" "J3"
-			(at 26.67 33.02 0)
-			(effects
-				(font
-					(size 1.27 1.27)
-				)
+			(at 24.13 42.2657 0)
+			(effects
+				(font
+					(size 1.27 1.27)
+				)
+				(justify left)
 			)
 		)
 		(property "Value" "EN"
-			(at 26.67 35.56 0)
-			(effects
-				(font
-					(size 1.27 1.27)
-				)
+			(at 24.13 39.7257 0)
+			(effects
+				(font
+					(size 1.27 1.27)
+				)
+				(justify left)
 			)
 		)
 		(property "Footprint" "Connector_JST:JST_GH_SM02B-GHS-TB_1x02-1MP_P1.25mm_Horizontal"
-			(at 26.67 41.91 0)
+			(at 26.67 39.37 0)
 			(effects
 				(font
@@
 		)
 		(property "Datasheet" "~"
-			(at 26.67 41.91 0)
-			(effects
-				(font
-					(size 1.27 1.27)
-				)
-				(hide yes)
-			)
-		)
-		(property "Description" "Generic connector, single row, 01x02, script generated (kicad-library-utils/schlib/autogen/connector/)"
-			(at 26.67 41.91 0)
+			(at 26.67 39.37 0)
+			(effects
+				(font
+					(size 1.27 1.27)
+				)
+				(hide yes)
+			)
+		)
+		(property "Description" "Generic connectable mounting pin connector, single row, 01x02, script generated (kicad-library-utils/schlib/autogen/connector/)"
+			(at 26.67 39.37 0)
 			(effects
 				(font
@@
 		)
 		(property "Sim.Device" ""
-			(at 26.67 41.91 0)
+			(at 26.67 39.37 0)
 			(effects
 				(font
@@
 		)
 		(property "Sim.Pins" ""
-			(at 26.67 41.91 0)
+			(at 26.67 39.37 0)
 			(effects
 				(font
@@
 		)
 		(pin "2"
+		)
+		(pin "MP"
 		)
 		(instances
@@
 	)
 	(symbol
+		(lib_name "Conn_01x02_MountingPin_1")
 		(lib_id "Connector_Generic_MountingPin:Conn_01x02_MountingPin")
-		(at 222.25 130.81 0)
+		(at 222.25 133.35 0)
+		(mirror x)
 		(unit 1)
 		(exclude_from_sim no)
@@
 		(on_board yes)
 		(dnp no)
-		(fields_autoplaced yes)
 		(property "Reference" "J7"
-			(at 224.79 131.1655 0)
+			(at 224.79 132.9945 0)
 			(effects
 				(font
@@
 		)
 		(property "Value" "CAN"
-			(at 224.79 133.7055 0)
+			(at 224.79 130.4545 0)
 			(effects
 				(font
@@
 		)
 		(property "Footprint" "Connector_JST:JST_GH_SM02B-GHS-TB_1x02-1MP_P1.25mm_Horizontal"
-			(at 222.25 130.81 0)
+			(at 222.25 133.35 0)
 			(effects
 				(font
@@
 		)
 		(property "Datasheet" "~"
-			(at 222.25 130.81 0)
+			(at 222.25 133.35 0)
 			(effects
 				(font
@@
 		)
 		(property "Description" "Generic connectable mounting pin connector, single row, 01x02, script generated (kicad-library-utils/schlib/autogen/connector/)"
-			(at 222.25 130.81 0)
+			(at 222.25 133.35 0)
 			(effects
 				(font
@@
 		)
 		(property "Sim.Device" ""
-			(at 222.25 130.81 0)
+			(at 222.25 133.35 0)
 			(effects
 				(font
@@
 		)
 		(property "Sim.Pins" ""
-			(at 222.25 130.81 0)
+			(at 222.25 133.35 0)
 			(effects
 				(font
@@
 	(symbol
 		(lib_id "power:GND")
-		(at 222.25 138.43 0)
+		(at 217.17 120.65 0)
 		(unit 1)
 		(exclude_from_sim no)
@@
 		(fields_autoplaced yes)
 		(property "Reference" "#PWR011"
-			(at 222.25 144.78 0)
+			(at 217.17 127 0)
 			(effects
 				(font
@@
 		)
 		(property "Value" "GND"
-			(at 222.25 143.51 0)
+			(at 217.17 125.73 0)
 			(effects
 				(font
@@
 		)
 		(property "Footprint" ""
-			(at 222.25 138.43 0)
+			(at 217.17 120.65 0)
 			(effects
 				(font
@@
 		)
 		(property "Datasheet" ""
-			(at 222.25 138.43 0)
+			(at 217.17 120.65 0)
 			(effects
 				(font
@@
 		)
 		(property "Description" "Power symbol creates a global label with name \"GND\" , ground"
-			(at 222.25 138.43 0)
-			(effects
-				(font
+			(at 217.17 120.65 0)
+			(effects
+				(font

Commit message: Majority of layout placement done
Connections:
- net GND: no longer H4.1
- net BAT+: now reaches H2.1
- net Frontend/BAT+ renamed Frontend/BAT_F
- new net Frontend/PACK-: H4.1
- no-connect marks 4 -> 3
Other:
- sheet Frontend ports: added BAT_F; removed BAT+
Changed lines of the file:
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@@
-	)
-	(junction
-		(at 106.68 69.85)
-		(diameter 0)
-		(color 0 0 0 0)
 	)
 	(junction
@@
 	)
 	(no_connect
-		(at 25.4 59.69)
-	)
-	(no_connect
 		(at 196.85 60.96)
 	)
@@
 	(wire
 		(pts
-			(xy 100.33 69.85) (xy 106.68 69.85)
-		)
-		(stroke
-			(width 0)
-			(type default)
-		)
-	)
-	(wire
-		(pts
 			(xy 217.17 120.65) (xy 222.25 120.65)
 		)
@@
 	(wire
 		(pts
-			(xy 106.68 69.85) (xy 109.22 69.85)
+			(xy 100.33 69.85) (xy 109.22 69.85)
 		)
 		(stroke
@@
 	(label "USB_DP"
 		(at 195.58 76.2 180)
+		(effects
+			(font
+				(size 1.27 1.27)
+			)
+			(justify right bottom)
+		)
+	)
+	(label "BAT+"
+		(at 25.4 59.69 180)
 		(effects
 			(font
@@
 	)
 	(symbol
-		(lib_id "power:GND")
-		(at 106.68 69.85 0)
-		(unit 1)
-		(exclude_from_sim no)
-		(in_bom yes)
-		(on_board yes)
-		(dnp no)
-		(fields_autoplaced yes)
-		(property "Reference" "#PWR04"
-			(at 106.68 76.2 0)
-			(effects
-				(font
-					(size 1.27 1.27)
-				)
-				(hide yes)
-			)
-		)
-		(property "Value" "GND"
-			(at 106.68 74.93 0)
-			(effects
-				(font
-					(size 1.27 1.27)
-				)
-			)
-		)
-		(property "Footprint" ""
-			(at 106.68 69.85 0)
-			(effects
-				(font
-					(size 1.27 1.27)
-				)
-				(hide yes)
-			)
-		)
-		(property "Datasheet" ""
-			(at 106.68 69.85 0)
-			(effects
-				(font
-					(size 1.27 1.27)
-				)
-				(hide yes)
-			)
-		)
-		(property "Description" "Power symbol creates a global label with name \"GND\" , ground"
-			(at 106.68 69.85 0)
-			(effects
-				(font
-					(size 1.27 1.27)
-				)
-				(hide yes)
-			)
-		)
-		(pin "1"
-		)
-		(instances
-			(project ""
-				(path "/3e668e3e-3e16-4665-a807-4735962c41d3"
-					(reference "#PWR04")
-					(unit 1)
-				)
-			)
-		)
-	)
-	(symbol
 		(lib_name "Conn_01x02_MountingPin_1")
 		(lib_id "Connector_Generic_MountingPin:Conn_01x02_MountingPin")
@@
 			)
 		)
-		(pin "BAT+" input
-			(at 82.55 59.69 180)
-			(effects
-				(font
-					(size 1.27 1.27)
-				)
-				(justify left)
-			)
-		)
 		(pin "Shutdown" input
 			(at 82.55 78.74 180)
@@
 			)
 		)
+		(pin "BAT_F" input
+			(at 82.55 59.69 180)
+			(effects
+				(font
+					(size 1.27 1.27)
+				)
+				(justify left)
+			)
+		)
