File: hardware/power-supply.kicad_sch (KiCad schematic)
At the start: 3 parts, among them U3 TPS563200

Commit message: BAT to 12V converter
Parts:
- removed U3: TPS563200, Package_TO_SOT_SMD:SOT-23-6, symbol Regulator_Switching:TPS563200
- added C27: 2.2n, symbol Device:C_Small
- added C28: 3.3n, symbol Device:C_Small
- added C29: 56p, symbol Device:C_Small
- added J13: Conn_01x02, symbol Connector_Generic:Conn_01x02
- added L1: 68u, symbol Device:L
- added R12, R17: 453k, symbol Device:R_Small
- added R16: 49.9, symbol Device:R_Small
- added R18: 100k, symbol Device:R_Small
- added R19: 0, symbol Device:R_Small
- added U4: LM5164DDA, Package_SO:HSOP-8-1EP_3.9x4.9mm_P1.27mm_EP2.41x3.1mm_ThermalVias, symbol Regulator_Switching:LM5164DDA
Connections:
- net GND: now also J13.2 (Pin_2), R16.2, R18.2, U4.1 (GND)
- net BAT_UVLO: no longer names the net of C501.1, R501.2
- net BAT_UVLO: now also U4.2 (VIN), U4.3 (EN/UVLO)
- new net: C27.2, L1.1, R17.1, U4.8 (SW)
- new net: C28.2, L1.2, R12.1, R19.1
- new net: C28.1, C29.1, R17.2
- new net: C29.2, R12.2, R16.1, U4.5 (FB)
- new net: R18.1, U4.4 (RON)
- new net: C27.1, U4.7 (BST)
- new net +12V: J13.1 (Pin_1), R19.2
- no-connect marks 0 -> 1
Other:
- note removed: "5V buck converter"
- company: (none) -> GreenMobi
- title: (none) -> GreenMobi BMS
- moved on the sheet: C501, R501

Commit message: Add missing files
Parts:
- added U3: TPS563200, Package_TO_SOT_SMD:SOT-23-6, symbol Regulator_Switching:TPS563200
Changed lines of the file:
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@@
+    )
+  )
+  (symbol (lib_id "Regulator_Switching:TPS563200") (at 85.09 80.01 0) (unit 1)
+    (in_bom yes) (on_board yes) (dnp no) (fields_autoplaced)
+    (property "Reference" "U3" (at 85.09 69.85 0)
+      (effects (font (size 1.27 1.27)))
+    )
+    (property "Value" "TPS563200" (at 85.09 72.39 0)
+      (effects (font (size 1.27 1.27)))
+    )
+    (property "Footprint" "Package_TO_SOT_SMD:SOT-23-6" (at 86.36 86.36 0)
+      (effects (font (size 1.27 1.27)) (justify left) hide)
+    )
+    (property "Datasheet" "http://www.ti.com/lit/ds/symlink/tps563200.pdf" (at 85.09 80.01 0)
+      (effects (font (size 1.27 1.27)) hide)
+    )
+    (pin "5")
+    (pin "1")
+    (pin "2")
+    (pin "3")
+    (pin "6")
+    (pin "4")
+    (instances
+      (project "greenmobi-bms"
+        (path "/3e668e3e-3e16-4665-a807-4735962c41d3/600d3fd5-a2c8-411e-91ac-e4cbb4ace0f8"
+          (reference "U3") (unit 1)
+        )
+      )
     )
   )

Commit message: Voltage regulators
Parts:
- added C30, C36, C37: 22u, symbol Device:C_Small
- added C31: 2.2u, Capacitor_SMD:C_0603_1608Metric, symbol Device:C_Small
- added C32, C33: 10u, symbol Device:C_Small
- added C34, C35: 100n, symbol Device:C_Small
- added C38: 47u, symbol Device:C_Small
- added L2: 3.3u, symbol Device:L
- added R20: 56.2k, symbol Device:R_Small
- added R21: 10k, symbol Device:R_Small
- added U7: AMS1117-3.3, Package_TO_SOT_SMD:SOT-223-3_TabPin2, symbol Regulator_Linear:AMS1117-3.3
Connections:
- net +12V: now also U3.3 (VIN), U3.5 (EN), C32.1, C33.1, C34.1
- net GND: now also U3.1 (GND), C30.2, C31.2, C32.2, C33.2, C34.2, C36.2, C37.2, C38.2, R21.2, U7.1 (GND)
- net at C28.2, L1.2, R12.1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: now also C38.1
- net at U3.2 (SW): now also C35.1
- net at U3.4 (VFB): now also R20.2, R21.1
- net at U3.6 (VBST): now also C35.2, L2.1
- new net +3.3V: C30.1, U7.2 (VO)
- new net +5V: C31.1, C36.1, C37.1, L2.2, R20.1, U7.3 (VI)
Other:
- moved on the sheet: C27, C28, C29, C501, J13, L1, R12, R16, R17, R18, R19, R501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

Commit message: Fix some ERC issues
Parts:
- renumbered C32 to C14, C33 to C15, C501 to C16, C34 to C17, C35 to C18, C36 to C19, C27 to C20, C37 to C21, C29 to C22, C28 to C23, C38 to C24, C31 to C25, C30 to C26, L2 to L1, L1 to L2, R501 to R16, R18 to R17, R17 to R18, R20 to R19, R21 to R20, R12 to R21, R16 to R22, R19 to R23, U3 to U6, U4 to U7, U7 to U8

Commit message: Remove BLE module to increase efficiency
Connections:
- net GND: now also U7.9 (EP)
Changed lines of the file:
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@@
   (junction (at 99.06 107.95) (diameter 0) (color 0 0 0 0)
   )
+  (junction (at 121.92 72.39) (diameter 0) (color 0 0 0 0)
+  )
   (junction (at 156.21 110.49) (diameter 0) (color 0 0 0 0)
   )
@@
   )
   (junction (at 146.05 57.15) (diameter 0) (color 0 0 0 0)
+  )
+  (junction (at 194.31 57.15) (diameter 0) (color 0 0 0 0)
   )
   (junction (at 88.9 107.95) (diameter 0) (color 0 0 0 0)
@@
     (stroke (width 0) (type default))
   )
+  (wire (pts (xy 121.92 72.39) (xy 127 72.39))
+    (stroke (width 0) (type default))
+  )
   (wire (pts (xy 153.67 72.39) (xy 153.67 73.66))
     (stroke (width 0) (type default))
@@
     (stroke (width 0) (type default))
   )
+  (wire (pts (xy 194.31 57.15) (xy 198.12 57.15))
+    (stroke (width 0) (type default))
+  )
   (wire (pts (xy 137.16 57.15) (xy 139.7 57.15))
     (stroke (width 0) (type default))
@@
     (stroke (width 0) (type default))
   )
-  (wire (pts (xy 190.5 57.15) (xy 198.12 57.15))
+  (wire (pts (xy 190.5 57.15) (xy 194.31 57.15))
     (stroke (width 0) (type default))
   )
@@
   (hierarchical_label "Power_in" (shape input) (at 73.66 52.07 180) (fields_autoplaced)
     (effects (font (size 1.27 1.27)) (justify right))
+  )
+  (symbol (lib_id "power:PWR_FLAG") (at 82.55 52.07 0) (unit 1)
+    (in_bom yes) (on_board yes) (dnp no) (fields_autoplaced)
+    (property "Reference" "#FLG05" (at 82.55 50.165 0)
+      (effects (font (size 1.27 1.27)) hide)
+    )
+    (property "Value" "PWR_FLAG" (at 82.55 46.99 0)
+      (effects (font (size 1.27 1.27)) hide)
+    )
+    (property "Footprint" "" (at 82.55 52.07 0)
+      (effects (font (size 1.27 1.27)) hide)
+    )
+    (property "Datasheet" "~" (at 82.55 52.07 0)
+      (effects (font (size 1.27 1.27)) hide)
+    )
+    (pin "1")
+    (instances
+      (project "greenmobi-bms"
+        (path "/3e668e3e-3e16-4665-a807-4735962c41d3/600d3fd5-a2c8-411e-91ac-e4cbb4ace0f8"
+          (reference "#FLG05") (unit 1)
+        )
+      )
+    )
   )
   (symbol (lib_id "power:GND") (at 121.92 74.93 0) (unit 1)
@@
         (path "/3e668e3e-3e16-4665-a807-4735962c41d3/600d3fd5-a2c8-411e-91ac-e4cbb4ace0f8"
           (reference "#PWR058") (unit 1)
+        )
+      )
+    )
+  )
+  (symbol (lib_id "power:PWR_FLAG") (at 156.21 110.49 270) (unit 1)
+    (in_bom yes) (on_board yes) (dnp no) (fields_autoplaced)
+    (property "Reference" "#FLG06" (at 158.115 110.49 0)
+      (effects (font (size 1.27 1.27)) hide)
+    )
+    (property "Value" "PWR_FLAG" (at 161.29 110.49 0)
+      (effects (font (size 1.27 1.27)) hide)
+    )
+    (property "Footprint" "" (at 156.21 110.49 0)
+      (effects (font (size 1.27 1.27)) hide)
+    )
+    (property "Datasheet" "~" (at 156.21 110.49 0)
+      (effects (font (size 1.27 1.27)) hide)
+    )
+    (pin "1")
+    (instances
+      (project "greenmobi-bms"
+        (path "/3e668e3e-3e16-4665-a807-4735962c41d3/600d3fd5-a2c8-411e-91ac-e4cbb4ace0f8"
+          (reference "#FLG06") (unit 1)
         )
       )
@@
         )
       )
+    )
+  )
+  (symbol (lib_id "power:PWR_FLAG") (at 194.31 57.15 180) (unit 1)
+    (in_bom yes) (on_board yes) (dnp no) (fields_autoplaced)
+    (property "Reference" "#FLG04" (at 194.31 59.055 0)
+      (effects (font (size 1.27 1.27)) hide)
+    )
+    (property "Value" "PWR_FLAG" (at 194.31 62.23 0)
+      (effects (font (size 1.27 1.27)) hide)
+    )
+    (property "Footprint" "" (at 194.31 57.15 0)
+      (effects (font (size 1.27 1.27)) hide)
+    )
+    (property "Datasheet" "~" (at 194.31 57.15 0)
+      (effects (font (size 1.27 1.27)) hide)
+    )
+    (pin "1")
+    (instances
+      (project "greenmobi-bms"
+        (path "/3e668e3e-3e16-4665-a807-4735962c41d3/600d3fd5-a2c8-411e-91ac-e4cbb4ace0f8"
+          (reference "#FLG04") (unit 1)
+        )
+      )

Commit message: Assigned some footprints
Parts:
- C14: footprint (none) -> Capacitor_SMD:C_0402_1005Metric
- C15: footprint (none) -> Capacitor_SMD:C_0805_2012Metric
- C16: value 2.2u -> 100n; footprint Capacitor_SMD:C_0603_1608Metric -> Capacitor_SMD:C_1206_3216Metric
- C25: footprint Capacitor_SMD:C_0603_1608Metric -> (none)
- renumbered J13 to J12, U6 to U5, U7 to U6, U8 to U7
