File: hardware/power-supply.kicad_sch (KiCad schematic)
At the start: 17 parts, among them U3 LM5164DDA, U4 TPS70933

Commit message: Prettyfy Schematic
Parts:
- removed R10: 0, Resistor_SMD:R_0402_1005Metric, symbol Device:R_Small
Connections:
- net Power_in is gone; now on net BAT: C19.1, U3.2 (VIN)
- net BAT: now reaches U3.3 (EN/UVLO)
- net +3.3V renamed 3.3V
- net +5V renamed 5V
Other:
- note added: "5V to 3.3V LDO"
- note added: "BAT to 5V buck"
- note added: "Logic Power"
- note added: "Main Buck"
- moved on the sheet: C19, C20, C21, C22, C23, C24, C25, C26, L4, R11, R12, R13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

Commit message: Reanotate schematic
Parts:
- renumbered C24 to C23, C23 to C24, R11 to R10, R12 to R11, R13 to R12, R14 to R13, R15 to R14

Commit message: Improvements to main buck and load switch
Parts:
- removed R14: 0, Resistor_SMD:R_0402_1005Metric, symbol Device:R_Small
- added C52, C53: 4.7u, Capacitor_SMD:C_0805_2012Metric, symbol Device:C_Small
- C23: value 56p -> 100p
- C25: value 3.3n -> 1.5n
- C26: value 47u -> 4.7u; footprint Capacitor_SMD:C_0603_1608Metric -> Capacitor_SMD:C_0805_2012Metric
- L4: footprint (none) -> Inductor_SMD:L_KOHERelec_MDA7030; LCSC (none) -> C2894721
- R10: value 100k -> 82.5k
- R11: value 316k -> 523k
- R12: value 316k -> 200k
- R13: value 100k -> 63.4k
- U3: value LM5164DDA -> LM5163DDA; LCSC (none) -> C2873264
Connections:
- net 5V: now also C26.1, C52.1, C53.1
- net BAT: no longer U3.3 (EN/UVLO)
- net GND: now also C52.2, C53.2
- new net EN: U3.3 (EN/UVLO)
Other:
- moved on the sheet: C19, C21, C23, C25, C26, L4, R10, R11, R12, R13, U3

Commit message: Reanotate schematic
Parts:
- renumbered C23 to C22, C22 to C23, C25 to C24, C24 to C25, C52 to C27, C53 to C28
Changed lines of the file:
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@@
 		(dnp no)
 		(fields_autoplaced yes)
-		(property "Reference" "#PWR038"
+		(property "Reference" "#PWR037"
 			(at 125.73 95.25 0)
 			(effects
@@
 			(project "greenmobi-bms"
 				(path "/3e668e3e-3e16-4665-a807-4735962c41d3/600d3fd5-a2c8-411e-91ac-e4cbb4ace0f8"
-					(reference "#PWR038")
+					(reference "#PWR037")
 					(unit 1)
 				)
@@
 		(dnp no)
 		(fields_autoplaced yes)
-		(property "Reference" "C23"
+		(property "Reference" "C22"
 			(at 160.02 82.5562 0)
 			(effects
@@
 			(project "greenmobi-bms"
 				(path "/3e668e3e-3e16-4665-a807-4735962c41d3/600d3fd5-a2c8-411e-91ac-e4cbb4ace0f8"
-					(reference "C23")
+					(reference "C22")
 					(unit 1)
 				)
@@
 		(dnp no)
 		(fields_autoplaced yes)
-		(property "Reference" "C53"
+		(property "Reference" "C28"
 			(at 204.47 81.2862 0)
 			(effects
@@
 			(project "greenmobi-bms"
 				(path "/3e668e3e-3e16-4665-a807-4735962c41d3/600d3fd5-a2c8-411e-91ac-e4cbb4ace0f8"
-					(reference "C53")
+					(reference "C28")
 					(unit 1)
 				)
@@
 		(dnp no)
 		(fields_autoplaced yes)
-		(property "Reference" "#PWR047"
+		(property "Reference" "#PWR044"
 			(at 193.04 101.6 0)
 			(effects
@@
 			(project "greenmobi-bms"
 				(path "/3e668e3e-3e16-4665-a807-4735962c41d3/600d3fd5-a2c8-411e-91ac-e4cbb4ace0f8"
-					(reference "#PWR047")
+					(reference "#PWR044")
 					(unit 1)
 				)
@@
 		(dnp no)
 		(fields_autoplaced yes)
-		(property "Reference" "C22"
+		(property "Reference" "C23"
 			(at 160.02 124.4663 0)
 			(effects
@@
 			(project "greenmobi-bms"
 				(path "/3e668e3e-3e16-4665-a807-4735962c41d3/600d3fd5-a2c8-411e-91ac-e4cbb4ace0f8"
-					(reference "C22")
+					(reference "C23")
 					(unit 1)
 				)
@@
 		(dnp no)
 		(fields_autoplaced yes)
-		(property "Reference" "#PWR048"
+		(property "Reference" "#PWR045"
 			(at 201.93 101.6 0)
 			(effects
@@
 			(project "greenmobi-bms"
 				(path "/3e668e3e-3e16-4665-a807-4735962c41d3/600d3fd5-a2c8-411e-91ac-e4cbb4ace0f8"
-					(reference "#PWR048")
+					(reference "#PWR045")
 					(unit 1)
 				)
@@
 		(dnp no)
 		(fields_autoplaced yes)
-		(property "Reference" "C24"
+		(property "Reference" "C25"
 			(at 168.91 124.4663 0)
 			(effects
@@
 			(project "greenmobi-bms"
 				(path "/3e668e3e-3e16-4665-a807-4735962c41d3/600d3fd5-a2c8-411e-91ac-e4cbb4ace0f8"
-					(reference "C24")
+					(reference "C25")
 					(unit 1)
 				)
@@
 		(on_board yes)
 		(dnp no)
-		(property "Reference" "C25"
+		(property "Reference" "C24"
 			(at 161.29 73.66 90)
 			(effects
@@
 			(project "greenmobi-bms"
 				(path "/3e668e3e-3e16-4665-a807-4735962c41d3/600d3fd5-a2c8-411e-91ac-e4cbb4ace0f8"
-					(reference "C25")
+					(reference "C24")
 					(unit 1)
 				)
@@
 		(dnp no)
 		(fields_autoplaced yes)
-		(property "Reference" "#PWR037"
+		(property "Reference" "#PWR038"
 			(at 129.54 135.89 0)
 			(effects
@@
 			(project "greenmobi-bms"
 				(path "/3e668e3e-3e16-4665-a807-4735962c41d3/600d3fd5-a2c8-411e-91ac-e4cbb4ace0f8"
-					(reference "#PWR037")
+					(reference "#PWR038")
 					(unit 1)
 				)
@@
 		(dnp no)
 		(fields_autoplaced yes)
-		(property "Reference" "C52"
+		(property "Reference" "C27"
 			(at 195.58 81.2862 0)
 			(effects
@@
 			(project "greenmobi-bms"
 				(path "/3e668e3e-3e16-4665-a807-4735962c41d3/600d3fd5-a2c8-411e-91ac-e4cbb4ace0f8"
-					(reference "C52")
-					(unit 1)
-				)
+					(reference "C27")
+					(unit 1)
+				)

Commit message: BAT connector change
Parts:
- added C58: 2.2u, Capacitor_SMD:C_1206_3216Metric, symbol Device:C_Small
- C19: LCSC (none) -> C1945
- C21: footprint (none) -> Capacitor_SMD:C_0402_1005Metric; LCSC (none) -> C106861
Connections:
- net BAT: now also C58.2
- net GND: now also C58.1
Changed lines of the file:
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@@
 	)
 	(rectangle
-		(start 79.375 51.435)
+		(start 73.66 51.435)
 		(end 213.36 105.41)
 		(stroke
@@
 	(text "Main Buck"
 		(exclude_from_sim no)
-		(at 90.932 55.372 0)
+		(at 85.09 54.864 0)
 		(effects
 			(font
@@
 	(text "BAT to 5V buck"
 		(exclude_from_sim no)
-		(at 89.408 58.674 0)
+		(at 83.566 58.166 0)
 		(effects
 			(font
@@
 	)
 	(junction
+		(at 86.36 66.04)
+		(diameter 0)
+		(color 0 0 0 0)
+	)
+	(junction
 		(at 157.48 121.92)
 		(diameter 0)
@@
 	(wire
 		(pts
-			(xy 87.63 66.04) (xy 96.52 66.04)
+			(xy 81.28 66.04) (xy 86.36 66.04)
 		)
 		(stroke
@@
 	(wire
 		(pts
+			(xy 86.36 66.04) (xy 96.52 66.04)
+		)
+		(stroke
+			(width 0)
+			(type default)
+		)
+	)
+	(wire
+		(pts
 			(xy 107.95 78.74) (xy 115.57 78.74)
 		)
@@
 	(wire
 		(pts
+			(xy 86.36 66.04) (xy 86.36 74.93)
+		)
+		(stroke
+			(width 0)
+			(type default)
+		)
+	)
+	(wire
+		(pts
 			(xy 143.51 87.63) (xy 157.48 87.63)
 		)
@@
 		(pts
 			(xy 157.48 78.74) (xy 157.48 81.28)
+		)
+		(stroke
+			(width 0)
+			(type default)
+		)
+	)
+	(wire
+		(pts
+			(xy 86.36 80.01) (xy 86.36 88.9)
 		)
 		(stroke
@@
 	(hierarchical_label "BAT"
 		(shape input)
-		(at 87.63 66.04 180)
+		(at 81.28 66.04 180)
 		(effects
 			(font
@@
 	)
 	(symbol
+		(lib_id "Device:C_Small")
+		(at 86.36 77.47 180)
+		(unit 1)
+		(exclude_from_sim no)
+		(in_bom yes)
+		(on_board yes)
+		(dnp no)
+		(fields_autoplaced yes)
+		(property "Reference" "C58"
+			(at 88.9 76.1935 0)
+			(effects
+				(font
+					(size 1.27 1.27)
+				)
+				(justify right)
+			)
+		)
+		(property "Value" "2.2u"
+			(at 88.9 78.7335 0)
+			(effects
+				(font
+					(size 1.27 1.27)
+				)
+				(justify right)
+			)
+		)
+		(property "Footprint" "Capacitor_SMD:C_1206_3216Metric"
+			(at 86.36 77.47 0)
+			(effects
+				(font
+					(size 1.27 1.27)
+				)
+				(hide yes)
+			)
+		)
+		(property "Datasheet" "~"
+			(at 86.36 77.47 0)
+			(effects
+				(font
+					(size 1.27 1.27)
+				)
+				(hide yes)
+			)
+		)
+		(property "Description" "Unpolarized capacitor, small symbol"
+			(at 86.36 77.47 0)
+			(effects
+				(font
+					(size 1.27 1.27)
+				)
+				(hide yes)
+			)
+		)
+		(property "Sim.Device" ""
+			(at 86.36 77.47 0)
+			(effects
+				(font
+					(size 1.27 1.27)
+				)
+			)
+		)
+		(property "Sim.Pins" ""
+			(at 86.36 77.47 0)
+			(effects
+				(font
+					(size 1.27 1.27)
+				)
+			)
+		)
+		(property "LCSC" "C577211"
+			(at 86.36 77.47 0)
+			(effects
+				(font
+					(size 1.27 1.27)
+				)
+				(hide yes)
+			)
+		)
+		(pin "1"
+		)
+		(pin "2"
+		)
+		(instances
+			(project "greenmobi-bms"
+				(path "/3e668e3e-3e16-4665-a807-4735962c41d3/600d3fd5-a2c8-411e-91ac-e4cbb4ace0f8"
+					(reference "C58")
+					(unit 1)
+				)
+			)
+		)
+	)
+	(symbol
 		(lib_id "power:GND")
 		(at 166.37 129.54 0)
@@
 		(fields_autoplaced yes)
 		(property "Reference" "C21"
-			(at 146.05 67.3163 0)
+			(at 146.05 67.3162 0)
 			(effects
 				(font
@@
 		)
 		(property "Value" "2.2n"
-			(at 146.05 69.8563 0)
+			(at 146.05 69.8562 0)
 			(effects
 				(font
@@
 			)
 		)
-		(property "Footprint" ""
+		(property "Footprint" "Capacitor_SMD:C_0402_1005Metric"
 			(at 143.51 68.58 0)
 			(effects
@@
 					(size 1.27 1.27)
 				)
+				(hide yes)
 			)
 		)
@@
 					(size 1.27 1.27)
 				)
+				(hide yes)
+			)
+		)
+		(property "LCSC" "C106861"
+			(at 143.51 68.58 0)
+			(effects
+				(font
+					(size 1.27 1.27)
+				)
+				(hide yes)
 			)
 		)
@@
 				(path "/3e668e3e-3e16-4665-a807-4735962c41d3/600d3fd5-a2c8-411e-91ac-e4cbb4ace0f8"
 					(reference "C21")
+					(unit 1)
+				)
+			)
+		)
+	)
+	(symbol
+		(lib_id "power:GND")
+		(at 86.36 88.9 0)
+		(unit 1)
+		(exclude_from_sim no)
+		(in_bom yes)
+		(on_board yes)
+		(dnp no)
+		(fields_autoplaced yes)
+		(property "Reference" "#PWR061"
+			(at 86.36 95.25 0)
+			(effects
+				(font
+					(size 1.27 1.27)
+				)
+				(hide yes)
+			)
+		)
+		(property "Value" "GND"
+			(at 86.36 93.98 0)
+			(effects
+				(font
+					(size 1.27 1.27)
+				)
+			)
+		)
+		(property "Footprint" ""
+			(at 86.36 88.9 0)
+			(effects
+				(font
+					(size 1.27 1.27)
+				)
+				(hide yes)
+			)
+		)
+		(property "Datasheet" ""
+			(at 86.36 88.9 0)
+			(effects
+				(font
+					(size 1.27 1.27)
+				)
+				(hide yes)
+			)
+		)
+		(property "Description" "Power symbol creates a global label with name \"GND\" , ground"
+			(at 86.36 88.9 0)
+			(effects
+				(font
+					(size 1.27 1.27)
+				)
+				(hide yes)
+			)
+		)
+		(pin "1"
+		)
+		(instances
+			(project "greenmobi-bms"
+				(path "/3e668e3e-3e16-4665-a807-4735962c41d3/600d3fd5-a2c8-411e-91ac-e4cbb4ace0f8"
+					(reference "#PWR061")
 					(unit 1)
 				)
@@
 					(size 1.27 1.27)
 				)
+				(hide yes)
 			)
 		)
@@
 					(size 1.27 1.27)
 				)
-			)
-		)
+				(hide yes)
+			)
+		)
+		(property "LCSC" "C1945"
+			(at 96.52 77.47 0)
+			(effects
+				(font
+					(size 1.27 1.27)
+				)
+				(hide yes)
+			)
+		)
