File: hardware/oled.kicad_sch (KiCad schematic)
At the start: 1 part, among them J17 Conn_01x30

Commit message: OLED regulator
Parts:
- added C14, C18: 1u, symbol Device:C_Small
- added Q28: AO3400A, Package_TO_SOT_SMD:SOT-23, symbol Transistor_FET:AO3400A
- added Q29: AO3401A, Package_TO_SOT_SMD:SOT-23, symbol Transistor_FET:AO3401A
- added R91, R93: 47k, symbol Device:R_Small
- J17: LCSC (none) -> C2890596
Connections:
- net GND: now also J17.1 (Pin_1)
- net at J17.2 (Pin_2): now also C14.1
- net at J17.3 (Pin_3): now also C14.2
- net at J17.4 (Pin_4): now also C18.1
- net at J17.5 (Pin_5): now also C18.2
- net at J17.6 (Pin_6): now also Q29.3 (D)
- net at J17.8 (Pin_8): now also Q28.2 (S), R93.2
- new net: Q28.3 (D), Q29.1 (G), R91.2
- new net: Q28.1 (G), R93.1
- new net +3.3V: Q29.2 (S), R91.1
- no-connect marks 0 -> 1
Other:
- moved on the sheet: J17

Commit message: OLED interface complete
Parts:
- removed Q28: AO3400A, Package_TO_SOT_SMD:SOT-23, symbol Transistor_FET:AO3400A
- removed Q29: AO3401A, Package_TO_SOT_SMD:SOT-23, symbol Transistor_FET:AO3401A
- removed R91, R93: 47k, symbol Device:R_Small
- added C62, C65: 4.7u, symbol Device:C_Small
- added C64: 100n, symbol Device:C_Small
- added R99: 910k, symbol Device:R_Small
- C14: value 1u -> 100n; Notes 16V X5R -> (none)
- C18: value 1u -> 4.7u; Notes 16V X5R -> 16V X7R
Connections:
- net +3.3V: now also J17.11 (Pin_11), J17.6 (Pin_6), J17.9 (Pin_9), C64.1, C65.1
- net GND: now also C14.2, C18.2, J17.10 (Pin_10), J17.12 (Pin_12), J17.13 (Pin_13), J17.15 (Pin_15), J17.16 (Pin_16), J17.17 (Pin_17), J17.21 (Pin_21), J17.22 (Pin_22), J17.23 (Pin_23), J17.24 (Pin_24), J17.25 (Pin_25), J17.29 (Pin_29), J17.30 (Pin_30), J17.8 (Pin_8), C62.1, C64.2, C65.2, R99.1
- net SCL: now also J17.18 (Pin_18)
- net SDA: now also J17.19 (Pin_19), J17.20 (Pin_20)
- net at J17.2 (Pin_2): no longer C14.1
- net at J17.3 (Pin_3): no longer C14.2
- net at J17.4 (Pin_4): no longer C18.1
- net at J17.5 (Pin_5): no longer C18.2
- net ~{RESET}: now reaches J17.14 (Pin_14)
- net at J17.26 (Pin_26): now also R99.2
- net at J17.27 (Pin_27): now also C62.2
- net +9V: now reaches J17.28 (Pin_28)
- net +9V: now also C14.1, C18.1
- no-connect marks 1 -> 5
