File: hardware/oled.kicad_sch (KiCad schematic)
At the start: 7 parts, among them J17 Conn_01x30

Commit message: Initiated sourcing
Parts:
- C14: footprint (none) -> Capacitor_SMD:C_0603_1608Metric
- C64: footprint (none) -> Capacitor_SMD:C_0402_1005Metric
Changed lines of the file:
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@@
 			)
 		)
-		(property "Footprint" ""
+		(property "Footprint" "Capacitor_SMD:C_0402_1005Metric"
 			(at 153.67 83.82 0)
 			(effects
@@
 			)
 		)
-		(property "Footprint" ""
+		(property "Footprint" "Capacitor_SMD:C_0603_1608Metric"
 			(at 162.56 137.16 0)
 			(effects

Commit message: More sourcing components
Parts:
- C18, C62: footprint (none) -> Capacitor_SMD:C_0603_1608Metric
- C65: footprint (none) -> Capacitor_SMD:C_0402_1005Metric
- J17: LCSC C2890596 -> C18723026
Changed lines of the file:
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@@
 			)
 		)
-		(property "LCSC" "C2890596"
+		(property "LCSC" "C18723026"
 			(at 195.58 95.25 0)
 			(effects
@@
 			)
 		)
-		(property "Footprint" ""
+		(property "Footprint" "Capacitor_SMD:C_0603_1608Metric"
 			(at 153.67 137.16 0)
 			(effects
@@
 			)
 		)
-		(property "Footprint" ""
+		(property "Footprint" "Capacitor_SMD:C_0402_1005Metric"
 			(at 142.24 83.82 0)
 			(effects
@@
 			)
 		)
-		(property "Footprint" ""
+		(property "Footprint" "Capacitor_SMD:C_0603_1608Metric"
 			(at 143.51 137.16 0)
 			(effects
