File: hardware/mcu.kicad_sch (KiCad schematic)
At the start: 24 parts, among them J2001 USB_C_Receptacle_USB2.0_14P, J2002 CAN, Q2001 MMBT3904, Q2002 MMBT3904, SW2001 SW_Push, U2001 ESP32-C3, U2002 MCP2562-E-SN

Commit message: Connectors
Parts:
- J2002: footprint Connector_Phoenix_MC:PhoenixContact_MCV_1,5_2-G-3.5_1x02_P3.50mm_Vertical -> Connector_JST:JST_PH_B2B-PH-SM4-TB_1x02-1MP_P2.00mm_Vertical
Changed lines of the file:
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@@
 			)
 		)
-		(property "Footprint" "Connector_Phoenix_MC:PhoenixContact_MCV_1,5_2-G-3.5_1x02_P3.50mm_Vertical"
+		(property "Footprint" "Connector_JST:JST_PH_B2B-PH-SM4-TB_1x02-1MP_P2.00mm_Vertical"
 			(at 200.66 41.91 0)
 			(effects

Commit message: Update to KiCAD 9
Changed lines of the file:
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@@
 (kicad_sch
-	(version 20231120)
+	(version 20250114)
 	(generator "eeschema")
-	(generator_version "8.0")
+	(generator_version "9.0")
 	(paper "A4")
 	(title_block
@@
 		(company "GreenMobi")
 	)
+	(text "Reset button"
+		(exclude_from_sim no)
+		(at 146.05 68.58 0)
+		(effects
+			(font
+				(size 1.27 1.27)
+			)
+			(justify left bottom)
+		)
+	)
+	(text "USB"
+		(exclude_from_sim no)
+		(at 215.265 19.05 0)
+		(effects
+			(font
+				(size 1.27 1.27)
+			)
+			(justify left bottom)
+		)
+	)
+	(text "Microcontroller"
+		(exclude_from_sim no)
+		(at 29.21 27.94 0)
+		(effects
+			(font
+				(size 1.27 1.27)
+			)
+			(justify left bottom)
+		)
+	)
+	(text "Power supply decoupling"
+		(exclude_from_sim no)
+		(at 29.972 33.274 0)
+		(effects
+			(font
+				(size 1.27 1.27)
+			)
+			(justify left bottom)
+		)
+	)
+	(text "CAN interface"
+		(exclude_from_sim no)
+		(at 143.51 23.495 0)
+		(effects
+			(font
+				(size 1.27 1.27)
+			)
+			(justify left bottom)
+		)
+	)
+	(text "State information"
+		(exclude_from_sim no)
+		(at 146.05 119.38 0)
+		(effects
+			(font
+				(size 1.27 1.27)
+			)
+			(justify left bottom)
+		)
+	)
 	(junction
 		(at 111.76 151.13)
@@
 		)
 	)
-	(text "Reset button"
-		(exclude_from_sim no)
-		(at 146.05 68.58 0)
-		(effects
-			(font
-				(size 1.27 1.27)
-			)
-			(justify left bottom)
-		)
-	)
-	(text "USB"
-		(exclude_from_sim no)
-		(at 215.265 19.05 0)
-		(effects
-			(font
-				(size 1.27 1.27)
-			)
-			(justify left bottom)
-		)
-	)
-	(text "Microcontroller"
-		(exclude_from_sim no)
-		(at 29.21 27.94 0)
-		(effects
-			(font
-				(size 1.27 1.27)
-			)
-			(justify left bottom)
-		)
-	)
-	(text "Power supply decoupling"
-		(exclude_from_sim no)
-		(at 29.972 33.274 0)
-		(effects
-			(font
-				(size 1.27 1.27)
-			)
-			(justify left bottom)
-		)
-	)
-	(text "CAN interface"
-		(exclude_from_sim no)
-		(at 143.51 23.495 0)
-		(effects
-			(font
-				(size 1.27 1.27)
-			)
-			(justify left bottom)
-		)
-	)
-	(text "State information"
-		(exclude_from_sim no)
-		(at 146.05 119.38 0)
-		(effects
-			(font
-				(size 1.27 1.27)
-			)
-			(justify left bottom)
-		)
-	)
 	(label "LED_RED"
 		(at 125.73 162.56 0)
-		(fields_autoplaced yes)
 		(effects
 			(font
@@
 	(label "DP"
 		(at 246.38 53.34 0)
-		(fields_autoplaced yes)
 		(effects
 			(font
@@
 	(label "DP"
 		(at 54.61 91.44 180)
-		(fields_autoplaced yes)
 		(effects
 			(font
@@
 	(label "NRST"
 		(at 152.4 83.82 180)
-		(fields_autoplaced yes)
 		(effects
 			(font
@@
 	(label "VBUS"
 		(at 255.27 33.02 0)
-		(fields_autoplaced yes)
 		(effects
 			(font
@@
 	(label "CAN_RX"
 		(at 160.02 40.64 180)
-		(fields_autoplaced yes)
 		(effects
 			(font
@@
 	(label "CAN_RX"
 		(at 105.41 91.44 0)
-		(fields_autoplaced yes)
 		(effects
 			(font
@@
 	(label "CAN_TX"
 		(at 105.41 93.98 0)
-		(fields_autoplaced yes)
 		(effects
 			(font
@@
 	(label "NRST"
 		(at 111.76 156.21 180)
-		(fields_autoplaced yes)
 		(effects
 			(font
@@
 	(label "LED_GREEN"
 		(at 157.48 147.32 180)
-		(fields_autoplaced yes)
 		(effects
 			(font
@@
 	(label "CAN_EN"
 		(at 125.73 149.86 0)
-		(fields_autoplaced yes)
 		(effects
 			(font
@@
 	(label "USB"
 		(at 267.97 30.48 0)
-		(fields_autoplaced yes)
 		(effects
 			(font
@@
 	(label "LED_RED"
 		(at 195.58 147.32 180)
-		(fields_autoplaced yes)
 		(effects
 			(font
@@
 	(label "{VBUS DP DN}"
 		(at 266.7 30.48 90)
-		(fields_autoplaced yes)
 		(effects
 			(font
@@
 	(label "LED_GREEN"
 		(at 125.73 160.02 0)
-		(fields_autoplaced yes)
 		(effects
 			(font
@@
 	(label "SWDIO"
 		(at 92.71 161.29 0)
-		(fields_autoplaced yes)
 		(effects
 			(font
@@
 	(label "BOOT0"
 		(at 111.76 158.75 180)
-		(fields_autoplaced yes)
 		(effects
 			(font
@@
 	(label "DN"
 		(at 246.38 48.26 0)
-		(fields_autoplaced yes)
 		(effects
 			(font
@@
 	(label "USB"
 		(at 49.53 85.09 180)
-		(fields_autoplaced yes)
 		(effects
 			(font
@@
 	(label "CAN_TX"
 		(at 160.02 38.1 180)
-		(fields_autoplaced yes)
 		(effects
 			(font
@@
 	(label "SWDCLK"
 		(at 92.71 163.83 0)
-		(fields_autoplaced yes)
 		(effects
 			(font
@@
 	(label "CAN_EN"
 		(at 160.02 48.26 180)
-		(fields_autoplaced yes)
 		(effects
 			(font
@@
 	(label "DN"
 		(at 54.61 88.9 180)
-		(fields_autoplaced yes)
 		(effects
 			(font
@@
 	(label "Buzzer"
 		(at 114.3 161.29 0)
-		(fields_autoplaced yes)
 		(effects
 			(font
@@
 		(shape output)
 		(at 59.69 106.68 180)
-		(fields_autoplaced yes)
 		(effects
 			(font
@@
 		(shape input)
 		(at 125.73 139.7 0)
-		(fields_autoplaced yes)
 		(effects
 			(font
@@
 		(shape input)
 		(at 125.73 142.24 0)
-		(fields_autoplaced yes)
 		(effects
 			(font
@@
 		(shape bidirectional)
 		(at 113.03 151.13 0)
-		(fields_autoplaced yes)
 		(effects
 			(font
@@
 		(shape input)
 		(at 125.73 134.62 0)
-		(fields_autoplaced yes)
 		(effects
 			(font
@@
 		(shape input)
 		(at 86.36 153.67 180)
-		(fields_autoplaced yes)
 		(effects
 			(font
@@
 		(shape input)
 		(at 125.73 137.16 0)
-		(fields_autoplaced yes)
 		(effects
 			(font
@@
 		(shape input)
 		(at 86.36 156.21 180)
-		(fields_autoplaced yes)
 		(effects
 			(font
@@
 		(shape input)
 		(at 59.69 104.14 180)
-		(fields_autoplaced yes)
 		(effects
 			(font
@@
 		(shape bidirectional)
 		(at 256.54 55.88 0)
-		(fields_autoplaced yes)
 		(effects
 			(font
@@
 		(shape output)
 		(at 125.73 144.78 0)
-		(fields_autoplaced yes)
 		(effects
 			(font
@@
 		(shape input)
 		(at 86.36 151.13 180)
-		(fields_autoplaced yes)
 		(effects
 			(font
@@
 		(shape output)
 		(at 113.03 148.59 0)
-		(fields_autoplaced yes)
 		(effects
 			(font
@@
 		(shape input)
 		(at 125.73 157.48 0)
-		(fields_autoplaced yes)
-		(effects
-			(font
+		(effects
+			(font

Commit message: Simplified AFE
Parts:
- R2002, R2003: value 220 -> 100; footprint (none) -> Resistor_SMD:R_0603_1608Metric
Changed lines of the file:
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@@
 			)
 		)
-		(property "Value" "220"
+		(property "Value" "100"
 			(at 167.64 139.7 0)
 			(effects
@@
 			)
 		)
-		(property "Footprint" ""
+		(property "Footprint" "Resistor_SMD:R_0603_1608Metric"
 			(at 171.45 138.43 0)
 			(effects
@@
 			)
 		)
-		(property "Value" "220"
+		(property "Value" "100"
 			(at 205.74 139.7 0)
 			(effects
@@
 			)
 		)
-		(property "Footprint" ""
+		(property "Footprint" "Resistor_SMD:R_0603_1608Metric"
 			(at 209.55 138.43 0)
 			(effects

Commit message: Test CI
Parts:
- removed R2004, R2005: 4.7k, symbol Device:R_Small
- added R1, R2: 4.7k, Resistor_SMD:R_0402_1005Metric_Pad0.72x0.64mm_HandSolder, symbol Device:R_Small
Connections:
- net +3.3V: now also R1.1, R2.1
- net CAN_RX: no longer U2001.4 (XTAL_32K_P)
- net CAN_TX: no longer U2001.5 (XTAL_32K_N)
- net I2C_SCL: now reaches U2001.27 (U0RXD)
- net I2C_SCL: now also R2.2
- net I2C_SDA: now reaches U2001.28 (U0TXD)
- net I2C_SDA: now also R1.2
Other:
- moved on the sheet: U2001

Commit message: Reanotate
Parts:
- renumbered C2001 to C1, C2002 to C2, C2003 to C3, C2004 to C4, C2007 to C5, D2001 to D1, D2002 to D2, J2002 to J5, J2001 to J6, Q2001 to Q1, Q2002 to Q2, R2009 to R10, R2001 to R3, R2006 to R4, R2002 to R5, R2010 to R6, R2007 to R7, R2003 to R8, R2008 to R9, SW2001 to SW1, U2001 to U1, U2002 to U2

Commit message: MCU pinning
Connections:
- net CAN_EN: now also U1.15 (GPIO9)
- net CHG_EN: now also U1.10 (MTDI)
- net DSG_EN: now also U1.9 (MTMS)
- net HW_EN: now also U1.6 (GPIO2)
- net PCHG_EN: now also U1.14 (GPIO8)
- net PSW_EN: now reaches U1.16 (GPIO10)
- net DIV_CHG: now reaches U1.4 (XTAL_32K_P)
- net DIV_OUT: now reaches U1.5 (XTAL_32K_N)
- no-connect marks 0 -> 7
Other:
- moved on the sheet: R1, R2

Commit message: Remove Thermal reliefs from connectors MP and ESP32 Crystal
Parts:
- added C2, C4: xp, Capacitor_SMD:C_0402_1005Metric, symbol Device:C_Small
- added L1: 24n, Inductor_SMD:L_0402_1005Metric, symbol Device:L_Small
- added Y1: 40MHz, Crystal:Crystal_SMD_3225-4Pin_3.2x2.5mm, symbol Device:Crystal_GND24
- J5: value CAN -> Conn_01x02_MountingPin; symbol Connector_Generic:Conn_01x02 -> Connector_Generic_MountingPin:Conn_01x02_MountingPin
- renumbered C2 to C3, C3 to C5, C4 to C6, C5 to C7
Connections:
- net GND: now also J5.MP (MountPin), C2.2, C4.2, Y1.2, Y1.4
- net at U1.29 (XTAL_N): now also C2.1, Y1.1
- net at U1.30 (XTAL_P): now also L1.2
- new net: C4.1, L1.1, Y1.3

Commit message: Crystal Layout
Connections:
- net GND: now also U1.33 (GND)
Changed lines of the file:
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@@
+	)
+	(symbol
+		(lib_name "GND_3")
+		(lib_id "power:GND")
+		(at 93.98 120.65 0)
+		(unit 1)
+		(exclude_from_sim no)
+		(in_bom yes)
+		(on_board yes)
+		(dnp no)
+		(fields_autoplaced yes)
+		(property "Reference" "#PWR047"
+			(at 93.98 127 0)
+			(effects
+				(font
+					(size 1.27 1.27)
+				)
+				(hide yes)
+			)
+		)
+		(property "Value" "GND"
+			(at 93.98 125.73 0)
+			(effects
+				(font
+					(size 1.27 1.27)
+				)
+			)
+		)
+		(property "Footprint" ""
+			(at 93.98 120.65 0)
+			(effects
+				(font
+					(size 1.27 1.27)
+				)
+				(hide yes)
+			)
+		)
+		(property "Datasheet" ""
+			(at 93.98 120.65 0)
+			(effects
+				(font
+					(size 1.27 1.27)
+				)
+				(hide yes)
+			)
+		)
+		(property "Description" "Power symbol creates a global label with name \"GND\" , ground"
+			(at 93.98 120.65 0)
+			(effects
+				(font
+					(size 1.27 1.27)
+				)
+				(hide yes)
+			)
+		)
+		(pin "1"
+		)
+		(instances
+			(project ""
+				(path "/3e668e3e-3e16-4665-a807-4735962c41d3/1c5935ea-6f80-435f-8ae1-741f5546f8d9"
+					(reference "#PWR047")
+					(unit 1)
+				)
+			)
+		)
 	)
 	(symbol
@@
 		(dnp no)
 		(fields_autoplaced yes)
-		(property "Reference" "#PWR018"
+		(property "Reference" "#PWR019"
 			(at 209.55 132.08 0)
 			(effects
@@
 			(project "greenmobi-bms"
 				(path "/3e668e3e-3e16-4665-a807-4735962c41d3/1c5935ea-6f80-435f-8ae1-741f5546f8d9"
-					(reference "#PWR018")
+					(reference "#PWR019")
 					(unit 1)
 				)
@@
 		(dnp no)
 		(fields_autoplaced yes)
-		(property "Reference" "#PWR020"
+		(property "Reference" "#PWR021"
 			(at 229.87 80.01 0)
 			(effects
@@
 			(project "greenmobi-bms"
 				(path "/3e668e3e-3e16-4665-a807-4735962c41d3/1c5935ea-6f80-435f-8ae1-741f5546f8d9"
-					(reference "#PWR020")
+					(reference "#PWR021")
 					(unit 1)
 				)
@@
 		(dnp no)
 		(fields_autoplaced yes)
-		(property "Reference" "#PWR046"
+		(property "Reference" "#PWR018"
 			(at 200.66 55.88 0)
 			(effects
@@
 			(project ""
 				(path "/3e668e3e-3e16-4665-a807-4735962c41d3/1c5935ea-6f80-435f-8ae1-741f5546f8d9"
-					(reference "#PWR046")
+					(reference "#PWR018")
 					(unit 1)
 				)
@@
 		(dnp no)
 		(fields_autoplaced yes)
-		(property "Reference" "#PWR019"
+		(property "Reference" "#PWR020"
 			(at 209.55 158.75 0)
 			(effects
@@
 			(project "greenmobi-bms"
 				(path "/3e668e3e-3e16-4665-a807-4735962c41d3/1c5935ea-6f80-435f-8ae1-741f5546f8d9"
-					(reference "#PWR019")
+					(reference "#PWR020")
 					(unit 1)
 				)
@@
 		(dnp no)
 		(fields_autoplaced yes)
-		(property "Reference" "#PWR021"
+		(property "Reference" "#PWR022"
 			(at 265.43 55.88 0)
 			(effects
@@
 			(project "greenmobi-bms"
 				(path "/3e668e3e-3e16-4665-a807-4735962c41d3/1c5935ea-6f80-435f-8ae1-741f5546f8d9"
-					(reference "#PWR021")
-					(unit 1)
-				)
+					(reference "#PWR022")
+					(unit 1)
+				)
