File: hardware/mcu.kicad_sch (KiCad schematic)
At the start: 28 parts, among them J5 Conn_01x02_MountingPin, J6 USB_C_Receptacle_USB2.0_14P, Q1 MMBT3904, Q2 MMBT3904, SW1 SW_Push, U1 ESP32-C3, U2 MCP2562-E-SN, Y1 40MHz

Commit message: Various changes (can't remember)
Parts:
- removed J5: Conn_01x02_MountingPin, Connector_JST:JST_PH_B2B-PH-SM4-TB_1x02-1MP_P2.00mm_Vertical, symbol Connector_Generic_MountingPin:Conn_01x02_MountingPin
- removed J6: USB_C_Receptacle_USB2.0_14P, Connector_USB:USB_C_Receptacle_Palconn_UTC16-G, symbol Connector:USB_C_Receptacle_USB2.0_14P
- removed R10, R9: 5.1k, Resistor_SMD:R_0603_1608Metric, symbol Device:R
- removed R6: 120, Resistor_SMD:R_0603_1608Metric, symbol Device:R_Small
- removed U2: MCP2562-E-SN, Package_SO:SOIC-8_3.9x4.9mm_P1.27mm, symbol Interface_CAN_LIN:MCP2562-E-SN
- added AE1: Antenna, symbol Device:Antenna
- added C36, C37: C_Small, symbol Device:C_Small
- added L3: L_Small, symbol Device:L_Small
Connections:
- net +3.3V: no longer D1.2 (A), D2.2 (A)
- net GND: now also C36.2, C37.2
- net at U1.1 (LNA_IN): now also C37.1, L3.1
- net CAN_EN renamed ~{COM_EN}
- net DN renamed USB_DP
- net DP renamed USB_DN
- new net: AE1.1 (A), C36.1, L3.2
- new net +3.3VP: D1.2 (A), D2.2 (A)
Other:
- note removed: "CAN interface"
- note removed: "USB"
- moved on the sheet: C1, C3, C5, C6, C7, D1, D2, Q1, Q2, R1, R2, R3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

Commit message: ESP32 Decoupling
Parts:
- removed AE1: Antenna, symbol Device:Antenna
- added AE1: Antenna_Shield, RF_Antenna:Texas_SWRA117D_2.4GHz_Left, symbol Device:Antenna_Shield
- added C54, C55: 1u, Capacitor_SMD:C_0402_1005Metric, symbol Device:C
- added C56: 10n, Capacitor_SMD:C_0402_1005Metric, symbol Device:C
- added C57: 100n, Capacitor_SMD:C_0402_1005Metric, symbol Device:C
- added L4: 2n, symbol Device:L_Small
- C3: value 100n -> 1u
- C5: value 100n -> 10u
- C6: value 4.7u -> 100n
Connections:
- net +3.3V: now also U1.11 (VDD3P3_RTC), U1.17 (VDD3P3_CPU), U1.18 (VDD_SPI), U1.31 (VDDA), U1.32 (VDDA), C55.1, C56.1, C57.1, L4.1
- net GND: now also AE1.2 (Shield), C54.2, C55.2, C56.2, C57.2
- net at C36.1, L3.2: now also AE1.1 (A)
- net VDD_RF: now reaches U1.2 (VDD3P3), U1.3 (VDD3P3)
- net VDD_RF: now also C54.1, L4.2
Other:
- note added: "RF Power Decoupling"
- note added: "RTC"
- note added: "VDDA"
- note added: "VDD_CPU"
- note added: "VDD_SPI"
- moved on the sheet: C1, C2, C3, C36, C37, C4, C5, C6, L1, L3, R1, R2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

Commit message: RF Inductor sourcing
Parts:
- removed C36: C_Small, symbol Device:C_Small
- removed C7: 100n, Capacitor_SMD:C_0402_1005Metric, symbol Device:C_Small
- removed SW1: SW_Push, Button_Switch_SMD:SW_SPST_CK_RS282G05A3, symbol Switch:SW_Push
- added C58: 1u, Capacitor_SMD:C_0402_1005Metric, symbol Device:C
- added C59: 1.5pF, Capacitor_SMD:C_0402_1005Metric, symbol Device:C_Small
- C2, C4: value xp -> 16p
- C37: value C_Small -> 1.5pF; footprint (none) -> Capacitor_SMD:C_0402_1005Metric; LCSC (none) -> C282238
- L3: value L_Small -> 2.4n; footprint (none) -> Inductor_SMD:L_0402_1005Metric; LCSC (none) -> C97997
- R3: now fitted
- Y1: footprint Crystal:Crystal_SMD_3225-4Pin_3.2x2.5mm -> Crystal:Crystal_SMD_2520-4Pin_2.5x2.0mm; LCSC (none) -> C3007519
Connections:
- net GND: now also C58.2, C59.2
- net NRST: now also U1.7 (CHIP_EN), C58.1
- net at AE1.1 (A), L3.2: now also C59.1
Other:
- note removed: "Reset button"

Commit message: MCU circuit sourced complete
Parts:
- removed D1: Green, LED_SMD:LED_0805_2012Metric, symbol Device:LED_Small
- removed D2: Red, LED_SMD:LED_0805_2012Metric, symbol Device:LED_Small
- removed Q1, Q2: MMBT3904, Package_TO_SOT_SMD:SOT-23, symbol Transistor_BJT:MMBT3904
- removed R4, R7: 47k, Resistor_SMD:R_0402_1005Metric, symbol Device:R_Small
- removed R5, R8: 100, Resistor_SMD:R_0603_1608Metric, symbol Device:R_Small
- added C7: 1u, Capacitor_SMD:C_0402_1005Metric, symbol Device:C_Small
- added R23, R27, R29: 10k, Resistor_SMD:R_0603_1608Metric, symbol Device:R_Small
- added SW1: boot, Button_Switch_SMD:SW_Push_SPST_NO_Alps_SKRK, symbol Switch:SW_Push
- added SW2: reset, Button_Switch_SMD:SW_Push_SPST_NO_Alps_SKRK, symbol Switch:SW_Push
- added TP5: TestPoint, symbol Connector:TestPoint
Connections:
- net +3.3V: now also R23.1, R27.1, R29.1
- net GND: now also C7.2, SW1.1, SW2.1
- net HW_EN: now also R27.2
- net PCHG_EN: now also R29.2
- net ~{COM_EN}: now also C7.1, R23.2, SW1.2
- net at U1.8 (GPIO3): now also TP5.1
- net NRST: no longer names the net of C58.1, R3.2, U1.7 (CHIP_EN)
- net NRST: now also SW2.2
- no-connect marks 7 -> 6
Other:
- note added: "Needed to enter in USB download mode"
- note removed: "State information"
- moved on the sheet: AE1, C1, C2, C3, C37, C4, C5, C54, C55, C56, C57, C58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

Commit message: Thermistor conenctions
Parts:
- added AE2, AE3: Calib, Connector_Coaxial:U.FL_Hirose_U.FL-R-SMT-1_Vertical, symbol Device:Antenna_Shield
- added C36, C60: 100p, Capacitor_SMD:C_0402_1005Metric, symbol Device:C_Small
- added C61: 100p, symbol Device:C_Small
- added TP6, TP7: TestPoint, Capacitor_SMD:C_0402_1005Metric, symbol Connector:TestPoint
- AE1: value Antenna_Shield -> WiFi+BT
Connections:
- net GND: now also AE2.2 (Shield), AE3.2 (Shield), C61.2
- net at C37.1, L3.1: now also C36.1; no longer U1.1 (LNA_IN)
- net at C59.1, L3.2: now also C60.2; no longer AE1.1 (A)
- new net: AE3.1 (A), TP7.1
- new net: C36.2, U1.1 (LNA_IN)
- new net: AE1.1 (A), C60.1, C61.1
- new net: AE2.1 (A), TP6.1
Other:
- moved on the sheet: AE1, C37, C58, C59, L3, R3, SW2

Commit message: CAN transciever
Parts:
- renumbered AE2 to AE1, AE3 to AE2, AE1 to AE3, C7 to C1, C6 to C10, C36 to C11, C37 to C12, C54 to C13, C59 to C14, C58 to C15, C60 to C16, C61 to C17, C1 to C2, C2 to C3, C3 to C4, C4 to C5, C55 to C6, C56 to C7, C57 to C8, C5 to C9, L4 to L2, R23 to R4, R29 to R5, R1 to R6, R2 to R7, R27 to R8, R3 to R9, TP5 to TP1, TP6 to TP2, TP7 to TP3, U1 to U2

Commit message: IO reorganization
Parts:
- added TP4, TP5, TP7, TP8: TestPoint, symbol Connector:TestPoint
- R4, R5, R8, R9: value 10k -> 5.1k
- R6, R7: value 4.7k -> 5.1k
Connections:
- net CHG_EN: no longer names the net of U2.10 (MTDI)
- net CHG_EN: now also TP5.1
- net DSG_EN: no longer names the net of U2.9 (MTMS)
- net DSG_EN: now also TP4.1
- net HW_EN renamed EN
- net PCHG_EN: no longer names the net of R5.2, U2.14 (GPIO8)
- net PCHG_EN: now also TP7.1
- net PSW_EN: no longer names the net of U2.16 (GPIO10)
- net PSW_EN: now also TP8.1

Commit message: Add missing cell conection
Parts:
- added TP10, TP9: TestPoint, symbol Connector:TestPoint
Connections:
- net DIV_CHG: no longer names the net of U2.4 (XTAL_32K_P)
- net DIV_CHG: now also TP9.1
- net DIV_OUT: no longer names the net of U2.5 (XTAL_32K_N)
- net DIV_OUT: now also TP10.1
Changed lines of the file:
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@@
-		)
-	)
-	(hierarchical_label "DIV_OUT"
-		(shape input)
-		(at 128.27 119.38 180)
-		(effects
-			(font
-				(size 1.27 1.27)
-			)
-			(justify right)
 		)
 	)
@@
 		)
 	)
-	(hierarchical_label "DIV_CHG"
-		(shape input)
-		(at 128.27 116.84 180)
-		(effects
-			(font
-				(size 1.27 1.27)
-			)
-			(justify right)
-		)
-	)
 	(hierarchical_label "USB_DN"
 		(shape bidirectional)
@@
 	)
 	(symbol
+		(lib_id "Connector:TestPoint")
+		(at 128.27 116.84 90)
+		(unit 1)
+		(exclude_from_sim no)
+		(in_bom yes)
+		(on_board yes)
+		(dnp no)
+		(property "Reference" "TP9"
+			(at 123.698 116.84 90)
+			(effects
+				(font
+					(size 1.27 1.27)
+				)
+				(justify left)
+			)
+		)
+		(property "Value" "TestPoint"
+			(at 126.2379 114.3 0)
+			(effects
+				(font
+					(size 1.27 1.27)
+				)
+				(justify left)
+				(hide yes)
+			)
+		)
+		(property "Footprint" ""
+			(at 128.27 111.76 0)
+			(effects
+				(font
+					(size 1.27 1.27)
+				)
+				(hide yes)
+			)
+		)
+		(property "Datasheet" "~"
+			(at 128.27 111.76 0)
+			(effects
+				(font
+					(size 1.27 1.27)
+				)
+				(hide yes)
+			)
+		)
+		(property "Description" "test point"
+			(at 128.27 116.84 0)
+			(effects
+				(font
+					(size 1.27 1.27)
+				)
+				(hide yes)
+			)
+		)
+		(property "Sim.Device" ""
+			(at 128.27 116.84 0)
+			(effects
+				(font
+					(size 1.27 1.27)
+				)
+			)
+		)
+		(property "Sim.Pins" ""
+			(at 128.27 116.84 0)
+			(effects
+				(font
+					(size 1.27 1.27)
+				)
+			)
+		)
+		(pin "1"
+		)
+		(instances
+			(project "greenmobi-bms"
+				(path "/3e668e3e-3e16-4665-a807-4735962c41d3/1c5935ea-6f80-435f-8ae1-741f5546f8d9"
+					(reference "TP9")
+					(unit 1)
+				)
+			)
+		)
+	)
+	(symbol
 		(lib_id "Device:C")
 		(at 104.14 48.26 0)
@@
 					(unit 1)
 				)
+			)
+		)
+	)
+	(symbol
+		(lib_id "Connector:TestPoint")
+		(at 128.27 119.38 90)
+		(unit 1)
+		(exclude_from_sim no)
+		(in_bom yes)
+		(on_board yes)
+		(dnp no)
+		(property "Reference" "TP10"
+			(at 123.698 119.38 90)
+			(effects
+				(font
+					(size 1.27 1.27)
+				)
+				(justify left)
+			)
+		)
+		(property "Value" "TestPoint"
+			(at 126.2379 116.84 0)
+			(effects
+				(font
+					(size 1.27 1.27)
+				)
+				(justify left)
+				(hide yes)
+			)
+		)
+		(property "Footprint" ""
+			(at 128.27 114.3 0)
+			(effects
+				(font
+					(size 1.27 1.27)
+				)
+				(hide yes)
+			)
+		)
+		(property "Datasheet" "~"
+			(at 128.27 114.3 0)
+			(effects
+				(font
+					(size 1.27 1.27)
+				)
+				(hide yes)
+			)
+		)
+		(property "Description" "test point"
+			(at 128.27 119.38 0)
+			(effects
+				(font
+					(size 1.27 1.27)
+				)
+				(hide yes)
+			)
+		)
+		(property "Sim.Device" ""
+			(at 128.27 119.38 0)
+			(effects
+				(font
+					(size 1.27 1.27)
+				)
+			)
+		)
+		(property "Sim.Pins" ""
+			(at 128.27 119.38 0)
+			(effects
+				(font
+					(size 1.27 1.27)
+				)
+			)
+		)
+		(pin "1"
+		)
+		(instances
+			(project "greenmobi-bms"
+				(path "/3e668e3e-3e16-4665-a807-4735962c41d3/1c5935ea-6f80-435f-8ae1-741f5546f8d9"
+					(reference "TP10")
+					(unit 1)
+				)
