File: hardware/frontend.kicad_sch (KiCad schematic)
At the start: 33 parts, among them J5001 EXT_NTC, J5002 EXT_NTC, J5004 Conn_01x03, J5005 Conn_01x11, J5006 Conn_01x03, Q37 IPTC025N15NM6, Q45 BSS127S, Q5001 IPTC025N15NM6, U5002 BQ769x2

Commit message: Reanotate
Parts:
- renumbered C41 to C16, C40 to C17, C37 to C18, C42 to C19, C27 to C20, D5 to D3, D1 to D5, J5004 to J10, J5005 to J11, J5001 to J7, J5002 to J8, J5006 to J9, Q5001 to Q7, Q37 to Q8, Q45 to Q9, R173 to R31, R168 to R32, R169 to R33, R167 to R34, R166 to R35, R141 to R36, R143 to R37, R142 to R38, R170 to R39, R144 to R40, R172 to R41, R171 to R42, R99 to R43, TH5001 to TH1, U5002 to U5

Commit message: MCU pinning
Parts:
- C20: footprint (none) -> Capacitor_SMD:C_0402_1005Metric
- R43: footprint (none) -> Resistor_SMD:R_0402_1005Metric
Connections:
- net CEL_0: now also J11.11 (Pin_11)
- net CEL_1: now also J11.10 (Pin_10)
- net CEL_10: now also J11.1 (Pin_1)
- net CEL_11: now also J10.3 (Pin_3)
- net CEL_14: now also J9.3 (Pin_3)
- net CEL_15: now also J9.2 (Pin_2)
- net CEL_16: now also J9.1 (Pin_1)
- net CEL_2: now also J11.9 (Pin_9)
- net CEL_3: now also J11.8 (Pin_8)
- net CEL_4: now also J11.7 (Pin_7)
- net CEL_5: now also J11.6 (Pin_6)
- net CEL_6: now also J11.5 (Pin_5)
- net CEL_8: now also J11.3 (Pin_3)
- net CEL_9: now also J11.2 (Pin_2)
- net PDSG: now reaches U5.39 (PDSG)
- net PCHG: now reaches U5.40 (PCHG)
- net DSG: now reaches U5.43 (DSG)
- net CHG: now reaches U5.45 (CHG)
- net DCHG: no longer names the net of U5.31 (DCHG)
- net DDSG: no longer names the net of U5.32 (DDSG)
Other:
- moved on the sheet: J10, J11, J7, J8, J9, TH1

Commit message: Remove Thermal reliefs from connectors MP and ESP32 Crystal
Parts:
- removed J7: EXT_NTC, Connector_JST:JST_PH_S2B-PH-SM4-TB_1x02-1MP_P2.00mm_Horizontal, symbol Connector:Conn_01x02_Pin
- added J12: EXT_NTC, Connector_JST:JST_PH_S2B-PH-SM4-TB_1x02-1MP_P2.00mm_Horizontal, symbol Connector_Generic_MountingPin:Conn_01x02_MountingPin
- J10, J9: value Conn_01x03 -> Conn_01x03_MountingPin; symbol Connector_Generic:Conn_01x03 -> Connector_Generic_MountingPin:Conn_01x03_MountingPin
- J11: value Conn_01x11 -> Conn_01x11_MountingPin; symbol Connector_Generic:Conn_01x11 -> Connector_Generic_MountingPin:Conn_01x11_MountingPin
- J8: symbol Connector:Conn_01x02_Pin -> Connector_Generic_MountingPin:Conn_01x02_MountingPin
- renumbered C16 to C15, C17 to C16, C18 to C17, C19 to C18, C20 to C19, Q7 to Q4, Q8 to Q5, Q9 to Q6, R31 to R19, R32 to R20, R33 to R21, R34 to R22, R35 to R23, R36 to R24, R37 to R25, R38 to R26, R39 to R27, R40 to R28, R41 to R29, R42 to R30, R43 to R31
Connections:
- net CEL_0: now also J11.1 (Pin_1); no longer J11.11 (Pin_11)
- net CEL_1: now also J11.2 (Pin_2); no longer J11.10 (Pin_10)
- net CEL_10: now also J11.11 (Pin_11); no longer J11.1 (Pin_1)
- net CEL_11: now also J10.1 (Pin_1); no longer J10.3 (Pin_3)
- net CEL_14: now also J9.1 (Pin_1); no longer J9.3 (Pin_3)
- net CEL_16: now also J9.3 (Pin_3); no longer J9.1 (Pin_1)
- net CEL_2: now also J11.3 (Pin_3); no longer J11.9 (Pin_9)
- net CEL_3: now also J11.4 (Pin_4); no longer J11.8 (Pin_8)
- net CEL_4: now also J11.5 (Pin_5); no longer J11.7 (Pin_7)
- net CEL_6: now also J11.7 (Pin_7); no longer J11.5 (Pin_5)
- net CEL_8: now also J11.9 (Pin_9); no longer J11.3 (Pin_3)
- net CEL_9: now also J11.10 (Pin_10); no longer J11.2 (Pin_2)
- net GND: now also J10.MP (MountPin), J11.MP (MountPin), J8.MP (MountPin), J9.MP (MountPin), J12.2 (Pin_2), J12.MP (MountPin)
- net TS2: now also J12.1 (Pin_1)

Commit message: Crystal Layout
Parts:
- renumbered J12 to J7
Changed lines of the file:
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@@
 		(dnp no)
 		(fields_autoplaced yes)
-		(property "Reference" "#PWR040"
+		(property "Reference" "#PWR042"
 			(at 364.49 204.47 0)
 			(effects
@@
 			(project "greenmobi-bms"
 				(path "/3e668e3e-3e16-4665-a807-4735962c41d3/10854291-e499-47cf-bc6f-4ce26b968542"
-					(reference "#PWR040")
+					(reference "#PWR042")
 					(unit 1)
 				)
@@
 		(dnp no)
 		(fields_autoplaced yes)
-		(property "Reference" "#PWR044"
+		(property "Reference" "#PWR043"
 			(at 369.57 209.55 0)
 			(effects
@@
 			(project "greenmobi-bms"
 				(path "/3e668e3e-3e16-4665-a807-4735962c41d3/10854291-e499-47cf-bc6f-4ce26b968542"
-					(reference "#PWR044")
+					(reference "#PWR043")
 					(unit 1)
 				)
@@
 		(dnp no)
 		(fields_autoplaced yes)
-		(property "Reference" "#PWR045"
+		(property "Reference" "#PWR041"
 			(at 347.98 209.55 0)
 			(effects
@@
 			(project "greenmobi-bms"
 				(path "/3e668e3e-3e16-4665-a807-4735962c41d3/10854291-e499-47cf-bc6f-4ce26b968542"
-					(reference "#PWR045")
+					(reference "#PWR041")
 					(unit 1)
 				)
@@
 		(dnp no)
 		(fields_autoplaced yes)
-		(property "Reference" "#PWR042"
+		(property "Reference" "#PWR046"
 			(at 387.35 102.87 0)
 			(effects
@@
 			(project "greenmobi-bms"
 				(path "/3e668e3e-3e16-4665-a807-4735962c41d3/10854291-e499-47cf-bc6f-4ce26b968542"
-					(reference "#PWR042")
+					(reference "#PWR046")
 					(unit 1)
 				)
@@
 		(dnp no)
 		(fields_autoplaced yes)
-		(property "Reference" "#PWR038"
+		(property "Reference" "#PWR039"
 			(at 334.01 172.72 0)
 			(effects
@@
 			(project ""
 				(path "/3e668e3e-3e16-4665-a807-4735962c41d3/10854291-e499-47cf-bc6f-4ce26b968542"
-					(reference "#PWR038")
+					(reference "#PWR039")
 					(unit 1)
 				)
@@
 		(dnp no)
 		(fields_autoplaced yes)
-		(property "Reference" "#PWR037"
+		(property "Reference" "#PWR038"
 			(at 322.58 208.28 0)
 			(effects
@@
 			(project "greenmobi-bms"
 				(path "/3e668e3e-3e16-4665-a807-4735962c41d3/10854291-e499-47cf-bc6f-4ce26b968542"
-					(reference "#PWR037")
+					(reference "#PWR038")
 					(unit 1)
 				)
@@
 		(dnp no)
 		(fields_autoplaced yes)
-		(property "Reference" "#PWR043"
+		(property "Reference" "#PWR044"
 			(at 387.35 72.39 0)
 			(effects
@@
 			(project "greenmobi-bms"
 				(path "/3e668e3e-3e16-4665-a807-4735962c41d3/10854291-e499-47cf-bc6f-4ce26b968542"
-					(reference "#PWR043")
+					(reference "#PWR044")
 					(unit 1)
 				)
@@
 		(dnp no)
 		(fields_autoplaced yes)
-		(property "Reference" "#PWR036"
+		(property "Reference" "#PWR037"
 			(at 185.42 143.51 0)
 			(effects
@@
 			(project "greenmobi-bms"
 				(path "/3e668e3e-3e16-4665-a807-4735962c41d3/10854291-e499-47cf-bc6f-4ce26b968542"
-					(reference "#PWR036")
+					(reference "#PWR037")
 					(unit 1)
 				)
@@
 		(on_board yes)
 		(dnp no)
-		(property "Reference" "J12"
+		(property "Reference" "J7"
 			(at 351.536 194.564 0)
 			(effects
@@
 			(project "greenmobi-bms"
 				(path "/3e668e3e-3e16-4665-a807-4735962c41d3/10854291-e499-47cf-bc6f-4ce26b968542"
-					(reference "J12")
+					(reference "J7")
 					(unit 1)
 				)
@@
 		(dnp no)
 		(fields_autoplaced yes)
-		(property "Reference" "#PWR041"
+		(property "Reference" "#PWR045"
 			(at 387.35 87.63 0)
 			(effects
@@
 			(project ""
 				(path "/3e668e3e-3e16-4665-a807-4735962c41d3/10854291-e499-47cf-bc6f-4ce26b968542"
-					(reference "#PWR041")
+					(reference "#PWR045")
 					(unit 1)
 				)
@@
 		(dnp no)
 		(fields_autoplaced yes)
-		(property "Reference" "#PWR034"
+		(property "Reference" "#PWR035"
 			(at 153.67 196.85 0)
 			(effects
@@
 			(project ""
 				(path "/3e668e3e-3e16-4665-a807-4735962c41d3/10854291-e499-47cf-bc6f-4ce26b968542"
-					(reference "#PWR034")
+					(reference "#PWR035")
 					(unit 1)
 				)
@@
 		(dnp no)
 		(fields_autoplaced yes)
-		(property "Reference" "#PWR039"
+		(property "Reference" "#PWR040"
 			(at 342.9 204.47 0)
 			(effects
@@
 			(project "greenmobi-bms"
 				(path "/3e668e3e-3e16-4665-a807-4735962c41d3/10854291-e499-47cf-bc6f-4ce26b968542"
-					(reference "#PWR039")
+					(reference "#PWR040")
 					(unit 1)
 				)
@@
 		(dnp no)
 		(fields_autoplaced yes)
-		(property "Reference" "#PWR035"
+		(property "Reference" "#PWR036"
 			(at 175.26 143.51 0)
 			(effects
@@
 			(project ""
 				(path "/3e668e3e-3e16-4665-a807-4735962c41d3/10854291-e499-47cf-bc6f-4ce26b968542"
-					(reference "#PWR035")
-					(unit 1)
-				)
+					(reference "#PWR036")
+					(unit 1)
+				)

Commit message: Cell balancing sourcing and repositioning
Connections:
- net CEL_12: now also J10.2 (Pin_2)
- net CEL_13: now also J10.3 (Pin_3)
Changed lines of the file:
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@@
+	)
+	(junction
+		(at 350.52 87.63)
+		(diameter 0)
+		(color 0 0 0 0)
 	)
 	(junction
@@
 	)
 	(junction
-		(at 350.52 87.6153)
-		(diameter 0)
-		(color 0 0 0 0)
-	)
-	(junction
 		(at 350.52 97.79)
 		(diameter 0)
@@
 	)
 	(junction
+		(at 350.52 92.71)
+		(diameter 0)
+		(color 0 0 0 0)
+	)
+	(junction
 		(at 334.01 107.95)
 		(diameter 0)
@@
 	)
 	(junction
-		(at 350.52 92.48)
-		(diameter 0)
-		(color 0 0 0 0)
-	)
-	(junction
 		(at 334.01 123.19)
 		(diameter 0)
@@
 	(wire
 		(pts
-			(xy 350.52 92.48) (xy 350.52 90.17)
-		)
-		(stroke
-			(width 0)
-			(type default)
-		)
-	)
-	(wire
-		(pts
 			(xy 349.25 72.39) (xy 374.65 72.39)
 		)
@@
 	(wire
 		(pts
-			(xy 355.6 92.71) (xy 369.57 92.71)
-		)
-		(stroke
-			(width 0)
-			(type default)
-		)
-	)
-	(wire
-		(pts
-			(xy 350.52 87.63) (xy 350.52 87.6153)
+			(xy 350.52 85.09) (xy 350.52 87.63)
 		)
 		(stroke
@@
 	(wire
 		(pts
-			(xy 350.52 87.6153) (xy 355.6 87.6153)
-		)
-		(stroke
-			(width 0)
-			(type default)
-		)
-	)
-	(wire
-		(pts
 			(xy 180.34 193.04) (xy 180.34 203.2)
 		)
@@
 	(wire
 		(pts
-			(xy 370.84 87.63) (xy 355.6 87.63)
-		)
-		(stroke
-			(width 0)
-			(type default)
-		)
-	)
-	(wire
-		(pts
 			(xy 334.01 157.48) (xy 334.01 160.02)
 		)
@@
 	(wire
 		(pts
+			(xy 350.52 87.63) (xy 370.84 87.63)
+		)
+		(stroke
+			(width 0)
+			(type default)
+		)
+	)
+	(wire
+		(pts
 			(xy 364.49 118.11) (xy 364.49 115.57)
 		)
@@
 	(wire
 		(pts
-			(xy 350.52 87.6153) (xy 350.52 85.09)
-		)
-		(stroke
-			(width 0)
-			(type default)
-		)
-	)
-	(wire
-		(pts
 			(xy 349.25 138.43) (xy 350.52 138.43)
 		)
@@
 	(wire
 		(pts
-			(xy 350.52 92.48) (xy 355.6 92.48)
+			(xy 350.52 92.71) (xy 369.57 92.71)
 		)
 		(stroke
@@
 	(wire
 		(pts
-			(xy 350.52 92.71) (xy 350.52 92.48)
+			(xy 350.52 90.17) (xy 350.52 92.71)
 		)
 		(stroke
@@
 	)
 	(label "CEL_13"
-		(at 355.6 87.6153 0)
+		(at 355.6 87.63 0)
 		(effects
 			(font
@@
 	)
 	(label "CEL_12"
-		(at 355.6 92.48 0)
-		(effects
-			(font
+		(at 355.6 92.71 0)
+		(effects
+			(font

Commit message: Various changes (can't remember)
Parts:
- added TP1, TP2, TP3: TestPoint, symbol Connector:TestPoint
- Q4, Q5: value IPTC025N15NM6 -> AGM015N10LL
Connections:
- net at U5.31 (DCHG): now also TP2.1
- net at U5.32 (DDSG): now also TP1.1
- net EN: now reaches U5.33 (RST_SHUT)
- net ALERT: no longer names the net of U5.25 (ALERT)
- net ALERT: now also TP3.1
- net CFETOFF: no longer names the net of U5.29 (CFETOFF)
- net CHG: no longer names the net of U5.45 (CHG)
- net DFETOFF: no longer names the net of U5.30 (DFETOFF)
- net DSG: no longer names the net of U5.43 (DSG)
- net PCHG: no longer names the net of U5.40 (PCHG)
- net PDSG: no longer names the net of U5.39 (PDSG)
- no-connect marks 0 -> 7

Commit message: Choose MOSFET
Parts:
- Q4, Q5: value AGM015N10LL -> IPT015N10N5
Changed lines of the file:
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@@
 			)
 		)
-		(property "Value" "AGM015N10LL"
+		(property "Value" "IPT015N10N5"
 			(at 129.54 46.99 90)
 			(effects
@@
 			)
 		)
-		(property "Value" "AGM015N10LL"
+		(property "Value" "IPT015N10N5"
 			(at 149.86 46.99 90)
 			(effects
