File: hardware/frontend.kicad_sch (KiCad schematic)
At the start: 66 parts, among them J11 EXT_NTC, J12 EXT_NTC, J7 Conn_01x08_MountingPin, J8 Conn_01x08_MountingPin, Q2 IPT015N10N5, Q3 IPT015N10N5, Q4 IPT015N10N5, Q5 IPT015N10N5, Q6 IPT015N10N5, Q7 IPT015N10N5, Q8 IPT015N10N5, Q9 IPT015N10N5, U5 BQ769x2

Commit message: Add missing cell conection
Parts:
- removed J7, J8: Conn_01x08_MountingPin, Connector_JST:JST_PH_S8B-PH-SM4-TB_1x08-1MP_P2.00mm_Horizontal, symbol Connector_Generic_MountingPin:Conn_01x08_MountingPin
- added C47: 100n, Capacitor_SMD:C_0402_1005Metric, symbol Device:C_Small
- added J8: Conn_01x17_MountingPin, symbol Connector_Generic_MountingPin:Conn_01x17_MountingPin
- added R48: 120, Resistor_SMD:R_0402_1005Metric, symbol Device:R_Small
Connections:
- net CEL_0: now also J8.17 (Pin_17)
- net CEL_1: now also J8.16 (Pin_16)
- net CEL_10: now also J8.7 (Pin_7)
- net CEL_11: now also J8.6 (Pin_6)
- net CEL_12: now also J8.5 (Pin_5)
- net CEL_13: now also J8.4 (Pin_4)
- net CEL_14: now also J8.3 (Pin_3)
- net CEL_15: now also J8.2 (Pin_2)
- net CEL_2: now also J8.15 (Pin_15)
- net CEL_3: now also J8.14 (Pin_14)
- net CEL_4: now also J8.13 (Pin_13)
- net CEL_5: now also J8.12 (Pin_12)
- net CEL_6: now also J8.11 (Pin_11)
- net CEL_7: now also J8.10 (Pin_10)
- net CEL_8: now also J8.9 (Pin_9)
- net CEL_9: now also J8.8 (Pin_8)
- net GND: now also J8.MP (MountPin)
- net VC15: now also C47.2
- net VC16: now also C47.1, R48.1
- new net CEL_16: J8.1 (Pin_1), R48.2

Commit message: Change balancing to a unified connector
Parts:
- J8: footprint (none) -> Connector_JST:JST_PHD_S34B-PHDSS_2x17_P2.00mm_Horizontal
Changed lines of the file:
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@@
 			)
 		)
-		(property "Footprint" ""
+		(property "Footprint" "Connector_JST:JST_PHD_S34B-PHDSS_2x17_P2.00mm_Horizontal"
 			(at 91.44 137.16 0)
 			(effects

Commit message: Change balance current and set most of the footprints
Parts:
- removed R34, R35, R38, R48: 120, Resistor_SMD:R_0402_1005Metric, symbol Device:R_Small
- added R20, R21, R22, R36: 56, Resistor_SMD:R_1206_3216Metric, symbol Device:R_Small
- C44: footprint (none) -> Capacitor_SMD:C_0603_1608Metric
- C45: renamed from C42; footprint (none) -> Capacitor_SMD:C_0402_1005Metric
- C46: renamed from C43; footprint (none) -> Capacitor_SMD:C_0402_1005Metric
- C47: renamed from C45; footprint (none) -> Capacitor_SMD:C_0603_1608Metric
- J7: renamed from J8; footprint Connector_JST:JST_PHD_S34B-PHDSS_2x17_P2.00mm_Horizontal -> greenmobi-bms:JST_GH_SM17B-GHS-TB_1x17-1MP_P1.25mm_Horizontal; LCSC (none) -> C20617492
- R16: renamed from R19; footprint (none) -> Capacitor_SMD:C_0603_1608Metric
- R17: renamed from R20; footprint (none) -> Capacitor_SMD:C_0603_1608Metric
- R18: renamed from R21; footprint (none) -> Capacitor_SMD:C_0603_1608Metric
- R19: renamed from R22; footprint (none) -> Capacitor_SMD:C_0603_1608Metric
- R23, R24, R25, R26, R27, R28, R29, R30, R31, R32, R33: value 120 -> 56; footprint Resistor_SMD:R_0402_1005Metric -> Resistor_SMD:R_1206_3216Metric; LCSC (none) -> C2933788
- R34: renamed from R36; value 120 -> 56; footprint Resistor_SMD:R_0402_1005Metric -> Resistor_SMD:R_1206_3216Metric; LCSC (none) -> C2933788
- R35: renamed from R37; value 120 -> 56; footprint Resistor_SMD:R_0402_1005Metric -> Resistor_SMD:R_1206_3216Metric; LCSC (none) -> C2933788
- R37: renamed from R39; footprint (none) -> Capacitor_SMD:C_0603_1608Metric
- R38: renamed from R40; footprint (none) -> Capacitor_SMD:C_0603_1608Metric
- R39: renamed from R41; footprint (none) -> Capacitor_SMD:C_0603_1608Metric
- R40: renamed from R42; footprint (none) -> Capacitor_SMD:C_0603_1608Metric
- R41: renamed from R10; footprint (none) -> Resistor_SMD:R_0402_1005Metric
- R42: renamed from R17; footprint (none) -> Resistor_SMD:R_0402_1005Metric
- R43: footprint (none) -> Resistor_SMD:R_0402_1005Metric
- R44: renamed from R16; footprint (none) -> Resistor_SMD:R_0402_1005Metric
- R45: renamed from R47; footprint (none) -> Resistor_SMD:R_0402_1005Metric
- R46: renamed from R44; footprint Capacitor_SMD:C_0402_1005Metric -> Resistor_SMD:R_0402_1005Metric
- R47: renamed from R45; footprint (none) -> Resistor_SMD:R_Shunt_Vishay_WSR2_WSR3; LCSC (none) -> C4126121
- R48: renamed from R46; footprint Capacitor_SMD:C_0402_1005Metric -> Resistor_SMD:R_0402_1005Metric
- renumbered C47 to C27, C26 to C28, C27 to C29, C28 to C30, C29 to C31, C30 to C32, C31 to C33, C32 to C34, C33 to C35, C34 to C36, C35 to C37, C36 to C38, C37 to C39, C38 to C40, C39 to C41, C40 to C42, C41 to C43, J11 to J8, J12 to J9, Q2 to Q1, Q3 to Q2, Q4 to Q3, Q5 to Q4, Q6 to Q5, Q7 to Q6, Q8 to Q7, Q9 to Q8
Connections:
- net CEL_0: now also R36.2
- net CEL_10: now also R26.2; no longer R28.2
- net CEL_11: now also R25.2; no longer R27.2
- net CEL_12: now also R24.2; no longer R26.2
- net CEL_13: now also R23.2; no longer R25.2
- net CEL_14: now also R22.2; no longer R24.2
- net CEL_15: now also R21.2; no longer R23.2
- net CEL_16: now also R20.2
- net CEL_3: now also R33.2
- net CEL_4: now also R32.2
- net CEL_5: now also R31.2; no longer R33.2
- net CEL_6: now also R30.2; no longer R32.2
- net CEL_7: now also R29.2; no longer R31.2
- net CEL_8: now also R28.2; no longer R30.2
- net CEL_9: now also R27.2; no longer R29.2
- net VC0: now also R36.1
- net VC10: now also R26.1; no longer R28.1
- net VC11: now also R25.1; no longer R27.1
- net VC12: now also R24.1; no longer R26.1
- net VC13: now also R23.1; no longer R25.1
- net VC14: now also R22.1; no longer R24.1
- net VC15: now also R21.1; no longer R23.1
- net VC16: now also R20.1
- net VC3: now also R33.1
- net VC4: now also R32.1
- net VC5: now also R31.1; no longer R33.1
- net VC6: now also R30.1; no longer R32.1
- net VC7: now also R29.1; no longer R31.1
- net VC8: now also R28.1; no longer R30.1
- net VC9: now also R27.1; no longer R29.1

Commit message: Cleanup ERC errors
Parts:
- added TP12: TestPoint, TestPoint:TestPoint_Pad_D1.0mm, symbol Connector:TestPoint
- renumbered J9 to J10, J7 to J8, J8 to J9
Connections:
- net EN: no longer names the net of R43.2, U5.33 (RST_SHUT)
- net EN: now also TP12.1

Commit message: Connectors changed to JST GH
Parts:
- J10, J9: footprint Connector_JST:JST_PH_S2B-PH-SM4-TB_1x02-1MP_P2.00mm_Horizontal -> Connector_JST:JST_GH_SM02B-GHS-TB_1x02-1MP_P1.25mm_Horizontal
Changed lines of the file:
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@@
 			)
 		)
-		(property "Footprint" "Connector_JST:JST_PH_S2B-PH-SM4-TB_1x02-1MP_P2.00mm_Horizontal"
+		(property "Footprint" "Connector_JST:JST_GH_SM02B-GHS-TB_1x02-1MP_P1.25mm_Horizontal"
 			(at 152.4 114.3 0)
 			(effects
@@
 					(size 1.27 1.27)
 				)
+				(hide yes)
 			)
 		)
@@
 					(size 1.27 1.27)
 				)
+				(hide yes)
 			)
 		)
@@
 					(size 1.27 1.27)
 				)
+				(hide yes)
 			)
 		)
@@
 			)
 		)
-		(property "Footprint" "Connector_JST:JST_PH_S2B-PH-SM4-TB_1x02-1MP_P2.00mm_Horizontal"
+		(property "Footprint" "Connector_JST:JST_GH_SM02B-GHS-TB_1x02-1MP_P1.25mm_Horizontal"
 			(at 152.4 93.98 0)
 			(effects

Commit message: Prettyfy Schematic
Other:
- note added: "Cell voltages"
- note added: "Cells"
- note removed: "Balancing FETs"
- note removed: "Bus Switches"
- moved on the sheet: Q1, Q2, Q3, Q4, Q5, Q6, Q7, Q8, R16, R17, R18, R19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

Commit message: Add resistor to discharge load switches gates
Parts:
- added R10, R49: 10M, Resistor_SMD:R_0402_1005Metric, symbol Device:R_Small
- Q1, Q2, Q3, Q4, Q5, Q6, Q7, Q8: footprint Package_TO_SOT_SMD:Infineon_PG-HSOF-8-1_ThermalVias -> Package_TO_SOT_SMD:Infineon_PG-HSOF-8-1
Connections:
- net BAT+: now also R49.1
- net CHG: now also R49.2
- net DSG: now also R10.2
- net PACK+: now also R10.1
Other:
- note added: "AFE"
- note added: "Analog Frontend"
- note added: "High side switch"
- note added: "Load Switch"
- moved on the sheet: Q1, Q2, Q3, Q4, Q5, Q6, Q7, Q8, R16, R17, R18, R19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

Commit message: Reanotate schematic
Parts:
- renumbered R49 to R15, R10 to R41, R41 to R42, R42 to R43, R43 to R44, R44 to R45, R45 to R46, R46 to R47, R47 to R48, R48 to R49
Changed lines of the file:
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@@
 		(dnp no)
 		(fields_autoplaced yes)
-		(property "Reference" "R10"
+		(property "Reference" "R41"
 			(at 105.41 53.3399 0)
 			(effects
@@
 			(project ""
 				(path "/3e668e3e-3e16-4665-a807-4735962c41d3/10854291-e499-47cf-bc6f-4ce26b968542"
-					(reference "R10")
+					(reference "R41")
 					(unit 1)
 				)
@@
 		(dnp no)
 		(fields_autoplaced yes)
-		(property "Reference" "#PWR054"
+		(property "Reference" "#PWR051"
 			(at 184.15 96.52 0)
 			(effects
@@
 			(project ""
 				(path "/3e668e3e-3e16-4665-a807-4735962c41d3/10854291-e499-47cf-bc6f-4ce26b968542"
-					(reference "#PWR054")
+					(reference "#PWR051")
 					(unit 1)
 				)
@@
 		(on_board yes)
 		(dnp no)
-		(property "Reference" "R49"
+		(property "Reference" "R15"
 			(at 33.782 53.34 0)
 			(effects
@@
 			(project "greenmobi-bms"
 				(path "/3e668e3e-3e16-4665-a807-4735962c41d3/10854291-e499-47cf-bc6f-4ce26b968542"
-					(reference "R49")
+					(reference "R15")
 					(unit 1)
 				)
@@
 		(dnp no)
 		(fields_autoplaced yes)
-		(property "Reference" "R47"
+		(property "Reference" "R48"
 			(at 240.03 137.16 90)
 			(effects
@@
 			(project ""
 				(path "/3e668e3e-3e16-4665-a807-4735962c41d3/10854291-e499-47cf-bc6f-4ce26b968542"
-					(reference "R47")
+					(reference "R48")
 					(unit 1)
 				)
@@
 		(dnp no)
 		(fields_autoplaced yes)
-		(property "Reference" "#PWR053"
+		(property "Reference" "#PWR050"
 			(at 157.48 123.19 0)
 			(effects
@@
 			(project "greenmobi-bms"
 				(path "/3e668e3e-3e16-4665-a807-4735962c41d3/10854291-e499-47cf-bc6f-4ce26b968542"
-					(reference "#PWR053")
+					(reference "#PWR050")
 					(unit 1)
 				)
@@
 		(dnp no)
 		(fields_autoplaced yes)
-		(property "Reference" "#PWR047"
+		(property "Reference" "#PWR044"
 			(at 52.07 193.04 0)
 			(effects
@@
 			(project ""
 				(path "/3e668e3e-3e16-4665-a807-4735962c41d3/10854291-e499-47cf-bc6f-4ce26b968542"
-					(reference "#PWR047")
+					(reference "#PWR044")
 					(unit 1)
 				)
@@
 		(dnp no)
 		(fields_autoplaced yes)
-		(property "Reference" "#PWR055"
+		(property "Reference" "#PWR052"
 			(at 195.58 41.91 0)
 			(effects
@@
 			(project ""
 				(path "/3e668e3e-3e16-4665-a807-4735962c41d3/10854291-e499-47cf-bc6f-4ce26b968542"
-					(reference "#PWR055")
+					(reference "#PWR052")
 					(unit 1)
 				)
@@
 		(dnp no)
 		(fields_autoplaced yes)
-		(property "Reference" "R48"
+		(property "Reference" "R49"
 			(at 247.65 129.5399 0)
 			(effects
@@
 			(project "greenmobi-bms"
 				(path "/3e668e3e-3e16-4665-a807-4735962c41d3/10854291-e499-47cf-bc6f-4ce26b968542"
-					(reference "R48")
+					(reference "R49")
 					(unit 1)
 				)
@@
 		(dnp no)
 		(fields_autoplaced yes)
-		(property "Reference" "R41"
+		(property "Reference" "R42"
 			(at 185.42 54.61 90)
 			(effects
@@
 			(project ""
 				(path "/3e668e3e-3e16-4665-a807-4735962c41d3/10854291-e499-47cf-bc6f-4ce26b968542"
-					(reference "R41")
+					(reference "R42")
 					(unit 1)
 				)
@@
 		(dnp no)
 		(fields_autoplaced yes)
-		(property "Reference" "#PWR056"
+		(property "Reference" "#PWR053"
 			(at 198.12 95.25 0)
 			(effects
@@
 			(project ""
 				(path "/3e668e3e-3e16-4665-a807-4735962c41d3/10854291-e499-47cf-bc6f-4ce26b968542"
-					(reference "#PWR056")
+					(reference "#PWR053")
 					(unit 1)
 				)
@@
 		(dnp no)
 		(fields_autoplaced yes)
-		(property "Reference" "#PWR048"
+		(property "Reference" "#PWR045"
 			(at 91.44 168.91 0)
 			(effects
@@
 			(project ""
 				(path "/3e668e3e-3e16-4665-a807-4735962c41d3/10854291-e499-47cf-bc6f-4ce26b968542"
-					(reference "#PWR048")
+					(reference "#PWR045")
 					(unit 1)
 				)
@@
 		(dnp no)
 		(fields_autoplaced yes)
-		(property "Reference" "#PWR058"
+		(property "Reference" "#PWR055"
 			(at 218.44 119.38 0)
 			(effects
@@
 			(project ""
 				(path "/3e668e3e-3e16-4665-a807-4735962c41d3/10854291-e499-47cf-bc6f-4ce26b968542"
-					(reference "#PWR058")
+					(reference "#PWR055")
 					(unit 1)
 				)
@@
 		(on_board yes)
 		(dnp no)
-		(property "Reference" "R45"
+		(property "Reference" "R46"
 			(at 191.77 64.262 90)
 			(effects
@@
 			(project "greenmobi-bms"
 				(path "/3e668e3e-3e16-4665-a807-4735962c41d3/10854291-e499-47cf-bc6f-4ce26b968542"
-					(reference "R45")
+					(reference "R46")
 					(unit 1)
 				)
@@
 		(dnp no)
 		(fields_autoplaced yes)
-		(property "Reference" "#PWR059"
+		(property "Reference" "#PWR056"
 			(at 240.03 44.45 0)
 			(effects
@@
 			(project "greenmobi-bms"
 				(path "/3e668e3e-3e16-4665-a807-4735962c41d3/10854291-e499-47cf-bc6f-4ce26b968542"
-					(reference "#PWR059")
+					(reference "#PWR056")
 					(unit 1)
 				)
@@
 		(dnp no)
 		(fields_autoplaced yes)
-		(property "Reference" "#PWR060"
+		(property "Reference" "#PWR057"
 			(at 250.19 60.96 0)
 			(effects
@@
 			(project ""
 				(path "/3e668e3e-3e16-4665-a807-4735962c41d3/10854291-e499-47cf-bc6f-4ce26b968542"
-					(reference "#PWR060")
+					(reference "#PWR057")
 					(unit 1)
 				)
@@
 		(dnp no)
 		(fields_autoplaced yes)
-		(property "Reference" "#PWR050"
+		(property "Reference" "#PWR047"
 			(at 152.4 107.95 0)
 			(effects
@@
 			(project "greenmobi-bms"
 				(path "/3e668e3e-3e16-4665-a807-4735962c41d3/10854291-e499-47cf-bc6f-4ce26b968542"
-					(reference "#PWR050")
+					(reference "#PWR047")
 					(unit 1)
 				)
@@
 		(on_board yes)
 		(dnp no)
-		(property "Reference" "R43"
+		(property "Reference" "R44"
 			(at 189.23 90.17 90)
 			(effects
@@
 			(project ""
 				(path "/3e668e3e-3e16-4665-a807-4735962c41d3/10854291-e499-47cf-bc6f-4ce26b968542"
-					(reference "R43")
+					(reference "R44")
 					(unit 1)
 				)
@@
 		(dnp no)
 		(fields_autoplaced yes)
-		(property "Reference" "#PWR057"
+		(property "Reference" "#PWR054"
 			(at 218.44 30.48 0)
 			(effects
@@
 			(project "greenmobi-bms"
 				(path "/3e668e3e-3e16-4665-a807-4735962c41d3/10854291-e499-47cf-bc6f-4ce26b968542"
-					(reference "#PWR057")
+					(reference "#PWR054")
 					(unit 1)
 				)
@@
 		(dnp no)
 		(fields_autoplaced yes)
-		(property "Reference" "#PWR052"
+		(property "Reference" "#PWR049"
 			(at 157.48 102.87 0)
 			(effects
@@
 			(project "greenmobi-bms"
 				(path "/3e668e3e-3e16-4665-a807-4735962c41d3/10854291-e499-47cf-bc6f-4ce26b968542"
-					(reference "#PWR052")
+					(reference "#PWR049")
 					(unit 1)
 				)
@@
 		(dnp no)
 		(fields_autoplaced yes)
-		(property "Reference" "R46"
+		(property "Reference" "R47"
 			(at 237.49 129.5399 0)
 			(effects
@@
 			(project ""
 				(path "/3e668e3e-3e16-4665-a807-4735962c41d3/10854291-e499-47cf-bc6f-4ce26b968542"
-					(reference "R46")
+					(reference "R47")
 					(unit 1)
 				)
@@
 		(on_board yes)
 		(dnp no)
-		(property "Reference" "R42"
+		(property "Reference" "R43"
 			(at 185.42 64.262 90)
 			(effects
@@
 			(project "greenmobi-bms"
 				(path "/3e668e3e-3e16-4665-a807-4735962c41d3/10854291-e499-47cf-bc6f-4ce26b968542"
-					(reference "R42")
+					(reference "R43")
 					(unit 1)
 				)
@@
 		(dnp no)
 		(fields_autoplaced yes)
-		(property "Reference" "#PWR049"
+		(property "Reference" "#PWR046"
 			(at 148.59 90.17 0)
 			(effects
@@
 			(project "greenmobi-bms"
 				(path "/3e668e3e-3e16-4665-a807-4735962c41d3/10854291-e499-47cf-bc6f-4ce26b968542"
-					(reference "#PWR049")
+					(reference "#PWR046")
 					(unit 1)
 				)
@@
 		(dnp no)
 		(fields_autoplaced yes)
-		(property "Reference" "R44"
+		(property "Reference" "R45"
 			(at 191.77 54.61 90)
 			(effects
@@
 			(project "greenmobi-bms"
 				(path "/3e668e3e-3e16-4665-a807-4735962c41d3/10854291-e499-47cf-bc6f-4ce26b968542"
-					(reference "R44")
+					(reference "R45")
 					(unit 1)
 				)
@@
 		(dnp no)
 		(fields_autoplaced yes)
-		(property "Reference" "#PWR051"
+		(property "Reference" "#PWR048"
 			(at 152.4 128.27 0)
 			(effects
@@
 			(project "greenmobi-bms"
 				(path "/3e668e3e-3e16-4665-a807-4735962c41d3/10854291-e499-47cf-bc6f-4ce26b968542"
-					(reference "#PWR051")
+					(reference "#PWR048")
 					(unit 1)
 				)
