File: hardware/frontend.kicad_sch (KiCad schematic)
At the start: 70 parts, among them J10 EXT_NTC, J8 Conn_01x17_MountingPin, J9 EXT_NTC, Q1 IPT015N10N5, Q2 IPT015N10N5, Q3 IPT015N10N5, Q4 IPT015N10N5, Q5 IPT015N10N5, Q6 IPT015N10N5, Q7 IPT015N10N5, Q8 IPT015N10N5, U5 BQ769x2

Commit message: Improvements to main buck and load switch
Parts:
- removed Q1, Q2, Q3, Q4, Q5, Q6, Q7, Q8: IPT015N10N5, Package_TO_SOT_SMD:Infineon_PG-HSOF-8-1, symbol Transistor_FET:IPT015N10N5
- removed R15, R41: 10M, Resistor_SMD:R_0402_1005Metric, symbol Device:R_Small
- removed R16, R17, R18, R19, R37, R38, R39, R40: 75, Capacitor_SMD:C_0603_1608Metric, symbol Device:R_Small
Connections:
- net VC0: no longer names the net of C43.1, R36.1, U5.16 (VC0)
- net VC1: no longer names the net of C41.2, C42.1, R35.1, U5.15 (VC1)
- net VC10: no longer names the net of C32.2, C33.1, R26.1, U5.6 (VC10)
- net VC11: no longer names the net of C31.2, C32.1, R25.1, U5.5 (VC11)
- net VC12: no longer names the net of C30.2, C31.1, R24.1, U5.4 (VC12)
- net VC13: no longer names the net of C29.2, C30.1, R23.1, U5.3 (VC13)
- net VC14: no longer names the net of C28.2, C29.1, R22.1
- net VC14: now also U5.2 (VC14)
- net VC15: no longer names the net of C27.2, C28.1, R21.1, U5.1 (VC15)
- net VC15: no longer U5.2 (VC14)
- net VC16: no longer names the net of C27.1, R20.1, U5.48 (VC16)
- net VC2: no longer names the net of C40.2, C41.1, R34.1, U5.14 (VC2)
- net VC3: no longer names the net of C39.2, C40.1, R33.1, U5.13 (VC3)
- net VC4: no longer names the net of C38.2, C39.1, R32.1, U5.12 (VC4)
- net VC5: no longer names the net of C37.2, C38.1, R31.1, U5.11 (VC5)
- net VC6: no longer names the net of C36.2, C37.1, R30.1, U5.10 (VC6)
- net VC7: no longer names the net of C35.2, C36.1, R29.1, U5.9 (VC7)
- net VC8: no longer names the net of C34.2, C35.1, R28.1, U5.8 (VC8)
- net VC9: no longer names the net of C33.2, C34.1, R27.1, U5.7 (VC9)
Other:
- added sheet Load Switch (load_switch.kicad_sch)
- note removed: "Cell voltages"
- note removed: "Cells"
- note removed: "High side switch"
- note removed: "Load Switch"
- moved on the sheet: C27, C28, C29, C30, C31, C32, C33, C34, C35, C36, C37, C38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

Commit message: Reanotate schematic
Parts:
- renumbered C44 to C29, C45 to C30, C46 to C31, C47 to C32, C27 to C33, C28 to C34, C29 to C35, C30 to C36, C31 to C37, C32 to C38, C33 to C39, C34 to C40, C35 to C41, C36 to C42, C37 to C43, C38 to C44, C39 to C45, C40 to C46, C41 to C47, C42 to C48, C43 to C49, J8 to J10, J9 to J8, J10 to J9, R42 to R14, R43 to R15, R44 to R16, R45 to R17, R46 to R18, R47 to R19, R48 to R20, R49 to R21, R20 to R22, R21 to R23, R22 to R24, R23 to R25, R24 to R26, R25 to R27, R26 to R28, R27 to R29, R28 to R30, R29 to R31, R30 to R32, R31 to R33, R32 to R34, R33 to R35, R34 to R36, R35 to R37, R36 to R38

Commit message: Enable logic
Parts:
- added R49, R50, R51: 5.1k, Resistor_SMD:R_0402_1005Metric, symbol Device:R_Small
Connections:
- net BAT+: now also R49.1
- net at C33.1, R22.1, U5.48 (VC16): now also R49.2
- net at U5.22 (TS2): now also R51.2
- new net: R50.2, R51.1
- new net Shutdown: R50.1
- no-connect marks 7 -> 6
Other:
- sheet Load Switch ports: added FET_C; removed none
- moved on the sheet: J8

Commit message: Cell to BAT connection
Parts:
- added C54: 1u, symbol Device:C_Small
- added C55: 100p, symbol Device:C_Small
- added D3: 1N4148W, Diode_SMD:D_SOD-123, symbol Diode:1N4148W
- R49: value 5.1k -> 120; footprint Resistor_SMD:R_0402_1005Metric -> (none)
Connections:
- net BAT+: now also C54.1, C55.1
- net CEL_16: now also D3.2 (A)
- net GND: now also C54.2, C55.2
- net at C33.1, R22.1, U5.48 (VC16): no longer R49.2
- new net: D3.1 (K), R49.2

Commit message: BAT- to GND connection
Parts:
- added C56, C57: 100n, Capacitor_SMD:C_0402_1005Metric, symbol Device:C_Small
Connections:
- net CEL_0 is gone; now on net BAT-: J10.17 (Pin_17), R38.2
- net GND: now also C56.2, C57.1
- net at C30.1, C31.1, R19.1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: now also C57.2
- net at C30.2, C31.2, R21.1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: now also C56.1

Commit message: Replace Front end input diode for a Schotky
Parts:
- removed D3: 1N4148W, Diode_SMD:D_SOD-123, symbol Diode:1N4148W
- added D4: 1N5819WS, Diode_SMD:D_SOD-323, symbol Diode:1N5819WS
Connections:
- net CEL_16: now also D4.2 (A)
- net at R49.2: now also D4.1 (K)
Other:
- sheet Load Switch ports: added BAT_F; removed BAT+
Changed lines of the file:
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@@
 		)
 	)
-	(hierarchical_label "BAT+"
+	(hierarchical_label "BAT_F"
 		(shape input)
 		(at 95.25 166.37 180)
@@
 	)
 	(symbol
+		(lib_id "Diode:1N5819WS")
+		(at 167.64 31.75 0)
+		(unit 1)
+		(exclude_from_sim no)
+		(in_bom yes)
+		(on_board yes)
+		(dnp no)
+		(fields_autoplaced yes)
+		(property "Reference" "D4"
+			(at 167.3225 25.4 0)
+			(effects
+				(font
+					(size 1.27 1.27)
+				)
+			)
+		)
+		(property "Value" "1N5819WS"
+			(at 167.3225 27.94 0)
+			(effects
+				(font
+					(size 1.27 1.27)
+				)
+			)
+		)
+		(property "Footprint" "Diode_SMD:D_SOD-323"
+			(at 167.64 36.195 0)
+			(effects
+				(font
+					(size 1.27 1.27)
+				)
+				(hide yes)
+			)
+		)
+		(property "Datasheet" "https://datasheet.lcsc.com/lcsc/2204281430_Guangdong-Hottech-1N5819WS_C191023.pdf"
+			(at 167.64 31.75 0)
+			(effects
+				(font
+					(size 1.27 1.27)
+				)
+				(hide yes)
+			)
+		)
+		(property "Description" "40V 600mV@1A 1A SOD-323 Schottky Barrier Diodes, SOD-323"
+			(at 167.64 31.75 0)
+			(effects
+				(font
+					(size 1.27 1.27)
+				)
+				(hide yes)
+			)
+		)
+		(property "LCSC" "C191023"
+			(at 167.64 31.75 0)
+			(effects
+				(font
+					(size 1.27 1.27)
+				)
+				(hide yes)
+			)
+		)
+		(pin "1"
+		)
+		(pin "2"
+		)
+		(instances
+			(project ""
+				(path "/3e668e3e-3e16-4665-a807-4735962c41d3/10854291-e499-47cf-bc6f-4ce26b968542"
+					(reference "D4")
+					(unit 1)
+				)
+			)
+		)
+	)
+	(symbol
 		(lib_id "Device:C_Small")
 		(at 127 114.3 90)
@@
 	)
 	(symbol
-		(lib_id "Diode:1N4148W")
-		(at 167.64 31.75 0)
-		(unit 1)
-		(exclude_from_sim no)
-		(in_bom yes)
-		(on_board yes)
-		(dnp no)
-		(fields_autoplaced yes)
-		(property "Reference" "D3"
-			(at 167.64 25.4 0)
-			(effects
-				(font
-					(size 1.27 1.27)
-				)
-			)
-		)
-		(property "Value" "1N4148W"
-			(at 167.64 27.94 0)
-			(effects
-				(font
-					(size 1.27 1.27)
-				)
-			)
-		)
-		(property "Footprint" "Diode_SMD:D_SOD-123"
-			(at 167.64 36.195 0)
-			(effects
-				(font
-					(size 1.27 1.27)
-				)
-				(hide yes)
-			)
-		)
-		(property "Datasheet" "https://www.vishay.com/docs/85748/1n4148w.pdf"
-			(at 167.64 31.75 0)
-			(effects
-				(font
-					(size 1.27 1.27)
-				)
-				(hide yes)
-			)
-		)
-		(property "Description" "75V 0.15A Fast Switching Diode, SOD-123"
-			(at 167.64 31.75 0)
-			(effects
-				(font
-					(size 1.27 1.27)
-				)
-				(hide yes)
-			)
-		)
-		(property "Sim.Device" "D"
-			(at 167.64 31.75 0)
-			(effects
-				(font
-					(size 1.27 1.27)
-				)
-				(hide yes)
-			)
-		)
-		(property "Sim.Pins" "1=K 2=A"
-			(at 167.64 31.75 0)
-			(effects
-				(font
-					(size 1.27 1.27)
-				)
-				(hide yes)
-			)
-		)
-		(property "LCSC" "C81598"
-			(at 167.64 31.75 0)
-			(effects
-				(font
-					(size 1.27 1.27)
-				)
-				(hide yes)
-			)
-		)
-		(pin "2"
-		)
-		(pin "1"
-		)
-		(instances
-			(project ""
-				(path "/3e668e3e-3e16-4665-a807-4735962c41d3/10854291-e499-47cf-bc6f-4ce26b968542"
-					(reference "D3")
-					(unit 1)
-				)
-			)
-		)
-	)
-	(symbol
 		(lib_id "Device:R_Small")
 		(at 199.39 35.56 90)
@@
 			)
 		)
-		(pin "BAT+" input
-			(at 95.25 166.37 180)
-			(effects
-				(font
-					(size 1.27 1.27)
-				)
-				(justify left)
-			)
-		)
 		(pin "CHG" input
 			(at 95.25 173.99 180)
@@
 			(effects
 				(font
+					(size 1.27 1.27)
+				)
+				(justify left)
+			)
+		)
+		(pin "BAT_F" input
+			(at 95.25 166.37 180)
+			(effects
+				(font

Commit message: package sizes set and AFE layout
Parts:
- C54: footprint (none) -> Capacitor_SMD:C_1206_3216Metric
- C55: footprint (none) -> Capacitor_SMD:C_0603_1608Metric
- R49: footprint (none) -> Resistor_SMD:R_0402_1005Metric
Connections:
- net BAT-: no longer J10.17 (Pin_17), R38.2
- new net CEL_0: J10.17 (Pin_17), R38.2
Changed lines of the file:
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@@
 	)
 	(junction
-		(at 229.87 116.84)
-		(diameter 0)
-		(color 0 0 0 0)
-	)
-	(junction
 		(at 189.23 35.56)
 		(diameter 0)
@@
 	(wire
 		(pts
-			(xy 229.87 116.84) (xy 232.41 116.84)
-		)
-		(stroke
-			(width 0)
-			(type default)
-		)
-	)
-	(wire
-		(pts
 			(xy 226.06 71.12) (xy 233.68 71.12)
 		)
@@
 	(hierarchical_label "BAT-"
 		(shape input)
-		(at 232.41 116.84 0)
-		(effects
-			(font
-				(size 1.27 1.27)
-			)
-			(justify left)
-		)
-	)
-	(hierarchical_label "BAT-"
-		(shape input)
 		(at 140.97 142.24 0)
 		(effects
@@
 			)
 		)
-		(property "Footprint" ""
+		(property "Footprint" "Capacitor_SMD:C_1206_3216Metric"
 			(at 149.86 35.56 0)
 			(effects
@@
 			)
 		)
-		(property "Footprint" ""
+		(property "Footprint" "Capacitor_SMD:C_0603_1608Metric"
 			(at 139.7 35.56 0)
 			(effects
@@
 			)
 		)
-		(property "Footprint" ""
+		(property "Footprint" "Resistor_SMD:R_0402_1005Metric"
 			(at 157.48 31.75 0)
 			(effects

Commit message: Majority of layout placement done
Connections:
- net BAT+ is gone; now on net BAT_F: C29.1, C54.1, C55.1, R49.1, U5.47 (BAT)
- net CEL_0 is gone; now on net GND: J10.17 (Pin_17), R38.2
Changed lines of the file:
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@@
 	)
 	(junction
+		(at 229.87 116.84)
+		(diameter 0)
+		(color 0 0 0 0)
+	)
+	(junction
 		(at 132.08 124.46)
 		(diameter 0)
@@
 	(wire
 		(pts
+			(xy 229.87 125.73) (xy 229.87 116.84)
+		)
+		(stroke
+			(width 0)
+			(type default)
+		)
+	)
+	(wire
+		(pts
 			(xy 166.37 86.36) (xy 166.37 91.44)
 		)
@@
 		)
 	)
+	(hierarchical_label "BAT_F"
+		(shape input)
+		(at 149.86 57.15 0)
+		(effects
+			(font
+				(size 1.27 1.27)
+			)
+			(justify left)
+		)
+	)
 	(hierarchical_label "PACK+"
 		(shape output)
@@
 		)
 	)
-	(hierarchical_label "BAT+"
-		(shape input)
-		(at 149.86 57.15 0)
-		(effects
-			(font
-				(size 1.27 1.27)
-			)
-			(justify left)
-		)
-	)
 	(hierarchical_label "Shutdown"
 		(shape input)
@@
 					(unit 1)
 				)
+			)
+		)
+	)
+	(symbol
+		(lib_id "power:GND")
+		(at 229.87 125.73 0)
+		(unit 1)
+		(exclude_from_sim no)
+		(in_bom yes)
+		(on_board yes)
+		(dnp no)
+		(fields_autoplaced yes)
+		(property "Reference" "#PWR027"
+			(at 229.87 132.08 0)
+			(effects
+				(font
+					(size 1.27 1.27)
+				)
+				(hide yes)
+			)
+		)
+		(property "Value" "GND"
+			(at 229.87 130.81 0)
+			(effects
+				(font
+					(size 1.27 1.27)
+				)
+			)
+		)
+		(property "Footprint" ""
+			(at 229.87 125.73 0)
+			(effects
+				(font
+					(size 1.27 1.27)
+				)
+				(hide yes)
+			)
+		)
+		(property "Datasheet" ""
+			(at 229.87 125.73 0)
+			(effects
+				(font
+					(size 1.27 1.27)
+				)
+				(hide yes)
+			)
+		)
+		(property "Description" "Power symbol creates a global label with name \"GND\" , ground"
+			(at 229.87 125.73 0)
+			(effects
+				(font
+					(size 1.27 1.27)
+				)
+				(hide yes)
+			)
+		)
+		(pin "1"
+		)
+		(instances
+			(project "greenmobi-bms"
+				(path "/3e668e3e-3e16-4665-a807-4735962c41d3/10854291-e499-47cf-bc6f-4ce26b968542"
+					(reference "#PWR027")
+					(unit 1)
+				)
