File: hardware/cell.kicad_sch (KiCad schematic)
At the start: 6 parts, among them Q8 MMBT3904

Commit message: Test CI
Parts:
- C10: footprint (none) -> Capacitor_SMD:C_0402_1005Metric
- R27, R28: footprint (none) -> Resistor_SMD:R_0402_1005Metric
- R35, R40: footprint (none) -> Resistor_SMD:R_1206_3216Metric
Changed lines of the file:
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@@
 			)
 		)
-		(property "Footprint" ""
+		(property "Footprint" "Capacitor_SMD:C_0402_1005Metric"
 			(at 130.81 99.06 0)
 			(effects
@@
 			)
 		)
-		(property "Footprint" ""
+		(property "Footprint" "Resistor_SMD:R_1206_3216Metric"
 			(at 147.32 96.52 0)
 			(effects
@@
 			)
 		)
-		(property "Footprint" ""
+		(property "Footprint" "Resistor_SMD:R_0402_1005Metric"
 			(at 140.97 92.71 0)
 			(effects
@@
 			)
 		)
-		(property "Footprint" ""
+		(property "Footprint" "Resistor_SMD:R_1206_3216Metric"
 			(at 154.94 96.52 0)
 			(effects
@@
 			)
 		)
-		(property "Footprint" ""
+		(property "Footprint" "Resistor_SMD:R_0402_1005Metric"
 			(at 140.97 105.41 0)
 			(effects

Commit message: Reanotate
Parts:
- renumbered C10 to C6, Q8 to Q3, R27 to R11, R28 to R12, R35 to R13, R40 to R14

Commit message: Reorder Schematic pages
Parts:
- renumbered C6 to C7, Q3 to Q4, R11 to R15, R12 to R16, R13 to R17, R14 to R18
Changed lines of the file:
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@@
 		(dnp no)
 		(fields_autoplaced yes)
-		(property "Reference" "C6"
+		(property "Reference" "C7"
 			(at 133.35 97.7962 0)
 			(effects
@@
 		(dnp no)
 		(fields_autoplaced yes)
-		(property "Reference" "Q3"
+		(property "Reference" "Q4"
 			(at 153.67 104.1399 0)
 			(effects
@@
 		(dnp no)
 		(fields_autoplaced yes)
-		(property "Reference" "R13"
+		(property "Reference" "R17"
 			(at 149.86 95.2499 0)
 			(effects
@@
 		(on_board yes)
 		(dnp no)
-		(property "Reference" "R11"
+		(property "Reference" "R15"
 			(at 140.97 95.25 90)
 			(effects
@@
 		(dnp no)
 		(fields_autoplaced yes)
-		(property "Reference" "R14"
+		(property "Reference" "R18"
 			(at 157.48 95.2499 0)
 			(effects
@@
 		(dnp no)
 		(fields_autoplaced yes)
-		(property "Reference" "R12"
+		(property "Reference" "R16"
 			(at 140.97 100.33 90)
 			(effects

Commit message: Change discharge current
Parts:
- removed R17: 80, Resistor_SMD:R_1206_3216Metric, symbol Device:R_Small
- R18: value 80 -> 82
Other:
- moved on the sheet: R18
Changed lines of the file:
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@@
 	(paper "A4")
 	(junction
-		(at 147.32 92.71)
-		(diameter 0)
-		(color 0 0 0 0)
-	)
-	(junction
-		(at 151.13 100.33)
-		(diameter 0)
-		(color 0 0 0 0)
-	)
-	(junction
-		(at 154.94 92.71)
+		(at 151.13 92.71)
 		(diameter 0)
 		(color 0 0 0 0)
@@
 	(wire
 		(pts
-			(xy 147.32 92.71) (xy 147.32 93.98)
-		)
-		(stroke
-			(width 0)
-			(type default)
-		)
-	)
-	(wire
-		(pts
 			(xy 130.81 92.71) (xy 138.43 92.71)
 		)
@@
 	(wire
 		(pts
-			(xy 151.13 100.33) (xy 154.94 100.33)
-		)
-		(stroke
-			(width 0)
-			(type default)
-		)
-	)
-	(wire
-		(pts
-			(xy 147.32 99.06) (xy 147.32 100.33)
-		)
-		(stroke
-			(width 0)
-			(type default)
-		)
-	)
-	(wire
-		(pts
 			(xy 127 92.71) (xy 130.81 92.71)
 		)
@@
 	(wire
 		(pts
-			(xy 143.51 92.71) (xy 147.32 92.71)
-		)
-		(stroke
-			(width 0)
-			(type default)
-		)
-	)
-	(wire
-		(pts
-			(xy 147.32 92.71) (xy 154.94 92.71)
-		)
-		(stroke
-			(width 0)
-			(type default)
-		)
-	)
-	(wire
-		(pts
-			(xy 154.94 92.71) (xy 154.94 93.98)
+			(xy 143.51 92.71) (xy 151.13 92.71)
+		)
+		(stroke
+			(width 0)
+			(type default)
+		)
+	)
+	(wire
+		(pts
+			(xy 151.13 92.71) (xy 151.13 93.98)
 		)
 		(stroke
@@
 	(wire
 		(pts
+			(xy 151.13 92.71) (xy 161.29 92.71)
+		)
+		(stroke
+			(width 0)
+			(type default)
+		)
+	)
+	(wire
+		(pts
 			(xy 151.13 111.76) (xy 151.13 110.49)
 		)
@@
 	(wire
 		(pts
-			(xy 147.32 100.33) (xy 151.13 100.33)
-		)
-		(stroke
-			(width 0)
-			(type default)
-		)
-	)
-	(wire
-		(pts
-			(xy 154.94 92.71) (xy 161.29 92.71)
-		)
-		(stroke
-			(width 0)
-			(type default)
-		)
-	)
-	(wire
-		(pts
 			(xy 130.81 105.41) (xy 138.43 105.41)
 		)
@@
 	(wire
 		(pts
-			(xy 154.94 99.06) (xy 154.94 100.33)
+			(xy 151.13 99.06) (xy 151.13 100.33)
 		)
 		(stroke
@@
 	(symbol
 		(lib_id "Device:R_Small")
-		(at 147.32 96.52 0)
-		(unit 1)
-		(exclude_from_sim no)
-		(in_bom yes)
-		(on_board yes)
-		(dnp no)
-		(fields_autoplaced yes)
-		(property "Reference" "R17"
-			(at 149.86 95.2499 0)
-			(effects
-				(font
-					(size 1.27 1.27)
-				)
-				(justify left)
-			)
-		)
-		(property "Value" "80"
-			(at 149.86 97.7899 0)
-			(effects
-				(font
-					(size 1.27 1.27)
-				)
-				(justify left)
-			)
-		)
-		(property "Footprint" "Resistor_SMD:R_1206_3216Metric"
-			(at 147.32 96.52 0)
-			(effects
-				(font
-					(size 1.27 1.27)
-				)
-				(hide yes)
-			)
-		)
-		(property "Datasheet" "~"
-			(at 147.32 96.52 0)
-			(effects
-				(font
-					(size 1.27 1.27)
-				)
-				(hide yes)
-			)
-		)
-		(property "Description" "Resistor, small symbol"
-			(at 147.32 96.52 0)
-			(effects
-				(font
-					(size 1.27 1.27)
-				)
-				(hide yes)
-			)
-		)
-		(pin "2"
-		)
-		(pin "1"
-		)
-		(instances
-			(project "greenmobi-bms"
-				(path "/3e668e3e-3e16-4665-a807-4735962c41d3/10854291-e499-47cf-bc6f-4ce26b968542/5010d67a-4eb9-4f33-9977-d1ee68dbd349"
-					(reference "R13")
-					(unit 1)
-				)
-				(path "/3e668e3e-3e16-4665-a807-4735962c41d3/10854291-e499-47cf-bc6f-4ce26b968542/556c3299-3449-435c-9f39-b3e196eabb16"
-					(reference "R94")
-					(unit 1)
-				)
-				(path "/3e668e3e-3e16-4665-a807-4735962c41d3/10854291-e499-47cf-bc6f-4ce26b968542/7e93ed7a-308c-4a1a-8763-d1420a07707d"
-					(reference "R54")
-					(unit 1)
-				)
-				(path "/3e668e3e-3e16-4665-a807-4735962c41d3/10854291-e499-47cf-bc6f-4ce26b968542/8494e1b0-b853-4a02-b6a5-496b4f49debc"
-					(reference "R86")
-					(unit 1)
-				)
-				(path "/3e668e3e-3e16-4665-a807-4735962c41d3/10854291-e499-47cf-bc6f-4ce26b968542/986fe2c6-cb30-47f1-962f-cc34651f2eb9"
-					(reference "R62")
-					(unit 1)
-				)
-				(path "/3e668e3e-3e16-4665-a807-4735962c41d3/10854291-e499-47cf-bc6f-4ce26b968542/a725e1e0-ea70-434a-b15a-111295be3c88"
-					(reference "R70")
-					(unit 1)
-				)
-				(path "/3e668e3e-3e16-4665-a807-4735962c41d3/10854291-e499-47cf-bc6f-4ce26b968542/b13d811d-80fa-4639-9484-50994b19b392"
-					(reference "R46")
-					(unit 1)
-				)
-				(path "/3e668e3e-3e16-4665-a807-4735962c41d3/10854291-e499-47cf-bc6f-4ce26b968542/bb32a0a3-8e2d-4121-ad08-49e4139482ba"
-					(reference "R17")
-					(unit 1)
-				)
-				(path "/3e668e3e-3e16-4665-a807-4735962c41d3/10854291-e499-47cf-bc6f-4ce26b968542/d3ab348e-3785-4bc4-b32c-2adcbcfaa2d3"
-					(reference "R78")
-					(unit 1)
-				)
-				(path "/3e668e3e-3e16-4665-a807-4735962c41d3/10854291-e499-47cf-bc6f-4ce26b968542/d6d835c6-ad04-4883-a11c-fbbf281adcad"
-					(reference "R82")
-					(unit 1)
-				)
-				(path "/3e668e3e-3e16-4665-a807-4735962c41d3/10854291-e499-47cf-bc6f-4ce26b968542/d8aa5e74-302b-4613-97ad-fecd4e2f7374"
-					(reference "R90")
-					(unit 1)
-				)
-				(path "/3e668e3e-3e16-4665-a807-4735962c41d3/10854291-e499-47cf-bc6f-4ce26b968542/d9674d57-752a-4721-bef5-17721ea30e41"
-					(reference "R58")
-					(unit 1)
-				)
-				(path "/3e668e3e-3e16-4665-a807-4735962c41d3/10854291-e499-47cf-bc6f-4ce26b968542/e7cfac8f-8076-4840-88ff-208b5a92562b"
-					(reference "R21")
-					(unit 1)
-				)
-				(path "/3e668e3e-3e16-4665-a807-4735962c41d3/10854291-e499-47cf-bc6f-4ce26b968542/eb545c5b-f2f4-4863-b0b0-5b025d6f2818"
-					(reference "R50")
-					(unit 1)
-				)
-				(path "/3e668e3e-3e16-4665-a807-4735962c41d3/10854291-e499-47cf-bc6f-4ce26b968542/f412b0a3-3603-46ae-8fce-adda24336678"
-					(reference "R74")
-					(unit 1)
-				)
-				(path "/3e668e3e-3e16-4665-a807-4735962c41d3/10854291-e499-47cf-bc6f-4ce26b968542/ff5958fe-aab0-4b11-92a0-ba1b94420b27"
-					(reference "R66")
-					(unit 1)
-				)
-			)
-		)
-	)
-	(symbol
-		(lib_id "Device:R_Small")
 		(at 140.97 92.71 90)
 		(unit 1)
@@
 	(symbol
 		(lib_id "Device:R_Small")
-		(at 154.94 96.52 0)
+		(at 151.13 96.52 0)
 		(unit 1)
 		(exclude_from_sim no)
@@
 		(fields_autoplaced yes)
 		(property "Reference" "R18"
-			(at 157.48 95.2499 0)
-			(effects
-				(font
-					(size 1.27 1.27)
-				)
-				(justify left)
-			)
-		)
-		(property "Value" "80"
-			(at 157.48 97.7899 0)
+			(at 153.67 95.2499 0)
+			(effects
+				(font
+					(size 1.27 1.27)
+				)
+				(justify left)
+			)
+		)
+		(property "Value" "82"
+			(at 153.67 97.7899 0)
 			(effects
 				(font
@@
 		)
 		(property "Footprint" "Resistor_SMD:R_1206_3216Metric"
-			(at 154.94 96.52 0)
+			(at 151.13 96.52 0)
 			(effects
 				(font
@@
 		)
 		(property "Datasheet" "~"
-			(at 154.94 96.52 0)
+			(at 151.13 96.52 0)
 			(effects
 				(font
@@
 		)
 		(property "Description" "Resistor, small symbol"
-			(at 154.94 96.52 0)
-			(effects
-				(font
+			(at 151.13 96.52 0)
+			(effects
+				(font

Commit message: Remove Thermal reliefs from connectors MP and ESP32 Crystal
Parts:
- renumbered C7 to C20, Q4 to Q7, R15 to R32, R16 to R33, R18 to R34

Commit message: Increased Discharge Resistor size
Parts:
- R34: footprint Resistor_SMD:R_1206_3216Metric -> Resistor_SMD:R_1210_3225Metric
Changed lines of the file:
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@@
 			)
 		)
-		(property "Footprint" "Resistor_SMD:R_1206_3216Metric"
+		(property "Footprint" "Resistor_SMD:R_1210_3225Metric"
 			(at 151.13 96.52 0)
 			(effects

Commit message: Cell balancing sourcing and repositioning
Parts:
- R34: value 82 -> 36; LCSC (none) -> C3000629
Changed lines of the file:
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@@
 			)
 		)
-		(property "Value" "82"
+		(property "Value" "36"
 			(at 153.67 97.7899 0)
 			(effects
@@
 			(at 151.13 96.52 0)
 			(effects
+				(font
+					(size 1.27 1.27)
+				)
+				(hide yes)
+			)
+		)
+		(property "LCSC" "C3000629"
+			(at 151.13 96.52 0)
+			(effects
