File: hardware/greenmobi-bms.kicad_pcb (KiCad board)
At the start: 2 copper layers, 100 x 40 mm, 131 parts, among them J1 BAT+, J10 Conn_01x03, J11 Conn_01x11, J2 BAT-, J3 PACK+, J4 PACK-, J5 CAN, J6 USB_C_Receptacle_USB2.0_14P, J7 EXT_NTC, J8 EXT_NTC, J9 Conn_01x03, Q1 MMBT3904, Q10 MMBT3904, Q11 MMBT3904, Q12 MMBT3904, Q13 MMBT3904, Q14 MMBT3904, Q15 MMBT3904, Q16 MMBT3904, Q17 MMBT3904, Q18 MMBT3904, Q19 MMBT3904, Q2 MMBT3904, Q20 MMBT3904, Q21 MMBT3904, Q22 MMBT3904, Q3 MMBT3904, Q4 MMBT3904, Q5 MMBT3904, Q6 AO3401A, Q7 IPTC025N15NM6, Q8 IPTC025N15NM6, Q9 BSS127S, SW1 SW_Push, U1 ESP32-C3, U2 MCP2562-E-SN, U3 LM5164DDA, U4 TPS7A0533PDBZ, U5 BQ769x2

Commit message: Remove Thermal reliefs from connectors MP and ESP32 Crystal
Parts:
- removed the C6 at (227.5, 124.1)
- removed the C7 at (235.3, 134.1)
- removed the Q3 at (219.2, 114.2)
- removed the Q4 at (237.2, 106.9)
- removed R11, R15, R80, R84, R88, R92: 100, Resistor_SMD:R_0402_1005Metric
- removed R12, R16, R81, R85, R89, R93: 300, Resistor_SMD:R_0402_1005Metric
- removed R14, R18, R83, R87, R91, R95: 82, Resistor_SMD:R_1206_3216Metric
- added C2: xp, Capacitor_SMD:C_0402_1005Metric, F.Cu at (175.3, 104.9)
- added C34: 100n, Capacitor_SMD:C_0402_1005Metric, F.Cu at (127.1, 95.6)
- added C35: 100n, Capacitor_SMD:C_0402_1005Metric, F.Cu at (127.1, 92.2)
- added C4: xp, Capacitor_SMD:C_0402_1005Metric, F.Cu at (169.9, 104.9)
- added L1: 24n, Inductor_SMD:L_0402_1005Metric, F.Cu at (171.6, 107.6)
- added Q6: BSS127S, Package_TO_SOT_SMD:SOT-23, F.Cu at (90.5, 128.3)
- added Q8: MMBT3904, Package_TO_SOT_SMD:SOT-23, F.Cu at (122.0, 140.0)
- added R35: 100, Resistor_SMD:R_0402_1005Metric, F.Cu at (127.0, 139.1)
- added R36: 300, Resistor_SMD:R_0402_1005Metric, F.Cu at (125.0, 139.1)
- added R37: 82, Resistor_SMD:R_1206_3216Metric, F.Cu at (117.5, 140.2)
- added R38: 100, Resistor_SMD:R_0402_1005Metric, F.Cu at (127.0, 135.7)
- added R39: 300, Resistor_SMD:R_0402_1005Metric, F.Cu at (125.0, 135.7)
- added R40: 82, Resistor_SMD:R_1206_3216Metric, F.Cu at (117.5, 136.7)
- added R41: 100, Resistor_SMD:R_0402_1005Metric, F.Cu at (127.1, 132.2)
- added R42: 300, Resistor_SMD:R_0402_1005Metric, F.Cu at (125.1, 132.2)
- added R43: 82, Resistor_SMD:R_1206_3216Metric, F.Cu at (117.5, 133.2)
- added R46: 82, Resistor_SMD:R_1206_3216Metric, F.Cu at (117.5, 129.8)
- added R50: 100, Resistor_SMD:R_0402_1005Metric, F.Cu at (127.1, 121.9)
- added R54: 300, Resistor_SMD:R_0402_1005Metric, F.Cu at (125.1, 118.5)
- added R58: 82, Resistor_SMD:R_1206_3216Metric, F.Cu at (117.5, 116.2)
- added R62: 100, Resistor_SMD:R_0402_1005Metric, F.Cu at (127.1, 108.3)
- added R66: 300, Resistor_SMD:R_0402_1005Metric, F.Cu at (125.1, 104.9)
- added R70: 82, Resistor_SMD:R_1206_3216Metric, F.Cu at (117.6, 102.5)
- added R74: 100, Resistor_SMD:R_0402_1005Metric, F.Cu at (127.1, 94.6)
- added R78: 300, Resistor_SMD:R_0402_1005Metric, F.Cu at (125.1, 91.2)
- added Y1: 40MHz, Crystal:Crystal_SMD_3225-4Pin_3.2x2.5mm, F.Cu at (172.6, 104.9)
- J10, J9: value Conn_01x03 -> Conn_01x03_MountingPin
- J11: value Conn_01x11 -> Conn_01x11_MountingPin
- J5: value CAN -> Conn_01x02_MountingPin
- Q9: value BSS127S -> MMBT3904
- R47, R59, R71: value 82 -> 100; footprint Resistor_SMD:R_1206_3216Metric -> Resistor_SMD:R_0402_1005Metric
- R48, R60, R72: value 100 -> 300
- R49, R61, R73: value 300 -> 82; footprint Resistor_SMD:R_0402_1005Metric -> Resistor_SMD:R_1206_3216Metric
- R51, R63, R75: value 82 -> 300; footprint Resistor_SMD:R_1206_3216Metric -> Resistor_SMD:R_0402_1005Metric
- R52, R64, R76: value 100 -> 82; footprint Resistor_SMD:R_0402_1005Metric -> Resistor_SMD:R_1206_3216Metric
- R53, R65, R77: value 300 -> 100
- moved R1 156.0 mm to (83.2, 133.5)
- moved R2 156.0 mm to (83.2, 135.5)
- moved R5 156.0 mm to (79.5, 133.7)
- moved R8 156.0 mm to (79.5, 136.2)
- moved D3 145.0 mm to (91.2, 124.2)
- moved R67 141.2 mm to (117.6, 105.9)
- moved R64 137.9 mm to (117.5, 109.4)
- moved R73 135.2 mm to (117.6, 99.1)
- moved R75 132.4 mm to (125.1, 94.6), turned to 180 degrees
- moved R49 132.0 mm to (117.5, 126.4)
- moved R79 131.7 mm to (117.5, 92.2)
- moved R65 131.3 mm to (127.1, 104.9), turned to 180 degrees
- moved R76 128.5 mm to (117.6, 95.6)
- moved R72 127.9 mm to (125.2, 98.1), turned to 180 degrees
- moved C26 127.6 mm to (127.1, 122.9), turned to 180 degrees
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- renumbered C12 to C11, C15 to C14, C20 to C19, C8 to C20, C2 to C3, C3 to C5, C4 to C6, C5 to C7, C9 to C8, C10 to C9, Q6 to Q3, Q7 to Q4, Q8 to Q5, Q5 to Q7, R36 to R24, R38 to R26, R43 to R31, R19 to R32, R20 to R33, R22 to R34
Connections:
- C21 pad 1: /Frontend/VC4 -> /Frontend/VC2
- C21 pad 2: /Frontend/VC3 -> /Frontend/VC1
- C22 pad 1: /Frontend/VC5 -> /Frontend/VC3
- C22 pad 2: /Frontend/VC4 -> /Frontend/VC2
- C23 pad 1: /Frontend/VC6 -> /Frontend/VC4
- C23 pad 2: /Frontend/VC5 -> /Frontend/VC3
- C24 pad 1: /Frontend/VC7 -> /Frontend/VC5
- C24 pad 2: /Frontend/VC6 -> /Frontend/VC4
- C25 pad 1: /Frontend/VC8 -> /Frontend/VC6
- C25 pad 2: /Frontend/VC7 -> /Frontend/VC5
- C26 pad 1: /Frontend/VC9 -> /Frontend/VC7
- C26 pad 2: /Frontend/VC8 -> /Frontend/VC6
- C27 pad 1: /Frontend/VC10 -> /Frontend/VC8
- C27 pad 2: /Frontend/VC9 -> /Frontend/VC7
- C28 pad 1: /Frontend/VC11 -> /Frontend/VC9
- C28 pad 2: /Frontend/VC10 -> /Frontend/VC8
- C29 pad 1: /Frontend/VC12 -> /Frontend/VC10
- C29 pad 2: /Frontend/VC11 -> /Frontend/VC9
- C30 pad 1: /Frontend/VC13 -> /Frontend/VC11
- C30 pad 2: /Frontend/VC12 -> /Frontend/VC10
- C31 pad 1: /Frontend/VC14 -> /Frontend/VC12
- C31 pad 2: /Frontend/VC13 -> /Frontend/VC11
- C32 pad 1: /Frontend/VC15 -> /Frontend/VC13
- C32 pad 2: /Frontend/VC14 -> /Frontend/VC12
- C33 pad 1: /Frontend/VC16 -> /Frontend/VC14
- C33 pad 2: /Frontend/VC15 -> /Frontend/VC13
- J10 pad 1: unconnected-(J10-Pin_1-Pad1) -> /Frontend/CEL_11
- J10 pad 3: /Frontend/CEL_11 -> unconnected-(J10-Pin_3-Pad3)
- J10 pad MP: (no net) -> GND
- J11 pad 1: /Frontend/CEL_10 -> /Frontend/CEL_0
- J11 pad 10: /Frontend/CEL_1 -> /Frontend/CEL_9
- J11 pad 11: /Frontend/CEL_0 -> /Frontend/CEL_10
- J11 pad 2: /Frontend/CEL_9 -> /Frontend/CEL_1
- J11 pad 3: /Frontend/CEL_8 -> /Frontend/CEL_2
- J11 pad 4: unconnected-(J11-Pin_4-Pad4) -> /Frontend/CEL_3
- J11 pad 5: /Frontend/CEL_6 -> /Frontend/CEL_4
- J11 pad 7: /Frontend/CEL_4 -> /Frontend/CEL_6
- J11 pad 8: /Frontend/CEL_3 -> unconnected-(J11-Pin_8-Pad8)
- J11 pad 9: /Frontend/CEL_2 -> /Frontend/CEL_8
- J11 pad MP: (no net) -> GND
- J5 pad MP: (no net) -> GND
- J7 pad MP: (no net) -> GND
- J8 pad MP: (no net) -> GND
- J9 pad 1: /Frontend/CEL_16 -> /Frontend/CEL_14
- J9 pad 3: /Frontend/CEL_14 -> /Frontend/CEL_16
- J9 pad MP: (no net) -> GND
- Q9 pad 2: /PACK+ -> /Frontend/CEL_2
- R44 pad 1: /Frontend/VC4 -> /Frontend/VC5
- R44 pad 2: /Frontend/CEL_4 -> /Frontend/CEL_5
- R45 pad 1: /Frontend/VC3 -> /Frontend/VC4
- R45 pad 2: Net-(Q10-B) -> Net-(Q11-B)
- R47 pad 1: /Frontend/CEL_4 -> /Frontend/VC6
- R47 pad 2: Net-(Q10-C) -> /Frontend/CEL_6
- R48 pad 2: /Frontend/CEL_5 -> Net-(Q12-B)
- R49 pad 1: /Frontend/VC4 -> /Frontend/CEL_6
- R49 pad 2: Net-(Q11-B) -> Net-(Q12-C)
- R51 pad 1: /Frontend/CEL_5 -> /Frontend/VC6
- R51 pad 2: Net-(Q11-C) -> Net-(Q13-B)
- R52 pad 1: /Frontend/VC6 -> /Frontend/CEL_7
- R52 pad 2: /Frontend/CEL_6 -> Net-(Q13-C)
- R53 pad 1: /Frontend/VC5 -> /Frontend/VC8
- R53 pad 2: Net-(Q12-B) -> /Frontend/CEL_8
- R55 pad 1: /Frontend/CEL_6 -> /Frontend/CEL_8
- R55 pad 2: Net-(Q12-C) -> Net-(Q14-C)
- R56 pad 1: /Frontend/VC7 -> /Frontend/VC9
- R56 pad 2: /Frontend/CEL_7 -> /Frontend/CEL_9
- R57 pad 1: /Frontend/VC6 -> /Frontend/VC8
- R57 pad 2: Net-(Q13-B) -> Net-(Q15-B)
- R59 pad 1: /Frontend/CEL_7 -> /Frontend/VC10
- R59 pad 2: Net-(Q13-C) -> /Frontend/CEL_10
- R60 pad 1: /Frontend/VC8 -> /Frontend/VC9
- R60 pad 2: /Frontend/CEL_8 -> Net-(Q16-B)
- R61 pad 1: /Frontend/VC7 -> /Frontend/CEL_10
- R61 pad 2: Net-(Q14-B) -> Net-(Q16-C)
- R63 pad 1: /Frontend/CEL_8 -> /Frontend/VC10
- R63 pad 2: Net-(Q14-C) -> Net-(Q17-B)
- R64 pad 1: /Frontend/VC9 -> /Frontend/CEL_11
- R64 pad 2: /Frontend/CEL_9 -> Net-(Q17-C)
- R65 pad 1: /Frontend/VC8 -> /Frontend/VC12
- R65 pad 2: Net-(Q15-B) -> /Frontend/CEL_12
- R67 pad 1: /Frontend/CEL_9 -> /Frontend/CEL_12
- R67 pad 2: Net-(Q15-C) -> Net-(Q18-C)
- R68 pad 1: /Frontend/VC10 -> /Frontend/VC13
- R68 pad 2: /Frontend/CEL_10 -> /Frontend/CEL_13
- R69 pad 1: /Frontend/VC9 -> /Frontend/VC12
- R69 pad 2: Net-(Q16-B) -> Net-(Q19-B)
- R71 pad 1: /Frontend/CEL_10 -> /Frontend/VC14
- R71 pad 2: Net-(Q16-C) -> /Frontend/CEL_14
- R72 pad 1: /Frontend/VC11 -> /Frontend/VC13
- R72 pad 2: /Frontend/CEL_11 -> Net-(Q20-B)
- R73 pad 1: /Frontend/VC10 -> /Frontend/CEL_14
- R73 pad 2: Net-(Q17-B) -> Net-(Q20-C)
- R75 pad 1: /Frontend/CEL_11 -> /Frontend/VC14
- R75 pad 2: Net-(Q17-C) -> Net-(Q21-B)
- R76 pad 1: /Frontend/VC12 -> /Frontend/CEL_15
- R76 pad 2: /Frontend/CEL_12 -> Net-(Q21-C)
- R77 pad 1: /Frontend/VC11 -> /Frontend/VC16
- R77 pad 2: Net-(Q18-B) -> /Frontend/CEL_16
- R79 pad 1: /Frontend/CEL_12 -> /Frontend/CEL_16
- R79 pad 2: Net-(Q18-C) -> Net-(Q22-C)
- U1 pad 10: unconnected-(U1-MTDI-Pad10) -> /CHG_EN
- U1 pad 14: unconnected-(U1-GPIO8-Pad14) -> /PCHG_EN
- U1 pad 15: unconnected-(U1-GPIO9-Pad15) -> /MCU/CAN_EN
- U1 pad 16: unconnected-(U1-GPIO10-Pad16) -> /MCU/PSW_EN
- U1 pad 29: unconnected-(U1-XTAL_N-Pad29) -> Net-(U1-XTAL_N)
- U1 pad 30: unconnected-(U1-XTAL_P-Pad30) -> Net-(U1-XTAL_P)
- U1 pad 4: unconnected-(U1-XTAL_32K_P-Pad4) -> /MCU/DIV_CHG
- U1 pad 5: unconnected-(U1-XTAL_32K_N-Pad5) -> /MCU/DIV_OUT
- U1 pad 6: unconnected-(U1-GPIO2-Pad6) -> /HW_EN
- U1 pad 9: unconnected-(U1-MTMS-Pad9) -> /DSG_EN
- U5 pad 31: /Frontend/DCHG -> unconnected-(U5-DCHG-Pad31)
- U5 pad 32: /Frontend/DDSG -> unconnected-(U5-DDSG-Pad32)
- U5 pad 39: unconnected-(U5-PDSG-Pad39) -> /Frontend/PDSG
- U5 pad 40: unconnected-(U5-PCHG-Pad40) -> /Frontend/PCHG
- U5 pad 43: unconnected-(U5-DSG-Pad43) -> /Frontend/DSG
- U5 pad 45: unconnected-(U5-CHG-Pad45) -> /Frontend/CHG
Routing:
- net Net-(U1-XTAL_N): track 0.00 -> 7.68 mm
- net GND: track 0.00 -> 3.16 mm, vias 0 -> 2
- net Net-(C4-Pad1): track 0.00 -> 1.75 mm
- added copper zone on F.Cu, net GND
Other:
- board size 100 x 40 mm -> 100 x 60 mm

Commit message: Crystal Layout
Routing:
- net GND: track 3.16 -> 5.68 mm, vias 2 -> 4
- net Net-(C4-Pad1): track 1.75 -> 3.18 mm
- net Net-(U1-XTAL_P): track 0.00 -> 1.30 mm
Changed lines of the file:
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@@
+	)
+	(segment
+		(start 171.43 104.03)
+		(end 171 103.6)
+		(width 0.25)
+		(layer "F.Cu")
+		(net 2)
+	)
+	(segment
+		(start 170.2 103.6)
+		(end 170.1 103.5)
+		(width 0.25)
+		(layer "F.Cu")
+		(net 2)
 	)
 	(segment
@@
 	)
 	(segment
+		(start 171.5 104.03)
+		(end 171.43 104.03)
+		(width 0.25)
+		(layer "F.Cu")
+		(net 2)
+	)
+	(segment
 		(start 174.17 106.2)
 		(end 173.7 105.73)
@@
 	)
 	(segment
+		(start 169.9 104.4)
+		(end 169 104.4)
+		(width 0.25)
+		(layer "F.Cu")
+		(net 2)
+	)
+	(segment
 		(start 173.7 105.73)
 		(end 173.83 105.73)
+		(width 0.25)
+		(layer "F.Cu")
+		(net 2)
+	)
+	(segment
+		(start 171 103.6)
+		(end 170.2 103.6)
 		(width 0.25)
 		(layer "F.Cu")
@@
 		(net 2)
 	)
+	(via
+		(at 170.1 103.5)
+		(size 0.8)
+		(drill 0.4)
+		(layers "F.Cu" "B.Cu")
+		(net 2)
+	)
+	(via
+		(at 169 104.4)
+		(size 0.8)
+		(drill 0.4)
+		(layers "F.Cu" "B.Cu")
+		(net 2)
+	)
+	(segment
+		(start 171.5 107.015)
+		(end 171.6 107.115)
+		(width 0.25)
+		(layer "F.Cu")
+		(net 45)
+	)
 	(segment
 		(start 171.13 105.36)
@@
 		(layer "F.Cu")
 		(net 45)
+	)
+	(segment
+		(start 171.5 105.73)
+		(end 171.5 107.015)
+		(width 0.25)
+		(layer "F.Cu")
+		(net 45)
+	)
+	(segment
+		(start 171.8 108.285)
+		(end 171.8 109.3)
+		(width 0.25)
+		(layer "F.Cu")
+		(net 62)
+	)
+	(segment
+		(start 171.6 108.085)
+		(end 171.8 108.285)
+		(width 0.25)
+		(layer "F.Cu")
+		(net 62)
 	)
 	(segment
@@
 			)
 		)
+	)
+	(zone
+		(net 0)
+		(net_name "")
+		(layer "B.Cu")
+		(hatch edge 0.5)
+		(connect_pads
+			(clearance 0)
+		)
+		(min_thickness 0.25)
+		(filled_areas_thickness no)
+		(keepout
+			(tracks not_allowed)
+			(vias allowed)
+			(pads allowed)
+			(copperpour allowed)
+			(footprints allowed)
+		)
+		(placement
+			(enabled no)
+			(sheetname "/")
+		)
+		(fill
+			(thermal_gap 0.5)
+			(thermal_bridge_width 0.5)
+		)
+		(polygon
+			(pts
+				(xy 176 103) (xy 176 106.8) (xy 172.9 106.8) (xy 172.9 108.7) (xy 171 108.7) (xy 171 106.7) (xy 169.2 106.7)
+				(xy 169.2 103)
+			)
+		)

Commit message: Increased Discharge Resistor size
Parts:
- R34, R37, R40, R43, R46, R49, R52, R55, R58, R61, R64, R67, R70, R73, R76, R79: footprint Resistor_SMD:R_1206_3216Metric -> Resistor_SMD:R_1210_3225Metric
- moved D4 63.3 mm to (152.6, 142.9)
- moved Q6 53.9 mm to (143.7, 137.1)
- moved D3 53.9 mm to (144.4, 133.0)
- moved R1 53.9 mm to (136.4, 142.2)
- moved R2 53.9 mm to (136.4, 144.2)
- moved R5 53.9 mm to (132.8, 142.5)
- moved R8 53.9 mm to (132.8, 145.0)
- moved U2 48.4 mm to (152.5, 137.0)
- moved J4 19.1 mm to (170.5, 131.9)
- moved Q11 0.27 mm to (121.8, 129.7), turned to 180 degrees
- moved Q12 0.27 mm to (121.8, 126.3), turned to 180 degrees
- moved Q15 0.27 mm to (121.8, 116.1), turned to 180 degrees
- moved Q13 0.27 mm to (121.9, 122.9), turned to 180 degrees
- moved Q14 0.27 mm to (121.9, 119.5), turned to 180 degrees
- moved Q16 0.27 mm to (121.9, 112.7), turned to 180 degrees
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Connections:
- U1 pad 33: unconnected-(U1-GND-Pad33) -> GND

Commit message: Cell balancing sourcing and repositioning
Parts:
- R34, R37, R40, R43, R46, R49, R52, R55, R58, R61, R64, R67, R70, R73, R76, R79: value 82 -> 36
- moved Q22 1.22 mm to (120.6, 92.0)
- moved Q9 1.22 mm to (120.6, 136.4)
- moved R45 1.22 mm to (123.9, 128.5)
- moved R67 1.22 mm to (116.4, 105.7)
- moved C27 1.22 mm to (125.9, 119.3)
- moved C29 1.22 mm to (125.9, 112.5)
- moved C31 1.22 mm to (125.9, 105.7)
- moved Q17 1.22 mm to (120.6, 109.1)
- moved Q20 1.22 mm to (120.7, 98.9)
- moved R48 1.22 mm to (123.9, 125.1)
- moved R53 1.22 mm to (125.9, 118.3)
- moved R55 1.22 mm to (116.4, 119.4)
- moved R57 1.22 mm to (123.8, 114.9)
- moved R59 1.22 mm to (125.9, 111.5)
- moved R61 1.22 mm to (116.4, 112.6)
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- renumbered J9 to J10, J10 to J9
Connections:
- J10 pad 1: /Frontend/CEL_14 -> /Frontend/CEL_11
- J10 pad 2: /Frontend/CEL_15 -> /Frontend/CEL_12
- J10 pad 3: /Frontend/CEL_16 -> /Frontend/CEL_13
- J9 pad 1: /Frontend/CEL_11 -> /Frontend/CEL_14
- J9 pad 2: unconnected-(J10-Pin_2-Pad2) -> /Frontend/CEL_15
- J9 pad 3: unconnected-(J10-Pin_3-Pad3) -> /Frontend/CEL_16

Commit message: Layout test
Parts:
- removed J10, J9: Conn_01x03_MountingPin, Connector_JST:JST_PH_S3B-PH-SM4-TB_1x03-1MP_P2.00mm_Horizontal
- removed J11: Conn_01x11_MountingPin, Connector_JST:JST_PH_S11B-PH-SM4-TB_1x11-1MP_P2.00mm_Horizontal
- added C38: 100n, Capacitor_SMD:C_0402_1005Metric, F.Cu at (82.9, 110.0)
- added C39: 100n, Capacitor_SMD:C_0402_1005Metric, F.Cu at (72.4, 131.6)
- added C40: 100n, Capacitor_SMD:C_0402_1005Metric, F.Cu at (82.9, 131.6)
- added C41: 100n, Capacitor_SMD:C_0402_1005Metric, F.Cu at (93.4, 88.3)
- added C42: 100n, Capacitor_SMD:C_0402_1005Metric, F.Cu at (93.4, 120.8)
- added C43: 100n, Capacitor_SMD:C_0402_1005Metric, F.Cu at (93.4, 110.0)
- added C44: 100n, Capacitor_SMD:C_0402_1005Metric, F.Cu at (72.4, 99.1)
- added C45: 100n, Capacitor_SMD:C_0402_1005Metric, F.Cu at (58.7, 135.3)
- added C46: 100n, Capacitor_SMD:C_0402_1005Metric, F.Cu at (82.9, 99.1)
- added C47: 100n, Capacitor_SMD:C_0402_1005Metric, F.Cu at (48.2, 135.3)
- added C48: 100n, Capacitor_SMD:C_0402_1005Metric, F.Cu at (82.9, 120.8)
- added C49: 100n, Capacitor_SMD:C_0402_1005Metric, F.Cu at (82.9, 88.3)
- added C50: 100n, Capacitor_SMD:C_0402_1005Metric, F.Cu at (72.4, 88.3)
- added C51: 100n, Capacitor_SMD:C_0402_1005Metric, F.Cu at (72.4, 110.0)
- added C52: 100n, Capacitor_SMD:C_0402_1005Metric, F.Cu at (93.4, 99.1)
- added C53: 100n, Capacitor_SMD:C_0402_1005Metric, F.Cu at (72.4, 120.8)
- added J12: Conn_01x08_MountingPin, Connector_JST:JST_PH_S8B-PH-SM4-TB_1x08-1MP_P2.00mm_Horizontal, F.Cu at (107.7, 133.2)
- added J13: Conn_01x08_MountingPin, Connector_JST:JST_PH_S8B-PH-SM4-TB_1x08-1MP_P2.00mm_Horizontal, F.Cu at (107.9, 106.8)
- added J14: Conn_01x08_MountingPin, Connector_JST:JST_PH_S8B-PH-SM4-TB_1x08-1MP_P2.00mm_Horizontal, F.Cu at (52.3, 115.4)
- added J15: Conn_01x08_MountingPin, Connector_JST:JST_PH_S8B-PH-SM4-TB_1x08-1MP_P2.00mm_Horizontal, F.Cu at (52.3, 126.7)
- added Q23: MMBT3904, Package_TO_SOT_SMD:SOT-23, F.Cu at (54.1, 140.9)
- added Q24: MMBT3904, Package_TO_SOT_SMD:SOT-23, F.Cu at (78.3, 137.2)
- added Q25: MMBT3904, Package_TO_SOT_SMD:SOT-23, F.Cu at (88.8, 93.9)
- added Q26: MMBT3904, Package_TO_SOT_SMD:SOT-23, F.Cu at (88.8, 126.4)
- added Q27: MMBT3904, Package_TO_SOT_SMD:SOT-23, F.Cu at (88.8, 115.6)
- added Q28: MMBT3904, Package_TO_SOT_SMD:SOT-23, F.Cu at (67.8, 104.8)
- added Q29: MMBT3904, Package_TO_SOT_SMD:SOT-23, F.Cu at (78.3, 104.8)
- added Q30: MMBT3904, Package_TO_SOT_SMD:SOT-23, F.Cu at (67.8, 126.4)
- added Q31: MMBT3904, Package_TO_SOT_SMD:SOT-23, F.Cu at (78.3, 126.4)
- added Q32: MMBT3904, Package_TO_SOT_SMD:SOT-23, F.Cu at (43.6, 140.9)
- added Q33: MMBT3904, Package_TO_SOT_SMD:SOT-23, F.Cu at (78.3, 93.9)
- added Q34: MMBT3904, Package_TO_SOT_SMD:SOT-23, F.Cu at (67.8, 93.9)
- added Q35: MMBT3904, Package_TO_SOT_SMD:SOT-23, F.Cu at (67.8, 115.6)
- added Q36: MMBT3904, Package_TO_SOT_SMD:SOT-23, F.Cu at (88.8, 104.8)
- added Q37: MMBT3904, Package_TO_SOT_SMD:SOT-23, F.Cu at (78.3, 115.6)
- added Q38: MMBT3904, Package_TO_SOT_SMD:SOT-23, F.Cu at (67.8, 137.2)
- added R100: 300, Resistor_SMD:R_0402_1005Metric, F.Cu at (58.0, 141.5)
- added R101: 300, Resistor_SMD:R_0402_1005Metric, F.Cu at (82.2, 105.3)
- added R102: 300, Resistor_SMD:R_0402_1005Metric, F.Cu at (82.2, 116.2)
- added R103: 300, Resistor_SMD:R_0402_1005Metric, F.Cu at (71.7, 127.0)
- added R104: 300, Resistor_SMD:R_0402_1005Metric, F.Cu at (82.2, 137.8)
- added R105: 300, Resistor_SMD:R_0402_1005Metric, F.Cu at (47.5, 141.5)
- added R106: 300, Resistor_SMD:R_0402_1005Metric, F.Cu at (82.2, 127.0)
- added R107: 300, Resistor_SMD:R_0402_1005Metric, F.Cu at (92.7, 105.3)
- added R108: 300, Resistor_SMD:R_0402_1005Metric, F.Cu at (82.2, 94.5)
- added R109: 300, Resistor_SMD:R_0402_1005Metric, F.Cu at (92.7, 94.5)
- added R110: 300, Resistor_SMD:R_0402_1005Metric, F.Cu at (71.7, 94.5)
- added R111: 300, Resistor_SMD:R_0402_1005Metric, F.Cu at (71.7, 116.2)
- added R112: 36, Resistor_SMD:R_1210_3225Metric, F.Cu at (89.2, 89.4)
- added R113: 36, Resistor_SMD:R_1210_3225Metric, F.Cu at (89.2, 121.9)
- added R114: 36, Resistor_SMD:R_1210_3225Metric, F.Cu at (89.2, 111.1)
- added R115: 36, Resistor_SMD:R_1210_3225Metric, F.Cu at (78.7, 132.7)
- added R116: 36, Resistor_SMD:R_1210_3225Metric, F.Cu at (68.2, 100.2)
- added R117: 36, Resistor_SMD:R_1210_3225Metric, F.Cu at (54.4, 136.4)
- added R118: 36, Resistor_SMD:R_1210_3225Metric, F.Cu at (78.7, 100.2)
- added R119: 36, Resistor_SMD:R_1210_3225Metric, F.Cu at (68.2, 121.9)
- added R120: 36, Resistor_SMD:R_1210_3225Metric, F.Cu at (43.9, 136.4)
- added R121: 36, Resistor_SMD:R_1210_3225Metric, F.Cu at (78.7, 121.9)
- added R122: 36, Resistor_SMD:R_1210_3225Metric, F.Cu at (78.7, 89.4)
- added R123: 36, Resistor_SMD:R_1210_3225Metric, F.Cu at (68.2, 89.4)
- added R124: 36, Resistor_SMD:R_1210_3225Metric, F.Cu at (68.2, 111.1)
- added R125: 36, Resistor_SMD:R_1210_3225Metric, F.Cu at (89.2, 100.2)
- added R126: 36, Resistor_SMD:R_1210_3225Metric, F.Cu at (78.7, 111.1)
- added R127: 36, Resistor_SMD:R_1210_3225Metric, F.Cu at (68.2, 132.7)
- added R80: 100, Resistor_SMD:R_0402_1005Metric, F.Cu at (71.7, 92.5)
- added R81: 100, Resistor_SMD:R_0402_1005Metric, F.Cu at (82.2, 92.5)
- added R82: 100, Resistor_SMD:R_0402_1005Metric, F.Cu at (92.7, 92.5)
- added R83: 100, Resistor_SMD:R_0402_1005Metric, F.Cu at (82.2, 125.0)
- added R84: 100, Resistor_SMD:R_0402_1005Metric, F.Cu at (47.5, 139.5)
- added R85: 100, Resistor_SMD:R_0402_1005Metric, F.Cu at (71.7, 125.0)
- added R86: 100, Resistor_SMD:R_0402_1005Metric, F.Cu at (92.7, 125.0)
- added R87: 100, Resistor_SMD:R_0402_1005Metric, F.Cu at (82.2, 103.3)
- added R88: 100, Resistor_SMD:R_0402_1005Metric, F.Cu at (58.0, 139.5)
- added R89: 100, Resistor_SMD:R_0402_1005Metric, F.Cu at (71.7, 103.3)
- added R90: 100, Resistor_SMD:R_0402_1005Metric, F.Cu at (92.7, 114.2)
- added R91: 100, Resistor_SMD:R_0402_1005Metric, F.Cu at (71.7, 135.8)
- added R92: 100, Resistor_SMD:R_0402_1005Metric, F.Cu at (71.7, 114.2)
- added R93: 100, Resistor_SMD:R_0402_1005Metric, F.Cu at (82.2, 135.8)
- added R94: 100, Resistor_SMD:R_0402_1005Metric, F.Cu at (82.2, 114.2)
- added R95: 100, Resistor_SMD:R_0402_1005Metric, F.Cu at (92.7, 103.3)
- added R96: 300, Resistor_SMD:R_0402_1005Metric, F.Cu at (92.7, 127.0)
- added R97: 300, Resistor_SMD:R_0402_1005Metric, F.Cu at (71.7, 105.3)
- added R98: 300, Resistor_SMD:R_0402_1005Metric, F.Cu at (71.7, 137.8)
- added R99: 300, Resistor_SMD:R_0402_1005Metric, F.Cu at (92.7, 116.2)
- added U6: BQ769x2, Package_QFP:TQFP-48_7x7mm_P0.5mm, F.Cu at (70.9, 150.8)
- J5: value Conn_01x02_MountingPin -> CAN
- Q4, Q5: value IPTC025N15NM6 -> IPT015N10N5
Connections:
- net /Frontend/ALERT renamed Net-(U5-ALERT)
- D1 pad 2: +3.3V -> +3.3VP
- D2 pad 2: +3.3V -> +3.3VP
- J6 pad A4: /MCU/VBUS -> unconnected-(J6-VBUS-PadA4)_1
- J6 pad A6: /MCU/DP -> /USB_DN
- J6 pad A7: /MCU/DN -> /USB_DP
- J6 pad A9: /MCU/VBUS -> unconnected-(J6-VBUS-PadA4)
- J6 pad B4: /MCU/VBUS -> unconnected-(J6-VBUS-PadA4)_2
- J6 pad B6: /MCU/DP -> /USB_DN
- J6 pad B7: /MCU/DN -> /USB_DP
- J6 pad B9: /MCU/VBUS -> unconnected-(J6-VBUS-PadA4)_3
- U1 pad 1: unconnected-(U1-LNA_IN-Pad1) -> Net-(U1-LNA_IN)
- U1 pad 15: /MCU/CAN_EN -> /MCU/~{COM_EN}
- U1 pad 25: /MCU/DN -> /MCU/USB_DP
- U1 pad 26: /MCU/DP -> /MCU/USB_DN
- U2 pad 1: /MCU/CAN_TX -> /CAN_TX
- U2 pad 4: /MCU/CAN_RX -> /CAN_RX
- U2 pad 8: /MCU/CAN_EN -> /CAN_EN
- U5 pad 29: /Frontend/CFETOFF -> unconnected-(U5-CFETOFF-Pad29)
- U5 pad 30: /Frontend/DFETOFF -> unconnected-(U5-DFETOFF-Pad30)
- U5 pad 31: unconnected-(U5-DCHG-Pad31) -> Net-(U5-DCHG)
- U5 pad 32: unconnected-(U5-DDSG-Pad32) -> Net-(U5-DDSG)
- U5 pad 33: unconnected-(U5-RST_SHUT-Pad33) -> /Frontend/EN
- U5 pad 39: /Frontend/PDSG -> unconnected-(U5-PDSG-Pad39)
- U5 pad 40: /Frontend/PCHG -> unconnected-(U5-PCHG-Pad40)
- U5 pad 43: /Frontend/DSG -> unconnected-(U5-DSG-Pad43)
- U5 pad 45: /Frontend/CHG -> unconnected-(U5-CHG-Pad45)
Other:
- board size 100 x 60 mm -> 100 x 56 mm

Commit message: Charge and Discharge FETs
Parts:
- removed D3, D4: BZV55C16, Diode_SMD:D_MiniMELF
- removed Q6: BSS127S, Package_TO_SOT_SMD:SOT-23
- added Q39: IPT015N10N5, Package_TO_SOT_SMD:Infineon_PG-HSOF-8-1_ThermalVias, F.Cu at (152.2, 15.8)
- added Q40: IPT015N10N5, Package_TO_SOT_SMD:Infineon_PG-HSOF-8-1_ThermalVias, F.Cu at (152.2, 27.5)
- added Q41: IPT015N10N5, Package_TO_SOT_SMD:Infineon_PG-HSOF-8-1_ThermalVias, F.Cu at (152.2, 39.2)
- added Q42: IPT015N10N5, Package_TO_SOT_SMD:Infineon_PG-HSOF-8-1_ThermalVias, F.Cu at (152.2, 50.9)
- added Q43: IPT015N10N5, Package_TO_SOT_SMD:Infineon_PG-HSOF-8-1_ThermalVias, F.Cu at (152.2, 62.5)
- added Q44: IPT015N10N5, Package_TO_SOT_SMD:Infineon_PG-HSOF-8-1_ThermalVias, F.Cu at (152.2, 74.2)
- added U8: ISO1540, Package_SO:SOIC-8_3.9x4.9mm_P1.27mm, F.Cu at (163.8, 13.3)
- Q4, Q5: footprint Package_TO_SOT_SMD:Infineon_PG-HSOF-8-1 -> Package_TO_SOT_SMD:Infineon_PG-HSOF-8-1_ThermalVias
- moved Q5 66.2 mm to (130.3, 51.3), turned to 90 degrees
- moved Q4 58.5 mm to (132.6, 70.3), turned to -90 degrees
- moved J13 0.10 mm to (107.9, 106.7)
Connections:
- U6 pad 26: unconnected-(U6-SCL-Pad26) -> /Frontend/I2C_SCL_TOP
- U6 pad 27: unconnected-(U6-SDA-Pad27) -> /Frontend/I2C_SDA_TOP

Commit message: FET layout study
Parts:
- J14, J15: moved to B.Cu
- R10, R6, R9: footprint Resistor_SMD:R_0603_1608Metric -> Resistor_SMD:R_0402_1005Metric
- moved Q39 95.0 mm to (152.5, 110.8)
- moved Q40 94.4 mm to (152.5, 121.9)
- moved Q41 94.0 mm to (152.5, 133.1)
- moved C11 80.7 mm to (234.3, 53.5)
- moved C9 80.7 mm to (234.3, 51.5)
- moved J2 80.7 mm to (218.0, 73.6)
- moved J4 80.7 mm to (218.0, 66.6)
- moved J6 80.7 mm to (194.4, 30.1)
- moved J7 80.7 mm to (244.2, 75.1)
- moved Q1 80.7 mm to (233.2, 34.3)
- moved Q2 80.7 mm to (233.2, 38.9)
- moved R10 80.7 mm to (237.6, 38.2)
- moved R4 80.7 mm to (203.6, 27.9)
- moved TH1 80.7 mm to (213.0, 31.0)
- moved U2 80.7 mm to (200.0, 71.7)
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Connections:
- net /Frontend/EN renamed Net-(U5-RST_SHUT)
- J14 pad 1: unconnected-(J14-Pin_1-Pad1) -> /Frontend/CEL_23
- J14 pad 2: unconnected-(J14-Pin_2-Pad2) -> /Frontend/CEL_22
- J14 pad 3: unconnected-(J14-Pin_3-Pad3) -> /Frontend/CEL_21
- J14 pad 4: unconnected-(J14-Pin_4-Pad4) -> /Frontend/CEL_20
- J14 pad 5: unconnected-(J14-Pin_5-Pad5) -> /Frontend/CEL_19
- J14 pad 6: unconnected-(J14-Pin_6-Pad6) -> /Frontend/CEL_18
- J14 pad 7: unconnected-(J14-Pin_7-Pad7) -> /Frontend/CEL_17
- J14 pad 8: unconnected-(J14-Pin_8-Pad8) -> /Frontend/CEL_16
- J15 pad 1: unconnected-(J15-Pin_1-Pad1) -> /Frontend/CEL_31
- J15 pad 2: unconnected-(J15-Pin_2-Pad2) -> /Frontend/CEL_30
- J15 pad 3: unconnected-(J15-Pin_3-Pad3) -> /Frontend/CEL_29
- J15 pad 4: unconnected-(J15-Pin_4-Pad4) -> /Frontend/CEL_28
- J15 pad 5: unconnected-(J15-Pin_5-Pad5) -> /Frontend/CEL_27
- J15 pad 6: unconnected-(J15-Pin_6-Pad6) -> /Frontend/CEL_26
- J15 pad 7: unconnected-(J15-Pin_7-Pad7) -> /Frontend/CEL_25
- J15 pad 8: unconnected-(J15-Pin_8-Pad8) -> /Frontend/CEL_24
- U6 pad 17: GND -> GND2
- U6 pad 33: unconnected-(U6-RST_SHUT-Pad33) -> Net-(U6-RST_SHUT)
- U8 pad 1: +3.3V -> +3.3VP
Routing:
- added copper zone on B.Cu, net GND
- added copper zone on In1.Cu, net GND
Other:
- copper layers 2 -> 4

Commit message: ESP32 Decoupling
Parts:
- added AE1: Antenna_Shield, RF_Antenna:Texas_SWRA117D_2.4GHz_Left, F.Cu at (205.3, 101.0)
- C3: value 100n -> 1u
- C5: value 100n -> 10u
- C6: value 4.7u -> 100n
- Q23, Q24, Q25, Q26, Q27, Q28, Q29, Q30, Q31, Q32, Q33, Q34, Q35, Q36, Q37, Q38, R112, R113, R114, R115, R116, R117, R118, R119, R120, R121, R122, R123, R124, R125, R126, R127: moved to B.Cu
- U4: value TPS7A0533PDBZ -> AMS1117-3.3; footprint Package_TO_SOT_SMD:SOT-23 -> Package_TO_SOT_SMD:SOT-223-3_TabPin2
- moved R115 103.7 mm to (116.2, 143.2)
- moved Q24 103.3 mm to (120.5, 143.2)
- moved U8 101.8 mm to (222.7, 96.4)
- moved R113 91.9 mm to (116.2, 136.4)
- moved Q26 91.3 mm to (120.5, 136.4)
- moved Q27 82.4 mm to (120.6, 133.0)
- moved R114 81.2 mm to (116.2, 132.9)
- moved Q30 80.9 mm to (120.5, 119.3)
- moved R119 79.5 mm to (116.2, 119.3)
- moved R112 71.0 mm to (116.2, 139.8)
- moved Q25 70.7 mm to (120.6, 139.8)
- moved Q32 70.3 mm to (120.6, 116.0)
- moved Q37 69.4 mm to (120.7, 95.4)
- moved R120 69.1 mm to (116.3, 115.9)
- moved Q29 68.1 mm to (120.5, 122.8)
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Connections:
- U1 pad 17: unconnected-(U1-VDD3P3_CPU-Pad17) -> +3.3V
- U1 pad 18: unconnected-(U1-VDD_SPI-Pad18) -> +3.3V
