File: hardware/greenmobi-bms.kicad_pcb (KiCad board)
At the start: 4 copper layers, 90 x 40 mm, 144 parts, among them J1 BAT+, J10 EXT_NTC, J2 BAT-, J3 Conn_01x02, J4 PACK+, J5 PACK-, J6 USB_C_Receptacle_USB2.0_14P, J7 CAN, J8 Conn_01x17_MountingPin, J9 EXT_NTC, Q1 IPT015N10N5, Q2 IPT015N10N5, Q3 IPT015N10N5, Q4 IPT015N10N5, Q5 IPT015N10N5, Q6 IPT015N10N5, Q7 IPT015N10N5, Q8 IPT015N10N5, U1 TJA1042T-3, U2 ESP32-C3, U3 LM5163DDA, U4 TPS70933, U5 BQ769x2, Y1 40MHz

Commit message: Update PCB
Parts:
- removed C22, C24: 1u, Capacitor_SMD:C_0402_1005Metric
- removed C50, C51: 100n, Capacitor_SMD:C_1210_3225Metric
- removed the R37 at (84.0, 111.6)
- removed the R38 at (84.0, 114.1)
- removed R49: 120, Resistor_SMD:R_0402_1005Metric
- added C25: 1u, Capacitor_SMD:C_0402_1005Metric, F.Cu at (89.8, 128.9)
- added R20: 0.2m, Resistor_SMD:R_Shunt_Vishay_WSR2_WSR3, F.Cu at (65.2, 97.9)
- added R21: 120, Resistor_SMD:R_0402_1005Metric, F.Cu at (59.3, 115.1)
- C23: value 56p -> 1u
- C26: value 47u -> 4.7u; footprint Capacitor_SMD:C_0603_1608Metric -> Capacitor_SMD:C_0805_2012Metric
- C27, C28: value 100n -> 4.7u; footprint Capacitor_SMD:C_0402_1005Metric -> Capacitor_SMD:C_0805_2012Metric
- C29: value 100n -> 470n; footprint Capacitor_SMD:C_0402_1005Metric -> Capacitor_SMD:C_0603_1608Metric
- C30: value 100n -> 100p
- C32: value 100n -> 2.2u; footprint Capacitor_SMD:C_0402_1005Metric -> Capacitor_SMD:C_0603_1608Metric
- C44: value 470n -> 100n; footprint Capacitor_SMD:C_0603_1608Metric -> Capacitor_SMD:C_0402_1005Metric
- C45: value 100p -> 100n
- C47: value 2.2u -> 100n; footprint Capacitor_SMD:C_0603_1608Metric -> Capacitor_SMD:C_0402_1005Metric
- C48, C49: footprint Capacitor_SMD:C_1210_3225Metric -> Capacitor_SMD:C_0402_1005Metric
- R10: value 100k -> 82.5k
- R11: value 316k -> 523k
- R12: value 316k -> 200k
- R13: value 100k -> 63.4k
- R14: value 0 -> 5.1k
- R15: value 10M -> 5.1k
- R16, R17, R18: value 75 -> 5.1k; footprint Capacitor_SMD:C_0603_1608Metric -> Resistor_SMD:R_0402_1005Metric
- R19: value 75 -> 120; footprint Capacitor_SMD:C_0603_1608Metric -> Resistor_SMD:R_0402_1005Metric
- R39: value 75 -> 10M; footprint Capacitor_SMD:C_0603_1608Metric -> Resistor_SMD:R_0402_1005Metric
- R41: value 10M -> 75; footprint Resistor_SMD:R_0402_1005Metric -> Capacitor_SMD:C_0603_1608Metric
- R42, R43, R44, R45, R46: value 5.1k -> 75; footprint Resistor_SMD:R_0402_1005Metric -> Capacitor_SMD:C_0603_1608Metric
- R47: value 120 -> 75; footprint Resistor_SMD:R_0402_1005Metric -> Capacitor_SMD:C_0603_1608Metric
- R48: value 0.2m -> 10M; footprint Resistor_SMD:R_Shunt_Vishay_WSR2_WSR3 -> Resistor_SMD:R_0402_1005Metric
- moved D1 42.2 mm to (82.2, 95.3)
- moved D2 42.2 mm to (82.2, 98.7)
- moved R8 39.6 mm to (59.3, 131.1)
- moved R9 39.6 mm to (59.3, 133.0)
- moved R5 36.4 mm to (59.3, 125.1)
- moved C28 36.2 mm to (83.2, 131.5)
- moved C27 35.3 mm to (83.2, 128.5)
- moved C1 35.1 mm to (96.8, 100.6)
- moved U4 34.5 mm to (78.0, 129.7)
- moved C12 34.2 mm to (65.1, 131.1)
- moved C13 34.2 mm to (65.1, 133.0)
- moved R13 34.1 mm to (86.9, 130.9)
- moved L2 30.0 mm to (59.3, 119.1)
- moved L3 30.0 mm to (59.3, 121.1)
- moved C20 29.9 mm to (89.8, 125.0)
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- renumbered J8 to J10, J9 to J8, J10 to J9, R20 to R22, R21 to R23, R22 to R24, R23 to R25, R24 to R26, R25 to R27, R26 to R28, R27 to R29, R28 to R30, R29 to R31, R30 to R32, R31 to R33, R32 to R34, R33 to R35, R34 to R36, R35 to R37, R36 to R38
Connections:
- C23 pad 1: Net-(C23-Pad1) -> +3.3V
- C23 pad 2: Net-(U3-FB) -> GND
- C26 pad 1: Net-(C26-Pad1) -> +5V
- C27 pad 1: /Frontend/VC16 -> +5V
- C27 pad 2: /Frontend/VC15 -> GND
- C28 pad 1: /Frontend/VC15 -> +5V
- C28 pad 2: /Frontend/VC14 -> GND
- C29 pad 1: /Frontend/VC14 -> /Frontend/BAT+
- C29 pad 2: /Frontend/VC13 -> Net-(U5-CP1)
- C30 pad 1: /Frontend/VC13 -> Net-(U5-SRN)
- C30 pad 2: /Frontend/VC12 -> Net-(U5-SRP)
- C31 pad 1: /Frontend/VC12 -> Net-(U5-SRN)
- C31 pad 2: /Frontend/VC11 -> Net-(U5-SRP)
- C32 pad 1: /Frontend/VC11 -> GND
- C32 pad 2: /Frontend/VC10 -> Net-(U5-REG18)
- C33 pad 1: /Frontend/VC10 -> Net-(U5-VC16)
- C33 pad 2: /Frontend/VC9 -> Net-(U5-VC15)
- C34 pad 1: /Frontend/VC9 -> Net-(U5-VC15)
- C34 pad 2: /Frontend/VC8 -> Net-(U5-VC14)
- C35 pad 1: /Frontend/VC8 -> Net-(U5-VC14)
- C35 pad 2: /Frontend/VC7 -> Net-(U5-VC13)
- C36 pad 1: /Frontend/VC7 -> Net-(U5-VC13)
- C36 pad 2: /Frontend/VC6 -> Net-(U5-VC12)
- C37 pad 1: /Frontend/VC6 -> Net-(U5-VC12)
- C37 pad 2: /Frontend/VC5 -> Net-(U5-VC11)
- C38 pad 1: /Frontend/VC5 -> Net-(U5-VC11)
- C38 pad 2: /Frontend/VC4 -> Net-(U5-VC10)
- C39 pad 1: /Frontend/VC4 -> Net-(U5-VC10)
- C39 pad 2: /Frontend/VC3 -> Net-(U5-VC9)
- C40 pad 1: /Frontend/VC3 -> Net-(U5-VC9)
- C40 pad 2: /Frontend/VC2 -> Net-(U5-VC8)
- C41 pad 1: /Frontend/VC2 -> Net-(U5-VC8)
- C41 pad 2: /Frontend/VC1 -> Net-(U5-VC7)
- C42 pad 1: /Frontend/VC1 -> Net-(U5-VC7)
- C42 pad 2: GND -> Net-(U5-VC6)
- C43 pad 1: /Frontend/VC0 -> Net-(U5-VC6)
- C43 pad 2: GND -> Net-(U5-VC5)
- C44 pad 1: /Frontend/BAT+ -> Net-(U5-VC5)
- C44 pad 2: Net-(U5-CP1) -> Net-(U5-VC4)
- C45 pad 1: Net-(U5-SRN) -> Net-(U5-VC4)
- C45 pad 2: Net-(U5-SRP) -> Net-(U5-VC3)
- C46 pad 1: Net-(U5-SRN) -> Net-(U5-VC3)
- C46 pad 2: Net-(U5-SRP) -> Net-(U5-VC2)
- C47 pad 1: GND -> Net-(U5-VC2)
- C47 pad 2: Net-(U5-REG18) -> Net-(U5-VC1)
- C48 pad 1: /Frontend/Load Switch/BAT+ -> Net-(U5-VC1)
- C48 pad 2: Net-(C48-Pad2) -> GND
- C49 pad 1: Net-(C48-Pad2) -> Net-(U5-VC0)
- C49 pad 2: /Frontend/Load Switch/PACK+ -> GND
- D1 pad 1: /Frontend/Load Switch/DSG -> /Frontend/CHG
- D1 pad 2: /Frontend/Load Switch/PACK+ -> /Frontend/BAT+
- D2 pad 1: /Frontend/Load Switch/CHG -> /Frontend/DSG
- D2 pad 2: /Frontend/Load Switch/BAT+ -> /Frontend/PACK+
- Q1 pad 2: /Frontend/Load Switch/BAT+ -> /Frontend/BAT+
- Q2 pad 2: /Frontend/Load Switch/BAT+ -> /Frontend/BAT+
- Q3 pad 2: /Frontend/Load Switch/BAT+ -> /Frontend/BAT+
- Q4 pad 2: /Frontend/Load Switch/BAT+ -> /Frontend/BAT+
- Q5 pad 2: /Frontend/Load Switch/PACK+ -> /Frontend/PACK+
- Q6 pad 2: /Frontend/Load Switch/PACK+ -> /Frontend/PACK+
- Q7 pad 2: /Frontend/Load Switch/PACK+ -> /Frontend/PACK+
- Q8 pad 2: /Frontend/Load Switch/PACK+ -> /Frontend/PACK+
- R11 pad 2: Net-(C23-Pad1) -> Net-(C22-Pad1)
- R14 pad 1: +5V -> /Frontend/PACK+
- R14 pad 2: Net-(C26-Pad1) -> Net-(R14-Pad2)
- R15 pad 1: /Frontend/Load Switch/BAT+ -> /Frontend/PACK+
- R15 pad 2: /Frontend/Load Switch/CHG -> Net-(R15-Pad2)
- R16 pad 1: Net-(Q1-G) -> GND
- R16 pad 2: /Frontend/Load Switch/CHG -> Net-(U5-RST_SHUT)
- R17 pad 1: Net-(Q2-G) -> Net-(R14-Pad2)
- R17 pad 2: /Frontend/Load Switch/CHG -> Net-(U5-PACK)
- R18 pad 1: Net-(Q3-G) -> Net-(R15-Pad2)
- R18 pad 2: /Frontend/Load Switch/CHG -> Net-(U5-LD)
- R19 pad 1: Net-(Q4-G) -> Net-(U5-SRN)
- R19 pad 2: /Frontend/Load Switch/CHG -> GND
- R22 pad 1: /Frontend/VC16 -> Net-(U5-VC16)
- R23 pad 1: /Frontend/VC15 -> Net-(U5-VC15)
- R24 pad 1: /Frontend/VC14 -> Net-(U5-VC14)
- R25 pad 1: /Frontend/VC13 -> Net-(U5-VC13)
- R26 pad 1: /Frontend/VC12 -> Net-(U5-VC12)
- R27 pad 1: /Frontend/VC11 -> Net-(U5-VC11)
- R28 pad 1: /Frontend/VC10 -> Net-(U5-VC10)
- R29 pad 1: /Frontend/VC9 -> Net-(U5-VC9)
- R30 pad 1: /Frontend/VC8 -> Net-(U5-VC8)
- R31 pad 1: /Frontend/VC7 -> Net-(U5-VC7)
- R32 pad 1: /Frontend/VC6 -> Net-(U5-VC6)
- R33 pad 1: /Frontend/VC5 -> Net-(U5-VC5)
- R34 pad 1: /Frontend/VC4 -> Net-(U5-VC4)
- R35 pad 1: /Frontend/VC3 -> Net-(U5-VC3)
- R36 pad 1: /Frontend/VC2 -> Net-(U5-VC2)
- R37 pad 1: /Frontend/VC1 -> Net-(U5-VC1)
- R38 pad 1: /Frontend/VC0 -> Net-(U5-VC0)
- R39 pad 1: Net-(Q7-G) -> /Frontend/BAT+
- R39 pad 2: /Frontend/Load Switch/DSG -> /Frontend/CHG
- R40 pad 1: Net-(Q8-G) -> Net-(Q1-G)
- R40 pad 2: /Frontend/Load Switch/DSG -> /Frontend/CHG
- R41 pad 1: /Frontend/Load Switch/PACK+ -> Net-(Q2-G)
- R41 pad 2: /Frontend/Load Switch/DSG -> /Frontend/CHG
- R42 pad 1: /Frontend/PACK+ -> Net-(Q3-G)
- R42 pad 2: Net-(R42-Pad2) -> /Frontend/CHG
- R43 pad 1: /Frontend/PACK+ -> Net-(Q4-G)
- R43 pad 2: Net-(R43-Pad2) -> /Frontend/CHG
- R44 pad 1: GND -> Net-(Q5-G)
- R44 pad 2: Net-(U5-RST_SHUT) -> /Frontend/DSG
- R45 pad 1: Net-(R42-Pad2) -> Net-(Q6-G)
- R45 pad 2: Net-(U5-PACK) -> /Frontend/DSG
- R46 pad 1: Net-(R43-Pad2) -> Net-(Q7-G)
- R46 pad 2: Net-(U5-LD) -> /Frontend/DSG
- R47 pad 1: Net-(U5-SRN) -> Net-(Q8-G)
- R47 pad 2: GND -> /Frontend/DSG
- R48 pad 1: GND -> /Frontend/PACK+
- R48 pad 2: /Frontend/BAT- -> /Frontend/DSG
- U3 pad 3: /Frontend/BAT+ -> /Power Supply/EN
- U5 pad 1: /Frontend/VC15 -> Net-(U5-VC15)
- U5 pad 10: /Frontend/VC6 -> Net-(U5-VC6)
- U5 pad 11: /Frontend/VC5 -> Net-(U5-VC5)
- U5 pad 12: /Frontend/VC4 -> Net-(U5-VC4)
- U5 pad 13: /Frontend/VC3 -> Net-(U5-VC3)
- U5 pad 14: /Frontend/VC2 -> Net-(U5-VC2)
- U5 pad 15: /Frontend/VC1 -> Net-(U5-VC1)
- U5 pad 16: /Frontend/VC0 -> Net-(U5-VC0)
- U5 pad 2: /Frontend/VC15 -> Net-(U5-VC14)
- U5 pad 3: /Frontend/VC13 -> Net-(U5-VC13)
- U5 pad 4: /Frontend/VC12 -> Net-(U5-VC12)
- U5 pad 48: /Frontend/VC16 -> Net-(U5-VC16)
- U5 pad 5: /Frontend/VC11 -> Net-(U5-VC11)
- U5 pad 6: /Frontend/VC10 -> Net-(U5-VC10)
- U5 pad 7: /Frontend/VC9 -> Net-(U5-VC9)
- U5 pad 8: /Frontend/VC8 -> Net-(U5-VC8)
- U5 pad 9: /Frontend/VC7 -> Net-(U5-VC7)

Commit message: Enable logic
Parts:
- added Q9: MMBT3904, Package_TO_SOT_SMD:SOT-23, F.Cu at (141.9, 86.3)
Connections:
- net Net-(Q1-D) renamed /Frontend/FET_C
- U5 pad 34: GND -> unconnected-(U5-REG2-Pad34)
- U5 pad 35: GND -> unconnected-(U5-REG1-Pad35)
- U5 pad 36: GND -> unconnected-(U5-REGIN-Pad36)
- U5 pad 37: GND -> unconnected-(U5-BREG-Pad37)

Commit message: Automotive fuse
Parts:
- removed J1: BAT+, TestPoint:TestPoint_Pad_4.0x4.0mm
- removed J4: PACK+, TestPoint:TestPoint_Pad_4.0x4.0mm
- removed Q9: MMBT3904, Package_TO_SOT_SMD:SOT-23
- added D3: 1N4148W, Diode_SMD:D_SOD-123, F.Cu at (164.6, 138.1)
- added H1: Fuse, greenmobi-bms:Automotive_Fuse, F.Cu at (187.1, 94.7)
- added H2: Fuse, greenmobi-bms:Automotive_Fuse, F.Cu at (158.8, 94.5)
- added R50: 5.1k, Resistor_SMD:R_0402_1005Metric, F.Cu at (163.1, 140.8)
- added R51: 5.1k, Resistor_SMD:R_0402_1005Metric, F.Cu at (163.1, 142.8)
- added R52: 5.1k, Resistor_SMD:R_0402_1005Metric, F.Cu at (158.2, 137.5)
- J3: value Conn_01x02 -> EN; footprint Connector_PinHeader_1.00mm:PinHeader_1x02_P1.00mm_Vertical -> Connector_JST:JST_GH_SM02B-GHS-TB_1x02-1MP_P1.25mm_Horizontal
- moved Q2 4.50 mm to (164.4, 120.6)
- moved Q3 4.50 mm to (175.5, 120.6)
- moved Q6 4.50 mm to (164.4, 106.5)
- moved Q7 4.50 mm to (175.6, 106.5)
- moved Q1 4.50 mm to (153.2, 120.7)
- moved Q4 4.50 mm to (186.7, 120.6)
- moved Q5 4.50 mm to (153.2, 106.5)
- moved Q8 4.50 mm to (186.7, 106.5)
Connections:
- C1 pad 1: /MCU/EN -> /Frontend/Shutdown
- J3 pad 2: /MCU/EN -> /Frontend/Shutdown
- R8 pad 2: /MCU/EN -> Net-(U2-GPIO2)
- U2 pad 6: /MCU/EN -> Net-(U2-GPIO2)
- U3 pad 3: /Power Supply/EN -> /Frontend/Shutdown
- U5 pad 22: unconnected-(U5-TS2-Pad22) -> Net-(U5-TS2)
- U5 pad 34: unconnected-(U5-REG2-Pad34) -> GND
- U5 pad 35: unconnected-(U5-REG1-Pad35) -> GND
- U5 pad 36: unconnected-(U5-REGIN-Pad36) -> GND
- U5 pad 37: unconnected-(U5-BREG-Pad37) -> GND

Commit message: BAT connector change
Parts:
- removed J2: BAT-, TestPoint:TestPoint_Pad_4.0x4.0mm
- removed J5: PACK-, TestPoint:TestPoint_Pad_4.0x4.0mm
- added C21: 2.2n, Capacitor_SMD:C_0402_1005Metric, F.Cu at (94.9, 154.7)
- added C50: 100n, Capacitor_SMD:C_1206_3216Metric, F.Cu at (96.3, 136.6)
- added C51: 100n, Capacitor_SMD:C_1206_3216Metric, F.Cu at (96.3, 139.9)
- added C52: 100n, Capacitor_SMD:C_1206_3216Metric, F.Cu at (96.3, 143.3)
- added C53: 100n, Capacitor_SMD:C_1206_3216Metric, F.Cu at (96.3, 146.7)
- added C56: 100n, Capacitor_SMD:C_0402_1005Metric, F.Cu at (94.9, 158.6)
- added C57: 100n, Capacitor_SMD:C_0402_1005Metric, F.Cu at (94.9, 160.6)
- added C58: 2.2u, Capacitor_SMD:C_1206_3216Metric, F.Cu at (96.3, 152.0)
- added H3: BAT-, greenmobi-bms:Automotive_Fuse, F.Cu at (175.2, 141.6)
- added H4: PACK-, greenmobi-bms:Automotive_Fuse, F.Cu at (198.4, 141.5)
- added H5: PACK+, greenmobi-bms:Automotive_Fuse, F.Cu at (196.9, 94.5)
- H2: value Fuse -> BAT+
- Q1, Q2, Q3, Q4, Q5, Q6, Q7, Q8: footprint Package_TO_SOT_SMD:Infineon_PG-HSOF-8-1 -> Package_TO_SOT_SMD:Infineon_PG-HSOF-8-1_ThermalVias
- moved R20 129.2 mm to (186.8, 141.6), turned to 180 degrees
- moved AE3 50.5 mm to (127.0, 145.1), turned to 180 degrees
- moved H1 45.2 mm to (161.8, 132.1)
- moved J6 35.0 mm to (106.4, 137.2), turned to -90 degrees
- moved D3 28.3 mm to (136.3, 138.8)
- moved U3 23.2 mm to (79.0, 139.9)
- moved R51 20.0 mm to (143.2, 140.1)
- moved R50 20.0 mm to (143.2, 138.2)
- moved R52 20.0 mm to (138.3, 134.8)
- moved C19 16.3 mm to (71.9, 140.7), turned to 90 degrees
- moved J3 16.0 mm to (130.2, 126.7), turned to 0 degrees
- moved Q1 11.3 mm to (164.6, 120.2)
- moved Q5 11.3 mm to (164.6, 106.3)
- moved Q6 10.8 mm to (175.2, 106.4)
- moved Q2 10.7 mm to (175.2, 120.2)
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Connections:
- H2 pad 1: Net-(J1-Pin_1) -> unconnected-(H2-Pad1)
- J10 pad 17: /Frontend/CEL_0 -> GND
- R19 pad 2: GND -> /Frontend/PACK-
- R20 pad 1: GND -> /Frontend/PACK-
- R20 pad 2: /Frontend/BAT- -> GND
- R21 pad 2: /Frontend/BAT- -> GND
- R38 pad 2: /Frontend/CEL_0 -> GND
Routing:
- added copper zone on B.Cu, net /Frontend/FET_C
- added copper zone on F.Cu, net /Frontend/FET_C
- added copper zone on In1.Cu, net /Frontend/FET_C
- added copper zone on In2.Cu, net /Frontend/FET_C
Other:
- board size 90 x 40 mm -> 100 x 62.3 mm

Commit message: Replace Front end input diode for a Schotky
Parts:
- moved H5 16.6 mm to (180.4, 94.7)
- moved H2 3.61 mm to (150.4, 94.7)
Connections:
- H3 pad 1: GND -> /Frontend/CEL_0
- H4 pad 1: /Frontend/PACK- -> GND
- J10 pad 17: GND -> /Frontend/CEL_0
- R19 pad 2: /Frontend/PACK- -> GND
- R20 pad 1: /Frontend/PACK- -> GND
- R20 pad 2: GND -> /Frontend/CEL_0
- R21 pad 2: GND -> /Frontend/CEL_0
- R38 pad 2: GND -> /Frontend/CEL_0
Changed lines of the file:
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@@
 	(net 121 "Net-(R50-Pad2)")
 	(net 122 "Net-(U5-TS2)")
-	(net 123 "/Frontend/PACK-")
+	(net 123 "/Frontend/CEL_0")
 	(net 124 "unconnected-(H2-Pad1)")
 	(footprint "Inductor_SMD:L_0402_1005Metric"
@@
 			(layers "F.Cu" "F.Mask" "F.Paste")
 			(roundrect_rratio 0.222222)
-			(net 2 "GND")
+			(net 123 "/Frontend/CEL_0")
 			(pintype "passive")
 		)
@@
 			(layers "F.Cu" "F.Mask" "F.Paste")
 			(roundrect_rratio 0.25)
-			(net 2 "GND")
+			(net 123 "/Frontend/CEL_0")
 			(pinfunction "Pin_17")
 			(pintype "passive")
@@
 			(layers "*.Cu" "*.Mask")
 			(remove_unused_layers no)
-			(net 2 "GND")
+			(net 123 "/Frontend/CEL_0")
 			(pinfunction "1")
 			(pintype "input")
@@
 	(footprint "greenmobi-bms:Automotive_Fuse"
 		(layer "F.Cu")
-		(at 153.95 94.05)
+		(at 150.4 94.7)
 		(descr "Mounting Hole 6.5mm")
 		(tags "mounting hole 6.5mm")
@@
 			(layers "*.Cu" "*.Mask")
 			(remove_unused_layers no)
-			(net 123 "/Frontend/PACK-")
+			(net 2 "GND")
 			(pinfunction "1")
 			(pintype "input")
@@
 			(size 3.94 5.84)
 			(layers "F.Cu" "F.Mask" "F.Paste")
-			(net 123 "/Frontend/PACK-")
+			(net 2 "GND")
 			(pintype "passive")
 		)
@@
 			(size 3.94 5.84)
 			(layers "F.Cu" "F.Mask" "F.Paste")
-			(net 2 "GND")
+			(net 123 "/Frontend/CEL_0")
 			(pintype "passive")
 		)
@@
 	(footprint "greenmobi-bms:Automotive_Fuse"
 		(layer "F.Cu")
-		(at 196.95 94.5)
+		(at 180.4 94.7)
 		(descr "Mounting Hole 6.5mm")
 		(tags "mounting hole 6.5mm")
@@
 			(layers "F.Cu" "F.Mask" "F.Paste")
 			(roundrect_rratio 0.25)
-			(net 123 "/Frontend/PACK-")
+			(net 2 "GND")
 			(pintype "passive")
 		)
@@
 			(layers "F.Cu" "F.Mask" "F.Paste")
 			(roundrect_rratio 0.25)
-			(net 2 "GND")
+			(net 123 "/Frontend/CEL_0")
 			(pintype "passive")
 		)

Commit message: package sizes set and AFE layout
Parts:
- removed D3: 1N4148W, Diode_SMD:D_SOD-123
- added C22: 100p, Capacitor_SMD:C_0603_1608Metric, F.Cu at (76.7, 96.4)
- added C24: 1.5n, Capacitor_SMD:C_0603_1608Metric, F.Cu at (76.7, 98.9)
- added C54: 1u, Capacitor_SMD:C_1206_3216Metric, F.Cu at (83.5, 110.6)
- added C55: 100p, Capacitor_SMD:C_0603_1608Metric, F.Cu at (91.3, 111.4)
- added D4: 1N5819WS, Diode_SMD:D_SOD-323, F.Cu at (95.5, 106.6)
- added R49: 120, Resistor_SMD:R_0402_1005Metric, F.Cu at (93.7, 100.2)
- J6: value USB_C_Receptacle_USB2.0_14P -> USB
- moved H4 91.3 mm to (107.3, 136.1), turned to 180 degrees
- moved J6 75.7 mm to (140.3, 69.5)
- moved R20 68.2 mm to (118.9, 136.1), turned to 0 degrees
- moved U1 64.5 mm to (146.0, 130.9), turned to -90 degrees
- moved R50 61.2 mm to (93.7, 102.1)
- moved R51 61.2 mm to (93.7, 104.1)
- moved C58 57.3 mm to (71.9, 100.2)
- moved AE3 56.5 mm to (135.6, 89.2), turned to 0 degrees
- moved C56 53.1 mm to (87.9, 106.0)
- moved C57 53.1 mm to (87.9, 108.0)
- moved C21 51.6 mm to (76.7, 106.4)
- moved R52 47.6 mm to (92.1, 123.6)
- moved H3 45.1 mm to (130.4, 136.1), turned to 180 degrees
- moved C19 43.8 mm to (71.9, 96.8), turned to 0 degrees
- moved R21 38.3 mm to (93.7, 98.2)
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Connections:
- C50 pad 1: /Frontend/BAT+ -> /Frontend/BAT_F
- D1 pad 2: /Frontend/BAT+ -> /Frontend/BAT_F
- H3 pad 1: /Frontend/CEL_0 -> /Frontend/BAT-
- J3 pad 1: GND -> /Frontend/Shutdown
- J3 pad 2: /Frontend/Shutdown -> GND
- J3 pad MP: (no net) -> GND
- J6 pad A8: (no net) -> unconnected-(J6-SBU1-PadA8)
- J6 pad B8: (no net) -> unconnected-(J6-SBU2-PadB8)
- J7 pad 1: Net-(J7-Pin_1) -> /CAN-
- J7 pad 2: Net-(J7-Pin_2) -> /CAN+
- Q1 pad 2: /Frontend/BAT+ -> /Frontend/BAT_F
- Q2 pad 2: /Frontend/BAT+ -> /Frontend/BAT_F
- Q3 pad 2: /Frontend/BAT+ -> /Frontend/BAT_F
- Q4 pad 2: /Frontend/BAT+ -> /Frontend/BAT_F
- R20 pad 2: /Frontend/CEL_0 -> /Frontend/BAT-
- R21 pad 2: /Frontend/CEL_0 -> /Frontend/BAT-
- R3 pad 1: Net-(J7-Pin_1) -> /CAN+
- R3 pad 2: Net-(J7-Pin_2) -> /CAN-
- R39 pad 1: /Frontend/BAT+ -> /Frontend/BAT_F
- U1 pad 6: Net-(J7-Pin_2) -> /CAN-
- U1 pad 7: Net-(J7-Pin_1) -> /CAN+
Routing:
- net Net-(U5-VC0): track 0.00 -> 20.0 mm
- net Net-(U5-VC1): track 0.00 -> 17.5 mm
- net Net-(U5-VC2): track 0.00 -> 15.0 mm
- net Net-(U5-VC16): track 0.00 -> 14.9 mm
- net Net-(U5-VC15): track 0.00 -> 12.9 mm
- net Net-(U5-VC3): track 0.00 -> 12.1 mm
- net Net-(U5-VC14): track 0.00 -> 11.4 mm
- net Net-(U5-VC4): track 0.00 -> 11.3 mm
- net Net-(U5-VC13): track 0.00 -> 9.63 mm
- net Net-(U5-VC5): track 0.00 -> 9.55 mm
- net Net-(U5-VC12): track 0.00 -> 7.89 mm
- net Net-(U5-VC6): track 0.00 -> 7.81 mm
- net Net-(U5-VC11): track 0.00 -> 6.16 mm
- net Net-(U5-VC7): track 0.00 -> 6.09 mm
- net Net-(U5-VC10): track 0.00 -> 4.42 mm
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Other:
- board size 100 x 62.3 mm -> 100 x 58.8 mm

Commit message: Change MCU footprint to GND vias on EPAD
Parts:
- U2: footprint Package_DFN_QFN:QFN-32-1EP_5x5mm_P0.5mm_EP3.7x3.7mm -> Package_DFN_QFN:QFN-32-1EP_5x5mm_P0.5mm_EP3.7x3.7mm_ThermalVias
- moved TP5 58.0 mm to (81.5, 83.6)
- moved TP7 58.0 mm to (81.5, 89.7)
- moved TP6 58.0 mm to (81.5, 86.7)
- moved TP1 58.0 mm to (78.5, 86.7)
- moved TP10 58.0 mm to (78.5, 89.7)
- moved TP2 58.0 mm to (84.6, 83.6)
- moved TP3 58.0 mm to (84.6, 86.7)
- moved TP4 58.0 mm to (84.6, 89.7)
- moved TP8 58.0 mm to (78.5, 83.6)
- moved TP12 58.0 mm to (87.5, 89.4)

Commit message: ESP32 layout
Parts:
- removed AE1: Calib, Connector_Coaxial:U.FL_Hirose_U.FL-R-SMT-1_Vertical
- removed C12, C18: 100p, Capacitor_SMD:C_0402_1005Metric
- removed TP9: TestPoint, TestPoint:TestPoint_Pad_D1.0mm
- TP11: footprint TestPoint:TestPoint_Pad_D1.0mm -> TestPoint:TestPoint_Pad_1.0x1.0mm
- moved L3 83.5 mm to (143.0, 135.0), turned to -90 degrees
- moved C13 75.8 mm to (142.5, 133.6), turned to 180 degrees
- moved C15 73.7 mm to (142.5, 136.4), turned to 180 degrees
- moved AE2 70.7 mm to (138.6, 138.2), turned to 180 degrees
- moved J7 64.5 mm to (164.9, 76.6), turned to 180 degrees
- moved J3 61.9 mm to (156.4, 76.5), turned to 180 degrees
- moved AE3 53.2 mm to (142.2, 142.0), turned to 180 degrees
- moved U1 50.6 mm to (164.9, 83.9), turned to 90 degrees
- moved C17 49.2 mm to (143.0, 137.8), turned to 90 degrees
- moved D4 31.5 mm to (123.1, 91.4), turned to 180 degrees
- moved U2 30.1 mm to (144.8, 129.7), turned to 90 degrees
- moved L1 26.3 mm to (140.6, 130.6), turned to 0 degrees
- moved C6 25.3 mm to (138.3, 131.9), turned to 180 degrees
- moved Y1 22.7 mm to (138.1, 129.6), turned to -90 degrees
- moved C4 20.3 mm to (137.8, 127.3), turned to 0 degrees
Connections:
- C13 pad 1: Net-(C12-Pad1) -> Net-(U2-LNA_IN)
- L3 pad 1: Net-(C12-Pad1) -> Net-(U2-LNA_IN)
Other:
- outline, holes or cut-outs redrawn
