File: hardware/greenmobi-bms.kicad_pcb (KiCad board)
At the start: 4 copper layers, 90 x 50 mm, 150 parts, among them J10 Conn_01x17_MountingPin, J3 EN, J6 USB, J7 CAN, J8 EXT_NTC, J9 EXT_NTC, Q1 IPT015N10N5, Q2 IPT015N10N5, Q3 IPT015N10N5, Q5 IPT015N10N5, Q6 IPT015N10N5, Q7 IPT015N10N5, U1 TJA1042T-3, U2 ESP32-C3, U3 LM5163DDA, U4 TPS70933, U5 BQ769x2, Y1 40MHz

Commit message: First Layout placement
Parts:
- removed C30: 100p, Capacitor_SMD:C_0402_1005Metric
- removed C56, C57: 100n, Capacitor_SMD:C_0402_1005Metric
- removed R14, R15, R50: 5.1k, Resistor_SMD:R_0402_1005Metric
- AE3: footprint RF_Antenna:Texas_SWRA117D_2.4GHz_Left -> RF_Antenna:Texas_SWRA117D_2.4GHz_Right
- R40, R41, R42, R44, R45, R46: footprint Capacitor_SMD:C_0603_1608Metric -> Capacitor_SMD:C_0402_1005Metric
- moved R44 112.8 mm to (192.9, 99.6), turned to -90 degrees
- moved R45 111.1 mm to (192.9, 110.1), turned to -90 degrees
- moved R46 109.9 mm to (192.9, 120.7), turned to -90 degrees
- moved C51 108.1 mm to (187.0, 122.5)
- moved R4 92.1 mm to (153.0, 124.0), turned to -90 degrees
- moved C50 89.8 mm to (168.6, 122.6)
- moved C2 89.2 mm to (153.0, 126.0), turned to -90 degrees
- moved R40 85.1 mm to (164.2, 90.2), turned to 90 degrees
- moved D1 83.7 mm to (159.3, 108.5)
- moved C52 83.2 mm to (161.9, 120.3)
- moved R41 82.8 mm to (164.2, 100.8), turned to 90 degrees
- moved D2 82.6 mm to (159.7, 117.9)
- moved R42 81.3 mm to (164.2, 111.3), turned to 90 degrees
- moved C53 78.8 mm to (157.3, 120.3)
- moved R6 77.5 mm to (135.7, 105.3), turned to 135 degrees
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Connections:
- C29 pad 1: /Frontend/BAT_F -> Net-(U5-BAT)
- C54 pad 1: /Frontend/BAT_F -> Net-(U5-BAT)
- C55 pad 1: /Frontend/BAT_F -> Net-(U5-BAT)
- R17 pad 1: Net-(R14-Pad2) -> /Frontend/PACK+
- R18 pad 1: Net-(R15-Pad2) -> /Frontend/PACK+
- R49 pad 1: /Frontend/BAT_F -> Net-(U5-BAT)
- R51 pad 1: Net-(R50-Pad2) -> /Frontend/Shutdown
- U5 pad 47: /Frontend/BAT_F -> Net-(U5-BAT)
Routing:
- net /USB_DP: track 0.00 -> 14.0 mm
- net /USB_DN: track 0.00 -> 13.6 mm
- net Net-(AE3-A): track 0.00 -> 10.7 mm
- net Net-(U5-VC3): track 0.00 -> 1.47 mm
- net Net-(U5-VC4): track 0.00 -> 1.39 mm
- removed copper zone on In1.Cu, net /Frontend/FET_C
- removed copper zone on In2.Cu, net /Frontend/FET_C
- removed copper zone on In1.Cu, net GND
Other:
- outline, holes or cut-outs redrawn
- copper layers 4 -> 2

Commit message: heatsink interface
Parts:
- removed TP1, TP10, TP2: TestPoint, TestPoint:TestPoint_Pad_D1.0mm
- moved C14 0.14 mm to (128.0, 97.5)
- moved C10 0.14 mm to (126.0, 96.1)
- moved C11 0.14 mm to (126.7, 96.8)
- moved C16 0.14 mm to (126.6, 98.9)
- moved L2 0.14 mm to (127.3, 98.1)
Connections:
- R16 pad 1: GND -> unconnected-(R16-Pad1)
- R16 pad 2: Net-(U5-RST_SHUT) -> unconnected-(R16-Pad2)

Commit message: Remove U.fL connector and improve layout
Parts:
- removed AE2: Calib, Connector_Coaxial:U.FL_Hirose_U.FL-R-SMT-1_Vertical
- removed C17: 100p, Capacitor_SMD:C_0402_1005Metric
- removed TP11: TestPoint, greenmobi-bms:TestPoint_Pad_0.55x0.62mm
- moved L2 5.19 mm to (125.7, 93.2)
- moved C10 4.87 mm to (123.6, 91.9), turned to -135 degrees
- moved C11 4.84 mm to (124.3, 92.6), turned to -135 degrees
- moved C5 4.00 mm to (131.5, 100.4)
- moved Y1 4.00 mm to (134.2, 92.6)
- moved C16 4.00 mm to (125.0, 95.3)
- moved C9 4.00 mm to (126.0, 99.7)
- moved L3 4.00 mm to (126.8, 92.3)
- moved C4 4.00 mm to (135.9, 94.1)
- moved C8 4.00 mm to (130.8, 92.8)
- moved C7 4.00 mm to (130.1, 92.2)
- moved R5 4.00 mm to (132.6, 103.1)
- moved R9 4.00 mm to (127.2, 101.7)
- moved C13 4.00 mm to (128.2, 93.0)
- moved C15 4.00 mm to (126.2, 91.0)
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Connections:
- net Net-(U2-LNA_IN) renamed /MCU/MCU_CLC
- AE3 pad 1: Net-(AE3-A) -> /MCU/Ant_CLC
- C15 pad 1: Net-(C15-Pad1) -> /MCU/Ant_CLC
- L3 pad 2: Net-(C15-Pad1) -> /MCU/Ant_CLC
Routing:
- net +5V: track 0.00 -> 11.0 mm, vias 0 -> 2
- net Net-(AE3-A): track 10.7 -> 0.00 mm
- net /MCU/Ant_CLC: track 0.00 -> 9.36 mm
- net /USB_DN: track 13.6 -> 18.3 mm
- net /USB_DP: track 14.0 -> 18.7 mm
- net +3.3V: track 0.00 -> 4.53 mm
- net /MCU/VDD_RF: track 0.00 -> 3.45 mm
- net /MCU/MCU_CLC: track 0.00 -> 2.41 mm
- net GND: track 1.60 -> 3.72 mm, vias 2 -> 42
- added copper zone on F.Cu, net +5V

Commit message: Zone fills
Parts:
- removed C52, C53: 100n, Capacitor_SMD:C_1206_3216Metric
- removed D4: 1N5819WS, Diode_SMD:D_SOD-323
- added kibuzzard-6861C75B: G***, kibuzzard-6861C75B, F.Cu at (125.4, 110.7)
- moved D1 18.2 mm to (153.5, 91.2)
- moved R40 18.2 mm to (153.5, 92.9)
- moved R47 2.29 mm to (159.4, 119.7)
- moved R23 0.20 mm to (121.6, 94.7)
- moved R28 0.20 mm to (121.6, 106.3)
- moved R33 0.20 mm to (121.6, 117.8)
- moved R38 0.20 mm to (121.6, 129.4)
- moved R39 0.20 mm to (121.6, 131.8)
- moved R24 0.20 mm to (121.6, 97.0)
- moved R25 0.20 mm to (121.6, 99.3)
- moved R26 0.20 mm to (121.6, 101.6)
- moved R27 0.20 mm to (121.6, 103.9)
- moved R29 0.20 mm to (121.6, 108.6)
- moved R30 0.20 mm to (121.6, 110.9)
- moved R31 0.20 mm to (121.6, 113.2)
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- renumbered AE3 to AE1, C13 to C12, C14 to C13, C15 to C14, C16 to C15, C58 to C16, C19 to C17, C20 to C18, C21 to C19, C22 to C20, C23 to C21, C24 to C22, C25 to C23, C26 to C24, C27 to C25, C28 to C26, C29 to C27, C31 to C28, C32 to C29, C55 to C30, C54 to C31, C33 to C32, C34 to C33, C35 to C34, C36 to C35, C37 to C36, C38 to C37, C39 to C38, C40 to C39, C41 to C40, C42 to C41, C43 to C42, C44 to C43, C45 to C44, C46 to C45, C47 to C46, C48 to C47, C49 to C48, C50 to C49, C51 to C50, H2 to H1, H1 to H2, H5 to H4, H4 to H5, J3 to J1, J6 to J2, J7 to J3, J8 to J4, J9 to J5, J10 to J6, Q5 to Q4, Q6 to Q5, Q7 to Q6, R52 to R1, R9 to R10, R10 to R11, R11 to R12, R12 to R13, R13 to R14, R51 to R15, R1 to R2, R49 to R22, R22 to R23, R23 to R24, R24 to R25, R25 to R26, R26 to R27, R27 to R28, R28 to R29, R2 to R3, R29 to R30, R30 to R31, R31 to R32, R32 to R33, R33 to R34, R34 to R35, R35 to R36, R36 to R37, R37 to R38, R38 to R39, R3 to R4, R39 to R40, R40 to R41, R41 to R42, R42 to R43, R48 to R47, R4 to R5, R5 to R6, R6 to R7, R7 to R8, R8 to R9, TP3 to TP1, TP4 to TP2, TP5 to TP3, TP6 to TP4, TP7 to TP5, TP8 to TP6, TP12 to TP7
Connections:
- R22 pad 2: Net-(D4-K) -> /Frontend/CEL_16
Routing:
- net /Frontend/CEL_16: track 0.00 -> 9.85 mm
- net GND: track 3.72 -> 13.4 mm
- net /Frontend/CEL_15: track 0.00 -> 9.14 mm
- net /Frontend/CEL_1: track 0.00 -> 9.07 mm
- net /Frontend/CEL_14: track 0.00 -> 8.22 mm
- net /Frontend/CEL_2: track 0.00 -> 8.03 mm
- net /Frontend/CEL_13: track 0.00 -> 7.23 mm
- net /Frontend/CEL_3: track 0.00 -> 7.15 mm
- net /Frontend/CEL_12: track 0.00 -> 6.14 mm
- net /Frontend/CEL_4: track 0.00 -> 6.08 mm
- net /Frontend/CEL_11: track 0.00 -> 5.32 mm
- net /Frontend/CEL_5: track 0.00 -> 5.24 mm
- net /Frontend/BAT_F: track 0.00 -> 4.85 mm
- net /Frontend/CEL_6: track 0.00 -> 4.18 mm
- net /Frontend/CEL_10: track 0.00 -> 3.85 mm
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- added copper zone on F.Cu, net /Frontend/BAT-
- added copper zone on F.Cu, net /Frontend/BAT_F
- added copper zone on F.Cu, net /Frontend/PACK+
- added copper zone on F.Cu, net /Frontend/PACK-
- added copper zone on F.Cu, net Net-(C49-Pad2)
- added copper zone on F.Cu, net Net-(U3-SW)
Other:
- board text added: "<<hash>>"

Commit message: PCB work
Parts:
- moved C11 1.55 mm to (125.0, 93.9), turned to -45 degrees
- moved C15 0.61 mm to (125.1, 95.9), turned to -135 degrees
- moved C10 0.59 mm to (123.8, 92.4), turned to 180 degrees
Routing:
- net GND: track 13.4 -> 13.9 mm, vias 42 -> 44

Commit message: Fix connection
Parts:
- moved H2 0.71 mm to (159.0, 98.0)
- moved H1 0.71 mm to (159.0, 128.0)
Connections:
- R16 pad 1: unconnected-(R16-Pad1) -> GND
- R16 pad 2: unconnected-(R16-Pad2) -> Net-(U5-RST_SHUT)

Commit message: Change product label
Parts:
- removed kibuzzard-6861C75B: G***, kibuzzard-6861C75B
- added kibuzzard-688328D2: G***, kibuzzard-688328D2, F.Cu at (125.4, 110.7)
Routing:
- net /Frontend/CEL_5: track 5.24 -> 4.56 mm

Commit message: Changed to charge only BMS
Parts:
- removed D2: BZT52Bxx, Diode_SMD:D_SOD-123F
- removed Q2, Q3, Q4, Q5, Q6: IPT015N10N5, Package_TO_SOT_SMD:Infineon_PG-HSOF-8-1_ThermalVias
- removed R42, R43, R44, R45, R46: 75, Capacitor_SMD:C_0402_1005Metric
- removed R47: 10M, Resistor_SMD:R_0402_1005Metric
- added F1: 20A, Fuse:Fuse_Littelfuse-NANO2-451_453, F.Cu at (180.4, 82.0)
- added H6: MountingHole_Pad, MountingHole:MountingHole_3.2mm_M3_Pad, F.Cu at (213.4, 72.0)
- added H7: MountingHole_Pad, MountingHole:MountingHole_3.2mm_M3_Pad, F.Cu at (213.4, 80.0)
- added H8: MountingHole_Pad, MountingHole:MountingHole_3.2mm_M3_Pad, F.Cu at (213.4, 87.9)
- added JP1: Cell_shunt, Jumper:SolderJumper-2_P1.3mm_Open_Pad1.0x1.5mm, B.Cu at (116.6, 102.2)
- added JP10: Cell_shunt, Jumper:SolderJumper-2_P1.3mm_Open_Pad1.0x1.5mm, B.Cu at (190.4, 123.0)
- added JP11: Cell_shunt, Jumper:SolderJumper-2_P1.3mm_Open_Pad1.0x1.5mm, B.Cu at (108.3, 104.6)
- added JP12: Cell_shunt, Jumper:SolderJumper-2_P1.3mm_Open_Pad1.0x1.5mm, B.Cu at (116.6, 106.4)
- added JP13: Cell_shunt, Jumper:SolderJumper-2_P1.3mm_Open_Pad1.0x1.5mm, B.Cu at (191.5, 92.4)
- added JP2: Cell_shunt, Jumper:SolderJumper-2_P1.3mm_Open_Pad1.0x1.5mm, B.Cu at (116.6, 105.7)
- added JP3: Cell_shunt, Jumper:SolderJumper-2_P1.3mm_Open_Pad1.0x1.5mm, B.Cu at (116.6, 109.3)
- added JP4: Cell_shunt, Jumper:SolderJumper-2_P1.3mm_Open_Pad1.0x1.5mm, B.Cu at (116.6, 112.8)
- added JP5: Cell_shunt, Jumper:SolderJumper-2_P1.3mm_Open_Pad1.0x1.5mm, B.Cu at (116.6, 116.4)
- added JP6: Cell_shunt, Jumper:SolderJumper-2_P1.3mm_Open_Pad1.0x1.5mm, B.Cu at (176.2, 123.0)
- added JP7: Cell_shunt, Jumper:SolderJumper-2_P1.3mm_Open_Pad1.0x1.5mm, B.Cu at (179.7, 123.0)
- added JP8: Cell_shunt, Jumper:SolderJumper-2_P1.3mm_Open_Pad1.0x1.5mm, B.Cu at (183.3, 123.0)
- added JP9: Cell_shunt, Jumper:SolderJumper-2_P1.3mm_Open_Pad1.0x1.5mm, B.Cu at (186.8, 123.0)
- AE1: footprint RF_Antenna:Texas_SWRA117D_2.4GHz_Right -> RF_Antenna:Texas_SWRA117D_2.4GHz_Left
- H1, H3: footprint greenmobi-bms:Automotive_Fuse -> Connector_Wire:SolderWire-2sqmm_1x01_D2mm_OD3.9mm
- H2: value Fuse -> MountingHole_Pad; footprint greenmobi-bms:Automotive_Fuse -> MountingHole:MountingHole_3.2mm_M3_Pad
- H4: value PACK+ -> CHG+; footprint greenmobi-bms:Automotive_Fuse -> Connector_Wire:SolderWire-2sqmm_1x01_D2mm_OD3.9mm
- H5: value PACK- -> CHG-; footprint greenmobi-bms:Automotive_Fuse -> Connector_Wire:SolderWire-2sqmm_1x01_D2mm_OD3.9mm
- R20: footprint Resistor_SMD:R_Shunt_Vishay_WSR2_WSR3 -> Resistor_SMD:R_1206_3216Metric
- moved J5 82.5 mm to (198.0, 129.4), turned to 0 degrees
- moved AE1 80.2 mm to (197.6, 88.5)
- moved R39 78.8 mm to (200.0, 123.2), turned to -90 degrees
- moved R38 76.3 mm to (197.7, 123.2), turned to -90 degrees
- moved R37 73.8 mm to (195.4, 123.2), turned to -90 degrees
- moved C10 73.4 mm to (197.2, 91.6), turned to 135 degrees
- moved C14 72.6 mm to (198.7, 93.5), turned to -45 degrees
- moved R36 71.4 mm to (193.0, 123.2), turned to -90 degrees
- moved L2 70.8 mm to (196.5, 93.0), turned to -135 degrees
- moved C11 70.8 mm to (195.8, 92.3), turned to -135 degrees
- moved L3 70.6 mm to (197.4, 94.1), turned to 45 degrees
- moved R35 69.1 mm to (190.7, 123.2), turned to -90 degrees
- moved C15 68.8 mm to (193.8, 92.4), turned to 135 degrees
- moved C13 68.7 mm to (195.1, 93.7), turned to 135 degrees
- moved C12 68.6 mm to (196.8, 95.4), turned to -45 degrees
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Connections:
- net /Frontend/PACK- renamed /Frontend/CHG-
- C16 pad 2: /Frontend/BAT_F -> /Frontend/BAT+
- C17 pad 1: /Frontend/BAT_F -> /Frontend/BAT+
- C49 pad 1: /Frontend/BAT_F -> /Frontend/BAT+
- C50 pad 2: /Frontend/PACK+ -> /Frontend/CHG+
- D1 pad 2: /Frontend/BAT_F -> /Frontend/BAT+
- H2 pad 1: /Frontend/BAT_F -> GND
- H4 pad 1: /Frontend/PACK+ -> /Frontend/CHG+
- Q1 pad 2: /Frontend/BAT_F -> /Frontend/BAT+
- Q1 pad 3: /Frontend/FET_C -> /Frontend/CHG+
- R17 pad 1: /Frontend/PACK+ -> /Frontend/BAT+
- R18 pad 1: /Frontend/PACK+ -> /Frontend/BAT+
- R40 pad 1: /Frontend/BAT_F -> /Frontend/BAT+
- U3 pad 2: /Frontend/BAT_F -> /Frontend/BAT+
Routing:
- net /MCU/Ant_CLC: track 9.36 -> 0.00 mm
- net /Frontend/BAT_F: track 4.85 -> 0.00 mm
- net /Frontend/BAT+: track 0.00 -> 4.85 mm
- net +3.3V: track 4.79 -> 2.55 mm
- net /USB_DN: track 18.3 -> 17.6 mm
- net /USB_DP: track 18.7 -> 17.9 mm
- added copper zone on In1.Cu, net GND
- added copper zone on In2.Cu, net GND
- removed copper zone on F.Cu, net /Frontend/BAT-
- removed copper zone on F.Cu, net /Frontend/BAT_F
- removed copper zone on F.Cu, net /Frontend/CHG-
- removed copper zone on B.Cu, net /Frontend/FET_C
- removed copper zone on F.Cu, net /Frontend/FET_C
- removed copper zone on F.Cu, net /Frontend/PACK+
- removed copper zone on F.Cu, net Net-(C49-Pad2)
Other:
- outline, holes or cut-outs redrawn
- copper layers 2 -> 4
