File: hardware/frontend/afe.kicad_sch (KiCad schematic)
At the start: 57 parts, among them J301 ISOSPI_OUT, J302 ISOSPI_IN, J303 Conn_01x19_Male, Q301 MMBT3904, U301 LTC6813-1

Commit message: Split the design into front end and controller
Parts:
- C302, C303, C305, C306, C307, C308, C309, C310, J301, J302, TR301: now fitted
Other:
- note added: "TODO: check if IBIAS connection is ok for daisy chain"
