File: hardware/frontend/greenmobi-bms-frontend.kicad_sch (KiCad schematic)
At the start: 57 parts, among them J301 ISOSPI_OUT, J302 ISOSPI_IN, J303 Conn_01x19_Male, Q301 MMBT3904, U301 LTC6813-1

Commit message: Set IBIAS resistors for daisy chain
Parts:
- R306: value 20k -> 1k; Notes (none) -> 1%
- R312: value 0 -> 3.01k; Notes (none) -> 1%
Other:
- note removed: "TODO: check if IBIAS connection is ok for daisy chain"
Changed lines of the file:
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@@
     (stroke (width 0) (type default))
-  )
-  (text "TODO: check if IBIAS connection\nis ok for daisy chain"
-    (at 118.11 76.2 0)
-    (effects (font (size 1.27 1.27)) (justify left bottom))
   )
   (text "filter battery input" (at 179.07 33.02 0)
     (effects (font (size 1.27 1.27)) (justify left bottom))
   )
+  (label "GPIO1" (at 173.99 106.68 180) (fields_autoplaced)
+    (effects (font (size 1.27 1.27)) (justify right bottom))
+  )
+  (label "GPIO9" (at 173.99 127 180) (fields_autoplaced)
+    (effects (font (size 1.27 1.27)) (justify right bottom))
+  )
+  (label "SDI" (at 173.99 99.06 180) (fields_autoplaced)
+    (effects (font (size 1.27 1.27)) (justify right bottom))
+  )
   (label "VREG" (at 124.46 88.9 180) (fields_autoplaced)
     (effects (font (size 1.27 1.27)) (justify right bottom))
   )
+  (label "GPIO6" (at 173.99 119.38 180) (fields_autoplaced)
+    (effects (font (size 1.27 1.27)) (justify right bottom))
+  )
   (label "VREG" (at 115.57 43.18 180) (fields_autoplaced)
     (effects (font (size 1.27 1.27)) (justify right bottom))
   )
+  (label "GPIO8" (at 173.99 124.46 180) (fields_autoplaced)
+    (effects (font (size 1.27 1.27)) (justify right bottom))
+  )
+  (label "SDO" (at 173.99 101.6 180) (fields_autoplaced)
+    (effects (font (size 1.27 1.27)) (justify right bottom))
+  )
+  (label "GPIO2" (at 173.99 109.22 180) (fields_autoplaced)
+    (effects (font (size 1.27 1.27)) (justify right bottom))
+  )
   (label "VREG" (at 143.51 45.72 180) (fields_autoplaced)
     (effects (font (size 1.27 1.27)) (justify right bottom))
@@
     (effects (font (size 1.27 1.27)) (justify left bottom))
   )
+  (label "GPIO5" (at 173.99 116.84 180) (fields_autoplaced)
+    (effects (font (size 1.27 1.27)) (justify right bottom))
+  )
   (label "VREG" (at 99.06 43.18 180) (fields_autoplaced)
     (effects (font (size 1.27 1.27)) (justify right bottom))
   )
+  (label "SCK" (at 173.99 96.52 180) (fields_autoplaced)
+    (effects (font (size 1.27 1.27)) (justify right bottom))
+  )
+  (label "GPIO7" (at 173.99 121.92 180) (fields_autoplaced)
+    (effects (font (size 1.27 1.27)) (justify right bottom))
+  )
+  (label "GPIO3" (at 173.99 111.76 180) (fields_autoplaced)
+    (effects (font (size 1.27 1.27)) (justify right bottom))
+  )
+  (label "CS" (at 173.99 93.98 180) (fields_autoplaced)
+    (effects (font (size 1.27 1.27)) (justify right bottom))
+  )
   (label "Vref2" (at 153.67 163.83 0) (fields_autoplaced)
     (effects (font (size 1.27 1.27)) (justify left bottom))
   )
+  (label "GPIO4" (at 173.99 114.3 180) (fields_autoplaced)
+    (effects (font (size 1.27 1.27)) (justify right bottom))
+  )
   (label "VREG" (at 173.99 58.42 180) (fields_autoplaced)
     (effects (font (size 1.27 1.27)) (justify right bottom))
   )
-  (hierarchical_label "GPIO4" (shape input) (at 173.99 114.3 180) (fields_autoplaced)
-    (effects (font (size 1.27 1.27)) (justify right))
-  )
-  (hierarchical_label "GPIO2" (shape input) (at 173.99 109.22 180) (fields_autoplaced)
-    (effects (font (size 1.27 1.27)) (justify right))
-  )
-  (hierarchical_label "GPIO3" (shape input) (at 173.99 111.76 180) (fields_autoplaced)
-    (effects (font (size 1.27 1.27)) (justify right))
-  )
-  (hierarchical_label "CS" (shape input) (at 173.99 93.98 180) (fields_autoplaced)
-    (effects (font (size 1.27 1.27)) (justify right))
-  )
-  (hierarchical_label "GPIO5" (shape input) (at 173.99 116.84 180) (fields_autoplaced)
-    (effects (font (size 1.27 1.27)) (justify right))
-  )
-  (hierarchical_label "SCK" (shape input) (at 173.99 96.52 180) (fields_autoplaced)
-    (effects (font (size 1.27 1.27)) (justify right))
-  )
-  (hierarchical_label "GPIO7" (shape input) (at 173.99 121.92 180) (fields_autoplaced)
-    (effects (font (size 1.27 1.27)) (justify right))
-  )
-  (hierarchical_label "SDO" (shape output) (at 173.99 101.6 180) (fields_autoplaced)
-    (effects (font (size 1.27 1.27)) (justify right))
-  )
-  (hierarchical_label "GPIO6" (shape input) (at 173.99 119.38 180) (fields_autoplaced)
-    (effects (font (size 1.27 1.27)) (justify right))
-  )
-  (hierarchical_label "SDI" (shape input) (at 173.99 99.06 180) (fields_autoplaced)
-    (effects (font (size 1.27 1.27)) (justify right))
-  )
-  (hierarchical_label "GPIO8" (shape input) (at 173.99 124.46 180) (fields_autoplaced)
-    (effects (font (size 1.27 1.27)) (justify right))
-  )
   (hierarchical_label "WDT" (shape output) (at 124.46 96.52 180) (fields_autoplaced)
-    (effects (font (size 1.27 1.27)) (justify right))
-  )
-  (hierarchical_label "GPIO9" (shape input) (at 173.99 127 180) (fields_autoplaced)
-    (effects (font (size 1.27 1.27)) (justify right))
-  )
-  (hierarchical_label "GPIO1" (shape input) (at 173.99 106.68 180) (fields_autoplaced)
     (effects (font (size 1.27 1.27)) (justify right))
   )
@@
       (effects (font (size 1.27 1.27)))
     )
-    (property "Value" "0" (at 125.73 83.82 90)
+    (property "Value" "3.01k" (at 125.73 83.82 90)
       (effects (font (size 1.27 1.27)))
     )
@@
     )
     (property "Datasheet" "~" (at 125.73 78.74 0)
+      (effects (font (size 1.27 1.27)) hide)
+    )
+    (property "Notes" "1%" (at 125.73 78.74 90)
       (effects (font (size 1.27 1.27)) hide)
     )
@@
       (effects (font (size 1.27 1.27)))
     )
-    (property "Value" "20k" (at 118.11 83.82 90)
+    (property "Value" "1k" (at 118.11 83.82 90)
       (effects (font (size 1.27 1.27)))
     )
@@
       (effects (font (size 1.27 1.27)) hide)
     )
+    (property "Notes" "1%" (at 118.11 78.74 90)
+      (effects (font (size 1.27 1.27)) hide)
+    )

Commit message: Filter frontend input voltage
Parts:
- added C35: 100n, symbol Device:C_Small
- added FB1: FerriteBead_Small, symbol Device:FerriteBead_Small
- added R89: 0, symbol Device:R_Small
- R313: value R_Small -> 100k
- R316: value R_Small -> 1k
Connections:
- net +BATT: now also FB1.1; no longer U301.1 (V+)
- net GND: now also C35.2
- new net: FB1.2, R89.1
- new net: C35.1, R89.2, U301.1 (V+)
Other:
- note removed: "filter battery input"
Changed lines of the file:
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@@
   (junction (at 203.2 91.44) (diameter 0) (color 0 0 0 0)
   )
+  (junction (at 186.69 33.02) (diameter 0) (color 0 0 0 0)
+  )
   (junction (at 203.2 137.16) (diameter 0) (color 0 0 0 0)
   )
@@
     (stroke (width 0) (type default))
   )
-  (wire (pts (xy 129.54 143.51) (xy 152.4 143.51))
+  (wire (pts (xy 133.35 143.51) (xy 152.4 143.51))
     (stroke (width 0) (type default))
   )
@@
     (stroke (width 0) (type default))
   )
-  (wire (pts (xy 129.54 116.84) (xy 147.32 116.84))
+  (wire (pts (xy 133.35 116.84) (xy 147.32 116.84))
     (stroke (width 0) (type default))
   )
@@
     (stroke (width 0) (type default))
   )
+  (wire (pts (xy 186.69 33.02) (xy 186.69 31.75))
+    (stroke (width 0) (type default))
+  )
   (wire (pts (xy 199.39 96.52) (xy 203.2 96.52))
     (stroke (width 0) (type default))
@@
     (stroke (width 0) (type default))
   )
-  (wire (pts (xy 129.54 147.32) (xy 154.94 147.32))
+  (wire (pts (xy 133.35 147.32) (xy 154.94 147.32))
     (stroke (width 0) (type default))
   )
@@
     (stroke (width 0) (type default))
   )
-  (wire (pts (xy 129.54 119.38) (xy 129.54 128.27))
+  (wire (pts (xy 133.35 119.38) (xy 133.35 128.27))
     (stroke (width 0) (type default))
   )
@@
     (stroke (width 0) (type default))
   )
-  (wire (pts (xy 124.46 106.68) (xy 129.54 106.68))
+  (wire (pts (xy 124.46 106.68) (xy 133.35 106.68))
     (stroke (width 0) (type default))
   )
@@
     (stroke (width 0) (type default))
   )
-  (wire (pts (xy 148.59 119.38) (xy 129.54 119.38))
+  (wire (pts (xy 148.59 119.38) (xy 133.35 119.38))
     (stroke (width 0) (type default))
   )
@@
     (stroke (width 0) (type default))
   )
+  (wire (pts (xy 172.72 33.02) (xy 186.69 33.02))
+    (stroke (width 0) (type default))
+  )
   (wire (pts (xy 203.2 60.96) (xy 212.09 60.96))
     (stroke (width 0) (type default))
@@
     (stroke (width 0) (type default))
   )
-  (wire (pts (xy 124.46 154.94) (xy 129.54 154.94))
+  (wire (pts (xy 124.46 154.94) (xy 133.35 154.94))
     (stroke (width 0) (type default))
   )
@@
     (stroke (width 0) (type default))
   )
+  (wire (pts (xy 186.69 33.02) (xy 186.69 40.64))
+    (stroke (width 0) (type default))
+  )
   (wire (pts (xy 240.03 55.88) (xy 252.73 55.88))
     (stroke (width 0) (type default))
@@
     (stroke (width 0) (type default))
   )
-  (wire (pts (xy 124.46 133.35) (xy 129.54 133.35))
+  (wire (pts (xy 124.46 133.35) (xy 133.35 133.35))
     (stroke (width 0) (type default))
   )
-  (wire (pts (xy 129.54 147.32) (xy 129.54 154.94))
+  (wire (pts (xy 133.35 147.32) (xy 133.35 154.94))
     (stroke (width 0) (type default))
   )
@@
     (stroke (width 0) (type default))
   )
-  (wire (pts (xy 129.54 133.35) (xy 129.54 143.51))
+  (wire (pts (xy 133.35 133.35) (xy 133.35 143.51))
     (stroke (width 0) (type default))
   )
@@
     (stroke (width 0) (type default))
   )
-  (wire (pts (xy 129.54 106.68) (xy 129.54 116.84))
+  (wire (pts (xy 133.35 106.68) (xy 133.35 116.84))
     (stroke (width 0) (type default))
   )
@@
     (stroke (width 0) (type default))
   )
-  (wire (pts (xy 124.46 128.27) (xy 129.54 128.27))
+  (wire (pts (xy 124.46 128.27) (xy 133.35 128.27))
     (stroke (width 0) (type default))
   )
@@
     (stroke (width 0) (type default))
   )
-  (text "filter battery input" (at 179.07 33.02 0)
-    (effects (font (size 1.27 1.27)) (justify left bottom))
-  )
   (label "GPIO1" (at 173.99 106.68 180) (fields_autoplaced)
     (effects (font (size 1.27 1.27)) (justify right bottom))
@@
     )
   )
+  (symbol (lib_name "GND_4") (lib_id "power:GND") (at 172.72 38.1 0) (unit 1)
+    (in_bom yes) (on_board yes) (dnp no) (fields_autoplaced)
+    (property "Reference" "#PWR020" (at 172.72 44.45 0)
+      (effects (font (size 1.27 1.27)) hide)
+    )
+    (property "Value" "GND" (at 172.72 43.18 0)
+      (effects (font (size 1.27 1.27)))
+    )
+    (property "Footprint" "" (at 172.72 38.1 0)
+      (effects (font (size 1.27 1.27)) hide)
+    )
+    (property "Datasheet" "" (at 172.72 38.1 0)
+      (effects (font (size 1.27 1.27)) hide)
+    )
+    (pin "1")
+    (instances
+      (project "greenmobi-bms-frontend"
+        (path "/4579673c-99f5-483a-a4b8-b709bd3e9950"
+          (reference "#PWR020") (unit 1)
+        )
+      )
+    )
+  )
   (symbol (lib_name "GND_2") (lib_id "power:GND") (at 153.67 180.34 0) (unit 1)
     (in_bom yes) (on_board yes) (dnp no) (fields_autoplaced)
@@
     )
   )
+  (symbol (lib_id "Device:R_Small") (at 186.69 29.21 0) (unit 1)
+    (in_bom yes) (on_board yes) (dnp no) (fields_autoplaced)
+    (property "Reference" "R89" (at 189.23 27.94 0)
+      (effects (font (size 1.27 1.27)) (justify left))
+    )
+    (property "Value" "0" (at 189.23 30.48 0)
+      (effects (font (size 1.27 1.27)) (justify left))
+    )
+    (property "Footprint" "" (at 186.69 29.21 0)
+      (effects (font (size 1.27 1.27)) hide)
+    )
+    (property "Datasheet" "~" (at 186.69 29.21 0)
+      (effects (font (size 1.27 1.27)) hide)
+    )
+    (pin "1")
+    (pin "2")
+    (instances
+      (project "greenmobi-bms-frontend"
+        (path "/4579673c-99f5-483a-a4b8-b709bd3e9950"
+          (reference "R89") (unit 1)
+        )
+      )
+    )
+  )
   (symbol (lib_id "Device:R_Small") (at 124.46 149.86 0) (unit 1)
     (in_bom yes) (on_board yes) (dnp no)
@@
   (symbol (lib_id "Device:R_Small") (at 153.67 168.91 0) (unit 1)
     (in_bom yes) (on_board yes) (dnp no) (fields_autoplaced)
-    (property "Reference" "R313" (at 156.21 168.275 0)
+    (property "Reference" "R313" (at 156.21 167.64 0)
       (effects (font (size 1.27 1.27)) (justify left))
     )
-    (property "Value" "R_Small" (at 156.21 170.815 0)
+    (property "Value" "100k" (at 156.21 170.18 0)
       (effects (font (size 1.27 1.27)) (justify left))
     )
@@
     )
   )
+  (symbol (lib_id "Device:C_Small") (at 172.72 35.56 0) (unit 1)
+    (in_bom yes) (on_board yes) (dnp no) (fields_autoplaced)
+    (property "Reference" "C35" (at 175.26 34.2963 0)
+      (effects (font (size 1.27 1.27)) (justify left))
+    )
+    (property "Value" "100n" (at 175.26 36.8363 0)
+      (effects (font (size 1.27 1.27)) (justify left))
+    )
+    (property "Footprint" "" (at 172.72 35.56 0)
+      (effects (font (size 1.27 1.27)) hide)
+    )
+    (property "Datasheet" "~" (at 172.72 35.56 0)
+      (effects (font (size 1.27 1.27)) hide)
+    )
+    (pin "2")
+    (pin "1")
+    (instances
+      (project "greenmobi-bms-frontend"
+        (path "/4579673c-99f5-483a-a4b8-b709bd3e9950"
+          (reference "C35") (unit 1)
+        )
+      )
+    )
+  )
   (symbol (lib_id "Device:R_Small") (at 99.06 45.72 0) (unit 1)
     (in_bom yes) (on_board yes) (dnp yes) (fields_autoplaced)
@@
     )
   )
+  (symbol (lib_id "Device:FerriteBead_Small") (at 186.69 24.13 0) (unit 1)
+    (in_bom yes) (on_board yes) (dnp no) (fields_autoplaced)
+    (property "Reference" "FB1" (at 189.23 22.8219 0)
+      (effects (font (size 1.27 1.27)) (justify left))
+    )
+    (property "Value" "FerriteBead_Small" (at 189.23 25.3619 0)
+      (effects (font (size 1.27 1.27)) (justify left))
+    )
+    (property "Footprint" "" (at 184.912 24.13 90)
+      (effects (font (size 1.27 1.27)) hide)
+    )
+    (property "Datasheet" "~" (at 186.69 24.13 0)
+      (effects (font (size 1.27 1.27)) hide)
+    )
+    (pin "2")
+    (pin "1")
+    (instances
+      (project "greenmobi-bms-frontend"
+        (path "/4579673c-99f5-483a-a4b8-b709bd3e9950"
+          (reference "FB1") (unit 1)
+        )
+      )
+    )
+  )
   (symbol (lib_id "Device:C_Small") (at 203.2 83.82 0) (unit 1)
     (in_bom yes) (on_board yes) (dnp no) (fields_autoplaced)
@@
       (effects (font (size 1.27 1.27)))
     )
-    (property "Value" "R_Small" (at 133.35 170.18 90)
+    (property "Value" "1k" (at 133.35 170.18 90)
       (effects (font (size 1.27 1.27)))
     )
@@
     )
   )
-  (symbol (lib_id "power:+BATT") (at 186.69 40.64 0) (unit 1)
+  (symbol (lib_id "power:+BATT") (at 186.69 21.59 0) (unit 1)
     (in_bom yes) (on_board yes) (dnp no) (fields_autoplaced)
-    (property "Reference" "#PWR0316" (at 186.69 44.45 0)
+    (property "Reference" "#PWR0316" (at 186.69 25.4 0)
       (effects (font (size 1.27 1.27)) hide)
     )
-    (property "Value" "+BATT" (at 186.69 35.56 0)
+    (property "Value" "+BATT" (at 186.69 16.51 0)
       (effects (font (size 1.27 1.27)))
     )
-    (property "Footprint" "" (at 186.69 40.64 0)
+    (property "Footprint" "" (at 186.69 21.59 0)
       (effects (font (size 1.27 1.27)) hide)
     )
-    (property "Datasheet" "" (at 186.69 40.64 0)
+    (property "Datasheet" "" (at 186.69 21.59 0)
       (effects (font (size 1.27 1.27)) hide)
     )

Commit message: Schematic finished
Parts:
- removed C312, C334: 100n, symbol Device:C_Small
- removed Q301: MMBT3904, Package_TO_SOT_SMD:SOT-23, symbol Transistor_BJT:MMBT3904
- removed R313: 100k, symbol Device:R_Small
- removed R316: 1k, symbol Device:R_Small
- added J10, J11, J4, J5, J6, J7, J8, J9: EXT_NTC, Connector_PinHeader_2.54mm:PinHeader_1x02_P2.54mm_Horizontal, symbol Connector:Conn_01x02_Pin
- added Q20: DZT5551, Package_TO_SOT_SMD:SOT-223-3_TabPin2, symbol greenmobi-bms:DZT5551
- C311, C35: footprint (none) -> Capacitor_SMD:C_0805_2012Metric
- C313, C314, FB1: footprint (none) -> Capacitor_SMD:C_0603_1608Metric
- J301: footprint (none) -> Connector_PinSocket_2.54mm:PinSocket_1x02_P2.54mm_Horizontal
- J302: footprint (none) -> Connector_PinHeader_2.54mm:PinHeader_1x02_P2.54mm_Horizontal
- J303: footprint Connector_Molex:Molex_Micro-Fit_3.0_43045-2000_2x10_P3.00mm_Horizontal -> Connector_PinHeader_2.54mm:PinHeader_1x19_P2.54mm_Horizontal
- R301, R302, R303, R304, R305, R306, R307, R308, R309, R310, R311, R312, R314, R315, R89, TH301: footprint (none) -> Resistor_SMD:R_0603_1608Metric
Connections:
- net GND: no longer TH301.2
- net VREG: now also Q20.3 (E)
- net Thermistor/NTC+: now reaches TH301.1
- net at U301.49 (DRIVE): now also Q20.1 (B)
- net at C311.1, R305.2: now also Q20.2 (C)
- new net Thermistor/NTC-: TH301.2
- new net Thermistor1/NTC+: J4.1 (Pin_1)
- new net Thermistor1/NTC-: J4.2 (Pin_2)
- new net Thermistor2/NTC+: J5.1 (Pin_1)
- new net Thermistor2/NTC-: J5.2 (Pin_2)
- new net Thermistor3/NTC+: J6.1 (Pin_1)
- new net Thermistor3/NTC-: J6.2 (Pin_2)
- new net Thermistor4/NTC+: J7.1 (Pin_1)
- new net Thermistor4/NTC-: J7.2 (Pin_2)
- new net Thermistor5/NTC+: J9.1 (Pin_1)
- new net Thermistor5/NTC-: J9.2 (Pin_2)
- new net Thermistor6/NTC+: J8.1 (Pin_1)
- new net Thermistor6/NTC-: J8.2 (Pin_2)
- new net Thermistor7/NTC+: J11.1 (Pin_1)
- new net Thermistor7/NTC-: J11.2 (Pin_2)
- new net Thermistor8/NTC+: J10.1 (Pin_1)
- new net Thermistor8/NTC-: J10.2 (Pin_2)
Other:
- added sheet Thermistor (thermistor.kicad_sch)
- added sheet Thermistor1 (thermistor.kicad_sch)
- added sheet Thermistor2 (thermistor.kicad_sch)
- added sheet Thermistor3 (thermistor.kicad_sch)
- added sheet Thermistor4 (thermistor.kicad_sch)
- added sheet Thermistor5 (thermistor.kicad_sch)
- added sheet Thermistor6 (thermistor.kicad_sch)
- added sheet Thermistor7 (thermistor.kicad_sch)
- added sheet Thermistor8 (thermistor.kicad_sch)
- title: (none) -> GreenMobi BMS
- moved on the sheet: C302, C303, C305, C306, C307, C308, C309, C310, J301, J302, R308, R309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
