File: hardware/frontend/balance_front_end.kicad_sch (KiCad schematic)
At the start: 6 parts, among them Q601 BSS308PE

Commit message: Split the design into front end and controller
Parts:
- renumbered F601 to F701, Q601 to Q701, R1504 to R2304, R601 to R701, R602 to R702, R603 to R703

Commit message: Set IBIAS resistors for daisy chain
Parts:
- renumbered F701 to F601, Q701 to Q601, R2304 to R1504, R701 to R601, R702 to R602, R703 to R603

Commit message: Filter frontend input voltage
Parts:
- renumbered F601 to F701, Q601 to Q701, R1504 to R2304, R601 to R701, R602 to R702, R603 to R703

Commit message: Schematic finished
Parts:
- removed F701: 1A, symbol Device:Fuse_Small
- R1504: renamed from R2304; footprint (none) -> Resistor_SMD:R_0603_1608Metric
- R601: renamed from R701; footprint (none) -> Resistor_SMD:R_0603_1608Metric
- R602: renamed from R702; footprint (none) -> Resistor_SMD:R_0603_1608Metric
- renumbered Q701 to Q601, R703 to R603
Connections:
- net CELL: now also Q601.3 (D)

Commit message: footprints assigned
Parts:
- R603: footprint (none) -> Resistor_SMD:R_2512_6332Metric
