File: hardware/controller/greenmobi-bms-controller.kicad_sch (KiCad schematic)
At the start: 11 parts, among them J101 CHG+, J102 BAT+, J103 OLED, J104 Barrel_Jack, J105 PACK-, J106 BAT-, U102 ACS724xLCTR-50AB

Commit message: Split the design into front end and controller
Parts:
- added J1: AFE, symbol Connector:Conn_01x04_Pin
- gave numbers to parts that had none: 3
Connections:
- net AFE/BAT+ renamed Charger monitoring/BAT+
- new net MCU/AFE_CS: J1.4 (Pin_4)
- new net MCU/AFE_MISO: J1.2 (Pin_2)
- new net MCU/AFE_MOSI: J1.1 (Pin_1)
- new net MCU/AFE_SCLK: J1.3 (Pin_3)
- no-connect marks 6 -> 0
Other:
- removed sheet AFE
- removed sheet Thermal
- note added: "TODO: isolated interface"

Commit message: Current sensors and ISOSPI interface
Parts:
- removed C2802: 1n, symbol Device:C_Small
- removed J1: AFE, symbol Connector:Conn_01x04_Pin
- removed U102: ACS724xLCTR-50AB, Package_SO:SOIC-8_3.9x4.9mm_P1.27mm, symbol Sensor_Current:ACS724xLCTR-50AB
- added J1: Power, symbol Connector_Generic:Conn_01x02
- added U2: ACS770xCB-200B-PFF, Sensor_Current:Allegro_CB_PFF, symbol Sensor_Current:ACS770xCB-200B-PFF
- renumbered C2801 to C101, C2804 to C103, R2802 to R101
Connections:
- net +3.3V: now also U2.1 (VCC)
- net GND: now also J1.2 (Pin_2), U2.2 (GND), U2.4 (IP+)
- net at R101.1: now also U2.3 (VIOUT)
- net at J106.1 (Pin_1): now also U2.5 (IP-)
- new net Power Supply/Power_in: J1.1 (Pin_1)
Other:
- added sheet ISOSPI interface (isospi_interface.kicad_sch)
- sheet Power Supply ports: added Power_in; removed none
- note removed: "TODO: isolated interface"
- moved on the sheet: J106
