File: hardware/controller/power-supply.kicad_sch (KiCad schematic)
At the start: 3 parts, among them U501 LM5164DDA

Commit message: Current sensors and ISOSPI interface
Parts:
- removed U501: LM5164DDA, Package_SO:HSOP-8-1EP_3.9x4.9mm_P1.27mm_EP2.41x3.1mm_ThermalVias, symbol Regulator_Switching:LM5164DDA
- added U3: TPS563200, Package_TO_SOT_SMD:SOT-23-6, symbol Regulator_Switching:TPS563200
Connections:
- net BAT_UVLO: now also U3.3 (VIN), U3.5 (EN)
- net GND: now also U3.1 (GND)
- net +BATT renamed Power_in
Changed lines of the file:
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@@
   (junction (at 67.31 81.28) (diameter 0) (color 0 0 0 0)
   )
-  (wire (pts (xy 55.88 81.28) (xy 59.69 81.28))
+  (wire (pts (xy 58.42 81.28) (xy 59.69 81.28))
     (stroke (width 0) (type default))
   )
@@
     (stroke (width 0) (type default))
   )
-  (wire (pts (xy 106.68 101.6) (xy 106.68 104.14))
+  (wire (pts (xy 106.68 91.44) (xy 106.68 104.14))
     (stroke (width 0) (type default))
   )
   (wire (pts (xy 67.31 87.63) (xy 67.31 104.14))
-    (stroke (width 0) (type default))
-  )
-  (wire (pts (xy 55.88 77.47) (xy 55.88 81.28))
     (stroke (width 0) (type default))
   )
@@
   )
   (hierarchical_label "BAT_UVLO" (shape output) (at 93.98 86.36 180) (fields_autoplaced)
+    (effects (font (size 1.27 1.27)) (justify right))
+  )
+  (hierarchical_label "Power_in" (shape input) (at 58.42 81.28 180) (fields_autoplaced)
     (effects (font (size 1.27 1.27)) (justify right))
   )
@@
     )
   )
-  (symbol (lib_id "Regulator_Switching:LM5164DDA") (at 109.22 88.9 0) (unit 1)
+  (symbol (lib_id "Regulator_Switching:TPS563200") (at 106.68 83.82 0) (unit 1)
     (in_bom yes) (on_board yes) (dnp no) (fields_autoplaced)
-    (property "Reference" "U501" (at 109.22 73.66 0)
+    (property "Reference" "U3" (at 106.68 73.66 0)
       (effects (font (size 1.27 1.27)))
     )
-    (property "Value" "LM5164DDA" (at 109.22 76.2 0)
+    (property "Value" "TPS563200" (at 106.68 76.2 0)
       (effects (font (size 1.27 1.27)))
     )
-    (property "Footprint" "Package_SO:HSOP-8-1EP_3.9x4.9mm_P1.27mm_EP2.41x3.1mm_ThermalVias" (at 110.49 100.33 0)
+    (property "Footprint" "Package_TO_SOT_SMD:SOT-23-6" (at 107.95 90.17 0)
+      (effects (font (size 1.27 1.27)) (justify left) hide)
+    )
+    (property "Datasheet" "http://www.ti.com/lit/ds/symlink/tps563200.pdf" (at 106.68 83.82 0)
       (effects (font (size 1.27 1.27)) hide)
     )
-    (property "Datasheet" "https://www.ti.com/lit/ds/symlink/lm5164.pdf?ts=1598311864250&ref_url=https%253A%252F%252Fwww.ti.com%252Fproduct%252FLM5164%253FHQS%253DTI-null-null-octopart-df-pf-null-wwe" (at 101.6 80.01 0)
-      (effects (font (size 1.27 1.27)) hide)
-    )
-    (property "LCSC" "C477928" (at 109.22 88.9 0)
-      (effects (font (size 1.27 1.27)) hide)
-    )
+    (pin "5")
     (pin "1")
     (pin "2")
     (pin "3")
+    (pin "6")
     (pin "4")
-    (pin "5")
-    (pin "6")
-    (pin "7")
-    (pin "8")
-    (pin "9")
     (instances
       (project "greenmobi-bms-controller"
         (path "/3e668e3e-3e16-4665-a807-4735962c41d3/600d3fd5-a2c8-411e-91ac-e4cbb4ace0f8"
-          (reference "U501") (unit 1)
+          (reference "U3") (unit 1)
         )
       )
-    )
-  )
-  (symbol (lib_id "power:+BATT") (at 55.88 77.47 0) (unit 1)
-    (in_bom yes) (on_board yes) (dnp no) (fields_autoplaced)
-    (property "Reference" "#PWR0501" (at 55.88 81.28 0)
-      (effects (font (size 1.27 1.27)) hide)
-    )
-    (property "Value" "+BATT" (at 55.88 72.39 0)
-      (effects (font (size 1.27 1.27)))
-    )
-    (property "Footprint" "" (at 55.88 77.47 0)
-      (effects (font (size 1.27 1.27)) hide)
-    )
-    (property "Datasheet" "" (at 55.88 77.47 0)
-      (effects (font (size 1.27 1.27)) hide)
-    )
-    (pin "1")
-    (instances
-      (project "greenmobi-bms-controller"
-        (path "/3e668e3e-3e16-4665-a807-4735962c41d3/600d3fd5-a2c8-411e-91ac-e4cbb4ace0f8"
-          (reference "#PWR0501") (unit 1)
-        )
-      )
